Commit message: Reducing spaghetti code
Introduced JointModule class to incapsulate most of the operations needed when adding new joint

File: urdf/ModularBot_Generated.urdf.xacro (robot description, xacro)
@@ -70,3 +70,3 @@
         </joint>
     </xacro:macro>
-<xacro:add_link a_i="0" alpha_i="0" d_i="${len1}" length="${len3}" suffix="1" theta_i="0" /><xacro:add_link a_i="${len3}" alpha_i="${-pi/2}" d_i="0" length="${len3}" suffix="2" theta_i="0" /><xacro:add_link a_i="${len3}" alpha_i="${pi/2}" d_i="0" length="${len3}" suffix="3" theta_i="0" /></robot>
+<xacro:add_link a_i="0" alpha_i="0" d_i="${len1}" length="0.8" suffix="1" theta_i="0" /><xacro:add_link a_i="0.8" alpha_i="${-pi/2}" d_i="0" length="0.8" suffix="2" theta_i="0" /><xacro:add_link a_i="0.8" alpha_i="${pi/2}" d_i="0" length="0.8" suffix="3" theta_i="0" /></robot>

File: urdf/ModularBot_new.urdf.xacro (robot description, xacro)
@@ -78,5 +78,5 @@
         </joint>
     </xacro:macro>
-    <xacro:macro name="add_link_angular" params="suffix p n x y z roll pitch yaw">
+    <xacro:macro name="add_link_elbow" params="suffix p n x y z roll pitch yaw">
         <link name="link_${suffix}">
             <visual>
