Commit message: Fixed rototranslation for non-elbow modules
-Add joint, elbow and link modules (YAML and URDF)
-YAML files also contain kin. param.
-Add capability to add also straight links

File: urdf/link_module.urdf (robot description, URDF)
Before this commit: robot link_module, 1 links, 0 joints
Links:
- link None: geometry collision box size=0.1 0.1 0.3; visual box size=0.1 0.1 0.3
