Commit message: Add master cube with connections for 2 branches

File: urdf/ModularBot_base.urdf (robot description, URDF)
Before this commit: robot ModularBot, 2 links, 1 joints
Links:
- removed link link_0
- added link L_0, mass 2; collision box size=0.4 0.4 0.4; visual box size=0.4 0.4 0.4
- added link L_0_A, mass 0.5; collision cylinder length=0.1 radius=0.06; visual cylinder length=0.1 radius=0.06
- added link L_0_B, mass 0.5; collision cylinder length=0.1 radius=0.06; visual cylinder length=0.1 radius=0.06
Joints:
- added joint fixed_A_branch: type fixed, parent L_0, child L_0_A, origin xyz=0 0.2 0.3 rpy=-1.57 0 0, axis 0 0 1
- added joint fixed_B_branch: type fixed, parent L_0, child L_0_B, origin xyz=0 -0.2 0.3 rpy=1.57 0 0, axis 0 0 1
- joint fixed: child link_0 -> L_0

File: urdf/ModularBot_new.urdf.xacro (robot description, xacro)
@@ -35,5 +35,5 @@
     </joint>
     <link name="base_link"/>
-    <link name="L_0">
+    <!-- <link name="L_0">
         <visual>
             <origin xyz="0 0 ${len1/2}" rpy="0 0 0" />
@@ -50,8 +50,76 @@
         </collision>
         <xacro:default_inertial mass="1"/>
-    </link>
+    </link> -->
     <joint name="fixed" type="fixed">
         <parent link="base_link"/>
         <child link="L_0"/>
+        <axis rpy="0 0 0" xyz="0 0 1"/>
+        <origin rpy="0.0 0.0 0.0" xyz="0.0 0.0 0.0"/>
+    </joint>
+    <link name="L_0">
+        <visual>
+            <origin rpy="0 0 0" xyz="0 0 0.2"/>
+            <geometry>
+                <box size="0.4 0.4 0.4"/>
+            </geometry>
+            <material name="black"/>
+        </visual>
+        <collision>
+            <geometry>
+                <box size="0.4 0.4 0.4"/>
+            </geometry>
+        </collision>
+        <inertial>
+            <mass value="2"/>
+            <inertia ixx="1.0" ixy="0.0" ixz="0.0" iyy="1.0" iyz="0.0" izz="1.0"/>
+        </inertial>
+    </link>
+    <link name="L_0_A">
+        <visual>
+            <origin rpy="0 0 0" xyz="0 0 0.05"/>
+            <geometry>
+                <cylinder length="0.1" radius="0.06"/>
+            </geometry>
+            <material name="black"/>
+        </visual>
+        <collision>
+            <geometry>
+                <cylinder length="0.1" radius="0.06"/>
+            </geometry>
+        </collision>
+        <inertial>
+            <mass value="0.5"/>
+            <inertia ixx="1.0" ixy="0.0" ixz="0.0" iyy="1.0" iyz="0.0" izz="1.0"/>
+        </inertial>
+    </link>
+    <link name="L_0_B">
+        <visual>
+            <origin rpy="0 0 0" xyz="0 0 0.05"/>
+            <geometry>
+                <cylinder length="0.1" radius="0.06"/>
+            </geometry>
+            <material name="black"/>
+        </visual>
+        <collision>
+            <geometry>
+                <cylinder length="0.1" radius="0.06"/>
+            </geometry>
+        </collision>
+        <inertial>
+            <mass value="0.5"/>
+            <inertia ixx="1.0" ixy="0.0" ixz="0.0" iyy="1.0" iyz="0.0" izz="1.0"/>
+        </inertial>
+    </link>
+    <joint name="fixed_A_branch" type="fixed">
+        <parent link="L_0"/>
+        <child link="L_0_A"/>
+        <axis rpy="0 0 0" xyz="0 0 1"/>
+        <origin rpy="-1.57 0 0" xyz="0 0.2 0.3"/>
+    </joint>
+    <joint name="fixed_B_branch" type="fixed">
+        <parent link="L_0"/>
+        <child link="L_0_B"/>
+        <axis rpy="0 0 0" xyz="0 0 1"/>
+        <origin rpy="1.57 0 0" xyz="0 -0.2 0.3"/>
     </joint>
     <!-- Macro for adding a straight link -->
