Commit message: Add URDF generator
python script that can be used to add links to the URDF tree

File: urdf/ModularBot.urdf.xacro (robot description, xacro)
@@ -25,5 +25,5 @@
     <link name="link_0">
         <visual>
-            <origin xyz="0 0 0.2" rpy="0 0 0" />
+            <origin xyz="0 0 ${len1/2}" rpy="0 0 0" />
             <geometry>
                 <cylinder radius="${width}" length="${len1}"/>
@@ -38,9 +38,4 @@
         <xacro:default_inertial mass="10"/>
     </link>
-    <!-- <joint name="fixed" type="fixed">
-        <parent link="base_link"/>
-        <child link="link_1"/>
-        <origin xyz="0 0 0.4" rpy="0 0 0" />
-    </joint> -->
     <joint name="fixed" type="fixed">
         <parent link="base_link"/>
@@ -54,5 +49,10 @@
             <box size="${length} ${width} ${width}"/>
             </geometry>
-            <material name="blue"/>
+            <xacro:if value="${suffix%2==0}">
+                <material name="white"/>
+            </xacro:if>
+            <xacro:unless value="${suffix%2==0}">
+                <material name="blue"/>
+            </xacro:unless>
         </visual>
         <collision>
@@ -78,6 +78,3 @@
         </joint>
     </xacro:macro>
-    <xacro:add_link suffix="1" length="${len3}" a_i="0" d_i="${len1}" alpha_i="${-pi/2}" theta_i="0"/>
-    <xacro:add_link suffix="2" length="${len3}" a_i="${len3}" d_i="0" alpha_i="${pi/2}" theta_i="0"/>
-    <xacro:add_link suffix="3" length="${len3}" a_i="${len3}" d_i="0" alpha_i="${-pi/2}" theta_i="0"/>
 </robot>

Commit message: update urdf generated files

File: urdf/ModularBot.urdf.xacro (robot description, xacro)
@@ -1,4 +1,8 @@
 <?xml version="1.0" ?>
 <robot name="ModularBot" xmlns:xacro="http://ros.org/wiki/xacro">
+  <xacro:include filename="$(find modular)/urdf/config.xacro"/>
+  <xacro:if value="${GAZEBO}">
+    <xacro:include filename="$(find modular)/urdf/modular.gazebo"/>
+  </xacro:if>
    <xacro:property name="size1" value="0.05"/>
    <xacro:property name="size2" value="0.055"/>
@@ -513,20 +517,7 @@
    <xacro:add_joint_stator name="J1_A_stator" size="3" size_y="0" size_z="0.2" type="joint_stator"/>
    <xacro:add_joint child="L_1_A" effort="35" father="J1_A_stator" lower_lim="-3.14" name="J1_A" pitch="-0.0" roll="0.0" type="joint" upper_lim="3.14" velocity="5.7" x="0.0" y="0.0" yaw="0.0" z="0.2"/>
-   <xacro:add_fixed_joint_stator child="J1_B_stator" father="L_0a_con3" name="fixed_J1_B" pitch="-0.0" roll="0.0" type="fixed_joint_stator" x="0.0" y="0.0" yaw="0.0" z="0.1"/>
-   <xacro:add_joint_stator name="J1_B_stator" size="3" size_y="0" size_z="0.2" type="joint_stator"/>
-   <xacro:add_joint child="L_1_B" effort="35" father="J1_B_stator" lower_lim="-3.14" name="J1_B" pitch="-0.0" roll="0.0" type="joint" upper_lim="3.14" velocity="5.7" x="0.0" y="0.0" yaw="0.0" z="0.2"/>
-   <xacro:add_link name="L_1_link_1_B" size="3" size_z="0.3" type="link"/>
-   <xacro:add_fixed_joint child="L_1_link_1_B" father="L_1_B" name="L_1_fixed_joint_1_B" pitch="-0.0" roll="0.0" type="fixed_joint" x="0.0" y="0.0" yaw="0.0" z="0.0"/>
-   <xacro:add_elbow name="L_1_elbow_2_B" size="3" size_y="0.2" size_z="0.2" type="elbow"/>
-   <xacro:add_fixed_joint child="L_1_elbow_2_B" father="L_1_link_1_B" name="L_1_fixed_joint_2_B" pitch="-0.0" roll="0.0" type="fixed_joint" x="0.0" y="0.0" yaw="0.0" z="0.3"/>
-   <xacro:add_fixed_joint_stator child="J2_B_stator" father="L_1_elbow_2_B" name="fixed_J2_B" pitch="-0.0" roll="-1.57" type="fixed_joint_stator" x="0.0" y="0.199999936586" yaw="0.0" z="0.200159265342"/>
-   <xacro:add_joint_stator name="J2_B_stator" size="3" size_y="0" size_z="0.2" type="joint_stator"/>
-   <xacro:add_joint child="L_2_B" effort="35" father="J2_B_stator" lower_lim="-3.14" name="J2_B" pitch="-0.0" roll="0.0" type="joint" upper_lim="3.14" velocity="5.7" x="0.0" y="0.0" yaw="0.0" z="0.2"/>
-   <xacro:add_elbow name="L_2_elbow_1_B" size="3" size_y="0.2" size_z="0.2" type="elbow"/>
-   <xacro:add_fixed_joint child="L_2_elbow_1_B" father="L_2_B" name="L_2_fixed_joint_1_B" pitch="-0.0" roll="0.0" type="fixed_joint" x="0.0" y="0.0" yaw="0.0" z="0.0"/>
-   <xacro:add_elbow name="L_2_elbow_2_B" size="3" size_y="0.2" size_z="0.2" type="elbow"/>
-   <xacro:add_fixed_joint child="L_2_elbow_2_B" father="L_2_elbow_1_B" name="L_2_fixed_joint_2_B" pitch="-0.0" roll="-1.57" type="fixed_joint" x="0.0" y="0.199999936586" yaw="0.0" z="0.200159265342"/>
-   <xacro:add_fixed_joint_stator child="J3_B_stator" father="L_2_elbow_2_B" name="fixed_J3_B" pitch="-0.0" roll="-1.57" type="fixed_joint_stator" x="0.0" y="0.199999936586" yaw="0.0" z="0.200159265342"/>
-   <xacro:add_joint_stator name="J3_B_stator" size="3" size_y="0" size_z="0.2" type="joint_stator"/>
-   <xacro:add_joint child="L_3_B" effort="35" father="J3_B_stator" lower_lim="-3.14" name="J3_B" pitch="-0.0" roll="0.0" type="joint" upper_lim="3.14" velocity="5.7" x="0.0" y="0.0" yaw="0.0" z="0.2"/>
+   <xacro:add_elbow name="L_1_elbow_1_A" size="3" size_y="0.2" size_z="0.2" type="elbow"/>
+   <xacro:add_fixed_joint child="L_1_elbow_1_A" father="L_1_A" name="L_1_fixed_joint_1_A" pitch="-0.0" roll="0.0" type="fixed_joint" x="0.0" y="0.0" yaw="0.0" z="0.0"/>
+   <xacro:add_link name="L_1_link_2_A" size="3" size_z="0.3" type="link"/>
+   <xacro:add_fixed_joint child="L_1_link_2_A" father="L_1_elbow_1_A" name="L_1_fixed_joint_2_A" pitch="-0.0" roll="-1.57" type="fixed_joint" x="0.0" y="0.199999936586" yaw="0.0" z="0.200159265342"/>
 </robot>

File: urdf/ModularBot_new.urdf.xacro (robot description, xacro)
@@ -1,4 +1,6 @@
 <?xml version="1.0"?>
 <robot name="ModularBot" xmlns:xacro="http://ros.org/wiki/xacro">
+    <!-- <xacro:include filename="$(find modular)/urdf/config.xacro" />
+    <xacro:include filename="$(find modular)/urdf/modular.gazebo" /> -->
     <xacro:property name="size1" value="0.05" />
     <xacro:property name="size2" value="0.055" />

File: urdf/ModularBot_test.urdf (robot description, URDF)
Before this commit: robot ModularBot, 3 links, 2 joints
Links:
- removed link L_0
- added link J1_A_stator, mass 0.5; collision cylinder length=0.2 radius=0.06; visual cylinder length=0.2 radius=0.06
- added link J1_B_stator, mass 0.5; collision cylinder length=0.2 radius=0.06; visual cylinder length=0.2 radius=0.06
- added link J2_B_stator, mass 0.5; collision cylinder length=0.2 radius=0.06; visual cylinder length=0.2 radius=0.06
- added link J3_B_stator, mass 0.5; collision cylinder length=0.2 radius=0.06; visual cylinder length=0.2 radius=0.06
- added link L_0a, mass 2; collision box size=0.4 0.4 0.4; visual box size=0.4 0.4 0.4
- added link L_0a_con1, mass 0.5; collision cylinder length=0.1 radius=0.06; visual cylinder length=0.1 radius=0.06
- added link L_0a_con2, mass 0.5; collision cylinder length=0.1 radius=0.06; visual cylinder length=0.1 radius=0.06
- added link L_0a_con3, mass 0.5; collision cylinder length=0.1 radius=0.06; visual cylinder length=0.1 radius=0.06
- added link L_0a_con4, mass 0.5; collision cylinder length=0.1 radius=0.06; visual cylinder length=0.1 radius=0.06
- added link L_1_A
- added link L_1_B
- added link L_1_elbow_2_B, mass 0.5; collision cylinder length=0.2 radius=0.06; collision cylinder length=0.2 radius=0.06
- added link L_1_link_1_B, mass 0.5; collision cylinder length=0.3 radius=0.06; visual cylinder length=0.3 radius=0.06
- added link L_2_B
- added link L_2_elbow_1_B, mass 0.5; collision cylinder length=0.2 radius=0.06; collision cylinder length=0.2 radius=0.06
- added link L_2_elbow_2_B, mass 0.5; collision cylinder length=0.2 radius=0.06; collision cylinder length=0.2 radius=0.06
- added link L_3_B
Joints:
- added joint J1_A: type revolute, parent J1_A_stator, child L_1_A, origin xyz=0.0 0.0 0.2 rpy=0.0 -0.0 0.0, axis 0 0 1, limit lower=-3.14 upper=3.14 effort=35 velocity=5.7
- added joint J1_B: type revolute, parent J1_B_stator, child L_1_B, origin xyz=0.0 0.0 0.2 rpy=0.0 -0.0 0.0, axis 0 0 1, limit lower=-3.14 upper=3.14 effort=35 velocity=5.7
- added joint J2_B: type revolute, parent J2_B_stator, child L_2_B, origin xyz=0.0 0.0 0.2 rpy=0.0 -0.0 0.0, axis 0 0 1, limit lower=-3.14 upper=3.14 effort=35 velocity=5.7
- added joint J3_B: type revolute, parent J3_B_stator, child L_3_B, origin xyz=0.0 0.0 0.2 rpy=0.0 -0.0 0.0, axis 0 0 1, limit lower=-3.14 upper=3.14 effort=35 velocity=5.7
- added joint L_0a_fixed_1: type fixed, parent L_0a, child L_0a_con1, origin xyz=0 0 0 rpy=3.14 0 0, axis 0 0 1
- added joint L_0a_fixed_2: type fixed, parent L_0a, child L_0a_con2, origin xyz=0 -0.2 0.2 rpy=1.57 0 0, axis 0 0 1
- added joint L_0a_fixed_3: type fixed, parent L_0a, child L_0a_con3, origin xyz=0 0 0.4 rpy=0 0 0, axis 0 0 1
- added joint L_0a_fixed_4: type fixed, parent L_0a, child L_0a_con4, origin xyz=0 0.2 0.2 rpy=-1.57 0 0, axis 0 0 1
- added joint L_1_fixed_joint_1_B: type fixed, parent L_1_B, child L_1_link_1_B, origin xyz=0.0 0.0 0.0 rpy=0.0 -0.0 0.0, axis 0 0 1
- added joint L_1_fixed_joint_2_B: type fixed, parent L_1_link_1_B, child L_1_elbow_2_B, origin xyz=0.0 0.0 0.3 rpy=0.0 -0.0 0.0, axis 0 0 1
- added joint L_2_fixed_joint_1_B: type fixed, parent L_2_B, child L_2_elbow_1_B, origin xyz=0.0 0.0 0.0 rpy=0.0 -0.0 0.0, axis 0 0 1
- added joint L_2_fixed_joint_2_B: type fixed, parent L_2_elbow_1_B, child L_2_elbow_2_B, origin xyz=0.0 0.199999936586 0.200159265342 rpy=-1.57 -0.0 0.0, axis 0 0 1
- added joint fixed_J1_A: type fixed, parent L_0a_con4, child J1_A_stator, origin xyz=0.0 0.0 0.1 rpy=0.0 -0.0 0.0, axis 0 0 1
- added joint fixed_J1_B: type fixed, parent L_0a_con3, child J1_B_stator, origin xyz=0.0 0.0 0.1 rpy=0.0 -0.0 0.0, axis 0 0 1
- added joint fixed_J2_B: type fixed, parent L_1_elbow_2_B, child J2_B_stator, origin xyz=0.0 0.199999936586 0.200159265342 rpy=-1.57 -0.0 0.0, axis 0 0 1
- added joint fixed_J3_B: type fixed, parent L_2_elbow_2_B, child J3_B_stator, origin xyz=0.0 0.199999936586 0.200159265342 rpy=-1.57 -0.0 0.0, axis 0 0 1
- joint fixed: axis (none) -> 0 0 1; child L_0 -> L_0a; origin (none) -> xyz=0.0 0.0 0.0 rpy=0.0 0.0 0.0
