Commit message: update files

File: urdf/ModularBot.urdf.xacro (robot description, xacro)
@@ -5,519 +5,762 @@
     <xacro:include filename="$(find modular)/urdf/modular.gazebo"/>
   </xacro:if>
-   <xacro:property name="size1" value="0.05"/>
-   <xacro:property name="size2" value="0.055"/>
-   <xacro:property name="size3" value="0.06"/>
-   <xacro:property name="len1" value="0.4"/>
-   <xacro:property name="len2" value="0.6"/>
-   <xacro:property name="len3" value="0.8"/>
-   <xacro:property name="mass" value="0.5"/>
    <material name="blue">
-      <color rgba="0 0 0.8 1"/>
-   </material>
-   <material name="black">
-      <color rgba="0 0 0 1"/>
-   </material>
-   <material name="white">
-      <color rgba="1 1 1 1"/>
-   </material>
-   <material name="grey">
-      <color rgba="0.5 0.5 0.5 1"/>
-   </material>
-   <xacro:macro name="default_inertial" params="mass">
-      <inertial>
-         <mass value="${mass}"/>
-         <inertia ixx="1.0" ixy="0.0" ixz="0.0" iyy="1.0" iyz="0.0" izz="1.0"/>
-      </inertial>
-   </xacro:macro>
-   <link name="world"/>
-   <joint name="world" type="fixed">
-      <parent link="world"/>
-      <child link="base_link"/>
-   </joint>
-   <link name="base_link"/>
-   <joint name="fixed" type="fixed">
-      <parent link="base_link"/>
-      <child link="L_0a"/>
-      <axis rpy="0 0 0" xyz="0 0 1"/>
-      <origin rpy="0.0 0.0 0.0" xyz="0.0 0.0 0.0"/>
-   </joint>
-   <link name="L_0a">
-      <visual>
-         <origin rpy="0 0 0" xyz="0 0 0.2"/>
-         <geometry>
-            <box size="0.4 0.4 0.4"/>
-         </geometry>
-         <material name="black"/>
-      </visual>
-      <collision>
-         <geometry>
-            <box size="0.4 0.4 0.4"/>
-         </geometry>
-      </collision>
-      <inertial>
-         <mass value="2"/>
-         <inertia ixx="1.0" ixy="0.0" ixz="0.0" iyy="1.0" iyz="0.0" izz="1.0"/>
-      </inertial>
-   </link>
-   <link name="L_0a_con1">
-      <visual>
-         <origin rpy="0 0 0" xyz="0 0 0.05"/>
-         <geometry>
-            <cylinder length="0.1" radius="0.06"/>
-         </geometry>
-         <material name="black"/>
-      </visual>
-      <collision>
-         <geometry>
-            <cylinder length="0.1" radius="0.06"/>
-         </geometry>
-      </collision>
-      <inertial>
-         <mass value="0.5"/>
-         <inertia ixx="1.0" ixy="0.0" ixz="0.0" iyy="1.0" iyz="0.0" izz="1.0"/>
-      </inertial>
-   </link>
-   <link name="L_0a_con2">
-      <visual>
-         <origin rpy="0 0 0" xyz="0 0 0.05"/>
-         <geometry>
-            <cylinder length="0.1" radius="0.06"/>
-         </geometry>
-         <material name="black"/>
-      </visual>
-      <collision>
-         <geometry>
-            <cylinder length="0.1" radius="0.06"/>
-         </geometry>
-      </collision>
-      <inertial>
-         <mass value="0.5"/>
-         <inertia ixx="1.0" ixy="0.0" ixz="0.0" iyy="1.0" iyz="0.0" izz="1.0"/>
-      </inertial>
-   </link>
-   <link name="L_0a_con3">
-      <visual>
-         <origin rpy="0 0 0" xyz="0 0 0.05"/>
-         <geometry>
-            <cylinder length="0.1" radius="0.06"/>
-         </geometry>
-         <material name="black"/>
-      </visual>
-      <collision>
-         <geometry>
-            <cylinder length="0.1" radius="0.06"/>
-         </geometry>
-      </collision>
-      <inertial>
-         <mass value="0.5"/>
-         <inertia ixx="1.0" ixy="0.0" ixz="0.0" iyy="1.0" iyz="0.0" izz="1.0"/>
-      </inertial>
-   </link>
-   <link name="L_0a_con4">
-      <visual>
-         <origin rpy="0 0 0" xyz="0 0 0.05"/>
-         <geometry>
-            <cylinder length="0.1" radius="0.06"/>
-         </geometry>
-         <material name="black"/>
-      </visual>
-      <collision>
-         <geometry>
-            <cylinder length="0.1" radius="0.06"/>
-         </geometry>
-      </collision>
-      <inertial>
-         <mass value="0.5"/>
-         <inertia ixx="1.0" ixy="0.0" ixz="0.0" iyy="1.0" iyz="0.0" izz="1.0"/>
-      </inertial>
-   </link>
-   <joint name="L_0a_fixed_1" type="fixed">
-      <parent link="L_0a"/>
-      <child link="L_0a_con1"/>
-      <axis rpy="0 0 0" xyz="0 0 1"/>
-      <origin rpy="3.14 0 0" xyz="0 0 0"/>
-   </joint>
-   <joint name="L_0a_fixed_2" type="fixed">
-      <parent link="L_0a"/>
-      <child link="L_0a_con2"/>
-      <axis rpy="0 0 0" xyz="0 0 1"/>
-      <origin rpy="1.57 0 0" xyz="0 -0.2 0.2"/>
-   </joint>
-   <joint name="L_0a_fixed_3" type="fixed">
-      <parent link="L_0a"/>
-      <child link="L_0a_con3"/>
-      <axis rpy="0 0 0" xyz="0 0 1"/>
-      <origin rpy="0 0 0" xyz="0 0 0.4"/>
-   </joint>
-   <joint name="L_0a_fixed_4" type="fixed">
-      <parent link="L_0a"/>
-      <child link="L_0a_con4"/>
-      <axis rpy="0 0 0" xyz="0 0 1"/>
-      <origin rpy="-1.57 0 0" xyz="0 0.2 0.2"/>
-   </joint>
-   <xacro:macro name="add_fixed_joint" params="type name father child x y z roll pitch yaw">
-      <joint name="${name}" type="fixed">
-         <axis rpy="0 0 0" xyz="0 0 1"/>
-         <parent link="${father}"/>
-         <child link="${child}"/>
-         <origin rpy="${roll} ${pitch} ${yaw}" xyz="${x} ${y} ${z}"/>
-      </joint>
-   </xacro:macro>
-   <xacro:macro name="add_slave_cube" params="name">
-      <link name="${name}">
-         <visual>
-            <origin rpy="0 0 0" xyz="0 0 0.2"/>
-            <geometry>
-               <box size="0.4 0.4 0.4"/>
-            </geometry>
-            <material name="black"/>
-         </visual>
-         <collision>
-            <geometry>
-               <box size="0.4 0.4 0.4"/>
-            </geometry>
-         </collision>
-         <inertial>
-            <mass value="2"/>
-            <inertia ixx="1.0" ixy="0.0" ixz="0.0" iyy="1.0" iyz="0.0" izz="1.0"/>
-         </inertial>
-      </link>
-      <link name="${name}_con1">
-         <visual>
-            <origin rpy="0 0 0" xyz="0 0 0.05"/>
-            <geometry>
-               <cylinder length="0.1" radius="0.06"/>
-            </geometry>
-            <material name="black"/>
-         </visual>
-         <collision>
-            <geometry>
-               <cylinder length="0.1" radius="0.06"/>
-            </geometry>
-         </collision>
-         <inertial>
-            <mass value="0.5"/>
-            <inertia ixx="1.0" ixy="0.0" ixz="0.0" iyy="1.0" iyz="0.0" izz="1.0"/>
-         </inertial>
-      </link>
-      <link name="${name}_con2">
-         <visual>
-            <origin rpy="0 0 0" xyz="0 0 0.05"/>
-            <geometry>
-               <cylinder length="0.1" radius="0.06"/>
-            </geometry>
-            <material name="black"/>
-         </visual>
-         <collision>
-            <geometry>
-               <cylinder length="0.1" radius="0.06"/>
-            </geometry>
-         </collision>
-         <inertial>
-            <mass value="0.5"/>
-            <inertia ixx="1.0" ixy="0.0" ixz="0.0" iyy="1.0" iyz="0.0" izz="1.0"/>
-         </inertial>
-      </link>
-      <link name="${name}_con3">
-         <visual>
-            <origin rpy="0 0 0" xyz="0 0 0.05"/>
-            <geometry>
-               <cylinder length="0.1" radius="0.06"/>
-            </geometry>
-            <material name="black"/>
-         </visual>
-         <collision>
-            <geometry>
-               <cylinder length="0.1" radius="0.06"/>
-            </geometry>
-         </collision>
-         <inertial>
-            <mass value="0.5"/>
-            <inertia ixx="1.0" ixy="0.0" ixz="0.0" iyy="1.0" iyz="0.0" izz="1.0"/>
-         </inertial>
-      </link>
-      <link name="${name}_con4">
-         <visual>
-            <origin rpy="0 0 0" xyz="0 0 0.05"/>
-            <geometry>
-               <cylinder length="0.1" radius="0.06"/>
-            </geometry>
-            <material name="black"/>
-         </visual>
-         <collision>
-            <geometry>
-               <cylinder length="0.1" radius="0.06"/>
-            </geometry>
-         </collision>
-         <inertial>
-            <mass value="0.5"/>
-            <inertia ixx="1.0" ixy="0.0" ixz="0.0" iyy="1.0" iyz="0.0" izz="1.0"/>
-         </inertial>
-      </link>
-      <joint name="${name}_fixed_1" type="fixed">
-         <parent link="${name}_con1"/>
-         <child link="${name}"/>
-         <axis rpy="0 0 0" xyz="0 0 1"/>
-         <origin rpy="0 0 0" xyz="0 0 0.1"/>
-      </joint>
-      <joint name="${name}_fixed_2" type="fixed">
-         <parent link="${name}"/>
-         <child link="${name}_con2"/>
-         <axis rpy="0 0 0" xyz="0 0 1"/>
-         <origin rpy="1.57 0 0" xyz="0 -0.2 0.2"/>
-      </joint>
-      <joint name="${name}_fixed_3" type="fixed">
-         <parent link="${name}"/>
-         <child link="${name}_con3"/>
-         <axis rpy="0 0 0" xyz="0 0 1"/>
-         <origin rpy="0 0 0" xyz="0 0 0.4"/>
-      </joint>
-      <joint name="${name}_fixed_4" type="fixed">
-         <parent link="${name}"/>
-         <child link="${name}_con4"/>
-         <axis rpy="0 0 0" xyz="0 0 1"/>
-         <origin rpy="-1.57 0 0" xyz="0 0.2 0.2"/>
-      </joint>
-   </xacro:macro>
-   <xacro:macro name="add_link" params="name type size_z size">
-      <xacro:if value="${size==1}">
-         <xacro:property name="radius" value="${size1}"/>
-      </xacro:if>
-      <xacro:unless value="${size==1}">
-         <xacro:if value="${size==2}">
-            <xacro:property name="radius" value="${size2}"/>
-         </xacro:if>
-         <xacro:unless value="${size==2}">
-            <xacro:property name="radius" value="${size3}"/>
-         </xacro:unless>
-      </xacro:unless>
-      <link name="${name}">
-         <visual>
-            <origin rpy="0 0 0" xyz="0 0 ${size_z/2}"/>
-            <geometry>
-               <cylinder length="${size_z}" radius="${radius}"/>
-            </geometry>
-            <material name="black"/>
-         </visual>
-         <collision>
-            <origin rpy="0 0 0" xyz="0 0 ${size_z/2}"/>
-            <geometry>
-               <cylinder length="${size_z}" radius="${radius}"/>
-            </geometry>
-         </collision>
-         <inertial>
-            <origin rpy="0 0 0" xyz="0 0 ${size_z/2}"/>
-            <mass value="${mass}"/>
-            <inertia ixx="${mass / 12.0 * (3*radius*radius + size_z*size_z)}" ixy="0.0" ixz="0.0" iyy="${mass / 12.0 * (size_z*size_z + 3*radius*radius)}" iyz="0.0" izz="${mass / 2.0 * (radius*radius)}"/>
-         </inertial>
-      </link>
-      <gazebo reference="${name}">
-         <mu1>0.2</mu1>
-         <mu2>0.2</mu2>
-         <kp>1000000.0</kp>
-         <kd>1.0</kd>
-         <maxVel>0.0</maxVel>
-         <minDepth>0.0001</minDepth>
-         <material>Gazebo/White</material>
-      </gazebo>
-   </xacro:macro>
-   <xacro:macro name="add_size_adapter" params="type name size_z size_in size_out">
-      <xacro:if value="${size_in==3}">
-         <xacro:property name="radius1" value="${size3}"/>
-      </xacro:if>
-      <xacro:unless value="${size_in==3}">
-         <xacro:if value="${size_in==2}">
-            <xacro:property name="radius1" value="${size2}"/>
-         </xacro:if>
-         <xacro:unless value="${size_in==2}">
-            </xacro:unless>
-      </xacro:unless>
-      <xacro:if value="${size_out==3}">
-        </xacro:if>
-      <xacro:unless value="${size_out==3}">
-         <xacro:if value="${size_out==2}">
-            <xacro:property name="radius2" value="${size2}"/>
-         </xacro:if>
-         <xacro:unless value="${size_out==2}">
-            <xacro:property name="radius2" value="${size1}"/>
-         </xacro:unless>
-      </xacro:unless>
-      <link name="${name}">
-         <visual>
-            <origin rpy="0 0 0" xyz="0 0 ${size_z/4}"/>
-            <geometry>
-               <cylinder length="${size_z/2}" radius="${radius1}"/>
-            </geometry>
-            <material name="grey"/>
-         </visual>
-         <visual>
-            <origin rpy="0 0 0" xyz="0 0 ${3*size_z/4}"/>
-            <geometry>
-               <cylinder length="${size_z/2}" radius="${radius2}"/>
-            </geometry>
-            <material name="grey"/>
-         </visual>
-         <collision>
-            <origin rpy="0 0 0" xyz="0 0 ${size_z/4}"/>
-            <geometry>
-               <cylinder length="${size_z/2}" radius="${radius1}"/>
-            </geometry>
-         </collision>
-         <collision>
-            <origin rpy="0 0 0" xyz="0 0 ${3*size_z/4}"/>
-            <geometry>
-               <cylinder length="${size_z/2}" radius="${radius2}"/>
-            </geometry>
-         </collision>
-         <inertial>
-            <origin rpy="0 0 0" xyz="0 0 ${size_z/2}"/>
-            <mass value="${mass}"/>
-            <inertia ixx="${mass / 12.0 * (3*radius1*radius1 + 4*size_z/2*size_z/2) + mass / 12.0 * (3*radius2*radius2 + 4*size_z/2*size_z/2)}" ixy="0.0" ixz="0.0" iyy="${mass / 12.0 * (3*radius1*radius1 + 4*size_z/2*size_z/2) + mass / 12.0 * (3*radius2*radius2 + 4*size_z/2*size_z/2)}" iyz="0.0" izz="${mass / 4.0 * (radius1*radius1) + mass / 4.0 * (radius2*radius2)}"/>
-         </inertial>
-      </link>
-      <gazebo reference="${name}">
-         <mu1>0.2</mu1>
-         <mu2>0.2</mu2>
-         <kp>1000000.0</kp>
-         <kd>1.0</kd>
-         <maxVel>0.0</maxVel>
-         <minDepth>0.0001</minDepth>
-         <material>Gazebo/Grey</material>
-      </gazebo>
-   </xacro:macro>
-   <xacro:macro name="add_elbow" params="type name size_y size_z size">
-      <xacro:if value="${size==1}">
-         <xacro:property name="radius" value="${size1}"/>
-      </xacro:if>
-      <xacro:unless value="${size==1}">
-         <xacro:if value="${size==2}">
-            <xacro:property name="radius" value="${size2}"/>
-         </xacro:if>
-         <xacro:unless value="${size==2}">
-            <xacro:property name="radius" value="${size3}"/>
-         </xacro:unless>
-      </xacro:unless>
-      <link name="${name}">
-         <visual>
-            <origin rpy="0 0 0" xyz="0 0 ${size_z/2}"/>
-            <geometry>
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