Commit message: update ModularBot files used for control

File: urdf/ModularBot.urdf.xacro (robot description, xacro)
@@ -1,9 +1,14 @@
 <?xml version="1.0" ?>
+<!-- =================================================================================== -->
+<!-- |    This document was autogenerated by xacro from /home/edoardo/advr-superbuild/external/modular/urdf/ModularBot_test.urdf.xacro | -->
+<!-- |    EDITING THIS FILE BY HAND IS NOT RECOMMENDED                                 | -->
+<!-- =================================================================================== -->
 <robot name="ModularBot" xmlns:xacro="http://ros.org/wiki/xacro">
-  <xacro:include filename="$(find modular)/urdf/config.xacro"/>
-  <xacro:if value="${GAZEBO}">
-    <xacro:include filename="$(find modular)/urdf/modular.gazebo"/>
-  </xacro:if>
-   <material name="blue">
+  <gazebo>
+    <plugin filename="libGazeboXBotPlugin.so" name="gazebo_xbot_plugin">
+      <path_to_config_file>configs/ADVR_shared/ModularBot/configs/config_ModularBot.yaml</path_to_config_file>
+    </plugin>
+  </gazebo>
+  <material name="blue">
     <color rgba="0 0 0.8 1"/>
   </material>
@@ -18,52 +23,51 @@
   </material>
   <link name="world"/>
+  <joint name="world" type="fixed">
+    <parent link="world"/>
+    <child link="base_link"/>
+  </joint>
+  <link name="base_link"/>
   <joint name="fixed" type="fixed">
-    <parent link="world"/>
-    <child link="L_0a"/>
-  </joint>
-  <!-- <link name="base_link">
-    <visual>
-      <origin rpy="0 0 0" xyz="0 0 0.05"/>
-      <geometry>
-        <cylinder length="0.1" radius="0.06"/>
-      </geometry>
-      <material name="black"/>
-    </visual>
-    <collision>
-      <geometry>
-        <cylinder length="0.1" radius="0.06"/>
-      </geometry>
-    </collision>
-    <inertial>
-      <mass value="0.5"/>
-      <inertia ixx="1.0" ixy="0.0" ixz="0.0" iyy="1.0" iyz="0.0" izz="1.0"/>
-    </inertial>
-  </link>
-  <joint name="J0" type="revolute">
     <parent link="base_link"/>
     <child link="L_0a"/>
     <axis rpy="0 0 0" xyz="0 0 1"/>
-    <origin rpy="0.0 0.0 0.0" xyz="0.0 0.0 0.1"/>
-    <limit effort="35" lower="-0.001" upper="0.001" velocity="5.7"/>
-  </joint> -->
+    <origin rpy="0.0 0.0 0.0" xyz="0.0 0.0 0.0"/>
+  </joint>
   <link name="L_0a">
     <visual>
-      <origin rpy="0 0 0" xyz="0 0 1"/>
-      <geometry>
-        <box size="0.4 0.4 2"/>
-      </geometry>
-      <material name="black"/>
-    </visual>
-    <collision>
-      <origin rpy="0 0 0" xyz="0 0 1"/>
-      <geometry>
-        <box size="0.4 0.4 2"/>
-      </geometry>
-    </collision>
-    <inertial>
-      <mass value="50"/>
+      <origin rpy="0 0 0" xyz="0 0 0.2"/>
+      <geometry>
+        <box size="0.4 0.4 0.4"/>
+      </geometry>
+      <material name="black"/>
+    </visual>
+    <collision>
+      <geometry>
+        <box size="0.4 0.4 0.4"/>
+      </geometry>
+    </collision>
+    <inertial>
+      <mass value="2"/>
       <inertia ixx="1.0" ixy="0.0" ixz="0.0" iyy="1.0" iyz="0.0" izz="1.0"/>
     </inertial>
   </link>
+  <link name="L_0a_con1">
+    <visual>
+      <origin rpy="0 0 0" xyz="0 0 0.05"/>
+      <geometry>
+        <cylinder length="0.1" radius="0.06"/>
+      </geometry>
+      <material name="black"/>
+    </visual>
+    <collision>
+      <geometry>
+        <cylinder length="0.1" radius="0.06"/>
+      </geometry>
+    </collision>
+    <inertial>
+      <mass value="0.5"/>
+      <inertia ixx="1.0" ixy="0.0" ixz="0.0" iyy="1.0" iyz="0.0" izz="1.0"/>
+    </inertial>
+  </link>
   <link name="L_0a_con2">
     <visual>
@@ -75,8 +79,25 @@
     </visual>
     <collision>
+      <geometry>
+        <cylinder length="0.1" radius="0.06"/>
+      </geometry>
+    </collision>
+    <inertial>
+      <mass value="0.5"/>
+      <inertia ixx="1.0" ixy="0.0" ixz="0.0" iyy="1.0" iyz="0.0" izz="1.0"/>
+    </inertial>
+  </link>
+  <link name="L_0a_con3">
+    <visual>
       <origin rpy="0 0 0" xyz="0 0 0.05"/>
       <geometry>
         <cylinder length="0.1" radius="0.06"/>
       </geometry>
+      <material name="black"/>
+    </visual>
+    <collision>
+      <geometry>
+        <cylinder length="0.1" radius="0.06"/>
+      </geometry>
     </collision>
     <inertial>
@@ -94,5 +115,4 @@
     </visual>
     <collision>
-      <origin rpy="0 0 0" xyz="0 0 0.05"/>
       <geometry>
         <cylinder length="0.1" radius="0.06"/>
@@ -104,9 +124,21 @@
     </inertial>
   </link>
+  <joint name="L_0a_fixed_1" type="fixed">
+    <parent link="L_0a"/>
+    <child link="L_0a_con1"/>
+    <axis rpy="0 0 0" xyz="0 0 1"/>
+    <origin rpy="3.14 0 0" xyz="0 0 0.0"/>
+  </joint>
   <joint name="L_0a_fixed_2" type="fixed">
     <parent link="L_0a"/>
     <child link="L_0a_con2"/>
     <axis rpy="0 0 0" xyz="0 0 1"/>
-    <origin rpy="1.57 3.14 0" xyz="0 -0.2 1.8"/>
+    <origin rpy="1.57 0 0" xyz="0 -0.2 0.2"/>
+  </joint>
+  <joint name="L_0a_fixed_3" type="fixed">
+    <parent link="L_0a"/>
+    <child link="L_0a_con3"/>
+    <axis rpy="0 0 0" xyz="0 0 1"/>
+    <origin rpy="0 0 0" xyz="0 0 0.4"/>
   </joint>
   <joint name="L_0a_fixed_4" type="fixed">
@@ -114,22 +146,221 @@
     <child link="L_0a_con4"/>
     <axis rpy="0 0 0" xyz="0 0 1"/>
-    <origin rpy="-1.57 0 0" xyz="0 0.2 1.8"/>
-  </joint>
-  <gazebo reference="L_0a">
-    <mu1>1000000</mu1>
-    <mu2>1000000</mu2>
-    <kp>1000000000.0</kp>
-    <kd>1.0</kd>
-    <maxVel>0.0</maxVel>
-    <minDepth>0.0001</minDepth>
-  </gazebo>
-  <!-- <joint name="J1_A" type="revolute">
+    <origin rpy="-1.57 0 0" xyz="0 0.2 0.2"/>
+  </joint>
+  <joint name="fixed_J1_A" type="fixed">
     <axis rpy="0 0 0" xyz="0 0 1"/>
     <parent link="L_0a_con4"/>
-    <child link="L_1_elbow_1_A"/>
-    <origin rpy="0.0 0.0 0.0" xyz="0.0 0.0 0.1"/>
-    <limit effort="300" lower="-3.14" upper="3.14" velocity="5.7"/>
-  </joint>
-  <link name="L_1_elbow_1_A">
+    <child link="J1_A_stator"/>
+    <origin rpy="0.0 -0.0 0.0" xyz="0.0 0.0 0.1"/>
+  </joint>
+  <link name="J1_A_stator">
+    <visual>
+      <origin rpy="3.14 0 1.57" xyz="0 0 0"/>
+      <geometry>
+        <mesh filename="package://modular/meshes/asm0001.stl" scale="0.001 0.001 0.001"/>
+      </geometry>
+    </visual>
+    <collision>
+      <origin rpy="3.14 0 1.57" xyz="0 0 0"/>
+      <geometry>
+        <mesh filename="package://modular/meshes/asm0001.stl" scale="0.001 0.001 0.001"/>
+      </geometry>
+    </collision>
+    <inertial>
+      <origin rpy="3.14 0 1.57" xyz="0 0 0.0296308777857"/>
+      <mass value="0.5"/>
+      <inertia ixx="0.0023807995811" ixy="0.0" ixz="0.0" iyy="0.00184565189114" iyz="0.0" izz="0.00143514768996"/>
+    </inertial>
+  </link>
+  <gazebo reference="J1_A_stator">
+    <mu1>0.2</mu1>
+    <mu2>0.2</mu2>
+    <kp>1000000.0</kp>
+    <kd>1.0</kd>
+    <maxVel>0.0</maxVel>
+    <minDepth>0.0001</minDepth>
+    <material>Gazebo/Blue</material>
+  </gazebo>
+  <joint name="J1_A" type="revolute">
+    <axis rpy="0 0 0" xyz="0 0 1"/>
+    <parent link="J1_A_stator"/>
+    <child link="L_1_A"/>
+    <origin rpy="-1.57 -0.0 0.0" xyz="0.0 0.0955079697175 0.0592617555715"/>
+    <limit effort="35" lower="-3.14" upper="3.14" velocity="5.7"/>
+  </joint>
+  <link name="L_1_A">
+    <inertial>
+      <origin rpy="0 0 0" xyz="0 0 -0.0635"/>
+      <mass value="0.5"/>
+      <inertia ixx="0.00268816666667" ixy="0.0" ixz="0.0" iyy="0.00268816666667" iyz="0.0" izz="0.0000148"/>
+    </inertial>
+  </link>
+  <link name="L_1_link_1_A">
+    <visual>
+      <origin rpy="0 0 0" xyz="0 0 0.15"/>
+      <geometry>
+        <cylinder length="0.3" radius="0.06"/>
+      </geometry>
+      <material name="black"/>
+    </visual>
+    <collision>
+      <origin rpy="0 0 0" xyz="0 0 0.15"/>
+      <geometry>
+        <cylinder length="0.3" radius="0.06"/>
+      </geometry>
+    </collision>
+    <inertial>
+      <origin rpy="0 0 0" xyz="0 0 0.15"/>
+      <mass value="0.5"/>
+      <inertia ixx="0.0042" ixy="0.0" ixz="0.0" iyy="0.0042" iyz="0.0" izz="0.0009"/>
+    </inertial>
+  </link>
+  <gazebo reference="L_1_link_1_A">
+    <mu1>0.2</mu1>
+    <mu2>0.2</mu2>
+    <kp>1000000.0</kp>
+    <kd>1.0</kd>
+    <maxVel>0.0</maxVel>
+    <minDepth>0.0001</minDepth>
+    <material>Gazebo/White</material>
+  </gazebo>
+  <joint name="L_1_fixed_joint_1_A" type="fixed">
+    <axis rpy="0 0 0" xyz="0 0 1"/>
+    <parent link="L_1_A"/>
+    <child link="L_1_link_1_A"/>
+    <origin rpy="0.0 -0.0 0.0" xyz="0.0 0.0 0.0"/>
+  </joint>
+  <joint name="fixed_J2_A" type="fixed">
+    <axis rpy="0 0 0" xyz="0 0 1"/>
+    <parent link="L_1_link_1_A"/>
+    <child link="J2_A_stator"/>
+    <origin rpy="0.0 -0.0 0.0" xyz="0.0 0.0 0.3"/>
+  </joint>
+  <link name="J2_A_stator">
+    <visual>
+      <origin rpy="3.14 0 1.57" xyz="0 0 0"/>
+      <geometry>
+        <mesh filename="package://modular/meshes/asm0001.stl" scale="0.001 0.001 0.001"/>
+      </geometry>
+    </visual>
+    <collision>
+      <origin rpy="3.14 0 1.57" xyz="0 0 0"/>
+      <geometry>
+        <mesh filename="package://modular/meshes/asm0001.stl" scale="0.001 0.001 0.001"/>
+      </geometry>
+    </collision>
+    <inertial>
+      <origin rpy="3.14 0 1.57" xyz="0 0 0.0296308777857"/>
+      <mass value="0.5"/>
+      <inertia ixx="0.0023807995811" ixy="0.0" ixz="0.0" iyy="0.00184565189114" iyz="0.0" izz="0.00143514768996"/>
+    </inertial>
+  </link>
+  <gazebo reference="J2_A_stator">
+    <mu1>0.2</mu1>
+    <mu2>0.2</mu2>
+    <kp>1000000.0</kp>
+    <kd>1.0</kd>
+    <maxVel>0.0</maxVel>
+    <minDepth>0.0001</minDepth>
+    <material>Gazebo/Blue</material>
+  </gazebo>
+  <joint name="J2_A" type="revolute">
+    <axis rpy="0 0 0" xyz="0 0 1"/>
+    <parent link="J2_A_stator"/>
+    <child link="L_2_A"/>
+    <origin rpy="-1.57 -0.0 0.0" xyz="0.0 0.0955079697175 0.0592617555715"/>
+    <limit effort="35" lower="-3.14" upper="3.14" velocity="5.7"/>
+  </joint>
+  <link name="L_2_A">
+    <inertial>
+      <origin rpy="0 0 0" xyz="0 0 -0.0635"/>
+      <mass value="0.5"/>
+      <inertia ixx="0.00268816666667" ixy="0.0" ixz="0.0" iyy="0.00268816666667" iyz="0.0" izz="0.0000148"/>
+    </inertial>
+  </link>
+  <link name="L_2_link_1_A">
+    <visual>
+      <origin rpy="0 0 0" xyz="0 0 0.15"/>
+      <geometry>
+        <cylinder length="0.3" radius="0.06"/>
+      </geometry>
+      <material name="black"/>
+    </visual>
+    <collision>
+      <origin rpy="0 0 0" xyz="0 0 0.15"/>
+      <geometry>
+        <cylinder length="0.3" radius="0.06"/>
+      </geometry>
+    </collision>
+    <inertial>
+      <origin rpy="0 0 0" xyz="0 0 0.15"/>
+      <mass value="0.5"/>
+      <inertia ixx="0.0042" ixy="0.0" ixz="0.0" iyy="0.0042" iyz="0.0" izz="0.0009"/>
+    </inertial>
+  </link>
+  <gazebo reference="L_2_link_1_A">
+    <mu1>0.2</mu1>
+    <mu2>0.2</mu2>
+    <kp>1000000.0</kp>
+    <kd>1.0</kd>
+    <maxVel>0.0</maxVel>
+    <minDepth>0.0001</minDepth>
+    <material>Gazebo/White</material>
+  </gazebo>
+  <joint name="L_2_fixed_joint_1_A" type="fixed">
+    <axis rpy="0 0 0" xyz="0 0 1"/>
+    <parent link="L_2_A"/>
+    <child link="L_2_link_1_A"/>
+    <origin rpy="0.0 -0.0 0.0" xyz="0.0 0.0 0.0"/>
+  </joint>
+  <joint name="fixed_J3_A" type="fixed">
+    <axis rpy="0 0 0" xyz="0 0 1"/>
+    <parent link="L_2_link_1_A"/>
+    <child link="J3_A_stator"/>
+    <origin rpy="0.0 -0.0 0.0" xyz="0.0 0.0 0.3"/>
+  </joint>
+  <link name="J3_A_stator">
+    <visual>
+      <origin rpy="3.14 0 1.57" xyz="0 0 0"/>
+      <geometry>
+        <mesh filename="package://modular/meshes/asm0001.stl" scale="0.001 0.001 0.001"/>
+      </geometry>
+    </visual>
+    <collision>
+      <origin rpy="3.14 0 1.57" xyz="0 0 0"/>
+      <geometry>
+        <mesh filename="package://modular/meshes/asm0001.stl" scale="0.001 0.001 0.001"/>
+      </geometry>
+    </collision>
+    <inertial>
+      <origin rpy="3.14 0 1.57" xyz="0 0 0.0296308777857"/>
+      <mass value="0.5"/>
+      <inertia ixx="0.0023807995811" ixy="0.0" ixz="0.0" iyy="0.00184565189114" iyz="0.0" izz="0.00143514768996"/>
+    </inertial>
+  </link>
+  <gazebo reference="J3_A_stator">
+    <mu1>0.2</mu1>
+    <mu2>0.2</mu2>
+    <kp>1000000.0</kp>
+    <kd>1.0</kd>
+    <maxVel>0.0</maxVel>
+    <minDepth>0.0001</minDepth>
+    <material>Gazebo/Blue</material>
+  </gazebo>
+  <joint name="J3_A" type="revolute">
+    <axis rpy="0 0 0" xyz="0 0 1"/>
+    <parent link="J3_A_stator"/>
+    <child link="L_3_A"/>
+    <origin rpy="-1.57 -0.0 0.0" xyz="0.0 0.0955079697175 0.0592617555715"/>
+    <limit effort="35" lower="-3.14" upper="3.14" velocity="5.7"/>
+  </joint>
+  <link name="L_3_A">
+    <inertial>
+      <origin rpy="0 0 0" xyz="0 0 -0.0635"/>
+      <mass value="0.5"/>
+      <inertia ixx="0.00268816666667" ixy="0.0" ixz="0.0" iyy="0.00268816666667" iyz="0.0" izz="0.0000148"/>
+    </inertial>
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