Commit message: Fixed problem with straight links on Gazebo
- straight links do not throw an error anymore on Gazebo
- also, added <gazebo> element tags in the urdf to improve simulation

File: urdf/ModularBot_new.urdf.xacro (robot description, xacro)
@@ -6,4 +6,5 @@
     <xacro:property name="len2" value="0.6" />
     <xacro:property name="len3" value="0.8" />
+    <xacro:property name="mass" value="1" />
     <!-- <xacro:property name="pi" value="3.1415" /> -->
     <material name="blue">
@@ -48,5 +49,5 @@
         <child link="link_0"/>
     </joint>
-    <xacro:macro name="add_link" params="suffix size_y size_z">
+    <xacro:macro name="add_link" params="suffix size_z">
         <link name="link_${suffix}">
             <visual>
@@ -55,4 +56,5 @@
                     <box size="${width} ${width} ${size_z}"/>
                 </geometry>
+                <material name="black"/>
                 <!-- <xacro:if value="${suffix%2==0}">
                     <material name="white"/>
@@ -62,4 +64,44 @@
                 </xacro:unless> -->
             </visual>
+            <collision>
+                <origin xyz="0 0 ${size_z/2}" rpy="0 0 0" />
+                <geometry>
+                    <box size="${width} ${width} ${size_z}"/>
+                </geometry>
+            </collision>
+            <inertial>
+                <origin xyz="0 0 ${size_z/2}" rpy="0 0 0"/>
+                <mass value="${mass}"/>
+                <inertia
+                ixx="${mass / 12.0 * (width*width + size_z*size_z)}" ixy="0.0" ixz="0.0"
+                iyy="${mass / 12.0 * (size_z*size_z + width*width)}" iyz="0.0"
+                izz="${mass / 12.0 * (width*width + width*width)}"/>
+            </inertial>
+        </link>
+        <gazebo reference="link_${suffix}">
+            <mu1>0.2</mu1>
+            <mu2>0.2</mu2>
+            <kp>1000000.0</kp>
+            <kd>1.0</kd>
+            <maxVel>0.0</maxVel>
+            <minDepth>0.0001</minDepth>
+            <material>Gazebo/White</material>
+        </gazebo>
+    </xacro:macro>
+    <xacro:macro name="add_elbow" params="suffix size_y size_z">
+        <link name="link_${suffix}">
+            <visual>
+                <origin xyz="0 0 ${size_z/2}" rpy="0 0 0" />
+                <geometry>
+                    <box size="${width} ${width} ${size_z}"/>
+                </geometry>
+                <material name="white"/>
+                <!-- <xacro:if value="${suffix%2==0}">
+                    <material name="white"/>
+                </xacro:if>
+                <xacro:unless value="${suffix%2==0}">
+                    <material name="blue"/>
+                </xacro:unless> -->
+            </visual>
             <visual>
                 <origin xyz="0 ${size_y/2} ${size_z}" rpy="0 0 0" />
@@ -67,4 +109,5 @@
                 <box size="${width} ${size_y} ${width}"/>
                 </geometry>
+                <material name="white"/>
                 <!-- <xacro:if value="${suffix%2==0}">
                     <material name="white"/>
@@ -80,5 +123,12 @@
                 </geometry>
             </collision>
-            <xacro:default_inertial mass="1"/>
+            <inertial>
+                <origin xyz="0 0 ${size_z/2}" rpy="0 0 0"/>
+                <mass value="${mass}"/>
+                <inertia
+                ixx="${mass / 12.0 * (width*width + size_z*size_z)}" ixy="0.0" ixz="0.0"
+                iyy="${mass / 12.0 * (size_z*size_z + width*width)}" iyz="0.0"
+                izz="${mass / 12.0 * (width*width + width*width)}"/>
+            </inertial>
             <collision>
                 <origin xyz="0 ${size_y/2} ${size_z}" rpy="0 0 0" />
@@ -88,7 +138,16 @@
             </collision>
         </link>
+        <gazebo reference="link_${suffix}">
+            <mu1>0.2</mu1>
+            <mu2>0.2</mu2>
+            <kp>1000000.0</kp>
+            <kd>1.0</kd>
+            <maxVel>0.0</maxVel>
+            <minDepth>0.0001</minDepth>
+            <material>Gazebo/White</material>
+        </gazebo>
     </xacro:macro>
     <xacro:macro name="add_fixed_joint" params="suffix x y z roll pitch yaw">
-        <joint name="fixed_joint_${suffix}_bis" type="fixed">
+        <joint name="fixed_joint_${suffix}" type="fixed">
             <axis xyz="0 0 1" rpy="0 0 0" />
             <parent link="link_${suffix}"/>
@@ -123,9 +182,25 @@
                 </geometry>
             </collision>
-            <xacro:default_inertial mass="1"/>
-        </link>
+            <inertial>
+                <origin xyz="0 0 ${size_z/2}" rpy="0 0 0"/>
+                <mass value="${mass}"/>
+                <inertia
+                ixx="${mass / 12.0 * (width*width + size_z*size_z)}" ixy="0.0" ixz="0.0"
+                iyy="${mass / 12.0 * (size_z*size_z + width*width)}" iyz="0.0"
+                izz="${mass / 12.0 * (width*width + width*width)}"/>
+            </inertial>
+        </link>
+        <gazebo reference="link_stator_joint_${suffix}">
+            <mu1>0.2</mu1>
+            <mu2>0.2</mu2>
+            <kp>1000000.0</kp>
+            <kd>1.0</kd>
+            <maxVel>0.0</maxVel>
+            <minDepth>0.0001</minDepth>
+            <material>Gazebo/Blue</material>
+        </gazebo>
     </xacro:macro>
     <xacro:macro name="add_fixed_joint_stator" params="suffix suffix_bis x y z roll pitch yaw">
-        <joint name="fixed_joint_${suffix_bis}_bis" type="fixed">
+        <joint name="fixed_joint_${suffix_bis}" type="fixed">
             <axis xyz="0 0 1" rpy="0 0 0" />
             <parent link="link_${suffix_bis}"/>

File: urdf/ModularBot_test.urdf (robot description, URDF)
Before this commit: robot ModularBot, 10 links, 9 joints
Links:
- added link link_1_bis, mass 1; collision box size=0.1 0.1 0.3; visual box size=0.1 0.1 0.3
- added link link_2_bis, mass 1; collision box size=0.1 0.1 0.3; visual box size=0.1 0.1 0.3
Joints:
- removed joint fixed_joint_0_bis
- removed joint fixed_joint_3_bis
- added joint fixed_joint_0: type fixed, parent link_0, child link_stator_joint_1, origin xyz=0.0 0.0 0.4 rpy=0.0 -0.0 0.0, axis 0 0 1
- added joint fixed_joint_1: type fixed, parent link_1, child link_1_bis, origin xyz=0.0 0.199999936586 0.200159265342 rpy=-1.57 -0.0 0.0, axis 0 0 1
- added joint fixed_joint_2: type fixed, parent link_2, child link_2_bis, origin xyz=0.0 0.199999936586 0.200159265342 rpy=-1.57 -0.0 0.0, axis 0 0 1
- added joint fixed_joint_3: type fixed, parent link_3, child link_3_bis, origin xyz=0.0 0.199999936586 0.200159265342 rpy=-1.57 -0.0 0.0, axis 0 0 1
- joint fixed_joint_1_bis: origin xyz=0.0 0.199999936586 0.200159265342 rpy=-1.57 -0.0 0.0 -> xyz=0.0 0.0 0.3 rpy=0.0 -0.0 0.0; parent link_1 -> link_1_bis
- joint fixed_joint_2_bis: origin xyz=0.0 0.199999936586 0.200159265342 rpy=-1.57 -0.0 0.0 -> xyz=0.0 0.0 0.3 rpy=0.0 -0.0 0.0; parent link_2 -> link_2_bis

File: urdf/ModularBot_test.urdf.xacro (robot description, xacro)
@@ -5,4 +5,5 @@
    <xacro:property name="len2" value="0.6"/>
    <xacro:property name="len3" value="0.8"/>
+   <xacro:property name="mass" value="1"/>
    <material name="blue">
       <color rgba="0 0 0.8 1"/>
@@ -20,5 +21,4 @@
       </inertial>
    </xacro:macro>
-   <link name="base_link"/>
    <link name="world"/>
    <joint name="world" type="fixed">
@@ -26,4 +26,5 @@
       <child link="base_link"/>
    </joint>
+   <link name="base_link"/>
    <link name="link_0">
       <visual>
@@ -45,5 +46,5 @@
       <child link="link_0"/>
    </joint>
-   <xacro:macro name="add_link" params="suffix size_y size_z">
+   <xacro:macro name="add_link" params="suffix size_z">
       <link name="link_${suffix}">
          <visual>
@@ -52,10 +53,5 @@
                <box size="${width} ${width} ${size_z}"/>
             </geometry>
-         </visual>
-         <visual>
-            <origin rpy="0 0 0" xyz="0 ${size_y/2} ${size_z}"/>
-            <geometry>
-               <box size="${width} ${size_y} ${width}"/>
-            </geometry>
+            <material name="black"/>
          </visual>
          <collision>
@@ -65,5 +61,47 @@
             </geometry>
          </collision>
-         <xacro:default_inertial mass="1"/>
+         <inertial>
+            <origin rpy="0 0 0" xyz="0 0 ${size_z/2}"/>
+            <mass value="${mass}"/>
+            <inertia ixx="${mass / 12.0 * (width*width + size_z*size_z)}" ixy="0.0" ixz="0.0" iyy="${mass / 12.0 * (size_z*size_z + width*width)}" iyz="0.0" izz="${mass / 12.0 * (width*width + width*width)}"/>
+         </inertial>
+      </link>
+      <gazebo reference="link_${suffix}">
+         <mu1>0.2</mu1>
+         <mu2>0.2</mu2>
+         <kp>1000000.0</kp>
+         <kd>1.0</kd>
+         <maxVel>0.0</maxVel>
+         <minDepth>0.0001</minDepth>
+         <material>Gazebo/White</material>
+      </gazebo>
+   </xacro:macro>
+   <xacro:macro name="add_elbow" params="suffix size_y size_z">
+      <link name="link_${suffix}">
+         <visual>
+            <origin rpy="0 0 0" xyz="0 0 ${size_z/2}"/>
+            <geometry>
+               <box size="${width} ${width} ${size_z}"/>
+            </geometry>
+            <material name="white"/>
+         </visual>
+         <visual>
+            <origin rpy="0 0 0" xyz="0 ${size_y/2} ${size_z}"/>
+            <geometry>
+               <box size="${width} ${size_y} ${width}"/>
+            </geometry>
+            <material name="white"/>
+         </visual>
+         <collision>
+            <origin rpy="0 0 0" xyz="0 0 ${size_z/2}"/>
+            <geometry>
+               <box size="${width} ${width} ${size_z}"/>
+            </geometry>
+         </collision>
+         <inertial>
+            <origin rpy="0 0 0" xyz="0 0 ${size_z/2}"/>
+            <mass value="${mass}"/>
+            <inertia ixx="${mass / 12.0 * (width*width + size_z*size_z)}" ixy="0.0" ixz="0.0" iyy="${mass / 12.0 * (size_z*size_z + width*width)}" iyz="0.0" izz="${mass / 12.0 * (width*width + width*width)}"/>
+         </inertial>
          <collision>
             <origin rpy="0 0 0" xyz="0 ${size_y/2} ${size_z}"/>
@@ -73,7 +111,16 @@
          </collision>
       </link>
+      <gazebo reference="link_${suffix}">
+         <mu1>0.2</mu1>
+         <mu2>0.2</mu2>
+         <kp>1000000.0</kp>
+         <kd>1.0</kd>
+         <maxVel>0.0</maxVel>
+         <minDepth>0.0001</minDepth>
+         <material>Gazebo/White</material>
+      </gazebo>
    </xacro:macro>
    <xacro:macro name="add_fixed_joint" params="suffix x y z roll pitch yaw">
-      <joint name="fixed_joint_${suffix}_bis" type="fixed">
+      <joint name="fixed_joint_${suffix}" type="fixed">
          <axis rpy="0 0 0" xyz="0 0 1"/>
          <parent link="link_${suffix}"/>
@@ -106,9 +153,22 @@
             </geometry>
          </collision>
-         <xacro:default_inertial mass="1"/>
+         <inertial>
+            <origin rpy="0 0 0" xyz="0 0 ${size_z/2}"/>
+            <mass value="${mass}"/>
+            <inertia ixx="${mass / 12.0 * (width*width + size_z*size_z)}" ixy="0.0" ixz="0.0" iyy="${mass / 12.0 * (size_z*size_z + width*width)}" iyz="0.0" izz="${mass / 12.0 * (width*width + width*width)}"/>
+         </inertial>
       </link>
+      <gazebo reference="link_stator_joint_${suffix}">
+         <mu1>0.2</mu1>
+         <mu2>0.2</mu2>
+         <kp>1000000.0</kp>
+         <kd>1.0</kd>
+         <maxVel>0.0</maxVel>
+         <minDepth>0.0001</minDepth>
+         <material>Gazebo/Blue</material>
+      </gazebo>
    </xacro:macro>
    <xacro:macro name="add_fixed_joint_stator" params="suffix suffix_bis x y z roll pitch yaw">
-      <joint name="fixed_joint_${suffix_bis}_bis" type="fixed">
+      <joint name="fixed_joint_${suffix_bis}" type="fixed">
          <axis rpy="0 0 0" xyz="0 0 1"/>
          <parent link="link_${suffix_bis}"/>
@@ -120,14 +180,18 @@
    <xacro:add_joint_stator size_y="0" size_z="0.2" suffix="1"/>
    <xacro:add_joint effort="35" lower_lim="-3.14" pitch="-0.0" roll="0.0" suffix="1" upper_lim="3.14" velocity="5.7" x="0.0" y="0.0" yaw="0.0" z="0.2"/>
-   <xacro:add_link size_y="0.2" size_z="0.2" suffix="1"/>
-   <xacro:add_fixed_joint_stator pitch="-0.0" roll="-1.57" suffix="2" suffix_bis="1" x="0.0" y="0.199999936586" yaw="0.0" z="0.200159265342"/>
+   <xacro:add_elbow size_y="0.2" size_z="0.2" suffix="1"/>
+   <xacro:add_fixed_joint pitch="-0.0" roll="-1.57" suffix="1" x="0.0" y="0.199999936586" yaw="0.0" z="0.200159265342"/>
+   <xacro:add_link size_z="0.3" suffix="1_bis"/>
+   <xacro:add_fixed_joint_stator pitch="-0.0" roll="0.0" suffix="2" suffix_bis="1_bis" x="0.0" y="0.0" yaw="0.0" z="0.3"/>
    <xacro:add_joint_stator size_y="0" size_z="0.2" suffix="2"/>
    <xacro:add_joint effort="35" lower_lim="-3.14" pitch="-0.0" roll="0.0" suffix="2" upper_lim="3.14" velocity="5.7" x="0.0" y="0.0" yaw="0.0" z="0.2"/>
-   <xacro:add_link size_y="0.2" size_z="0.2" suffix="2"/>
-   <xacro:add_fixed_joint_stator pitch="-0.0" roll="-1.57" suffix="3" suffix_bis="2" x="0.0" y="0.199999936586" yaw="0.0" z="0.200159265342"/>
+   <xacro:add_elbow size_y="0.2" size_z="0.2" suffix="2"/>
+   <xacro:add_fixed_joint pitch="-0.0" roll="-1.57" suffix="2" x="0.0" y="0.199999936586" yaw="0.0" z="0.200159265342"/>
+   <xacro:add_link size_z="0.3" suffix="2_bis"/>
+   <xacro:add_fixed_joint_stator pitch="-0.0" roll="0.0" suffix="3" suffix_bis="2_bis" x="0.0" y="0.0" yaw="0.0" z="0.3"/>
    <xacro:add_joint_stator size_y="0" size_z="0.2" suffix="3"/>
    <xacro:add_joint effort="35" lower_lim="-3.14" pitch="-0.0" roll="0.0" suffix="3" upper_lim="3.14" velocity="5.7" x="0.0" y="0.0" yaw="0.0" z="0.2"/>
-   <xacro:add_link size_y="0.2" size_z="0.2" suffix="3"/>
+   <xacro:add_elbow size_y="0.2" size_z="0.2" suffix="3"/>
    <xacro:add_fixed_joint pitch="-0.0" roll="-1.57" suffix="3" x="0.0" y="0.199999936586" yaw="0.0" z="0.200159265342"/>
-   <xacro:add_link size_y="0.2" size_z="0.2" suffix="3_bis"/>
+   <xacro:add_elbow size_y="0.2" size_z="0.2" suffix="3_bis"/>
 </robot>

Commit message: Add updateURDF method, remove kin. computations from JS
- URDF_viewer.js now receives directly the newly generated urdf from URDF_writer.py.
- The kinematic computations are now done only in Python

File: urdf/ModularBot_new.urdf.xacro (robot description, xacro)
@@ -166,4 +166,5 @@
             <limit lower="${lower_lim}" upper="${upper_lim}" effort="${effort}" velocity="${velocity}"/>
         </joint>
+        <link name="link_${suffix}"/>
     </xacro:macro>
     <xacro:macro name="add_joint_stator" params="suffix size_y size_z">
