Commit message: Add size adapters and "size logic"
Also, buttons for adding modules are shown/hidden only when is possible to add the relative module

File: urdf/ModularBot_new.urdf.xacro (robot description, xacro)
@@ -1,5 +1,7 @@
 <?xml version="1.0"?>
 <robot name="ModularBot" xmlns:xacro="http://ros.org/wiki/xacro">
-    <xacro:property name="width" value="0.1" />
+    <xacro:property name="size1" value="0.05" />
+    <xacro:property name="size2" value="0.055" />
+    <xacro:property name="size3" value="0.06" />
     <!-- <xacro:property name="leglen" value="0.3" /> -->
     <xacro:property name="len1" value="0.4" />
@@ -17,4 +19,7 @@
         <color rgba="1 1 1 1"/>
     </material>
+    <material name="grey">
+        <color rgba="0.5 0.5 0.5 1"/>
+    </material>
     <xacro:macro name="default_inertial" params="mass">
         <inertial>
@@ -23,5 +28,5 @@
         </inertial>
     </xacro:macro>
-    <!-- adding world lin for Gazebo simulation -->
+    <!-- adding world link for Gazebo simulation -->
     <link name="world"/>
     <joint name="world" type="fixed">
@@ -34,5 +39,5 @@
             <origin xyz="0 0 ${len1/2}" rpy="0 0 0" />
             <geometry>
-                <cylinder radius="${width}" length="${len1}"/>
+                <cylinder radius="${size1}" length="${len1}"/>
             </geometry>
             <material name="black"/>
@@ -40,5 +45,5 @@
         <collision>
             <geometry>
-                <cylinder radius="${width}" length="${len1}"/>
+                <cylinder radius="${size1}" length="${len1}"/>
             </geometry>
         </collision>
@@ -49,10 +54,22 @@
         <child link="link_0"/>
     </joint>
-    <xacro:macro name="add_link" params="suffix size_z">
+    <xacro:macro name="add_link" params="suffix size_z size">
+        <xacro:if value="${size==1}">
+            <xacro:property name="radius" value="${size1}" />
+        </xacro:if>
+        <xacro:unless value="${size==1}">
+            <xacro:if value="${size==2}">
+                <xacro:property name="radius" value="${size2}" />
+            </xacro:if>
+            <xacro:unless value="${size==2}">
+                <xacro:property name="radius" value="${size3}" />
+            </xacro:unless>
+        </xacro:unless>
         <link name="link_${suffix}">
             <visual>
                 <origin xyz="0 0 ${size_z/2}" rpy="0 0 0" />
                 <geometry>
-                    <box size="${width} ${width} ${size_z}"/>
+                    <!-- <box size="${radius} ${radius} ${size_z}"/> -->
+                    <cylinder radius="${radius}" length="${size_z}"/>
                 </geometry>
                 <material name="black"/>
@@ -67,5 +84,6 @@
                 <origin xyz="0 0 ${size_z/2}" rpy="0 0 0" />
                 <geometry>
-                    <box size="${width} ${width} ${size_z}"/>
+                    <!-- <box size="${radius} ${radius} ${size_z}"/> -->
+                    <cylinder radius="${radius}" length="${size_z}"/>
                 </geometry>
             </collision>
@@ -74,7 +92,7 @@
                 <mass value="${mass}"/>
                 <inertia
-                ixx="${mass / 12.0 * (width*width + size_z*size_z)}" ixy="0.0" ixz="0.0"
-                iyy="${mass / 12.0 * (size_z*size_z + width*width)}" iyz="0.0"
-                izz="${mass / 12.0 * (width*width + width*width)}"/>
+                ixx="${mass / 12.0 * (radius*radius + size_z*size_z)}" ixy="0.0" ixz="0.0"
+                iyy="${mass / 12.0 * (size_z*size_z + radius*radius)}" iyz="0.0"
+                izz="${mass / 12.0 * (radius*radius + radius*radius)}"/>
             </inertial>
         </link>
@@ -89,36 +107,47 @@
         </gazebo>
     </xacro:macro>
-    <xacro:macro name="add_elbow" params="suffix size_y size_z">
+    <xacro:macro name="add_size_adapter" params="suffix size_z size">
+        <xacro:if value="${size==3}">
+            <xacro:property name="radius1" value="${size3}" />
+            <xacro:property name="radius2" value="${size2}" />
+        </xacro:if>
+        <xacro:unless value="${size==3}">
+            <xacro:if value="${size==2}">
+                <xacro:property name="radius1" value="${size2}" />
+                <xacro:property name="radius2" value="${size1}" />
+            </xacro:if>
+            <xacro:unless value="${size==2}">
+                <!-- ERROR! -->
+            </xacro:unless>
+        </xacro:unless>
         <link name="link_${suffix}">
             <visual>
-                <origin xyz="0 0 ${size_z/2}" rpy="0 0 0" />
-                <geometry>
-                    <box size="${width} ${width} ${size_z}"/>
-                </geometry>
-                <material name="white"/>
-                <!-- <xacro:if value="${suffix%2==0}">
-                    <material name="white"/>
-                </xacro:if>
-                <xacro:unless value="${suffix%2==0}">
-                    <material name="blue"/>
-                </xacro:unless> -->
-            </visual>
-            <visual>
-                <origin xyz="0 ${size_y/2} ${size_z}" rpy="0 0 0" />
-                <geometry>
-                <box size="${width} ${size_y} ${width}"/>
-                </geometry>
-                <material name="white"/>
-                <!-- <xacro:if value="${suffix%2==0}">
-                    <material name="white"/>
-                </xacro:if>
-                <xacro:unless value="${suffix%2==0}">
-                    <material name="blue"/>
-                </xacro:unless> -->
-            </visual>
-            <collision>
-                <origin xyz="0 0 ${size_z/2}" rpy="0 0 0" />
-                <geometry>
-                    <box size="${width} ${width} ${size_z}"/>
+                <origin xyz="0 0 ${size_z/4}" rpy="0 0 0" />
+                <geometry>
+                    <!-- <box size="${radius} ${radius} ${size_z}"/> -->
+                    <cylinder radius="${radius1}" length="${size_z/2}"/>
+                </geometry>
+                <material name="grey"/>
+            </visual>
+            <visual>
+                <origin xyz="0 0 ${3*size_z/4}" rpy="0 0 0" />
+                <geometry>
+                    <!-- <box size="${radius} ${radius} ${size_z}"/> -->
+                    <cylinder radius="${radius2}" length="${size_z/2}"/>
+                </geometry>
+                <material name="grey"/>
+            </visual>
+            <collision>
+                <origin xyz="0 0 ${size_z/4}" rpy="0 0 0" />
+                <geometry>
+                    <!-- <box size="${radius} ${radius} ${size_z}"/> -->
+                    <cylinder radius="${radius1}" length="${size_z/2}"/>
+                </geometry>
+            </collision>
+            <collision>
+                <origin xyz="0 0 ${3*size_z/4}" rpy="0 0 0" />
+                <geometry>
+                    <!-- <box size="${radius} ${radius} ${size_z}"/> -->
+                    <cylinder radius="${radius2}" length="${size_z/2}"/>
                 </geometry>
             </collision>
@@ -127,12 +156,93 @@
                 <mass value="${mass}"/>
                 <inertia
-                ixx="${mass / 12.0 * (width*width + size_z*size_z)}" ixy="0.0" ixz="0.0"
-                iyy="${mass / 12.0 * (size_z*size_z + width*width)}" iyz="0.0"
-                izz="${mass / 12.0 * (width*width + width*width)}"/>
+                ixx="${mass / 12.0 * (radius1*radius1 + size_z*size_z)}" ixy="0.0" ixz="0.0"
+                iyy="${mass / 12.0 * (size_z*size_z + radius1*radius1)}" iyz="0.0"
+                izz="${mass / 12.0 * (radius1*radius1 + radius1*radius1)}"/>
             </inertial>
-            <collision>
-                <origin xyz="0 ${size_y/2} ${size_z}" rpy="0 0 0" />
-                <geometry>
-                <box size="${width} ${size_y} ${width}"/>
+        </link>
+        <gazebo reference="link_${suffix}">
+            <mu1>0.2</mu1>
+            <mu2>0.2</mu2>
+            <kp>1000000.0</kp>
+            <kd>1.0</kd>
+            <maxVel>0.0</maxVel>
+            <minDepth>0.0001</minDepth>
+            <material>Gazebo/Grey</material>
+        </gazebo>
+    </xacro:macro>
+    <xacro:macro name="add_elbow" params="suffix size_y size_z size">
+        <xacro:if value="${size==1}">
+            <xacro:property name="radius" value="${size1}" />
+        </xacro:if>
+        <xacro:unless value="${size==1}">
+            <xacro:if value="${size==2}">
+                <xacro:property name="radius" value="${size2}" />
+            </xacro:if>
+            <xacro:unless value="${size==2}">
+                <xacro:property name="radius" value="${size3}" />
+            </xacro:unless>
+        </xacro:unless>
+        <link name="link_${suffix}">
+            <visual>
+                <origin xyz="0 0 ${size_z/2}" rpy="0 0 0" />
+                <geometry>
+                    <!-- <box size="${radius} ${radius} ${size_z}"/> -->
+                    <cylinder radius="${radius}" length="${size_z}"/>
+                </geometry>
+                <material name="white"/>
+                <!-- <xacro:if value="${suffix%2==0}">
+                    <material name="white"/>
+                </xacro:if>
+                <xacro:unless value="${suffix%2==0}">
+                    <material name="blue"/>
+                </xacro:unless> -->
+            </visual>
+            <visual>
+                <origin xyz="0 ${size_y/2} ${size_z}" rpy="1.57 0 0" />
+                <geometry>
+                    <!-- <box size="${radius} ${size_y} ${radius}"/> -->
+                    <cylinder radius="${radius}" length="${size_y}"/>
+                </geometry>
+                <material name="white"/>
+                <!-- <xacro:if value="${suffix%2==0}">
+                    <material name="white"/>
+                </xacro:if>
+                <xacro:unless value="${suffix%2==0}">
+                    <material name="blue"/>
+                </xacro:unless> -->
+            </visual>
+            <visual>
+                <origin xyz="0 0 ${size_z}" rpy="0 0 0" />
+                <geometry>
+                    <sphere radius="${radius}" />
+                </geometry>
+                <material name="white"/>
+            </visual>
+            <collision>
+                <origin xyz="0 0 ${size_z/2}" rpy="0 0 0" />
+                <geometry>
+                    <!-- <box size="${radius} ${radius} ${size_z}"/> -->
+                    <cylinder radius="${radius}" length="${size_z}"/>
+                </geometry>
+            </collision>
+            <inertial>
+                <origin xyz="0 0 ${size_z/2}" rpy="0 0 0"/>
+                <mass value="${mass}"/>
+                <inertia
+                ixx="${mass / 12.0 * (radius*radius + size_z*size_z)}" ixy="0.0" ixz="0.0"
+                iyy="${mass / 12.0 * (size_z*size_z + radius*radius)}" iyz="0.0"
+                izz="${mass / 12.0 * (radius*radius + radius*radius)}"/>
+            </inertial>
+            <collision>
+                <origin xyz="0 ${size_y/2} ${size_z}" rpy="1.57 0 0" />
+                <geometry>
+                    <!-- <box size="${radius} ${size_y} ${radius}"/> -->
+                    <cylinder radius="${radius}" length="${size_y}"/>
+                </geometry>
+            </collision>
+            <collision>
+                <origin xyz="0 0 ${size_z}" rpy="0 0 0" />
+                <geometry>
+                    <sphere radius="${radius}" />
                 </geometry>
             </collision>
@@ -168,10 +278,21 @@
         <link name="link_${suffix}"/>
     </xacro:macro>
-    <xacro:macro name="add_joint_stator" params="suffix size_y size_z">
+    <xacro:macro name="add_joint_stator" params="suffix size_y size_z size">
+        <xacro:if value="${size==1}">
+            <xacro:property name="radius" value="${size1}" />
+        </xacro:if>
+        <xacro:unless value="${size==1}">
+            <xacro:if value="${size==2}">
+                <xacro:property name="radius" value="${size2}" />
+            </xacro:if>
+            <xacro:unless value="${size==2}">
+                <xacro:property name="radius" value="${size3}" />
+            </xacro:unless>
+        </xacro:unless>
         <link name="link_stator_joint_${suffix}">
             <visual>
                 <origin xyz="0 0 ${size_z/2}" rpy="0 0 0" />
                 <geometry>
-                    <cylinder radius="${width}" length="${size_z}"/>
+                    <cylinder radius="${radius}" length="${size_z}"/>
                 </geometry>
                 <material name="blue"/>
@@ -180,5 +301,5 @@
                 <origin xyz="0 0 ${size_z/2}" rpy="0 0 0" />
                 <geometry>
-                    <cylinder radius="${width}" length="${size_z}"/>
+                    <cylinder radius="${radius}" length="${size_z}"/>
                 </geometry>
             </collision>
@@ -187,7 +308,7 @@
                 <mass value="${mass}"/>
                 <inertia
-                ixx="${mass / 12.0 * (width*width + size_z*size_z)}" ixy="0.0" ixz="0.0"
-                iyy="${mass / 12.0 * (size_z*size_z + width*width)}" iyz="0.0"
-                izz="${mass / 12.0 * (width*width + width*width)}"/>
+                ixx="${mass / 12.0 * (radius*radius + size_z*size_z)}" ixy="0.0" ixz="0.0"
+                iyy="${mass / 12.0 * (size_z*size_z + radius*radius)}" iyz="0.0"
+                izz="${mass / 12.0 * (radius*radius + radius*radius)}"/>
             </inertial>
         </link>
@@ -216,5 +337,5 @@
                 <origin xyz="0 0 ${p/2}" rpy="0 0 0" />
                 <geometry>
-                <box size="${width} ${width} ${p}"/>
+                <box size="${size1} ${size1} ${p}"/>
                 </geometry>
                 <xacro:if value="${suffix%2==0}">
@@ -228,5 +349,5 @@
                 <origin xyz="0 ${n/2} ${p}" rpy="0 0 0" />
                 <geometry>
-                <box size="${width} ${n} ${width}"/>
+                <box size="${size1} ${n} ${size1}"/>
                 </geometry>
                 <xacro:if value="${suffix%2==0}">
@@ -240,5 +361,5 @@
                 <origin xyz="0 0 -0.05" rpy="0 0 0" />
                 <geometry>
-                <box size="${width} ${width} 0.1"/>
+                <box size="${size1} ${size1} 0.1"/>
                 </geometry>
                 <material name="black"/>
@@ -247,5 +368,5 @@
                 <origin xyz="0 0 ${p/2}" rpy="0 0 0" />
                 <geometry>
-                <box size="${width} ${width} ${p}"/>
+                <box size="${size1} ${size1} ${p}"/>
                 </geometry>
             </collision>
@@ -253,5 +374,5 @@
                 <origin xyz="0 ${n/2} ${p}" rpy="0 0 0" />
                 <geometry>
-                <box size="${width} ${n} ${width}"/>
+                <box size="${size1} ${n} ${size1}"/>
                 </geometry>
             </collision>
@@ -259,5 +380,5 @@
                 <origin xyz="0 0 -0.05" rpy="0 0 0" />
                 <geometry>
-                <box size="${width} ${width} 0.1"/>
+                <box size="${size1} ${size1} 0.1"/>
                 </geometry>
                 <material name="black"/>
