Commit message: Add a YAML file for each module and size combination
"size" is now a global variable used to select the correct YAML file and show the correct buttons

File: urdf/ModularBot_new.urdf.xacro (robot description, xacro)
@@ -54,4 +54,5 @@
         <child link="link_0"/>
     </joint>
+    <!-- Macro for adding a straight link -->
     <xacro:macro name="add_link" params="suffix size_z size">
         <xacro:if value="${size==1}">
@@ -70,19 +71,11 @@
                 <origin xyz="0 0 ${size_z/2}" rpy="0 0 0" />
                 <geometry>
-                    <!-- <box size="${radius} ${radius} ${size_z}"/> -->
                     <cylinder radius="${radius}" length="${size_z}"/>
                 </geometry>
                 <material name="black"/>
-                <!-- <xacro:if value="${suffix%2==0}">
-                    <material name="white"/>
-                </xacro:if>
-                <xacro:unless value="${suffix%2==0}">
-                    <material name="blue"/>
-                </xacro:unless> -->
-            </visual>
-            <collision>
-                <origin xyz="0 0 ${size_z/2}" rpy="0 0 0" />
-                <geometry>
-                    <!-- <box size="${radius} ${radius} ${size_z}"/> -->
+            </visual>
+            <collision>
+                <origin xyz="0 0 ${size_z/2}" rpy="0 0 0" />
+                <geometry>
                     <cylinder radius="${radius}" length="${size_z}"/>
                 </geometry>
@@ -92,7 +85,7 @@
                 <mass value="${mass}"/>
                 <inertia
-                ixx="${mass / 12.0 * (radius*radius + size_z*size_z)}" ixy="0.0" ixz="0.0"
-                iyy="${mass / 12.0 * (size_z*size_z + radius*radius)}" iyz="0.0"
-                izz="${mass / 12.0 * (radius*radius + radius*radius)}"/>
+                ixx="${mass / 12.0 * (3*radius*radius + size_z*size_z)}" ixy="0.0" ixz="0.0"
+                iyy="${mass / 12.0 * (size_z*size_z + 3*radius*radius)}" iyz="0.0"
+                izz="${mass / 2.0 * (radius*radius)}"/>
             </inertial>
         </link>
@@ -107,16 +100,26 @@
         </gazebo>
     </xacro:macro>
-    <xacro:macro name="add_size_adapter" params="suffix size_z size">
-        <xacro:if value="${size==3}">
+    <!-- Macro for adding a size adapter -->
+    <xacro:macro name="add_size_adapter" params="suffix size_z size_in size_out">
+        <xacro:if value="${size_in==3}">
             <xacro:property name="radius1" value="${size3}" />
-            <xacro:property name="radius2" value="${size2}" />
-        </xacro:if>
-        <xacro:unless value="${size==3}">
-            <xacro:if value="${size==2}">
+        </xacro:if>
+        <xacro:unless value="${size_in==3}">
+            <xacro:if value="${size_in==2}">
                 <xacro:property name="radius1" value="${size2}" />
+            </xacro:if>
+            <xacro:unless value="${size_in==2}">
+                <!-- ERROR! -->
+            </xacro:unless>
+        </xacro:unless>
+        <xacro:if value="${size_out==3}">
+            <!-- ERROR! -->
+        </xacro:if>
+        <xacro:unless value="${size_out==3}">
+            <xacro:if value="${size_out==2}">
+                <xacro:property name="radius2" value="${size2}" />
+            </xacro:if>
+            <xacro:unless value="${size_out==2}">
                 <xacro:property name="radius2" value="${size1}" />
-            </xacro:if>
-            <xacro:unless value="${size==2}">
-                <!-- ERROR! -->
             </xacro:unless>
         </xacro:unless>
@@ -125,5 +128,4 @@
                 <origin xyz="0 0 ${size_z/4}" rpy="0 0 0" />
                 <geometry>
-                    <!-- <box size="${radius} ${radius} ${size_z}"/> -->
                     <cylinder radius="${radius1}" length="${size_z/2}"/>
                 </geometry>
@@ -133,5 +135,4 @@
                 <origin xyz="0 0 ${3*size_z/4}" rpy="0 0 0" />
                 <geometry>
-                    <!-- <box size="${radius} ${radius} ${size_z}"/> -->
                     <cylinder radius="${radius2}" length="${size_z/2}"/>
                 </geometry>
@@ -141,5 +142,4 @@
                 <origin xyz="0 0 ${size_z/4}" rpy="0 0 0" />
                 <geometry>
-                    <!-- <box size="${radius} ${radius} ${size_z}"/> -->
                     <cylinder radius="${radius1}" length="${size_z/2}"/>
                 </geometry>
@@ -148,5 +148,4 @@
                 <origin xyz="0 0 ${3*size_z/4}" rpy="0 0 0" />
                 <geometry>
-                    <!-- <box size="${radius} ${radius} ${size_z}"/> -->
                     <cylinder radius="${radius2}" length="${size_z/2}"/>
                 </geometry>
@@ -156,7 +155,7 @@
                 <mass value="${mass}"/>
                 <inertia
-                ixx="${mass / 12.0 * (radius1*radius1 + size_z*size_z)}" ixy="0.0" ixz="0.0"
-                iyy="${mass / 12.0 * (size_z*size_z + radius1*radius1)}" iyz="0.0"
-                izz="${mass / 12.0 * (radius1*radius1 + radius1*radius1)}"/>
+                ixx="${mass / 12.0 * (3*radius1*radius1 + 4*size_z/2*size_z/2) + mass / 12.0 * (3*radius2*radius2 + 4*size_z/2*size_z/2)}" ixy="0.0" ixz="0.0"
+                iyy="${mass / 12.0 * (3*radius1*radius1 + 4*size_z/2*size_z/2) + mass / 12.0 * (3*radius2*radius2 + 4*size_z/2*size_z/2)}" iyz="0.0"
+                izz="${mass / 2.0 * (radius1*radius1) + mass / 2.0 * (radius2*radius2)}"/>
             </inertial>
         </link>
@@ -171,4 +170,5 @@
         </gazebo>
     </xacro:macro>
+    <!-- Macro for adding an elbow module (90° link) -->
     <xacro:macro name="add_elbow" params="suffix size_y size_z size">
         <xacro:if value="${size==1}">
@@ -187,28 +187,14 @@
                 <origin xyz="0 0 ${size_z/2}" rpy="0 0 0" />
                 <geometry>
-                    <!-- <box size="${radius} ${radius} ${size_z}"/> -->
                     <cylinder radius="${radius}" length="${size_z}"/>
                 </geometry>
                 <material name="white"/>
-                <!-- <xacro:if value="${suffix%2==0}">
-                    <material name="white"/>
-                </xacro:if>
-                <xacro:unless value="${suffix%2==0}">
-                    <material name="blue"/>
-                </xacro:unless> -->
             </visual>
             <visual>
                 <origin xyz="0 ${size_y/2} ${size_z}" rpy="1.57 0 0" />
                 <geometry>
-                    <!-- <box size="${radius} ${size_y} ${radius}"/> -->
                     <cylinder radius="${radius}" length="${size_y}"/>
                 </geometry>
                 <material name="white"/>
-                <!-- <xacro:if value="${suffix%2==0}">
-                    <material name="white"/>
-                </xacro:if>
-                <xacro:unless value="${suffix%2==0}">
-                    <material name="blue"/>
-                </xacro:unless> -->
             </visual>
             <visual>
@@ -222,5 +208,4 @@
                 <origin xyz="0 0 ${size_z/2}" rpy="0 0 0" />
                 <geometry>
-                    <!-- <box size="${radius} ${radius} ${size_z}"/> -->
                     <cylinder radius="${radius}" length="${size_z}"/>
                 </geometry>
@@ -237,5 +222,4 @@
                 <origin xyz="0 ${size_y/2} ${size_z}" rpy="1.57 0 0" />
                 <geometry>
-                    <!-- <box size="${radius} ${size_y} ${radius}"/> -->
                     <cylinder radius="${radius}" length="${size_y}"/>
                 </geometry>
@@ -258,18 +242,18 @@
         </gazebo>
     </xacro:macro>
+    <!-- Macro for adding a fixed joint (rigid interconnection between links) -->
     <xacro:macro name="add_fixed_joint" params="suffix x y z roll pitch yaw">
         <joint name="fixed_joint_${suffix}" type="fixed">
             <axis xyz="0 0 1" rpy="0 0 0" />
             <parent link="link_${suffix}"/>
-            <!-- <parent link="base_link"/> -->
             <child link="link_${suffix}_bis"/>
             <origin xyz="${x} ${y} ${z}" rpy="${roll} ${pitch} ${yaw}"/>
         </joint>
     </xacro:macro>
+    <!-- Macro for adding the joint (it has no size) -->
     <xacro:macro name="add_joint" params="suffix x y z roll pitch yaw upper_lim lower_lim effort velocity">
         <joint name="joint_${suffix}" type="revolute">
             <axis xyz="0 0 1" rpy="0 0 0" />
             <parent link="link_stator_joint_${suffix}"/>
-            <!-- <parent link="base_link"/> -->
             <child link="link_${suffix}"/>
             <origin xyz="${x} ${y} ${z}" rpy="${roll} ${pitch} ${yaw}"/>
@@ -278,4 +262,5 @@
         <link name="link_${suffix}"/>
     </xacro:macro>
+    <!-- Macro for adding the physical module housing the actuator -->
     <xacro:macro name="add_joint_stator" params="suffix size_y size_z size">
         <xacro:if value="${size==1}">
@@ -323,73 +308,12 @@
         </gazebo>
     </xacro:macro>
+    <!-- Macro for adding a fixed joint (rigid interconnection between links and statoric part of the joint) -->
     <xacro:macro name="add_fixed_joint_stator" params="suffix suffix_bis x y z roll pitch yaw">
         <joint name="fixed_joint_${suffix_bis}" type="fixed">
             <axis xyz="0 0 1" rpy="0 0 0" />
             <parent link="link_${suffix_bis}"/>
-            <!-- <parent link="base_link"/> -->
             <child link="link_stator_joint_${suffix}"/>
             <origin xyz="${x} ${y} ${z}" rpy="${roll} ${pitch} ${yaw}"/>
         </joint>
     </xacro:macro>
-    <!-- <xacro:macro name="add_link_elbow" params="suffix p n x y z roll pitch yaw">
-        <link name="link_${suffix}">
-            <visual>
-                <origin xyz="0 0 ${p/2}" rpy="0 0 0" />
-                <geometry>
-                <box size="${size1} ${size1} ${p}"/>
-                </geometry>
-                <xacro:if value="${suffix%2==0}">
-                    <material name="white"/>
-                </xacro:if>
-                <xacro:unless value="${suffix%2==0}">
-                    <material name="blue"/>
-                </xacro:unless>
-            </visual>
-            <visual>
-                <origin xyz="0 ${n/2} ${p}" rpy="0 0 0" />
-                <geometry>
-                <box size="${size1} ${n} ${size1}"/>
-                </geometry>
-                <xacro:if value="${suffix%2==0}">
-                    <material name="white"/>
-                </xacro:if>
-                <xacro:unless value="${suffix%2==0}">
-                    <material name="blue"/>
-                </xacro:unless>
-            </visual>
-            <visual>
-                <origin xyz="0 0 -0.05" rpy="0 0 0" />
-                <geometry>
-                <box size="${size1} ${size1} 0.1"/>
-                </geometry>
-                <material name="black"/>
-            </visual>
-            <collision>
-                <origin xyz="0 0 ${p/2}" rpy="0 0 0" />
-                <geometry>
-                <box size="${size1} ${size1} ${p}"/>
-                </geometry>
-            </collision>
-            <collision>
-                <origin xyz="0 ${n/2} ${p}" rpy="0 0 0" />
-                <geometry>
-                <box size="${size1} ${n} ${size1}"/>
-                </geometry>
-            </collision>
-            <collision>
-                <origin xyz="0 0 -0.05" rpy="0 0 0" />
-                <geometry>
-                <box size="${size1} ${size1} 0.1"/>
-                </geometry>
-                <material name="black"/>
-            </collision>
-            <xacro:default_inertial mass="1"/>
-        </link>
-        <joint name="joint_${suffix-1}_${suffix}" type="continuous">
-            <axis xyz="0 0 1" rpy="0 0 0" />
-            <parent link="link_${suffix-1}"/>
-            <child link="link_${suffix}"/>
-            <origin xyz="${x} ${y} ${z}" rpy="${roll} ${pitch} ${yaw}"/>
-        </joint>
-    </xacro:macro> -->
 </robot>

File: urdf/ModularBot_test.urdf (robot description, URDF)
Before this commit: robot ModularBot, 12 links, 11 joints
Links:
- added link link_1_bis_bis, mass 1; collision cylinder length=0.2 radius=0.06; collision cylinder length=0.2 radius=0.06
- added link link_1_bis_bis_bis, mass 1; collision cylinder length=0.05 radius=0.055; collision cylinder length=0.05 radius=0.06
- added link link_2_bis_bis, mass 1; collision cylinder length=0.7 radius=0.055; visual cylinder length=0.7 radius=0.055
- added link link_2_bis_bis_bis, mass 1; collision cylinder length=0.05 radius=0.05; collision cylinder length=0.05 radius=0.055
- link link_0: geometry collision cylinder length=0.4 radius=0.05; visual cylinder length=0.4 radius=0.05
- link link_1: mass 1 -> None; geometry 
- link link_1_bis: geometry collision cylinder length=0.2 radius=0.06; collision cylinder length=0.2 radius=0.06
- link link_2: mass 1 -> None; geometry 
- link link_2_bis: geometry collision cylinder length=0.2 radius=0.055; collision cylinder length=0.2 radius=0.055
- link link_3: mass 1 -> None; geometry 
- link link_3_bis: geometry collision cylinder length=0.2 radius=0.05; collision cylinder length=0.2 radius=0.05
- link link_stator_joint_1: geometry collision cylinder length=0.2 radius=0.06; visual cylinder length=0.2 radius=0.06
- link link_stator_joint_2: geometry collision cylinder length=0.2 radius=0.055; visual cylinder length=0.2 radius=0.055
- link link_stator_joint_3: geometry collision cylinder length=0.2 radius=0.05; visual cylinder length=0.2 radius=0.05
Joints:
- added joint fixed_joint_1_bis_bis: type fixed, parent link_1_bis_bis, child link_1_bis_bis_bis, origin xyz=0.0 0.199999936586 0.200159265342 rpy=-1.57 -0.0 0.0, axis 0 0 1
- added joint fixed_joint_1_bis_bis_bis: type fixed, parent link_1_bis_bis_bis, child link_stator_joint_2, origin xyz=0.0 0.0 0.1 rpy=0.0 -0.0 0.0, axis 0 0 1
- added joint fixed_joint_2_bis_bis: type fixed, parent link_2_bis_bis, child link_2_bis_bis_bis, origin xyz=0.0 0.0 0.7 rpy=0.0 -0.0 0.0, axis 0 0 1
- added joint fixed_joint_2_bis_bis_bis: type fixed, parent link_2_bis_bis_bis, child link_stator_joint_3, origin xyz=0.0 0.0 0.1 rpy=0.0 -0.0 0.0, axis 0 0 1
- joint fixed_joint_1: origin xyz=0.0 0.199999936586 0.200159265342 rpy=-1.57 -0.0 0.0 -> xyz=0.0 0.0 0.0 rpy=0.0 -0.0 0.0
- joint fixed_joint_1_bis: child link_stator_joint_2 -> link_1_bis_bis; origin xyz=0.0 0.0 0.3 rpy=0.0 -0.0 0.0 -> xyz=0.0 0.199999936586 0.200159265342 rpy=-1.57 -0.0 0.0
- joint fixed_joint_2: origin xyz=0.0 0.199999936586 0.200159265342 rpy=-1.57 -0.0 0.0 -> xyz=0.0 0.0 0.0 rpy=0.0 -0.0 0.0
- joint fixed_joint_2_bis: child link_stator_joint_3 -> link_2_bis_bis; origin xyz=0.0 0.0 0.3 rpy=0.0 -0.0 0.0 -> xyz=0.0 0.199999936586 0.200159265342 rpy=-1.57 -0.0 0.0
- joint fixed_joint_3: origin xyz=0.0 0.199999936586 0.200159265342 rpy=-1.57 -0.0 0.0 -> xyz=0.0 0.0 0.0 rpy=0.0 -0.0 0.0
