Commit message: Fix collisions for Gazebo sim and update inertia matrices
Also, added fields for dynamic parameters in YAML files

File: urdf/ModularBot_new.urdf.xacro (robot description, xacro)
@@ -8,5 +8,5 @@
     <xacro:property name="len2" value="0.6" />
     <xacro:property name="len3" value="0.8" />
-    <xacro:property name="mass" value="1" />
+    <xacro:property name="mass" value="0.5" />
     <!-- <xacro:property name="pi" value="3.1415" /> -->
     <material name="blue">
@@ -44,9 +44,10 @@
         </visual>
         <collision>
+            <origin xyz="0 0 ${len1/2}" rpy="0 0 0" />
             <geometry>
                 <cylinder radius="${size1}" length="${len1}"/>
             </geometry>
         </collision>
-        <xacro:default_inertial mass="10"/>
+        <xacro:default_inertial mass="1"/>
     </link>
     <joint name="fixed" type="fixed">
@@ -157,5 +158,5 @@
                 ixx="${mass / 12.0 * (3*radius1*radius1 + 4*size_z/2*size_z/2) + mass / 12.0 * (3*radius2*radius2 + 4*size_z/2*size_z/2)}" ixy="0.0" ixz="0.0"
                 iyy="${mass / 12.0 * (3*radius1*radius1 + 4*size_z/2*size_z/2) + mass / 12.0 * (3*radius2*radius2 + 4*size_z/2*size_z/2)}" iyz="0.0"
-                izz="${mass / 2.0 * (radius1*radius1) + mass / 2.0 * (radius2*radius2)}"/>
+                izz="${mass / 4.0 * (radius1*radius1) + mass / 4.0 * (radius2*radius2)}"/>
             </inertial>
         </link>
@@ -215,7 +216,7 @@
                 <mass value="${mass}"/>
                 <inertia
-                ixx="${mass / 12.0 * (radius*radius + size_z*size_z)}" ixy="0.0" ixz="0.0"
-                iyy="${mass / 12.0 * (size_z*size_z + radius*radius)}" iyz="0.0"
-                izz="${mass / 12.0 * (radius*radius + radius*radius)}"/>
+                ixx="${mass / 2 *( 1 / 12.0 * (3*radius*radius + 4*size_y*size_y) + size_z*size_z) + mass / 24.0 * (3*radius*radius + 4*size_z*size_z)}" ixy="0.0" ixz="0.0"
+                iyy="${mass / 24.0 * (3*radius*radius + 4*size_z*size_z) + mass / 2 *( 1 / 2 *radius*radius + size_z*size_z)}" iyz="0.0"
+                izz="${mass / 4.0 * (radius*radius) + mass / 24.0 * (3*radius*radius + 4*size_y*size_y)}"/>
             </inertial>
             <collision>
@@ -293,7 +294,7 @@
                 <mass value="${mass}"/>
                 <inertia
-                ixx="${mass / 12.0 * (radius*radius + size_z*size_z)}" ixy="0.0" ixz="0.0"
-                iyy="${mass / 12.0 * (size_z*size_z + radius*radius)}" iyz="0.0"
-                izz="${mass / 12.0 * (radius*radius + radius*radius)}"/>
+                ixx="${mass / 12.0 * (3*radius*radius + size_z*size_z)}" ixy="0.0" ixz="0.0"
+                iyy="${mass / 12.0 * (size_z*size_z + 3*radius*radius)}" iyz="0.0"
+                izz="${mass / 2.0 * (radius*radius)}"/>
             </inertial>
         </link>

File: urdf/ModularBot_test.urdf (robot description, URDF)
Before this commit: robot ModularBot, 17 links, 16 joints
Links:
- removed link link_3_bis_bis
- added link link_4
- added link link_4_bis, mass 0.5; collision cylinder length=0.2 radius=0.05; collision cylinder length=0.2 radius=0.05
- added link link_5
- added link link_stator_joint_4, mass 0.5; collision cylinder length=0.2 radius=0.05; visual cylinder length=0.2 radius=0.05
- added link link_stator_joint_5, mass 0.5; collision cylinder length=0.2 radius=0.05; visual cylinder length=0.2 radius=0.05
- link link_0: mass 10 -> 1
- link link_1_bis: mass 1 -> 0.5; geometry collision cylinder length=0.7 radius=0.06; visual cylinder length=0.7 radius=0.06
- link link_1_bis_bis: mass 1 -> 0.5; geometry collision cylinder length=0.2 radius=0.06; collision cylinder length=0.2 radius=0.06
- link link_1_bis_bis_bis: mass 1 -> 0.5
- link link_2_bis: mass 1 -> 0.5
- link link_2_bis_bis: mass 1 -> 0.5
- link link_2_bis_bis_bis: mass 1 -> 0.5
- link link_3_bis: mass 1 -> 0.5
- link link_stator_joint_1: mass 1 -> 0.5
- link link_stator_joint_2: mass 1 -> 0.5
- link link_stator_joint_3: mass 1 -> 0.5
Joints:
- added joint fixed_joint_4: type fixed, parent link_4, child link_4_bis, origin xyz=0.0 0.0 0.0 rpy=0.0 -0.0 0.0, axis 0 0 1
- added joint fixed_joint_4_bis: type fixed, parent link_4_bis, child link_stator_joint_5, origin xyz=0.0 0.199999936586 0.200159265342 rpy=-1.57 -0.0 0.0, axis 0 0 1
- added joint joint_4: type revolute, parent link_stator_joint_4, child link_4, origin xyz=0.0 0.0 0.2 rpy=0.0 -0.0 0.0, axis 0 0 1, limit lower=-3.14 upper=3.14 effort=35 velocity=5.7
- added joint joint_5: type revolute, parent link_stator_joint_5, child link_5, origin xyz=0.0 0.0 0.2 rpy=0.0 -0.0 0.0, axis 0 0 1, limit lower=-3.14 upper=3.14 effort=35 velocity=5.7
- joint fixed_joint_1_bis: origin xyz=0.0 0.199999936586 0.200159265342 rpy=-1.57 -0.0 0.0 -> xyz=0.0 0.0 0.7 rpy=0.0 -0.0 0.0
- joint fixed_joint_1_bis_bis: origin xyz=0.0 0.0 0.3 rpy=0.0 -0.0 0.0 -> xyz=0.0 0.199999936586 0.200159265342 rpy=-1.57 -0.0 0.0
- joint fixed_joint_3_bis: child link_3_bis_bis -> link_stator_joint_4

File: urdf/ModularBot_test.urdf.xacro (robot description, xacro)
@@ -7,5 +7,5 @@
    <xacro:property name="len2" value="0.6"/>
    <xacro:property name="len3" value="0.8"/>
-   <xacro:property name="mass" value="1"/>
+   <xacro:property name="mass" value="0.5"/>
    <material name="blue">
       <color rgba="0 0 0.8 1"/>
@@ -41,9 +41,10 @@
       </visual>
       <collision>
+         <origin rpy="0 0 0" xyz="0 0 ${len1/2}"/>
          <geometry>
             <cylinder length="${len1}" radius="${size1}"/>
          </geometry>
       </collision>
-      <xacro:default_inertial mass="10"/>
+      <xacro:default_inertial mass="1"/>
    </link>
    <joint name="fixed" type="fixed">
@@ -144,5 +145,5 @@
             <origin rpy="0 0 0" xyz="0 0 ${size_z/2}"/>
             <mass value="${mass}"/>
-            <inertia ixx="${mass / 12.0 * (3*radius1*radius1 + 4*size_z/2*size_z/2) + mass / 12.0 * (3*radius2*radius2 + 4*size_z/2*size_z/2)}" ixy="0.0" ixz="0.0" iyy="${mass / 12.0 * (3*radius1*radius1 + 4*size_z/2*size_z/2) + mass / 12.0 * (3*radius2*radius2 + 4*size_z/2*size_z/2)}" iyz="0.0" izz="${mass / 2.0 * (radius1*radius1) + mass / 2.0 * (radius2*radius2)}"/>
+            <inertia ixx="${mass / 12.0 * (3*radius1*radius1 + 4*size_z/2*size_z/2) + mass / 12.0 * (3*radius2*radius2 + 4*size_z/2*size_z/2)}" ixy="0.0" ixz="0.0" iyy="${mass / 12.0 * (3*radius1*radius1 + 4*size_z/2*size_z/2) + mass / 12.0 * (3*radius2*radius2 + 4*size_z/2*size_z/2)}" iyz="0.0" izz="${mass / 4.0 * (radius1*radius1) + mass / 4.0 * (radius2*radius2)}"/>
          </inertial>
       </link>
@@ -200,5 +201,5 @@
             <origin rpy="0 0 0" xyz="0 0 ${size_z/2}"/>
             <mass value="${mass}"/>
-            <inertia ixx="${mass / 12.0 * (radius*radius + size_z*size_z)}" ixy="0.0" ixz="0.0" iyy="${mass / 12.0 * (size_z*size_z + radius*radius)}" iyz="0.0" izz="${mass / 12.0 * (radius*radius + radius*radius)}"/>
+            <inertia ixx="${mass / 2 *( 1 / 12.0 * (3*radius*radius + 4*size_y*size_y) + size_z*size_z) + mass / 24.0 * (3*radius*radius + 4*size_z*size_z)}" ixy="0.0" ixz="0.0" iyy="${mass / 24.0 * (3*radius*radius + 4*size_z*size_z) + mass / 2 *( 1 / 2 *radius*radius + size_z*size_z)}" iyz="0.0" izz="${mass / 4.0 * (radius*radius) + mass / 24.0 * (3*radius*radius + 4*size_y*size_y)}"/>
          </inertial>
          <collision>
@@ -272,5 +273,5 @@
             <origin rpy="0 0 0" xyz="0 0 ${size_z/2}"/>
             <mass value="${mass}"/>
-            <inertia ixx="${mass / 12.0 * (radius*radius + size_z*size_z)}" ixy="0.0" ixz="0.0" iyy="${mass / 12.0 * (size_z*size_z + radius*radius)}" iyz="0.0" izz="${mass / 12.0 * (radius*radius + radius*radius)}"/>
+            <inertia ixx="${mass / 12.0 * (3*radius*radius + size_z*size_z)}" ixy="0.0" ixz="0.0" iyy="${mass / 12.0 * (size_z*size_z + 3*radius*radius)}" iyz="0.0" izz="${mass / 2.0 * (radius*radius)}"/>
          </inertial>
       </link>
@@ -297,8 +298,8 @@
    <xacro:add_joint effort="35" lower_lim="-3.14" pitch="-0.0" roll="0.0" suffix="1" upper_lim="3.14" velocity="5.7" x="0.0" y="0.0" yaw="0.0" z="0.2"/>
    <xacro:add_fixed_joint pitch="-0.0" roll="0.0" suffix="1" x="0.0" y="0.0" yaw="0.0" z="0.0"/>
-   <xacro:add_elbow size="3" size_y="0.2" size_z="0.2" suffix="1_bis"/>
-   <xacro:add_fixed_joint pitch="-0.0" roll="-1.57" suffix="1_bis" x="0.0" y="0.199999936586" yaw="0.0" z="0.200159265342"/>
-   <xacro:add_link size="3" size_z="0.3" suffix="1_bis_bis"/>
-   <xacro:add_fixed_joint pitch="-0.0" roll="0.0" suffix="1_bis_bis" x="0.0" y="0.0" yaw="0.0" z="0.3"/>
+   <xacro:add_link size="3" size_z="0.7" suffix="1_bis"/>
+   <xacro:add_fixed_joint pitch="-0.0" roll="0.0" suffix="1_bis" x="0.0" y="0.0" yaw="0.0" z="0.7"/>
+   <xacro:add_elbow size="3" size_y="0.2" size_z="0.2" suffix="1_bis_bis"/>
+   <xacro:add_fixed_joint pitch="-0.0" roll="-1.57" suffix="1_bis_bis" x="0.0" y="0.199999936586" yaw="0.0" z="0.200159265342"/>
    <xacro:add_size_adapter size_in="3" size_out="2" size_z="0.1" suffix="1_bis_bis_bis"/>
    <xacro:add_fixed_joint_stator pitch="-0.0" roll="0.0" suffix="2" suffix_bis="1_bis_bis_bis" x="0.0" y="0.0" yaw="0.0" z="0.1"/>
@@ -316,5 +317,11 @@
    <xacro:add_fixed_joint pitch="-0.0" roll="0.0" suffix="3" x="0.0" y="0.0" yaw="0.0" z="0.0"/>
    <xacro:add_elbow size="1" size_y="0.2" size_z="0.2" suffix="3_bis"/>
-   <xacro:add_fixed_joint pitch="-0.0" roll="-1.57" suffix="3_bis" x="0.0" y="0.199999936586" yaw="0.0" z="0.200159265342"/>
-   <xacro:add_link size="1" size_z="0.3" suffix="3_bis_bis"/>
+   <xacro:add_fixed_joint_stator pitch="-0.0" roll="-1.57" suffix="4" suffix_bis="3_bis" x="0.0" y="0.199999936586" yaw="0.0" z="0.200159265342"/>
+   <xacro:add_joint_stator size="1" size_y="0" size_z="0.2" suffix="4"/>
+   <xacro:add_joint effort="35" lower_lim="-3.14" pitch="-0.0" roll="0.0" suffix="4" upper_lim="3.14" velocity="5.7" x="0.0" y="0.0" yaw="0.0" z="0.2"/>
+   <xacro:add_fixed_joint pitch="-0.0" roll="0.0" suffix="4" x="0.0" y="0.0" yaw="0.0" z="0.0"/>
+   <xacro:add_elbow size="1" size_y="0.2" size_z="0.2" suffix="4_bis"/>
+   <xacro:add_fixed_joint_stator pitch="-0.0" roll="-1.57" suffix="5" suffix_bis="4_bis" x="0.0" y="0.199999936586" yaw="0.0" z="0.200159265342"/>
+   <xacro:add_joint_stator size="1" size_y="0" size_z="0.2" suffix="5"/>
+   <xacro:add_joint effort="35" lower_lim="-3.14" pitch="-0.0" roll="0.0" suffix="5" upper_lim="3.14" velocity="5.7" x="0.0" y="0.0" yaw="0.0" z="0.2"/>
 </robot>
