Commit message: Add capability to remove modules
- remove_module() in URDF_writer.py now can remove the last added module from the URDF
- updateURDF now rebuilds completely the robot at every change, so it is easier to remove modules. before it was just adding the new stuff
- the way the modules are named has been changed to deal with the removal. names are now generated in python and not in xacro

File: urdf/ModularBot_new.urdf.xacro (robot description, xacro)
@@ -35,5 +35,5 @@
     </joint>
     <link name="base_link"/>
-    <link name="link_0">
+    <link name="L_0">
         <visual>
             <origin xyz="0 0 ${len1/2}" rpy="0 0 0" />
@@ -53,8 +53,8 @@
     <joint name="fixed" type="fixed">
         <parent link="base_link"/>
-        <child link="link_0"/>
+        <child link="L_0"/>
     </joint>
     <!-- Macro for adding a straight link -->
-    <xacro:macro name="add_link" params="suffix size_z size">
+    <xacro:macro name="add_link" params="name type size_z size">
         <xacro:if value="${size==1}">
             <xacro:property name="radius" value="${size1}" />
@@ -68,5 +68,5 @@
             </xacro:unless>
         </xacro:unless>
-        <link name="link_${suffix}">
+        <link name="${name}">
             <visual>
                 <origin xyz="0 0 ${size_z/2}" rpy="0 0 0" />
@@ -91,5 +91,5 @@
             </inertial>
         </link>
-        <gazebo reference="link_${suffix}">
+        <gazebo reference="${name}">
             <mu1>0.2</mu1>
             <mu2>0.2</mu2>
@@ -102,5 +102,5 @@
     </xacro:macro>
     <!-- Macro for adding a size adapter -->
-    <xacro:macro name="add_size_adapter" params="suffix size_z size_in size_out">
+    <xacro:macro name="add_size_adapter" params="type name size_z size_in size_out">
         <xacro:if value="${size_in==3}">
             <xacro:property name="radius1" value="${size3}" />
@@ -125,5 +125,5 @@
             </xacro:unless>
         </xacro:unless>
-        <link name="link_${suffix}">
+        <link name="${name}">
             <visual>
                 <origin xyz="0 0 ${size_z/4}" rpy="0 0 0" />
@@ -161,5 +161,5 @@
             </inertial>
         </link>
-        <gazebo reference="link_${suffix}">
+        <gazebo reference="${name}">
             <mu1>0.2</mu1>
             <mu2>0.2</mu2>
@@ -172,5 +172,5 @@
     </xacro:macro>
     <!-- Macro for adding an elbow module (90° link) -->
-    <xacro:macro name="add_elbow" params="suffix size_y size_z size">
+    <xacro:macro name="add_elbow" params="type name size_y size_z size">
         <xacro:if value="${size==1}">
             <xacro:property name="radius" value="${size1}" />
@@ -184,5 +184,5 @@
             </xacro:unless>
         </xacro:unless>
-        <link name="link_${suffix}">
+        <link name="${name}">
             <visual>
                 <origin xyz="0 0 ${size_z/2}" rpy="0 0 0" />
@@ -233,5 +233,5 @@
             </collision>
         </link>
-        <gazebo reference="link_${suffix}">
+        <gazebo reference="${name}">
             <mu1>0.2</mu1>
             <mu2>0.2</mu2>
@@ -244,25 +244,25 @@
     </xacro:macro>
     <!-- Macro for adding a fixed joint (rigid interconnection between links) -->
-    <xacro:macro name="add_fixed_joint" params="suffix x y z roll pitch yaw">
-        <joint name="fixed_joint_${suffix}" type="fixed">
+    <xacro:macro name="add_fixed_joint" params="type name father child x y z roll pitch yaw">
+        <joint name="${name}" type="fixed">
             <axis xyz="0 0 1" rpy="0 0 0" />
-            <parent link="link_${suffix}"/>
-            <child link="link_${suffix}_bis"/>
+            <parent link="${father}"/>
+            <child link="${child}"/>
             <origin xyz="${x} ${y} ${z}" rpy="${roll} ${pitch} ${yaw}"/>
         </joint>
     </xacro:macro>
     <!-- Macro for adding the joint (it has no size) -->
-    <xacro:macro name="add_joint" params="suffix x y z roll pitch yaw upper_lim lower_lim effort velocity">
-        <joint name="joint_${suffix}" type="revolute">
+    <xacro:macro name="add_joint" params="type name father child x y z roll pitch yaw upper_lim lower_lim effort velocity">
+        <joint name="${name}" type="revolute">
             <axis xyz="0 0 1" rpy="0 0 0" />
-            <parent link="link_stator_joint_${suffix}"/>
-            <child link="link_${suffix}"/>
+            <parent link="${father}"/>
+            <child link="${child}"/>
             <origin xyz="${x} ${y} ${z}" rpy="${roll} ${pitch} ${yaw}"/>
             <limit lower="${lower_lim}" upper="${upper_lim}" effort="${effort}" velocity="${velocity}"/>
         </joint>
-        <link name="link_${suffix}"/>
+        <link name="${child}"/>
     </xacro:macro>
     <!-- Macro for adding the physical module housing the actuator -->
-    <xacro:macro name="add_joint_stator" params="suffix size_y size_z size">
+    <xacro:macro name="add_joint_stator" params="type name size_y size_z size">
         <xacro:if value="${size==1}">
             <xacro:property name="radius" value="${size1}" />
@@ -276,5 +276,5 @@
             </xacro:unless>
         </xacro:unless>
-        <link name="link_stator_joint_${suffix}">
+        <link name="${name}">
             <visual>
                 <origin xyz="0 0 ${size_z/2}" rpy="0 0 0" />
@@ -299,5 +299,5 @@
             </inertial>
         </link>
-        <gazebo reference="link_stator_joint_${suffix}">
+        <gazebo reference="${name}">
             <mu1>0.2</mu1>
             <mu2>0.2</mu2>
@@ -310,9 +310,9 @@
     </xacro:macro>
     <!-- Macro for adding a fixed joint (rigid interconnection between links and statoric part of the joint) -->
-    <xacro:macro name="add_fixed_joint_stator" params="suffix suffix_bis x y z roll pitch yaw">
-        <joint name="fixed_joint_${suffix_bis}" type="fixed">
+    <xacro:macro name="add_fixed_joint_stator" params="type name father child x y z roll pitch yaw">
+        <joint name="${name}" type="fixed">
             <axis xyz="0 0 1" rpy="0 0 0" />
-            <parent link="link_${suffix_bis}"/>
-            <child link="link_stator_joint_${suffix}"/>
+            <parent link="${father}"/>
+            <child link="${child}"/>
             <origin xyz="${x} ${y} ${z}" rpy="${roll} ${pitch} ${yaw}"/>
         </joint>

File: urdf/ModularBot_test.urdf (robot description, URDF)
Before this commit: robot ModularBot, 21 links, 20 joints
Links:
- removed link link_0
- removed link link_1
- removed link link_1_bis
- removed link link_1_bis_bis
- removed link link_1_bis_bis_bis
- removed link link_2
- removed link link_2_bis
- removed link link_2_bis_bis
- removed link link_2_bis_bis_bis
- removed link link_3
- removed link link_3_bis
- removed link link_4
- removed link link_4_bis
- removed link link_5
- removed link link_stator_joint_1
- removed link link_stator_joint_2
- removed link link_stator_joint_3
- removed link link_stator_joint_4
- removed link link_stator_joint_5
- added link L_0, mass 1; collision cylinder length=0.4 radius=0.05; visual cylinder length=0.4 radius=0.05
Joints:
- removed joint fixed_joint_0
- removed joint fixed_joint_1
- removed joint fixed_joint_1_bis
- removed joint fixed_joint_1_bis_bis
- removed joint fixed_joint_1_bis_bis_bis
- removed joint fixed_joint_2
- removed joint fixed_joint_2_bis
- removed joint fixed_joint_2_bis_bis
- removed joint fixed_joint_2_bis_bis_bis
- removed joint fixed_joint_3
- removed joint fixed_joint_3_bis
- removed joint fixed_joint_4
- removed joint fixed_joint_4_bis
- removed joint joint_1
- removed joint joint_2
- removed joint joint_3
- removed joint joint_4
- removed joint joint_5
- joint fixed: child link_0 -> L_0

File: urdf/ModularBot_test.urdf.xacro (robot description, xacro)
@@ -32,5 +32,5 @@
    </joint>
    <link name="base_link"/>
-   <link name="link_0">
+   <link name="L_0">
       <visual>
          <origin rpy="0 0 0" xyz="0 0 ${len1/2}"/>
@@ -50,7 +50,7 @@
    <joint name="fixed" type="fixed">
       <parent link="base_link"/>
-      <child link="link_0"/>
+      <child link="L_0"/>
    </joint>
-   <xacro:macro name="add_link" params="suffix size_z size">
+   <xacro:macro name="add_link" params="name type size_z size">
       <xacro:if value="${size==1}">
          <xacro:property name="radius" value="${size1}"/>
@@ -64,5 +64,5 @@
          </xacro:unless>
       </xacro:unless>
-      <link name="link_${suffix}">
+      <link name="${name}">
          <visual>
             <origin rpy="0 0 0" xyz="0 0 ${size_z/2}"/>
@@ -84,5 +84,5 @@
          </inertial>
       </link>
-      <gazebo reference="link_${suffix}">
+      <gazebo reference="${name}">
          <mu1>0.2</mu1>
          <mu2>0.2</mu2>
@@ -94,5 +94,5 @@
       </gazebo>
    </xacro:macro>
-   <xacro:macro name="add_size_adapter" params="suffix size_z size_in size_out">
+   <xacro:macro name="add_size_adapter" params="type name size_z size_in size_out">
       <xacro:if value="${size_in==3}">
          <xacro:property name="radius1" value="${size3}"/>
@@ -115,5 +115,5 @@
          </xacro:unless>
       </xacro:unless>
-      <link name="link_${suffix}">
+      <link name="${name}">
          <visual>
             <origin rpy="0 0 0" xyz="0 0 ${size_z/4}"/>
@@ -148,5 +148,5 @@
          </inertial>
       </link>
-      <gazebo reference="link_${suffix}">
+      <gazebo reference="${name}">
          <mu1>0.2</mu1>
          <mu2>0.2</mu2>
@@ -158,5 +158,5 @@
       </gazebo>
    </xacro:macro>
-   <xacro:macro name="add_elbow" params="suffix size_y size_z size">
+   <xacro:macro name="add_elbow" params="type name size_y size_z size">
       <xacro:if value="${size==1}">
          <xacro:property name="radius" value="${size1}"/>
@@ -170,5 +170,5 @@
          </xacro:unless>
       </xacro:unless>
-      <link name="link_${suffix}">
+      <link name="${name}">
          <visual>
             <origin rpy="0 0 0" xyz="0 0 ${size_z/2}"/>
@@ -216,5 +216,5 @@
          </collision>
       </link>
-      <gazebo reference="link_${suffix}">
+      <gazebo reference="${name}">
          <mu1>0.2</mu1>
          <mu2>0.2</mu2>
@@ -226,23 +226,23 @@
       </gazebo>
    </xacro:macro>
-   <xacro:macro name="add_fixed_joint" params="suffix x y z roll pitch yaw">
-      <joint name="fixed_joint_${suffix}" type="fixed">
+   <xacro:macro name="add_fixed_joint" params="type name father child x y z roll pitch yaw">
+      <joint name="${name}" type="fixed">
          <axis rpy="0 0 0" xyz="0 0 1"/>
-         <parent link="link_${suffix}"/>
-         <child link="link_${suffix}_bis"/>
+         <parent link="${father}"/>
+         <child link="${child}"/>
          <origin rpy="${roll} ${pitch} ${yaw}" xyz="${x} ${y} ${z}"/>
       </joint>
    </xacro:macro>
-   <xacro:macro name="add_joint" params="suffix x y z roll pitch yaw upper_lim lower_lim effort velocity">
-      <joint name="joint_${suffix}" type="revolute">
+   <xacro:macro name="add_joint" params="type name father child x y z roll pitch yaw upper_lim lower_lim effort velocity">
+      <joint name="${name}" type="revolute">
          <axis rpy="0 0 0" xyz="0 0 1"/>
-         <parent link="link_stator_joint_${suffix}"/>
-         <child link="link_${suffix}"/>
+         <parent link="${father}"/>
+         <child link="${child}"/>
          <origin rpy="${roll} ${pitch} ${yaw}" xyz="${x} ${y} ${z}"/>
          <limit effort="${effort}" lower="${lower_lim}" upper="${upper_lim}" velocity="${velocity}"/>
       </joint>
-      <link name="link_${suffix}"/>
-   </xacro:macro>
-   <xacro:macro name="add_joint_stator" params="suffix size_y size_z size">
+      <link name="${child}"/>
+   </xacro:macro>
+   <xacro:macro name="add_joint_stator" params="type name size_y size_z size">
       <xacro:if value="${size==1}">
          <xacro:property name="radius" value="${size1}"/>
@@ -256,5 +256,5 @@
          </xacro:unless>
       </xacro:unless>
-      <link name="link_stator_joint_${suffix}">
+      <link name="${name}">
          <visual>
             <origin rpy="0 0 0" xyz="0 0 ${size_z/2}"/>
@@ -276,5 +276,5 @@
          </inertial>
       </link>
-      <gazebo reference="link_stator_joint_${suffix}">
+      <gazebo reference="${name}">
          <mu1>0.2</mu1>
          <mu2>0.2</mu2>
@@ -286,42 +286,11 @@
       </gazebo>
    </xacro:macro>
-   <xacro:macro name="add_fixed_joint_stator" params="suffix suffix_bis x y z roll pitch yaw">
-      <joint name="fixed_joint_${suffix_bis}" type="fixed">
+   <xacro:macro name="add_fixed_joint_stator" params="type name father child x y z roll pitch yaw">
+      <joint name="${name}" type="fixed">
          <axis rpy="0 0 0" xyz="0 0 1"/>
-         <parent link="link_${suffix_bis}"/>
-         <child link="link_stator_joint_${suffix}"/>
+         <parent link="${father}"/>
+         <child link="${child}"/>
          <origin rpy="${roll} ${pitch} ${yaw}" xyz="${x} ${y} ${z}"/>
       </joint>
    </xacro:macro>
-   <xacro:add_fixed_joint_stator pitch="-0.0" roll="0.0" suffix="1" suffix_bis="0" x="0.0" y="0.0" yaw="0.0" z="0.4"/>
-   <xacro:add_joint_stator size="3" size_y="0" size_z="0.2" suffix="1"/>
-   <xacro:add_joint effort="35" lower_lim="-3.14" pitch="-0.0" roll="0.0" suffix="1" upper_lim="3.14" velocity="5.7" x="0.0" y="0.0" yaw="0.0" z="0.2"/>
-   <xacro:add_fixed_joint pitch="-0.0" roll="0.0" suffix="1" x="0.0" y="0.0" yaw="0.0" z="0.0"/>
-   <xacro:add_link size="3" size_z="0.7" suffix="1_bis"/>
-   <xacro:add_fixed_joint pitch="-0.0" roll="0.0" suffix="1_bis" x="0.0" y="0.0" yaw="0.0" z="0.7"/>
-   <xacro:add_elbow size="3" size_y="0.2" size_z="0.2" suffix="1_bis_bis"/>
-   <xacro:add_fixed_joint pitch="-0.0" roll="-1.57" suffix="1_bis_bis" x="0.0" y="0.199999936586" yaw="0.0" z="0.200159265342"/>
-   <xacro:add_size_adapter size_in="3" size_out="2" size_z="0.1" suffix="1_bis_bis_bis"/>
-   <xacro:add_fixed_joint_stator pitch="-0.0" roll="0.0" suffix="2" suffix_bis="1_bis_bis_bis" x="0.0" y="0.0" yaw="0.0" z="0.1"/>
-   <xacro:add_joint_stator size="2" size_y="0" size_z="0.2" suffix="2"/>
-   <xacro:add_joint effort="35" lower_lim="-3.14" pitch="-0.0" roll="0.0" suffix="2" upper_lim="3.14" velocity="5.7" x="0.0" y="0.0" yaw="0.0" z="0.2"/>
-   <xacro:add_fixed_joint pitch="-0.0" roll="0.0" suffix="2" x="0.0" y="0.0" yaw="0.0" z="0.0"/>
-   <xacro:add_link size="2" size_z="0.5" suffix="2_bis"/>
-   <xacro:add_fixed_joint pitch="-0.0" roll="0.0" suffix="2_bis" x="0.0" y="0.0" yaw="0.0" z="0.5"/>
-   <xacro:add_elbow size="2" size_y="0.2" size_z="0.2" suffix="2_bis_bis"/>
-   <xacro:add_fixed_joint pitch="-0.0" roll="-1.57" suffix="2_bis_bis" x="0.0" y="0.199999936586" yaw="0.0" z="0.200159265342"/>
-   <xacro:add_size_adapter size_in="2" size_out="1" size_z="0.1" suffix="2_bis_bis_bis"/>
-   <xacro:add_fixed_joint_stator pitch="-0.0" roll="0.0" suffix="3" suffix_bis="2_bis_bis_bis" x="0.0" y="0.0" yaw="0.0" z="0.1"/>
-   <xacro:add_joint_stator size="1" size_y="0" size_z="0.2" suffix="3"/>
-   <xacro:add_joint effort="35" lower_lim="-3.14" pitch="-0.0" roll="0.0" suffix="3" upper_lim="3.14" velocity="5.7" x="0.0" y="0.0" yaw="0.0" z="0.2"/>
-   <xacro:add_fixed_joint pitch="-0.0" roll="0.0" suffix="3" x="0.0" y="0.0" yaw="0.0" z="0.0"/>
-   <xacro:add_elbow size="1" size_y="0.2" size_z="0.2" suffix="3_bis"/>
-   <xacro:add_fixed_joint_stator pitch="-0.0" roll="-1.57" suffix="4" suffix_bis="3_bis" x="0.0" y="0.199999936586" yaw="0.0" z="0.200159265342"/>
-   <xacro:add_joint_stator size="1" size_y="0" size_z="0.2" suffix="4"/>
-   <xacro:add_joint effort="35" lower_lim="-3.14" pitch="-0.0" roll="0.0" suffix="4" upper_lim="3.14" velocity="5.7" x="0.0" y="0.0" yaw="0.0" z="0.2"/>
-   <xacro:add_fixed_joint pitch="-0.0" roll="0.0" suffix="4" x="0.0" y="0.0" yaw="0.0" z="0.0"/>
-   <xacro:add_elbow size="1" size_y="0.2" size_z="0.2" suffix="4_bis"/>
-   <xacro:add_fixed_joint_stator pitch="-0.0" roll="-1.57" suffix="5" suffix_bis="4_bis" x="0.0" y="0.199999936586" yaw="0.0" z="0.200159265342"/>
-   <xacro:add_joint_stator size="1" size_y="0" size_z="0.2" suffix="5"/>
-   <xacro:add_joint effort="35" lower_lim="-3.14" pitch="-0.0" roll="0.0" suffix="5" upper_lim="3.14" velocity="5.7" x="0.0" y="0.0" yaw="0.0" z="0.2"/>
 </robot>
