Commit message: Add capability to add/remove master cubes
remove still need some fixin

File: urdf/ModularBot_new.urdf.xacro (robot description, xacro)
@@ -53,9 +53,9 @@
     <joint name="fixed" type="fixed">
         <parent link="base_link"/>
-        <child link="L_0"/>
+        <child link="L_0a"/>
         <axis rpy="0 0 0" xyz="0 0 1"/>
         <origin rpy="0.0 0.0 0.0" xyz="0.0 0.0 0.0"/>
     </joint>
-    <link name="L_0">
+    <link name="L_0a">
         <visual>
             <origin rpy="0 0 0" xyz="0 0 0.2"/>
@@ -75,5 +75,5 @@
         </inertial>
     </link>
-    <link name="L_0_A">
+    <link name="L_0a_con1">
         <visual>
             <origin rpy="0 0 0" xyz="0 0 0.05"/>
@@ -93,5 +93,5 @@
         </inertial>
     </link>
-    <link name="L_0_B">
+    <link name="L_0a_con2">
         <visual>
             <origin rpy="0 0 0" xyz="0 0 0.05"/>
@@ -111,16 +111,190 @@
         </inertial>
     </link>
-    <joint name="fixed_A_branch" type="fixed">
-        <parent link="L_0"/>
-        <child link="L_0_A"/>
+    <link name="L_0a_con3">
+        <visual>
+            <origin rpy="0 0 0" xyz="0 0 0.05"/>
+            <geometry>
+                <cylinder length="0.1" radius="0.06"/>
+            </geometry>
+            <material name="black"/>
+        </visual>
+        <collision>
+            <geometry>
+                <cylinder length="0.1" radius="0.06"/>
+            </geometry>
+        </collision>
+        <inertial>
+            <mass value="0.5"/>
+            <inertia ixx="1.0" ixy="0.0" ixz="0.0" iyy="1.0" iyz="0.0" izz="1.0"/>
+        </inertial>
+    </link>
+    <link name="L_0a_con4">
+        <visual>
+            <origin rpy="0 0 0" xyz="0 0 0.05"/>
+            <geometry>
+                <cylinder length="0.1" radius="0.06"/>
+            </geometry>
+            <material name="black"/>
+        </visual>
+        <collision>
+            <geometry>
+                <cylinder length="0.1" radius="0.06"/>
+            </geometry>
+        </collision>
+        <inertial>
+            <mass value="0.5"/>
+            <inertia ixx="1.0" ixy="0.0" ixz="0.0" iyy="1.0" iyz="0.0" izz="1.0"/>
+        </inertial>
+    </link>
+    <joint name="L_0a_fixed_1" type="fixed">
+        <parent link="L_0a"/>
+        <child link="L_0a_con1"/>
         <axis rpy="0 0 0" xyz="0 0 1"/>
-        <origin rpy="-1.57 0 0" xyz="0 0.2 0.3"/>
+        <origin rpy="3.14 0 0" xyz="0 0 0"/>
     </joint>
-    <joint name="fixed_B_branch" type="fixed">
-        <parent link="L_0"/>
-        <child link="L_0_B"/>
+    <joint name="L_0a_fixed_2" type="fixed">
+        <parent link="L_0a"/>
+        <child link="L_0a_con2"/>
         <axis rpy="0 0 0" xyz="0 0 1"/>
-        <origin rpy="1.57 0 0" xyz="0 -0.2 0.3"/>
+        <origin rpy="1.57 0 0" xyz="0 -0.2 0.2"/>
     </joint>
+    <joint name="L_0a_fixed_3" type="fixed">
+        <parent link="L_0a"/>
+        <child link="L_0a_con3"/>
+        <axis rpy="0 0 0" xyz="0 0 1"/>
+        <origin rpy="0 0 0" xyz="0 0 0.4"/>
+    </joint>
+    <joint name="L_0a_fixed_4" type="fixed">
+        <parent link="L_0a"/>
+        <child link="L_0a_con4"/>
+        <axis rpy="0 0 0" xyz="0 0 1"/>
+        <origin rpy="-1.57 0 0" xyz="0 0.2 0.2"/>
+    </joint>
+    <!-- Macro for adding a fixed joint (rigid interconnection between links) -->
+    <xacro:macro name="add_fixed_joint" params="type name father child x y z roll pitch yaw">
+        <joint name="${name}" type="fixed">
+            <axis xyz="0 0 1" rpy="0 0 0" />
+            <parent link="${father}"/>
+            <child link="${child}"/>
+            <origin xyz="${x} ${y} ${z}" rpy="${roll} ${pitch} ${yaw}"/>
+        </joint>
+    </xacro:macro>
+    <!-- Macro for adding a slave cube -->
+    <xacro:macro name="add_slave_cube" params="name">
+        <link name="${name}">
+            <visual>
+                <origin rpy="0 0 0" xyz="0 0 0.2"/>
+                <geometry>
+                    <box size="0.4 0.4 0.4"/>
+                </geometry>
+                <material name="black"/>
+            </visual>
+            <collision>
+                <geometry>
+                    <box size="0.4 0.4 0.4"/>
+                </geometry>
+            </collision>
+            <inertial>
+                <mass value="2"/>
+                <inertia ixx="1.0" ixy="0.0" ixz="0.0" iyy="1.0" iyz="0.0" izz="1.0"/>
+            </inertial>
+        </link>
+        <link name="${name}_con1">
+            <visual>
+                <origin rpy="0 0 0" xyz="0 0 0.05"/>
+                <geometry>
+                    <cylinder length="0.1" radius="0.06"/>
+                </geometry>
+                <material name="black"/>
+            </visual>
+            <collision>
+                <geometry>
+                    <cylinder length="0.1" radius="0.06"/>
+                </geometry>
+            </collision>
+            <inertial>
+                <mass value="0.5"/>
+                <inertia ixx="1.0" ixy="0.0" ixz="0.0" iyy="1.0" iyz="0.0" izz="1.0"/>
+            </inertial>
+        </link>
+        <link name="${name}_con2">
+            <visual>
+                <origin rpy="0 0 0" xyz="0 0 0.05"/>
+                <geometry>
+                    <cylinder length="0.1" radius="0.06"/>
+                </geometry>
+                <material name="black"/>
+            </visual>
+            <collision>
+                <geometry>
+                    <cylinder length="0.1" radius="0.06"/>
+                </geometry>
+            </collision>
+            <inertial>
+                <mass value="0.5"/>
+                <inertia ixx="1.0" ixy="0.0" ixz="0.0" iyy="1.0" iyz="0.0" izz="1.0"/>
+            </inertial>
+        </link>
+        <link name="${name}_con3">
+            <visual>
+                <origin rpy="0 0 0" xyz="0 0 0.05"/>
+                <geometry>
+                    <cylinder length="0.1" radius="0.06"/>
+                </geometry>
+                <material name="black"/>
+            </visual>
+            <collision>
+                <geometry>
+                    <cylinder length="0.1" radius="0.06"/>
+                </geometry>
+            </collision>
+            <inertial>
+                <mass value="0.5"/>
+                <inertia ixx="1.0" ixy="0.0" ixz="0.0" iyy="1.0" iyz="0.0" izz="1.0"/>
+            </inertial>
+        </link>
+        <link name="${name}_con4">
+            <visual>
+                <origin rpy="0 0 0" xyz="0 0 0.05"/>
+                <geometry>
+                    <cylinder length="0.1" radius="0.06"/>
+                </geometry>
+                <material name="black"/>
+            </visual>
+            <collision>
+                <geometry>
+                    <cylinder length="0.1" radius="0.06"/>
+                </geometry>
+            </collision>
+            <inertial>
+                <mass value="0.5"/>
+                <inertia ixx="1.0" ixy="0.0" ixz="0.0" iyy="1.0" iyz="0.0" izz="1.0"/>
+            </inertial>
+        </link>
+        <joint name="${name}_fixed_1" type="fixed">
+            <parent link="${name}_con1"/>
+            <child link="${name}"/>
+            <axis rpy="0 0 0" xyz="0 0 1"/>
+            <origin rpy="0 0 0" xyz="0 0 0.1"/>
+        </joint>
+        <joint name="${name}_fixed_2" type="fixed">
+            <parent link="${name}"/>
+            <child link="${name}_con2"/>
+            <axis rpy="0 0 0" xyz="0 0 1"/>
+            <origin rpy="1.57 0 0" xyz="0 -0.2 0.2"/>
+        </joint>
+        <joint name="${name}_fixed_3" type="fixed">
+            <parent link="${name}"/>
+            <child link="${name}_con3"/>
+            <axis rpy="0 0 0" xyz="0 0 1"/>
+            <origin rpy="0 0 0" xyz="0 0 0.4"/>
+        </joint>
+        <joint name="${name}_fixed_4" type="fixed">
+            <parent link="${name}"/>
+            <child link="${name}_con4"/>
+            <axis rpy="0 0 0" xyz="0 0 1"/>
+            <origin rpy="-1.57 0 0" xyz="0 0.2 0.2"/>
+        </joint>
+    </xacro:macro>
     <!-- Macro for adding a straight link -->
     <xacro:macro name="add_link" params="name type size_z size">
@@ -311,13 +485,4 @@
         </gazebo>
     </xacro:macro>
-    <!-- Macro for adding a fixed joint (rigid interconnection between links) -->
-    <xacro:macro name="add_fixed_joint" params="type name father child x y z roll pitch yaw">
-        <joint name="${name}" type="fixed">
-            <axis xyz="0 0 1" rpy="0 0 0" />
-            <parent link="${father}"/>
-            <child link="${child}"/>
-            <origin xyz="${x} ${y} ${z}" rpy="${roll} ${pitch} ${yaw}"/>
-        </joint>
-    </xacro:macro>
     <!-- Macro for adding the joint (it has no size) -->
     <xacro:macro name="add_joint" params="type name father child x y z roll pitch yaw upper_lim lower_lim effort velocity">

Commit message: changes to the base xacro file
the first cube is no longer added by default

File: urdf/ModularBot_new.urdf.xacro (robot description, xacro)
@@ -53,5 +53,6 @@
         <xacro:default_inertial mass="1"/>
     </link> -->
-    <joint name="fixed" type="fixed">
+    <!-- L_0a first link -->
+    <!-- <joint name="fixed" type="fixed">
         <parent link="base_link"/>
         <child link="L_0a"/>
@@ -172,5 +173,5 @@
         <axis rpy="0 0 0" xyz="0 0 1"/>
         <origin rpy="-1.57 0 0" xyz="0 0.2 0.2"/>
-    </joint>
+    </joint> -->
     <!-- Macro for adding a fixed joint (rigid interconnection between links) -->
     <xacro:macro name="add_fixed_joint" params="type name father child x y z roll pitch yaw">
@@ -180,4 +181,127 @@
             <child link="${child}"/>
             <origin xyz="${x} ${y} ${z}" rpy="${roll} ${pitch} ${yaw}"/>
+        </joint>
+    </xacro:macro>
+    <!-- Macro for adding a master cube -->
+    <xacro:macro name="add_master_cube" params="name">
+        <joint name="fixed" type="fixed">
+            <parent link="base_link"/>
+            <child link="${name}"/>
+            <axis rpy="0 0 0" xyz="0 0 1"/>
+            <origin rpy="0.0 0.0 0.0" xyz="0.0 0.0 0.0"/>
+        </joint>
+        <link name="${name}">
+            <visual>
+                <origin rpy="0 0 0" xyz="0 0 0.2"/>
+                <geometry>
+                    <box size="0.4 0.4 0.4"/>
+                </geometry>
+                <material name="black"/>
+            </visual>
+            <collision>
+                <geometry>
+                    <box size="0.4 0.4 0.4"/>
+                </geometry>
+            </collision>
+            <inertial>
+                <mass value="2"/>
+                <inertia ixx="1.0" ixy="0.0" ixz="0.0" iyy="1.0" iyz="0.0" izz="1.0"/>
+            </inertial>
+        </link>
+        <link name="${name}_con1">
+            <visual>
+                <origin rpy="0 0 0" xyz="0 0 0.05"/>
+                <geometry>
+                    <cylinder length="0.1" radius="0.06"/>
+                </geometry>
+                <material name="black"/>
+            </visual>
+            <collision>
+                <geometry>
+                    <cylinder length="0.1" radius="0.06"/>
+                </geometry>
+            </collision>
+            <inertial>
+                <mass value="0.5"/>
+                <inertia ixx="1.0" ixy="0.0" ixz="0.0" iyy="1.0" iyz="0.0" izz="1.0"/>
+            </inertial>
+        </link>
+        <link name="${name}_con2">
+            <visual>
+                <origin rpy="0 0 0" xyz="0 0 0.05"/>
+                <geometry>
+                    <cylinder length="0.1" radius="0.06"/>
+                </geometry>
+                <material name="black"/>
+            </visual>
+            <collision>
+                <geometry>
+                    <cylinder length="0.1" radius="0.06"/>
+                </geometry>
+            </collision>
+            <inertial>
+                <mass value="0.5"/>
+                <inertia ixx="1.0" ixy="0.0" ixz="0.0" iyy="1.0" iyz="0.0" izz="1.0"/>
+            </inertial>
+        </link>
+        <link name="${name}_con3">
+            <visual>
+                <origin rpy="0 0 0" xyz="0 0 0.05"/>
+                <geometry>
+                    <cylinder length="0.1" radius="0.06"/>
+                </geometry>
+                <material name="black"/>
+            </visual>
+            <collision>
+                <geometry>
+                    <cylinder length="0.1" radius="0.06"/>
+                </geometry>
+            </collision>
+            <inertial>
+                <mass value="0.5"/>
+                <inertia ixx="1.0" ixy="0.0" ixz="0.0" iyy="1.0" iyz="0.0" izz="1.0"/>
+            </inertial>
+        </link>
+        <link name="${name}_con4">
+            <visual>
+                <origin rpy="0 0 0" xyz="0 0 0.05"/>
+                <geometry>
+                    <cylinder length="0.1" radius="0.06"/>
+                </geometry>
+                <material name="black"/>
+            </visual>
+            <collision>
+                <geometry>
+                    <cylinder length="0.1" radius="0.06"/>
+                </geometry>
+            </collision>
+            <inertial>
+                <mass value="0.5"/>
+                <inertia ixx="1.0" ixy="0.0" ixz="0.0" iyy="1.0" iyz="0.0" izz="1.0"/>
+            </inertial>
+        </link>
+        <joint name="${name}_fixed_1" type="fixed">
+            <parent link="${name}"/>
+            <child link="${name}_con1"/>
+            <axis rpy="0 0 0" xyz="0 0 1"/>
+            <origin rpy="3.14 0 0" xyz="0 0 0.0"/>
+        </joint>
+        <joint name="${name}_fixed_2" type="fixed">
+            <parent link="${name}"/>
+            <child link="${name}_con2"/>
+            <axis rpy="0 0 0" xyz="0 0 1"/>
+            <origin rpy="1.57 0 0" xyz="0 -0.2 0.2"/>
+        </joint>
+        <joint name="${name}_fixed_3" type="fixed">
+            <parent link="${name}"/>
+            <child link="${name}_con3"/>
+            <axis rpy="0 0 0" xyz="0 0 1"/>
+            <origin rpy="0 0 0" xyz="0 0 0.4"/>
+        </joint>
+        <joint name="${name}_fixed_4" type="fixed">
+            <parent link="${name}"/>
+            <child link="${name}_con4"/>
+            <axis rpy="0 0 0" xyz="0 0 1"/>
+            <origin rpy="-1.57 0 0" xyz="0 0.2 0.2"/>
         </joint>
     </xacro:macro>

Commit message: change to base xacro to integrate new elbow joint
- add a dummy link with no visual but with inertial parameters (the rotating part inertia) after the joint
- if statement to switch between normal joints and elbow joints
- integrate mesh file for elbow joint

File: urdf/ModularBot_new.urdf.xacro (robot description, xacro)
@@ -611,5 +611,5 @@
         </gazebo>
     </xacro:macro>
-    <!-- Macro for adding the joint (it has no size) -->
+    <!-- Macro for adding the joint. A dummy link is also added with no visual tag, but with inertial parameters corresponding to the rotating part -->
     <xacro:macro name="add_joint" params="type name father child x y z roll pitch yaw upper_lim lower_lim effort velocity">
         <joint name="${name}" type="revolute">
@@ -620,5 +620,15 @@
             <limit lower="${lower_lim}" upper="${upper_lim}" effort="${effort}" velocity="${velocity}"/>
         </joint>
-        <link name="${child}"/>
+        <link name="${child}">
+            <!-- inertial parameters for avocado rotating part. wrt a point on one end of the rod -->
+            <inertial>
+                <origin xyz="0 0 -0.0635" rpy="0 0 0"/>
+                <mass value="${mass}"/>
+                <inertia
+                ixx="${mass / 3.0 * (0.127*0.127)}" ixy="0.0" ixz="0.0"
+                iyy="${mass / 3.0 * (0.127*0.127)}" iyz="0.0"
+                izz="0.0000148"/>
+            </inertial>
+        </link>
     </xacro:macro>
     <!-- Macro for adding the physical module housing the actuator -->
@@ -635,27 +645,55 @@
             </xacro:unless>
         </xacro:unless>
-        <link name="${name}">
-            <visual>
-                <origin xyz="0 0 ${size_z/2}" rpy="0 0 0" />
-                <geometry>
-                    <cylinder radius="${radius}" length="${size_z}"/>
-                </geometry>
-                <material name="blue"/>
-            </visual>
-            <collision>
-                <origin xyz="0 0 ${size_z/2}" rpy="0 0 0" />
-                <geometry>
-                    <cylinder radius="${radius}" length="${size_z}"/>
-                </geometry>
-            </collision>
-            <inertial>
-                <origin xyz="0 0 ${size_z/2}" rpy="0 0 0"/>
-                <mass value="${mass}"/>
-                <inertia
-                ixx="${mass / 12.0 * (3*radius*radius + size_z*size_z)}" ixy="0.0" ixz="0.0"
-                iyy="${mass / 12.0 * (size_z*size_z + 3*radius*radius)}" iyz="0.0"
-                izz="${mass / 2.0 * (radius*radius)}"/>
-            </inertial>
-        </link>
+        <xacro:if value="${size_y==0}">
+            <link name="${name}">
+                <visual>
+                    <origin xyz="0 0 ${size_z/2}" rpy="0 0 0" />
+                    <geometry>
+                        <cylinder radius="${radius}" length="${size_z}"/>
+                    </geometry>
+                    <material name="blue"/>
+                </visual>
+                <collision>
+                    <origin xyz="0 0 ${size_z/2}" rpy="0 0 0" />
+                    <geometry>
+                        <cylinder radius="${radius}" length="${size_z}"/>
+                    </geometry>
+                </collision>
+                <inertial>
+                    <origin xyz="0 0 ${size_z/2}" rpy="0 0 0"/>
+                    <mass value="${mass}"/>
+                    <inertia
+                    ixx="${mass / 12.0 * (3*radius*radius + size_z*size_z)}" ixy="0.0" ixz="0.0"
+                    iyy="${mass / 12.0 * (size_z*size_z + 3*radius*radius)}" iyz="0.0"
+                    izz="${mass / 2.0 * (radius*radius)}"/>
+                </inertial>
+            </link>
+        </xacro:if>
+        <xacro:unless value="${size_y==0}">
+            <link name="${name}">
+                <visual>
+                    <!-- Load mesh. Rotate the origin frame (this is because of how the .stl was saved) -->
+                    <origin rpy="3.14 0 1.57" xyz="0 0 0"/>
+                    <geometry>
+                        <mesh filename="package://asm0001.stl" scale="0.001 0.001 0.001"/>
+                    </geometry>
+                </visual>
+                <collision>
+                    <origin rpy="3.14 0 1.57" xyz="0 0 0"/>
+                    <geometry>
+                        <mesh filename="package://asm0001.stl" scale="0.001 0.001 0.001"/>
+                    </geometry>
+                </collision>
+                <!-- TODO: change inertial parameters with the one from CAD. This will be the inertia tensor of only the housing/stator part -->
+                <inertial>
+                    <origin xyz="0 0 ${size_z/2}" rpy="3.14 0 1.57"/>
+                    <mass value="${mass}"/>
+                    <inertia
+                    ixx="${mass / 2 *( 1 / 12.0 * (3*radius*radius + 4*size_y*size_y) + size_z*size_z) + mass / 24.0 * (3*radius*radius + 4*size_z*size_z)}" ixy="0.0" ixz="0.0"
+                    iyy="${mass / 24.0 * (3*radius*radius + 4*size_z*size_z) + mass / 2 *( 1 / 2 *radius*radius + size_z*size_z)}" iyz="0.0"
+                    izz="${mass / 4.0 * (radius*radius) + mass / 24.0 * (3*radius*radius + 4*size_y*size_y)}"/>
+                </inertial>
+            </link>
+        </xacro:unless>
         <gazebo reference="${name}">
             <mu1>0.2</mu1>

Commit message: add Gazebo XBot plugin to base xacro
In this way the generated urdf can be controlled in Gazebo simulation via XBotCore

File: urdf/ModularBot_new.urdf.xacro (robot description, xacro)
@@ -3,4 +3,10 @@
     <!-- <xacro:include filename="$(find modular)/urdf/config.xacro" />
     <xacro:include filename="$(find modular)/urdf/modular.gazebo" /> -->
+    <gazebo>
+        <plugin name="gazebo_xbot_plugin" filename="libGazeboXBotPlugin.so">
+            <!-- <path_to_config_file>${xbot_config_file}</path_to_config_file> -->
+            <path_to_config_file>configs/ADVR_shared/ModularBot/configs/config_ModularBot.yaml</path_to_config_file>
+        </plugin>
+    </gazebo>
     <xacro:property name="size1" value="0.05" />
     <xacro:property name="size2" value="0.055" />
@@ -676,5 +682,5 @@
                     <origin rpy="3.14 0 1.57" xyz="0 0 0"/>
                     <geometry>
-                        <mesh filename="package://asm0001.stl" scale="0.001 0.001 0.001"/>
+                        <mesh filename="package://modular/meshes/asm0001.stl" scale="0.001 0.001 0.001"/>
                     </geometry>
                 </visual>
@@ -682,5 +688,5 @@
                     <origin rpy="3.14 0 1.57" xyz="0 0 0"/>
                     <geometry>
-                        <mesh filename="package://asm0001.stl" scale="0.001 0.001 0.001"/>
+                        <mesh filename="package://modular/meshes/asm0001.stl" scale="0.001 0.001 0.001"/>
                     </geometry>
                 </collision>

Commit message: fix collision ref. frame for master cube

File: urdf/ModularBot_new.urdf.xacro (robot description, xacro)
@@ -206,4 +206,5 @@
             </visual>
             <collision>
+                <origin rpy="0 0 0" xyz="0 0 0.2"/>
                 <geometry>
                     <box size="0.4 0.4 0.4"/>

Commit message: fixes to handle wrong orientation of mesh file
Warning: there are some hardcoded value to rotate the mesh. To be removed when correct meshes are taken.

File: urdf/ModularBot_new.urdf.xacro (robot description, xacro)
@@ -681,5 +681,5 @@
                 <visual>
                     <!-- Load mesh. Rotate the origin frame (this is because of how the .stl was saved) -->
-                    <origin rpy="3.14 0 1.57" xyz="0 0 0"/>
+                    <origin rpy="3.14 0 -1.57" xyz="0 0 0"/>
                     <geometry>
                         <mesh filename="package://modular/meshes/asm0001.stl" scale="0.001 0.001 0.001"/>
@@ -687,5 +687,5 @@
                 </visual>
                 <collision>
-                    <origin rpy="3.14 0 1.57" xyz="0 0 0"/>
+                    <origin rpy="3.14 0 -1.57" xyz="0 0 0"/>
                     <geometry>
                         <mesh filename="package://modular/meshes/asm0001.stl" scale="0.001 0.001 0.001"/>
@@ -694,5 +694,5 @@
                 <!-- TODO: change inertial parameters with the one from CAD. This will be the inertia tensor of only the housing/stator part -->
                 <inertial>
-                    <origin xyz="0 0 ${size_z/2}" rpy="3.14 0 1.57"/>
+                    <origin xyz="0 0 ${size_z/2}" rpy="0 0 0"/>
                     <mass value="${mass}"/>
                     <inertia
