Commit message: add backwards connection capability

File: urdf/ModularBot_new.urdf.xacro (robot description, xacro)
@@ -627,18 +627,61 @@
             <limit lower="${lower_lim}" upper="${upper_lim}" effort="${effort}" velocity="${velocity}"/>
         </joint>
-        <link name="${child}">
-            <!-- inertial parameters for avocado rotating part. wrt a point on one end of the rod -->
+        <!--<link name="${child}">-->
+            <!--<xacro:if value="${type==joint_mesh}">-->
+                <!--<visual>-->
+                    <!--&lt;!&ndash; Load mesh. Rotate the origin frame (this is because of how the .stl was saved) &ndash;&gt;-->
+                    <!--<origin rpy="${roll} ${pitch} ${yaw}" xyz="${x} ${y} ${z}"/>-->
+                    <!--<geometry>-->
+                        <!--<mesh filename="package://modular/meshes/asm0001.stl" scale="0.001 0.001 0.001"/>-->
+                    <!--</geometry>-->
+                <!--</visual>-->
+                <!--<collision>-->
+                    <!--<origin rpy="${roll} ${pitch} ${yaw}" xyz="${x} ${y} ${z}"/>-->
+                    <!--<geometry>-->
+                        <!--<mesh filename="package://modular/meshes/asm0001.stl" scale="0.001 0.001 0.001"/>-->
+                    <!--</geometry>-->
+                <!--</collision>-->
+            <!--</xacro:if>-->
+            <!--&lt;!&ndash; inertial parameters for avocado rotating part. wrt a point on one end of the rod &ndash;&gt;-->
+            <!--<inertial>-->
+                <!--<origin xyz="0 0 -0.0635" rpy="0 0 0"/>-->
+                <!--<mass value="${mass}"/>-->
+                <!--<inertia-->
+                <!--ixx="${mass / 3.0 * (0.127*0.127)}" ixy="0.0" ixz="0.0"-->
+                <!--iyy="${mass / 3.0 * (0.127*0.127)}" iyz="0.0"-->
+                <!--izz="0.0000148"/>-->
+            <!--</inertial>-->
+        <!--</link>-->
+    </xacro:macro>
+    <xacro:macro name="add_distal" params="type name mesh x y z roll pitch yaw">
+        <link name="${name}">
+            <xacro:unless value="${mesh == 0}">
+                <visual>
+                    <!-- Load mesh. Rotate the origin frame (this is because of how the .stl was saved) -->
+                    <origin rpy="${roll} ${pitch} ${yaw}" xyz="${x} ${y} ${z}"/>
+                    <geometry>
+                        <mesh filename="package://modular/meshes/asm0001.stl" scale="0.001 0.001 0.001"/>
+                    </geometry>
+                </visual>
+                <collision>
+                    <origin rpy="${roll} ${pitch} ${yaw}" xyz="${x} ${y} ${z}"/>
+                    <geometry>
+                        <mesh filename="package://modular/meshes/asm0001.stl" scale="0.001 0.001 0.001"/>
+                    </geometry>
+                </collision>
+            </xacro:unless>
+            <!--inertial parameters for avocado rotating part. wrt a point on one end of the rod-->
             <inertial>
                 <origin xyz="0 0 -0.0635" rpy="0 0 0"/>
                 <mass value="${mass}"/>
                 <inertia
-                ixx="${mass / 3.0 * (0.127*0.127)}" ixy="0.0" ixz="0.0"
-                iyy="${mass / 3.0 * (0.127*0.127)}" iyz="0.0"
-                izz="0.0000148"/>
+                        ixx="${mass / 3.0 * (0.127*0.127)}" ixy="0.0" ixz="0.0"
+                        iyy="${mass / 3.0 * (0.127*0.127)}" iyz="0.0"
+                        izz="0.0000148"/>
             </inertial>
         </link>
     </xacro:macro>
     <!-- Macro for adding the physical module housing the actuator -->
-    <xacro:macro name="add_joint_stator" params="type name size_y size_z size">
+    <xacro:macro name="add_joint_stator" params="type name size_y size_z size x y z roll pitch yaw">
         <xacro:if value="${size==1}">
             <xacro:property name="radius" value="${size1}" />
@@ -671,7 +714,7 @@
                     <mass value="${mass}"/>
                     <inertia
-                    ixx="${mass / 12.0 * (3*radius*radius + size_z*size_z)}" ixy="0.0" ixz="0.0"
-                    iyy="${mass / 12.0 * (size_z*size_z + 3*radius*radius)}" iyz="0.0"
-                    izz="${mass / 2.0 * (radius*radius)}"/>
+                            ixx="${mass / 12.0 * (3*radius*radius + size_z*size_z)}" ixy="0.0" ixz="0.0"
+                            iyy="${mass / 12.0 * (size_z*size_z + 3*radius*radius)}" iyz="0.0"
+                            izz="${mass / 2.0 * (radius*radius)}"/>
                 </inertial>
             </link>
@@ -681,5 +724,5 @@
                 <visual>
                     <!-- Load mesh. Rotate the origin frame (this is because of how the .stl was saved) -->
-                    <origin rpy="3.14 0 -1.57" xyz="0 0 0"/>
+                    <origin rpy="${roll} ${pitch} ${yaw}" xyz="${x} ${y} ${z}"/>
                     <geometry>
                         <mesh filename="package://modular/meshes/asm0001.stl" scale="0.001 0.001 0.001"/>
@@ -687,5 +730,5 @@
                 </visual>
                 <collision>
-                    <origin rpy="3.14 0 -1.57" xyz="0 0 0"/>
+                    <origin rpy="${roll} ${pitch} ${yaw}" xyz="${x} ${y} ${z}"/>
                     <geometry>
                         <mesh filename="package://modular/meshes/asm0001.stl" scale="0.001 0.001 0.001"/>
@@ -697,7 +740,7 @@
                     <mass value="${mass}"/>
                     <inertia
-                    ixx="${mass / 2 *( 1 / 12.0 * (3*radius*radius + 4*size_y*size_y) + size_z*size_z) + mass / 24.0 * (3*radius*radius + 4*size_z*size_z)}" ixy="0.0" ixz="0.0"
-                    iyy="${mass / 24.0 * (3*radius*radius + 4*size_z*size_z) + mass / 2 *( 1 / 2 *radius*radius + size_z*size_z)}" iyz="0.0"
-                    izz="${mass / 4.0 * (radius*radius) + mass / 24.0 * (3*radius*radius + 4*size_y*size_y)}"/>
+                            ixx="${mass / 2 *( 1 / 12.0 * (3*radius*radius + 4*size_y*size_y) + size_z*size_z) + mass / 24.0 * (3*radius*radius + 4*size_z*size_z)}" ixy="0.0" ixz="0.0"
+                            iyy="${mass / 24.0 * (3*radius*radius + 4*size_z*size_z) + mass / 2 *( 1 / 2 *radius*radius + size_z*size_z)}" iyz="0.0"
+                            izz="${mass / 4.0 * (radius*radius) + mass / 24.0 * (3*radius*radius + 4*size_y*size_y)}"/>
                 </inertial>
             </link>

Commit message: add add_rotor_fast to xacro and add YAML import
- add_rotor_fast is a macro to add a link whose inertia is computed by reflecting it to the link-side by the gear ratio

- add_distal and add_joint_stator now read inertia param. from YAML file and load meshes path from there as well

File: urdf/ModularBot_new.urdf.xacro (robot description, xacro)
@@ -29,4 +29,13 @@
     <material name="grey">
         <color rgba="0.5 0.5 0.5 1"/>
+    </material>
+    <material name="red">
+        <color rgba="1 0 0 1"/>
+    </material>
+    <material name="green">
+        <color rgba="0 1 0 1"/>
+    </material>
+    <material name="yellow">
+        <color rgba="1 1 0 1"/>
     </material>
     <xacro:macro name="default_inertial" params="mass">
@@ -449,5 +458,5 @@
                     <cylinder radius="${radius}" length="${size_z}"/>
                 </geometry>
-                <material name="black"/>
+                <material name="white"/>
             </visual>
             <collision>
@@ -565,5 +574,5 @@
                     <cylinder radius="${radius}" length="${size_z}"/>
                 </geometry>
-                <material name="white"/>
+                <material name="blue"/>
             </visual>
             <visual>
@@ -572,5 +581,5 @@
                     <cylinder radius="${radius}" length="${size_y}"/>
                 </geometry>
-                <material name="white"/>
+                <material name="blue"/>
             </visual>
             <visual>
@@ -579,5 +588,5 @@
                     <sphere radius="${radius}" />
                 </geometry>
-                <material name="white"/>
+                <material name="blue"/>
             </visual>
             <collision>
@@ -654,12 +663,31 @@
         <!--</link>-->
     </xacro:macro>
-    <xacro:macro name="add_distal" params="type name mesh x y z roll pitch yaw">
+    <xacro:macro name="add_rotor_fast" params="type name filename x y z roll pitch yaw">
+        <xacro:property name="module" value="${load_yaml(filename)}"/>
         <link name="${name}">
-            <xacro:unless value="${mesh == 0}">
+            <inertial>
+                <origin
+                        xyz="${module['dynamics']['body_2_fast']['CoM']['x']} ${module['dynamics']['body_2_fast']['CoM']['y']} ${module['dynamics']['body_2_fast']['CoM']['z']}"
+                        rpy="0 0 0"/>
+                    <mass value="${module['dynamics']['body_2_fast']['mass']}"/>
+                    <inertia
+                        ixx="${module['dynamics']['body_2_fast']['inertia_tensor']['I_xx']}"
+                        ixy="${module['dynamics']['body_2_fast']['inertia_tensor']['I_xy']}"
+                        iyy="${module['dynamics']['body_2_fast']['inertia_tensor']['I_yy']}"
+                        ixz="${module['control']['nu']} * ${module['dynamics']['body_2_fast']['inertia_tensor']['I_xz']}"
+                        iyz="${module['control']['nu']} * ${module['dynamics']['body_2_fast']['inertia_tensor']['I_yz']}"
+                        izz="${module['control']['nu']} * ${module['control']['nu']} * ${module['dynamics']['body_2_fast']['inertia_tensor']['I_zz']}"/>
+            </inertial>
+        </link>
+    </xacro:macro>
+    <xacro:macro name="add_distal" params="type name filename mesh_bool mesh x y z roll pitch yaw">
+        <xacro:property name="module" value="${load_yaml(filename)}"/>
+        <link name="${name}">
+            <xacro:unless value="${mesh_bool == 0}">
                 <visual>
                     <!-- Load mesh. Rotate the origin frame (this is because of how the .stl was saved) -->
                     <origin rpy="${roll} ${pitch} ${yaw}" xyz="${x} ${y} ${z}"/>
                     <geometry>
-                        <mesh filename="package://modular/meshes/asm0001.stl" scale="0.001 0.001 0.001"/>
+                        <mesh filename="${mesh}" scale="0.001 0.001 0.001"/>
                     </geometry>
                 </visual>
@@ -667,21 +695,35 @@
                     <origin rpy="${roll} ${pitch} ${yaw}" xyz="${x} ${y} ${z}"/>
                     <geometry>
-                        <mesh filename="package://modular/meshes/asm0001.stl" scale="0.001 0.001 0.001"/>
+                        <mesh filename="${mesh}" scale="0.001 0.001 0.001"/>
                     </geometry>
                 </collision>
             </xacro:unless>
             <!--inertial parameters for avocado rotating part. wrt a point on one end of the rod-->
-            <inertial>
-                <origin xyz="0 0 -0.0635" rpy="0 0 0"/>
-                <mass value="${mass}"/>
+            <!-- <inertial>
+                <origin xyz="0 0 -0.002265" rpy="0 0 0"/>
+                <mass value="0.153466"/>
                 <inertia
-                        ixx="${mass / 3.0 * (0.127*0.127)}" ixy="0.0" ixz="0.0"
-                        iyy="${mass / 3.0 * (0.127*0.127)}" iyz="0.0"
-                        izz="0.0000148"/>
+                        ixx="0.000034763" ixy="0.0" ixz="0.0"
+                        iyy="0.000034827" iyz="0.0"
+                        izz="0.000031822"/>
+            </inertial> -->
+            <inertial>
+                <origin
+                    xyz="${module['dynamics']['body_2']['CoM']['x']} ${module['dynamics']['body_2']['CoM']['y']} ${module['dynamics']['body_2']['CoM']['z']}"
+                    rpy="0 0 0"/>
+                <mass value="${module['dynamics']['body_2']['mass']}"/>
+                <inertia
+                    ixx="${module['dynamics']['body_2']['inertia_tensor']['I_xx']}"
+                    ixy="${module['dynamics']['body_2']['inertia_tensor']['I_xy']}"
+                    ixz="${module['dynamics']['body_2']['inertia_tensor']['I_xz']}"
+                    iyy="${module['dynamics']['body_2']['inertia_tensor']['I_yy']}"
+                    iyz="${module['dynamics']['body_2']['inertia_tensor']['I_yz']}"
+                    izz="${module['dynamics']['body_2']['inertia_tensor']['I_zz']}"/>
             </inertial>
         </link>
     </xacro:macro>
     <!-- Macro for adding the physical module housing the actuator -->
-    <xacro:macro name="add_joint_stator" params="type name size_y size_z size x y z roll pitch yaw">
+    <xacro:macro name="add_joint_stator" params="type name filename mesh_bool mesh size_y size_z size x y z roll pitch yaw">
+        <xacro:property name="module" value="${load_yaml(filename)}"/>
         <xacro:if value="${size==1}">
             <xacro:property name="radius" value="${size1}" />
@@ -695,5 +737,5 @@
             </xacro:unless>
         </xacro:unless>
-        <xacro:if value="${size_y==0}">
+        <xacro:if value="${mesh_bool==0}">
             <link name="${name}">
                 <visual>
@@ -720,5 +762,5 @@
             </link>
         </xacro:if>
-        <xacro:unless value="${size_y==0}">
+        <xacro:unless value="${mesh_bool == 0}">
             <link name="${name}">
                 <visual>
@@ -726,21 +768,27 @@
                     <origin rpy="${roll} ${pitch} ${yaw}" xyz="${x} ${y} ${z}"/>
                     <geometry>
-                        <mesh filename="package://modular/meshes/asm0001.stl" scale="0.001 0.001 0.001"/>
+                        <mesh filename="${mesh}" scale="0.001 0.001 0.001"/>
                     </geometry>
+                    <material name="grey"/>
                 </visual>
                 <collision>
                     <origin rpy="${roll} ${pitch} ${yaw}" xyz="${x} ${y} ${z}"/>
                     <geometry>
-                        <mesh filename="package://modular/meshes/asm0001.stl" scale="0.001 0.001 0.001"/>
+                        <mesh filename="${mesh}" scale="0.001 0.001 0.001"/>
                     </geometry>
                 </collision>
                 <!-- TODO: change inertial parameters with the one from CAD. This will be the inertia tensor of only the housing/stator part -->
                 <inertial>
-                    <origin xyz="0 0 ${size_z/2}" rpy="0 0 0"/>
-                    <mass value="${mass}"/>
+                    <origin
+                        xyz="${module['dynamics']['body_1']['CoM']['x']} ${module['dynamics']['body_1']['CoM']['y']} ${module['dynamics']['body_1']['CoM']['z']}"
+                        rpy="0 0 0"/>
+                    <mass value="${module['dynamics']['body_1']['mass']}"/>
                     <inertia
-                            ixx="${mass / 2 *( 1 / 12.0 * (3*radius*radius + 4*size_y*size_y) + size_z*size_z) + mass / 24.0 * (3*radius*radius + 4*size_z*size_z)}" ixy="0.0" ixz="0.0"
-                            iyy="${mass / 24.0 * (3*radius*radius + 4*size_z*size_z) + mass / 2 *( 1 / 2 *radius*radius + size_z*size_z)}" iyz="0.0"
-                            izz="${mass / 4.0 * (radius*radius) + mass / 24.0 * (3*radius*radius + 4*size_y*size_y)}"/>
+                        ixx="${module['dynamics']['body_1']['inertia_tensor']['I_xx']}"
+                        ixy="${module['dynamics']['body_1']['inertia_tensor']['I_xy']}"
+                        ixz="${module['dynamics']['body_1']['inertia_tensor']['I_xz']}"
+                        iyy="${module['dynamics']['body_1']['inertia_tensor']['I_yy']}"
+                        iyz="${module['dynamics']['body_1']['inertia_tensor']['I_yz']}"
+                        izz="${module['dynamics']['body_1']['inertia_tensor']['I_zz']}"/>
                 </inertial>
             </link>
@@ -757,5 +805,5 @@
     </xacro:macro>
     <!-- Macro for adding a fixed joint (rigid interconnection between links and statoric part of the joint) -->
-    <xacro:macro name="add_fixed_joint_stator" params="type name father child x y z roll pitch yaw">
+    <xacro:macro name="add_fixed_joint" params="type name father child x y z roll pitch yaw">
         <joint name="${name}" type="fixed">
             <axis xyz="0 0 1" rpy="0 0 0" />

Commit message: handle gear ratio and mesh orientation in distal_link (xacro)

File: urdf/ModularBot_new.urdf.xacro (robot description, xacro)
@@ -665,4 +665,5 @@
     <xacro:macro name="add_rotor_fast" params="type name filename x y z roll pitch yaw">
         <xacro:property name="module" value="${load_yaml(filename)}"/>
+        <xacro:property name="gear_ratio" value="${module['control']['nu']}"/>
         <link name="${name}">
             <inertial>
@@ -675,28 +676,37 @@
                         ixy="${module['dynamics']['body_2_fast']['inertia_tensor']['I_xy']}"
                         iyy="${module['dynamics']['body_2_fast']['inertia_tensor']['I_yy']}"
-                        ixz="${module['control']['nu']} * ${module['dynamics']['body_2_fast']['inertia_tensor']['I_xz']}"
-                        iyz="${module['control']['nu']} * ${module['dynamics']['body_2_fast']['inertia_tensor']['I_yz']}"
-                        izz="${module['control']['nu']} * ${module['control']['nu']} * ${module['dynamics']['body_2_fast']['inertia_tensor']['I_zz']}"/>
-            </inertial>
-        </link>
-    </xacro:macro>
-    <xacro:macro name="add_distal" params="type name filename mesh_bool mesh x y z roll pitch yaw">
+                        ixz="${ gear_ratio * module['dynamics']['body_2_fast']['inertia_tensor']['I_xz'] }"
+                        iyz="${ gear_ratio * module['dynamics']['body_2_fast']['inertia_tensor']['I_yz'] }"
+                        izz="${ gear_ratio * gear_ratio * module['dynamics']['body_2_fast']['inertia_tensor']['I_zz'] }"/>
+            </inertial>
+        </link>
+    </xacro:macro>
+    <xacro:macro name="add_distal" params="type name filename">
         <xacro:property name="module" value="${load_yaml(filename)}"/>
+        <!-- <xacro:property name="visual" value="${module['visual']['mesh_body_1']}"/> -->
+        <xacro:property name="mesh_bool" value="false"/>
+        <xacro:unless value="${ module['visual']['mesh_body_1'] == '' }">
+            <xacro:property name="mesh_bool" value="true"/>
+        </xacro:unless>
         <link name="${name}">
-            <xacro:unless value="${mesh_bool == 0}">
+            <xacro:if value="${ mesh_bool }">
                 <visual>
                     <!-- Load mesh. Rotate the origin frame (this is because of how the .stl was saved) -->
-                    <origin rpy="${roll} ${pitch} ${yaw}" xyz="${x} ${y} ${z}"/>
+                    <origin
+                        rpy="${module['visual']['tf_mesh_2']['roll']} ${module['visual']['tf_mesh_2']['pitch']} ${module['visual']['tf_mesh_2']['yaw']}"
+                        xyz="${module['visual']['tf_mesh_2']['x']} ${module['visual']['tf_mesh_2']['y']} ${module['visual']['tf_mesh_2']['z']}"/>
                     <geometry>
-                        <mesh filename="${mesh}" scale="0.001 0.001 0.001"/>
+                        <mesh filename="${module['visual']['mesh_body_2']}" scale="0.001 0.001 0.001"/>
                     </geometry>
                 </visual>
                 <collision>
-                    <origin rpy="${roll} ${pitch} ${yaw}" xyz="${x} ${y} ${z}"/>
+                    <origin
+                        rpy="${module['visual']['tf_mesh_2']['roll']} ${module['visual']['tf_mesh_2']['pitch']} ${module['visual']['tf_mesh_2']['yaw']}"
+                        xyz="${module['visual']['tf_mesh_2']['x']} ${module['visual']['tf_mesh_2']['y']} ${module['visual']['tf_mesh_2']['z']}"/>
                     <geometry>
-                        <mesh filename="${mesh}" scale="0.001 0.001 0.001"/>
+                        <mesh filename="${module['visual']['mesh_body_2']}" scale="0.001 0.001 0.001"/>
                     </geometry>
                 </collision>
-            </xacro:unless>
+            </xacro:if>
             <!--inertial parameters for avocado rotating part. wrt a point on one end of the rod-->
             <!-- <inertial>

Commit message: Now collision mesh is retrieved both from python and xacro

File: urdf/ModularBot_new.urdf.xacro (robot description, xacro)
@@ -705,5 +705,5 @@
                         xyz="${module['visual']['tf_mesh_2']['x']} ${module['visual']['tf_mesh_2']['y']} ${module['visual']['tf_mesh_2']['z']}"/>
                     <geometry>
-                        <mesh filename="${module['visual']['mesh_body_2']}" scale="0.001 0.001 0.001"/>
+                        <mesh filename="${module['visual']['mesh_collision_2']}" scale="0.001 0.001 0.001"/>
                     </geometry>
                 </collision>
@@ -734,5 +734,5 @@
     </xacro:macro>
     <!-- Macro for adding the physical module housing the actuator -->
-    <xacro:macro name="add_joint_stator" params="type name filename mesh_bool mesh size_y size_z size x y z roll pitch yaw">
+    <xacro:macro name="add_joint_stator" params="type name filename mesh_bool mesh_visual mesh_collision size_y size_z size x y z roll pitch yaw">
         <xacro:property name="module" value="${load_yaml(filename)}"/>
         <xacro:if value="${size==1}">
@@ -778,5 +778,5 @@
                     <origin rpy="${roll} ${pitch} ${yaw}" xyz="${x} ${y} ${z}"/>
                     <geometry>
-                        <mesh filename="${mesh}" scale="0.001 0.001 0.001"/>
+                        <mesh filename="${mesh_visual}" scale="0.001 0.001 0.001"/>
                     </geometry>
                     <material name="grey"/>
@@ -785,5 +785,5 @@
                     <origin rpy="${roll} ${pitch} ${yaw}" xyz="${x} ${y} ${z}"/>
                     <geometry>
-                        <mesh filename="${mesh}" scale="0.001 0.001 0.001"/>
+                        <mesh filename="${mesh_collision}" scale="0.001 0.001 0.001"/>
                     </geometry>
                 </collision>
