Commit message: removed crazy inertia values for cube link

File: urdf/ModularBot_new.urdf.xacro (robot description, xacro)
@@ -41,6 +41,6 @@
     <xacro:macro name="default_inertial" params="mass">
         <inertial>
-        <mass value="${mass}" />
-        <inertia ixx="1.0" ixy="0.0" ixz="0.0" iyy="1.0" iyz="0.0" izz="1.0" />
+            <mass value="${mass}" />
+            <inertia ixx="1.0e-03" ixy="0.0" ixz="0.0" iyy="1.0e-03" iyz="0.0" izz="1.0e-03" />
         </inertial>
     </xacro:macro>
@@ -52,141 +52,4 @@
     </joint>
     <link name="base_link"/>
-    <!-- <link name="L_0">
-        <visual>
-            <origin xyz="0 0 ${len1/2}" rpy="0 0 0" />
-            <geometry>
-                <cylinder radius="${size1}" length="${len1}"/>
-            </geometry>
-            <material name="black"/>
-        </visual>
-        <collision>
-            <origin xyz="0 0 ${len1/2}" rpy="0 0 0" />
-            <geometry>
-                <cylinder radius="${size1}" length="${len1}"/>
-            </geometry>
-        </collision>
-        <xacro:default_inertial mass="1"/>
-    </link> -->
-    <!-- L_0a first link -->
-    <!-- <joint name="fixed" type="fixed">
-        <parent link="base_link"/>
-        <child link="L_0a"/>
-        <axis rpy="0 0 0" xyz="0 0 1"/>
-        <origin rpy="0.0 0.0 0.0" xyz="0.0 0.0 0.0"/>
-    </joint>
-    <link name="L_0a">
-        <visual>
-            <origin rpy="0 0 0" xyz="0 0 0.2"/>
-            <geometry>
-                <box size="0.4 0.4 0.4"/>
-            </geometry>
-            <material name="black"/>
-        </visual>
-        <collision>
-            <geometry>
-                <box size="0.4 0.4 0.4"/>
-            </geometry>
-        </collision>
-        <inertial>
-            <mass value="2"/>
-            <inertia ixx="1.0" ixy="0.0" ixz="0.0" iyy="1.0" iyz="0.0" izz="1.0"/>
-        </inertial>
-    </link>
-    <link name="L_0a_con1">
-        <visual>
-            <origin rpy="0 0 0" xyz="0 0 0.05"/>
-            <geometry>
-                <cylinder length="0.1" radius="0.06"/>
-            </geometry>
-            <material name="black"/>
-        </visual>
-        <collision>
-            <geometry>
-                <cylinder length="0.1" radius="0.06"/>
-            </geometry>
-        </collision>
-        <inertial>
-            <mass value="0.5"/>
-            <inertia ixx="1.0" ixy="0.0" ixz="0.0" iyy="1.0" iyz="0.0" izz="1.0"/>
-        </inertial>
-    </link>
-    <link name="L_0a_con2">
-        <visual>
-            <origin rpy="0 0 0" xyz="0 0 0.05"/>
-            <geometry>
-                <cylinder length="0.1" radius="0.06"/>
-            </geometry>
-            <material name="black"/>
-        </visual>
-        <collision>
-            <geometry>
-                <cylinder length="0.1" radius="0.06"/>
-            </geometry>
-        </collision>
-        <inertial>
-            <mass value="0.5"/>
-            <inertia ixx="1.0" ixy="0.0" ixz="0.0" iyy="1.0" iyz="0.0" izz="1.0"/>
-        </inertial>
-    </link>
-    <link name="L_0a_con3">
-        <visual>
-            <origin rpy="0 0 0" xyz="0 0 0.05"/>
-            <geometry>
-                <cylinder length="0.1" radius="0.06"/>
-            </geometry>
-            <material name="black"/>
-        </visual>
-        <collision>
-            <geometry>
-                <cylinder length="0.1" radius="0.06"/>
-            </geometry>
-        </collision>
-        <inertial>
-            <mass value="0.5"/>
-            <inertia ixx="1.0" ixy="0.0" ixz="0.0" iyy="1.0" iyz="0.0" izz="1.0"/>
-        </inertial>
-    </link>
-    <link name="L_0a_con4">
-        <visual>
-            <origin rpy="0 0 0" xyz="0 0 0.05"/>
-            <geometry>
-                <cylinder length="0.1" radius="0.06"/>
-            </geometry>
-            <material name="black"/>
-        </visual>
-        <collision>
-            <geometry>
-                <cylinder length="0.1" radius="0.06"/>
-            </geometry>
-        </collision>
-        <inertial>
-            <mass value="0.5"/>
-            <inertia ixx="1.0" ixy="0.0" ixz="0.0" iyy="1.0" iyz="0.0" izz="1.0"/>
-        </inertial>
-    </link>
-    <joint name="L_0a_fixed_1" type="fixed">
-        <parent link="L_0a"/>
-        <child link="L_0a_con1"/>
-        <axis rpy="0 0 0" xyz="0 0 1"/>
-        <origin rpy="3.14 0 0" xyz="0 0 0"/>
-    </joint>
-    <joint name="L_0a_fixed_2" type="fixed">
-        <parent link="L_0a"/>
-        <child link="L_0a_con2"/>
-        <axis rpy="0 0 0" xyz="0 0 1"/>
-        <origin rpy="1.57 0 0" xyz="0 -0.2 0.2"/>
-    </joint>
-    <joint name="L_0a_fixed_3" type="fixed">
-        <parent link="L_0a"/>
-        <child link="L_0a_con3"/>
-        <axis rpy="0 0 0" xyz="0 0 1"/>
-        <origin rpy="0 0 0" xyz="0 0 0.4"/>
-    </joint>
-    <joint name="L_0a_fixed_4" type="fixed">
-        <parent link="L_0a"/>
-        <child link="L_0a_con4"/>
-        <axis rpy="0 0 0" xyz="0 0 1"/>
-        <origin rpy="-1.57 0 0" xyz="0 0.2 0.2"/>
-    </joint> -->
     <!-- Macro for adding a fixed joint (rigid interconnection between links) -->
     <xacro:macro name="add_fixed_joint" params="type name father child x y z roll pitch yaw">
@@ -220,8 +83,5 @@
                 </geometry>
             </collision>
-            <inertial>
-                <mass value="2"/>
-                <inertia ixx="1.0" ixy="0.0" ixz="0.0" iyy="1.0" iyz="0.0" izz="1.0"/>
-            </inertial>
+            <xacro:default_inertial mass="2"/>
         </link>
         <link name="${name}_con1">
@@ -238,8 +98,5 @@
                 </geometry>
             </collision>
-            <inertial>
-                <mass value="0.5"/>
-                <inertia ixx="1.0" ixy="0.0" ixz="0.0" iyy="1.0" iyz="0.0" izz="1.0"/>
-            </inertial>
+            <xacro:default_inertial mass="0.1"/>
         </link>
         <link name="${name}_con2">
@@ -256,8 +113,5 @@
                 </geometry>
             </collision>
-            <inertial>
-                <mass value="0.5"/>
-                <inertia ixx="1.0" ixy="0.0" ixz="0.0" iyy="1.0" iyz="0.0" izz="1.0"/>
-            </inertial>
+            <xacro:default_inertial mass="0.1"/>
         </link>
         <link name="${name}_con3">
@@ -274,8 +128,5 @@
                 </geometry>
             </collision>
-            <inertial>
-                <mass value="0.5"/>
-                <inertia ixx="1.0" ixy="0.0" ixz="0.0" iyy="1.0" iyz="0.0" izz="1.0"/>
-            </inertial>
+            <xacro:default_inertial mass="0.1"/>
         </link>
         <link name="${name}_con4">
@@ -292,8 +143,5 @@
                 </geometry>
             </collision>
-            <inertial>
-                <mass value="0.5"/>
-                <inertia ixx="1.0" ixy="0.0" ixz="0.0" iyy="1.0" iyz="0.0" izz="1.0"/>
-            </inertial>
+            <xacro:default_inertial mass="0.1"/>
         </link>
         <joint name="${name}_fixed_1" type="fixed">
@@ -337,8 +185,5 @@
                 </geometry>
             </collision>
-            <inertial>
-                <mass value="2"/>
-                <inertia ixx="1.0" ixy="0.0" ixz="0.0" iyy="1.0" iyz="0.0" izz="1.0"/>
-            </inertial>
+            <xacro:default_inertial mass="2.0"/>
         </link>
         <link name="${name}_con1">
@@ -355,8 +200,5 @@
                 </geometry>
             </collision>
-            <inertial>
-                <mass value="0.5"/>
-                <inertia ixx="1.0" ixy="0.0" ixz="0.0" iyy="1.0" iyz="0.0" izz="1.0"/>
-            </inertial>
+            <xacro:default_inertial mass="0.1"/>
         </link>
         <link name="${name}_con2">
@@ -373,8 +215,5 @@
                 </geometry>
             </collision>
-            <inertial>
-                <mass value="0.5"/>
-                <inertia ixx="1.0" ixy="0.0" ixz="0.0" iyy="1.0" iyz="0.0" izz="1.0"/>
-            </inertial>
+            <xacro:default_inertial mass="0.1"/>
         </link>
         <link name="${name}_con3">
@@ -391,8 +230,5 @@
                 </geometry>
             </collision>
-            <inertial>
-                <mass value="0.5"/>
-                <inertia ixx="1.0" ixy="0.0" ixz="0.0" iyy="1.0" iyz="0.0" izz="1.0"/>
-            </inertial>
+            <xacro:default_inertial mass="0.1"/>
         </link>
         <link name="${name}_con4">
@@ -409,8 +245,5 @@
                 </geometry>
             </collision>
-            <inertial>
-                <mass value="0.5"/>
-                <inertia ixx="1.0" ixy="0.0" ixz="0.0" iyy="1.0" iyz="0.0" izz="1.0"/>
-            </inertial>
+            <xacro:default_inertial mass="0.1"/>
         </link>
         <joint name="${name}_fixed_1" type="fixed">

Commit message: remove meshes from python

File: urdf/ModularBot_new.urdf.xacro (robot description, xacro)
@@ -567,6 +567,10 @@
     </xacro:macro>
     <!-- Macro for adding the physical module housing the actuator -->
-    <xacro:macro name="add_joint_stator" params="type name filename mesh_bool mesh_visual mesh_collision size_y size_z size x y z roll pitch yaw">
+    <xacro:macro name="add_joint_stator" params="type name filename size_y size_z size">
         <xacro:property name="module" value="${load_yaml(filename)}"/>
+        <xacro:property name="mesh_bool" value="false"/>
+        <xacro:unless value="${ module['visual']['mesh_body_1'] == '' }">
+            <xacro:property name="mesh_bool" value="true"/>
+        </xacro:unless>
         <xacro:if value="${size==1}">
             <xacro:property name="radius" value="${size1}" />
@@ -609,14 +613,18 @@
                 <visual>
                     <!-- Load mesh. Rotate the origin frame (this is because of how the .stl was saved) -->
-                    <origin rpy="${roll} ${pitch} ${yaw}" xyz="${x} ${y} ${z}"/>
+                    <origin
+                        rpy="${module['visual']['tf_mesh_1']['roll']} ${module['visual']['tf_mesh_1']['pitch']} ${module['visual']['tf_mesh_1']['yaw']}"
+                        xyz="${module['visual']['tf_mesh_1']['x']} ${module['visual']['tf_mesh_1']['y']} ${module['visual']['tf_mesh_1']['z']}"/>
                     <geometry>
-                        <mesh filename="${mesh_visual}" scale="0.001 0.001 0.001"/>
+                        <mesh filename="${module['visual']['mesh_body_1']}" scale="0.001 0.001 0.001"/>
                     </geometry>
                     <material name="grey"/>
                 </visual>
                 <collision>
-                    <origin rpy="${roll} ${pitch} ${yaw}" xyz="${x} ${y} ${z}"/>
+                    <origin
+                        rpy="${module['visual']['tf_mesh_1']['roll']} ${module['visual']['tf_mesh_1']['pitch']} ${module['visual']['tf_mesh_1']['yaw']}"
+                        xyz="${module['visual']['tf_mesh_1']['x']} ${module['visual']['tf_mesh_1']['y']} ${module['visual']['tf_mesh_1']['z']}"/>
                     <geometry>
-                        <mesh filename="${mesh_collision}" scale="0.001 0.001 0.001"/>
+                        <mesh filename="${module['visual']['mesh_collision_1']}" scale="0.001 0.001 0.001"/>
                     </geometry>
                 </collision>

Commit message: change xacro with cube mesh and read params from yaml

File: urdf/ModularBot_new.urdf.xacro (robot description, xacro)
@@ -62,5 +62,6 @@
     </xacro:macro>
     <!-- Macro for adding a master cube -->
-    <xacro:macro name="add_master_cube" params="name">
+    <xacro:macro name="add_master_cube" params="name filename">
+        <xacro:property name="module" value="${load_yaml(filename)}"/>
         <joint name="fixed" type="fixed">
             <parent link="base_link"/>
@@ -71,14 +72,16 @@
         <link name="${name}">
             <visual>
-                <origin rpy="0 0 0" xyz="0 0 0.2"/>
-                <geometry>
-                    <box size="0.4 0.4 0.4"/>
-                </geometry>
-                <material name="black"/>
-            </visual>
-            <collision>
-                <origin rpy="0 0 0" xyz="0 0 0.2"/>
-                <geometry>
-                    <box size="0.4 0.4 0.4"/>
+                <origin rpy="0 0 0" xyz="0 0 0.17"/>
+                <geometry>
+                    <!-- <box size="0.34 0.34 0.34"/> -->
+                    <mesh filename="${module['visual']['mesh_body_1']}" scale="0.001 0.001 0.001"/>
+                </geometry>
+                <!-- <material name="gray"/> -->
+            </visual>
+            <collision>
+                <origin rpy="0 0 0" xyz="0 0 0.17"/>
+                <geometry>
+                    <!-- <box size="0.34 0.34 0.34"/> -->
+                    <mesh filename="${module['visual']['mesh_collision_1']}" scale="0.001 0.001 0.001"/>
                 </geometry>
             </collision>
@@ -91,5 +94,5 @@
                     <cylinder length="0.1" radius="0.06"/>
                 </geometry>
-                <material name="black"/>
+                <material name="green"/>
             </visual>
             <collision>
@@ -106,5 +109,5 @@
                     <cylinder length="0.1" radius="0.06"/>
                 </geometry>
-                <material name="black"/>
+                <material name="green"/>
             </visual>
             <collision>
@@ -121,5 +124,5 @@
                     <cylinder length="0.1" radius="0.06"/>
                 </geometry>
-                <material name="black"/>
+                <material name="green"/>
             </visual>
             <collision>
@@ -136,5 +139,5 @@
                     <cylinder length="0.1" radius="0.06"/>
                 </geometry>
-                <material name="black"/>
+                <material name="green"/>
             </visual>
             <collision>
@@ -149,5 +152,6 @@
             <child link="${name}_con1"/>
             <axis rpy="0 0 0" xyz="0 0 1"/>
-            <origin rpy="3.14 0 0" xyz="0 0 0.0"/>
+            <origin rpy="${module['kinematics']['connector_1']['roll']} ${module['kinematics']['connector_1']['pitch']} ${module['kinematics']['connector_1']['yaw']}"
+                    xyz="${module['kinematics']['connector_1']['x']} ${module['kinematics']['connector_1']['y']} ${module['kinematics']['connector_1']['z']}"/>
         </joint>
         <joint name="${name}_fixed_2" type="fixed">
@@ -155,5 +159,6 @@
             <child link="${name}_con2"/>
             <axis rpy="0 0 0" xyz="0 0 1"/>
-            <origin rpy="1.57 0 0" xyz="0 -0.2 0.2"/>
+            <origin rpy="${module['kinematics']['connector_2']['roll']} ${module['kinematics']['connector_2']['pitch']} ${module['kinematics']['connector_2']['yaw']}"
+                    xyz="${module['kinematics']['connector_2']['x']} ${module['kinematics']['connector_2']['y']} ${module['kinematics']['connector_2']['z']}"/>
         </joint>
         <joint name="${name}_fixed_3" type="fixed">
@@ -161,5 +166,6 @@
             <child link="${name}_con3"/>
             <axis rpy="0 0 0" xyz="0 0 1"/>
-            <origin rpy="0 0 0" xyz="0 0 0.4"/>
+            <origin rpy="${module['kinematics']['connector_3']['roll']} ${module['kinematics']['connector_3']['pitch']} ${module['kinematics']['connector_3']['yaw']}"
+                    xyz="${module['kinematics']['connector_3']['x']} ${module['kinematics']['connector_3']['y']} ${module['kinematics']['connector_3']['z']}"/>
         </joint>
         <joint name="${name}_fixed_4" type="fixed">
@@ -167,20 +173,24 @@
             <child link="${name}_con4"/>
             <axis rpy="0 0 0" xyz="0 0 1"/>
-            <origin rpy="-1.57 0 0" xyz="0 0.2 0.2"/>
+            <origin rpy="${module['kinematics']['connector_4']['roll']} ${module['kinematics']['connector_4']['pitch']} ${module['kinematics']['connector_4']['yaw']}"
+                    xyz="${module['kinematics']['connector_4']['x']} ${module['kinematics']['connector_4']['y']} ${module['kinematics']['connector_4']['z']}"/>
         </joint>
     </xacro:macro>
     <!-- Macro for adding a slave cube -->
-    <xacro:macro name="add_slave_cube" params="name">
+    <xacro:macro name="add_slave_cube" params="name filename">
+        <xacro:property name="module" value="${load_yaml(filename)}"/>
         <link name="${name}">
             <visual>
-                <origin rpy="0 0 0" xyz="0 0 0.2"/>
-                <geometry>
-                    <box size="0.4 0.4 0.4"/>
-                </geometry>
-                <material name="black"/>
-            </visual>
-            <collision>
-                <geometry>
-                    <box size="0.4 0.4 0.4"/>
+                <origin rpy="0 0 0" xyz="0 0 0.17"/>
+                <geometry>
+                    <!-- <box size="0.34 0.34 0.34"/> -->
+                    <mesh filename="${module['visual']['mesh_body_1']}" scale="0.001 0.001 0.001"/>
+                </geometry>
+                <!-- <material name="grey"/> -->
+            </visual>
+            <collision>
+                <geometry>
+                    <!-- <box size="0.34 0.34 0.34"/> -->
+                    <mesh filename="${module['visual']['mesh_body_1']}" scale="0.001 0.001 0.001"/>
                 </geometry>
             </collision>
@@ -193,5 +203,5 @@
                     <cylinder length="0.1" radius="0.06"/>
                 </geometry>
-                <material name="black"/>
+                <material name="green"/>
             </visual>
             <collision>
@@ -208,5 +218,5 @@
                     <cylinder length="0.1" radius="0.06"/>
                 </geometry>
-                <material name="black"/>
+                <material name="green"/>
             </visual>
             <collision>
@@ -223,5 +233,5 @@
                     <cylinder length="0.1" radius="0.06"/>
                 </geometry>
-                <material name="black"/>
+                <material name="green"/>
             </visual>
             <collision>
@@ -238,5 +248,5 @@
                     <cylinder length="0.1" radius="0.06"/>
                 </geometry>
-                <material name="black"/>
+                <material name="green"/>
             </visual>
             <collision>
@@ -251,5 +261,5 @@
             <child link="${name}"/>
             <axis rpy="0 0 0" xyz="0 0 1"/>
-            <origin rpy="0 0 0" xyz="0 0 0.1"/>
+            <origin rpy="0 0 0" xyz="0 0 0.0"/>
         </joint>
         <joint name="${name}_fixed_2" type="fixed">
@@ -257,5 +267,6 @@
             <child link="${name}_con2"/>
             <axis rpy="0 0 0" xyz="0 0 1"/>
-            <origin rpy="1.57 0 0" xyz="0 -0.2 0.2"/>
+            <origin rpy="${module['kinematics']['connector_2']['roll']} ${module['kinematics']['connector_2']['pitch']} ${module['kinematics']['connector_2']['yaw']}"
+                    xyz="${module['kinematics']['connector_2']['x']} ${module['kinematics']['connector_2']['y']} ${module['kinematics']['connector_2']['z']}"/>
         </joint>
         <joint name="${name}_fixed_3" type="fixed">
@@ -263,5 +274,6 @@
             <child link="${name}_con3"/>
             <axis rpy="0 0 0" xyz="0 0 1"/>
-            <origin rpy="0 0 0" xyz="0 0 0.4"/>
+            <origin rpy="${module['kinematics']['connector_3']['roll']} ${module['kinematics']['connector_3']['pitch']} ${module['kinematics']['connector_3']['yaw']}"
+                    xyz="${module['kinematics']['connector_3']['x']} ${module['kinematics']['connector_3']['y']} ${module['kinematics']['connector_3']['z']}"/>
         </joint>
         <joint name="${name}_fixed_4" type="fixed">
@@ -269,5 +281,6 @@
             <child link="${name}_con4"/>
             <axis rpy="0 0 0" xyz="0 0 1"/>
-            <origin rpy="-1.57 0 0" xyz="0 0.2 0.2"/>
+            <origin rpy="${module['kinematics']['connector_4']['roll']} ${module['kinematics']['connector_4']['pitch']} ${module['kinematics']['connector_4']['yaw']}"
+                    xyz="${module['kinematics']['connector_4']['x']} ${module['kinematics']['connector_4']['y']} ${module['kinematics']['connector_4']['z']}"/>
         </joint>
     </xacro:macro>
