Commit message: change radius of "connectors"

File: urdf/ModularBot_new.urdf.xacro (robot description, xacro)
@@ -12,4 +12,5 @@
     <xacro:property name="size2" value="0.055" />
     <xacro:property name="size3" value="0.06" />
+    <xacro:property name="size_con" value="0.045" />
     <!-- <xacro:property name="leglen" value="0.3" /> -->
     <xacro:property name="len1" value="0.4" />
@@ -92,5 +93,5 @@
                 <origin rpy="0 0 0" xyz="0 0 0.05"/>
                 <geometry>
-                    <cylinder length="0.1" radius="0.06"/>
+                    <cylinder length="0.1" radius="${size_con}"/>
                 </geometry>
                 <material name="green"/>
@@ -98,5 +99,5 @@
             <collision>
                 <geometry>
-                    <cylinder length="0.1" radius="0.06"/>
+                    <cylinder length="0.1" radius="${size_con}"/>
                 </geometry>
             </collision>
@@ -107,5 +108,5 @@
                 <origin rpy="0 0 0" xyz="0 0 0.05"/>
                 <geometry>
-                    <cylinder length="0.1" radius="0.06"/>
+                    <cylinder length="0.1" radius="${size_con}"/>
                 </geometry>
                 <material name="green"/>
@@ -113,5 +114,5 @@
             <collision>
                 <geometry>
-                    <cylinder length="0.1" radius="0.06"/>
+                    <cylinder length="0.1" radius="${size_con}"/>
                 </geometry>
             </collision>
@@ -122,5 +123,5 @@
                 <origin rpy="0 0 0" xyz="0 0 0.05"/>
                 <geometry>
-                    <cylinder length="0.1" radius="0.06"/>
+                    <cylinder length="0.1" radius="${size_con}"/>
                 </geometry>
                 <material name="green"/>
@@ -128,5 +129,5 @@
             <collision>
                 <geometry>
-                    <cylinder length="0.1" radius="0.06"/>
+                    <cylinder length="0.1" radius="${size_con}"/>
                 </geometry>
             </collision>
@@ -137,5 +138,5 @@
                 <origin rpy="0 0 0" xyz="0 0 0.05"/>
                 <geometry>
-                    <cylinder length="0.1" radius="0.06"/>
+                    <cylinder length="0.1" radius="${size_con}"/>
                 </geometry>
                 <material name="green"/>
@@ -143,5 +144,5 @@
             <collision>
                 <geometry>
-                    <cylinder length="0.1" radius="0.06"/>
+                    <cylinder length="0.1" radius="${size_con}"/>
                 </geometry>
             </collision>
@@ -201,5 +202,5 @@
                 <origin rpy="0 0 0" xyz="0 0 0.05"/>
                 <geometry>
-                    <cylinder length="0.1" radius="0.06"/>
+                    <cylinder length="0.1" radius="${size_con}"/>
                 </geometry>
                 <material name="green"/>
@@ -207,5 +208,5 @@
             <collision>
                 <geometry>
-                    <cylinder length="0.1" radius="0.06"/>
+                    <cylinder length="0.1" radius="${size_con}"/>
                 </geometry>
             </collision>
@@ -216,5 +217,5 @@
                 <origin rpy="0 0 0" xyz="0 0 0.05"/>
                 <geometry>
-                    <cylinder length="0.1" radius="0.06"/>
+                    <cylinder length="0.1" radius="${size_con}"/>
                 </geometry>
                 <material name="green"/>
@@ -222,5 +223,5 @@
             <collision>
                 <geometry>
-                    <cylinder length="0.1" radius="0.06"/>
+                    <cylinder length="0.1" radius="${size_con}"/>
                 </geometry>
             </collision>
@@ -231,5 +232,5 @@
                 <origin rpy="0 0 0" xyz="0 0 0.05"/>
                 <geometry>
-                    <cylinder length="0.1" radius="0.06"/>
+                    <cylinder length="0.1" radius="${size_con}"/>
                 </geometry>
                 <material name="green"/>
@@ -237,5 +238,5 @@
             <collision>
                 <geometry>
-                    <cylinder length="0.1" radius="0.06"/>
+                    <cylinder length="0.1" radius="${size_con}"/>
                 </geometry>
             </collision>
@@ -246,5 +247,5 @@
                 <origin rpy="0 0 0" xyz="0 0 0.05"/>
                 <geometry>
-                    <cylinder length="0.1" radius="0.06"/>
+                    <cylinder length="0.1" radius="${size_con}"/>
                 </geometry>
                 <material name="green"/>
@@ -252,5 +253,5 @@
             <collision>
                 <geometry>
-                    <cylinder length="0.1" radius="0.06"/>
+                    <cylinder length="0.1" radius="${size_con}"/>
                 </geometry>
             </collision>

Commit message: remove inertias and collision from connections

File: urdf/ModularBot_new.urdf.xacro (robot description, xacro)
@@ -97,12 +97,15 @@
                 <material name="green"/>
             </visual>
-            <collision>
+        </link>
+        <link name="${name}_con2">
+            <visual>
+                <origin rpy="0 0 0" xyz="0 0 0.05"/>
                 <geometry>
                     <cylinder length="0.1" radius="${size_con}"/>
                 </geometry>
-            </collision>
-            <xacro:default_inertial mass="0.1"/>
-        </link>
-        <link name="${name}_con2">
+                <material name="green"/>
+            </visual>
+        </link>
+        <link name="${name}_con3">
             <visual>
                 <origin rpy="0 0 0" xyz="0 0 0.05"/>
@@ -112,40 +115,13 @@
                 <material name="green"/>
             </visual>
-            <collision>
+        </link>
+        <link name="${name}_con4">
+            <visual>
+                <origin rpy="0 0 0" xyz="0 0 0.05"/>
                 <geometry>
                     <cylinder length="0.1" radius="${size_con}"/>
                 </geometry>
-            </collision>
-            <xacro:default_inertial mass="0.1"/>
-        </link>
-        <link name="${name}_con3">
-            <visual>
-                <origin rpy="0 0 0" xyz="0 0 0.05"/>
-                <geometry>
-                    <cylinder length="0.1" radius="${size_con}"/>
-                </geometry>
-                <material name="green"/>
-            </visual>
-            <collision>
-                <geometry>
-                    <cylinder length="0.1" radius="${size_con}"/>
-                </geometry>
-            </collision>
-            <xacro:default_inertial mass="0.1"/>
-        </link>
-        <link name="${name}_con4">
-            <visual>
-                <origin rpy="0 0 0" xyz="0 0 0.05"/>
-                <geometry>
-                    <cylinder length="0.1" radius="${size_con}"/>
-                </geometry>
-                <material name="green"/>
-            </visual>
-            <collision>
-                <geometry>
-                    <cylinder length="0.1" radius="${size_con}"/>
-                </geometry>
-            </collision>
-            <xacro:default_inertial mass="0.1"/>
+                <material name="green"/>
+            </visual>
         </link>
         <joint name="${name}_fixed_1" type="fixed">
@@ -206,12 +182,15 @@
                 <material name="green"/>
             </visual>
-            <collision>
+        </link>
+        <link name="${name}_con2">
+            <visual>
+                <origin rpy="0 0 0" xyz="0 0 0.05"/>
                 <geometry>
                     <cylinder length="0.1" radius="${size_con}"/>
                 </geometry>
-            </collision>
-            <xacro:default_inertial mass="0.1"/>
-        </link>
-        <link name="${name}_con2">
+                <material name="green"/>
+            </visual>
+        </link>
+        <link name="${name}_con3">
             <visual>
                 <origin rpy="0 0 0" xyz="0 0 0.05"/>
@@ -221,40 +200,13 @@
                 <material name="green"/>
             </visual>
-            <collision>
+        </link>
+        <link name="${name}_con4">
+            <visual>
+                <origin rpy="0 0 0" xyz="0 0 0.05"/>
                 <geometry>
                     <cylinder length="0.1" radius="${size_con}"/>
                 </geometry>
-            </collision>
-            <xacro:default_inertial mass="0.1"/>
-        </link>
-        <link name="${name}_con3">
-            <visual>
-                <origin rpy="0 0 0" xyz="0 0 0.05"/>
-                <geometry>
-                    <cylinder length="0.1" radius="${size_con}"/>
-                </geometry>
-                <material name="green"/>
-            </visual>
-            <collision>
-                <geometry>
-                    <cylinder length="0.1" radius="${size_con}"/>
-                </geometry>
-            </collision>
-            <xacro:default_inertial mass="0.1"/>
-        </link>
-        <link name="${name}_con4">
-            <visual>
-                <origin rpy="0 0 0" xyz="0 0 0.05"/>
-                <geometry>
-                    <cylinder length="0.1" radius="${size_con}"/>
-                </geometry>
-                <material name="green"/>
-            </visual>
-            <collision>
-                <geometry>
-                    <cylinder length="0.1" radius="${size_con}"/>
-                </geometry>
-            </collision>
-            <xacro:default_inertial mass="0.1"/>
+                <material name="green"/>
+            </visual>
         </link>
         <joint name="${name}_fixed_1" type="fixed">

Commit message: split cube and connectors in xacro
in this way it is easier to remove them when deploying

File: urdf/ModularBot_new.urdf.xacro (robot description, xacro)
@@ -12,5 +12,5 @@
     <xacro:property name="size2" value="0.055" />
     <xacro:property name="size3" value="0.06" />
-    <xacro:property name="size_con" value="0.045" />
+    <xacro:property name="size_interface" value="0.045" />
     <!-- <xacro:property name="leglen" value="0.3" /> -->
     <xacro:property name="len1" value="0.4" />
@@ -63,5 +63,5 @@
     </xacro:macro>
     <!-- Macro for adding a master cube -->
-    <xacro:macro name="add_master_cube" params="name filename">
+    <xacro:macro name="add_master_cube" params="name filename type">
         <xacro:property name="module" value="${load_yaml(filename)}"/>
         <joint name="fixed" type="fixed">
@@ -89,9 +89,12 @@
             <xacro:default_inertial mass="2"/>
         </link>
+    </xacro:macro>
+    <xacro:macro name="add_connectors" params="name filename type">
+        <xacro:property name="module" value="${load_yaml(filename)}"/>
         <link name="${name}_con1">
             <visual>
                 <origin rpy="0 0 0" xyz="0 0 0.05"/>
                 <geometry>
-                    <cylinder length="0.1" radius="${size_con}"/>
+                    <cylinder length="0.1" radius="${size_interface}"/>
                 </geometry>
                 <material name="green"/>
@@ -102,5 +105,5 @@
                 <origin rpy="0 0 0" xyz="0 0 0.05"/>
                 <geometry>
-                    <cylinder length="0.1" radius="${size_con}"/>
+                    <cylinder length="0.1" radius="${size_interface}"/>
                 </geometry>
                 <material name="green"/>
@@ -111,5 +114,5 @@
                 <origin rpy="0 0 0" xyz="0 0 0.05"/>
                 <geometry>
-                    <cylinder length="0.1" radius="${size_con}"/>
+                    <cylinder length="0.1" radius="${size_interface}"/>
                 </geometry>
                 <material name="green"/>
@@ -120,5 +123,5 @@
                 <origin rpy="0 0 0" xyz="0 0 0.05"/>
                 <geometry>
-                    <cylinder length="0.1" radius="${size_con}"/>
+                    <cylinder length="0.1" radius="${size_interface}"/>
                 </geometry>
                 <material name="green"/>
@@ -155,5 +158,5 @@
     </xacro:macro>
     <!-- Macro for adding a slave cube -->
-    <xacro:macro name="add_slave_cube" params="name filename">
+    <xacro:macro name="add_slave_cube" params="name filename type">
         <xacro:property name="module" value="${load_yaml(filename)}"/>
         <link name="${name}">
@@ -178,5 +181,5 @@
                 <origin rpy="0 0 0" xyz="0 0 0.05"/>
                 <geometry>
-                    <cylinder length="0.1" radius="${size_con}"/>
+                    <cylinder length="0.1" radius="${size_interface}"/>
                 </geometry>
                 <material name="green"/>
@@ -187,5 +190,5 @@
                 <origin rpy="0 0 0" xyz="0 0 0.05"/>
                 <geometry>
-                    <cylinder length="0.1" radius="${size_con}"/>
+                    <cylinder length="0.1" radius="${size_interface}"/>
                 </geometry>
                 <material name="green"/>
@@ -196,5 +199,5 @@
                 <origin rpy="0 0 0" xyz="0 0 0.05"/>
                 <geometry>
-                    <cylinder length="0.1" radius="${size_con}"/>
+                    <cylinder length="0.1" radius="${size_interface}"/>
                 </geometry>
                 <material name="green"/>
@@ -205,5 +208,5 @@
                 <origin rpy="0 0 0" xyz="0 0 0.05"/>
                 <geometry>
-                    <cylinder length="0.1" radius="${size_con}"/>
+                    <cylinder length="0.1" radius="${size_interface}"/>
                 </geometry>
                 <material name="green"/>

Commit message: add tool_exchanger module & update config file writer

File: urdf/ModularBot_new.urdf.xacro (robot description, xacro)
@@ -532,4 +532,56 @@
                     iyz="${module['dynamics']['body_2']['inertia_tensor']['I_yz']}"
                     izz="${module['dynamics']['body_2']['inertia_tensor']['I_zz']}"/>
+            </inertial>
+        </link>
+    </xacro:macro>
+    <xacro:macro name="add_tool_exchanger" params="type name filename">
+        <xacro:property name="module" value="${load_yaml(filename)}"/>
+        <!-- <xacro:property name="visual" value="${module['visual']['mesh_body_1']}"/> -->
+        <xacro:property name="mesh_bool" value="false"/>
+        <xacro:unless value="${ module['visual']['mesh_body_1'] == '' }">
+            <xacro:property name="mesh_bool" value="true"/>
+        </xacro:unless>
+        <link name="${name}">
+            <xacro:if value="${ mesh_bool }">
+                <visual>
+                    <!-- Load mesh. Rotate the origin frame (this is because of how the .stl was saved) -->
+                    <origin
+                        rpy="${module['visual']['tf_mesh_1']['roll']} ${module['visual']['tf_mesh_1']['pitch']} ${module['visual']['tf_mesh_1']['yaw']}"
+                        xyz="${module['visual']['tf_mesh_1']['x']} ${module['visual']['tf_mesh_1']['y']} ${module['visual']['tf_mesh_1']['z']}"/>
+                    <geometry>
+                        <mesh filename="${module['visual']['mesh_body_1']}" scale="0.001 0.001 0.001"/>
+                    </geometry>
+                    <material name="yellow"/>
+                </visual>
+                <collision>
+                    <origin
+                        rpy="${module['visual']['tf_mesh_1']['roll']} ${module['visual']['tf_mesh_1']['pitch']} ${module['visual']['tf_mesh_1']['yaw']}"
+                        xyz="${module['visual']['tf_mesh_1']['x']} ${module['visual']['tf_mesh_1']['y']} ${module['visual']['tf_mesh_1']['z']}"/>
+                    <geometry>
+                        <mesh filename="${module['visual']['mesh_collision_1']}" scale="0.001 0.001 0.001"/>
+                    </geometry>
+                </collision>
+            </xacro:if>
+            <!--inertial parameters for avocado rotating part. wrt a point on one end of the rod-->
+            <!-- <inertial>
+                <origin xyz="0 0 -0.002265" rpy="0 0 0"/>
+                <mass value="0.153466"/>
+                <inertia
+                        ixx="0.000034763" ixy="0.0" ixz="0.0"
+                        iyy="0.000034827" iyz="0.0"
+                        izz="0.000031822"/>
+            </inertial> -->
+            <inertial>
+                <origin
+                    xyz="${module['dynamics']['body_1']['CoM']['x']} ${module['dynamics']['body_1']['CoM']['y']} ${module['dynamics']['body_1']['CoM']['z']}"
+                    rpy="0 0 0"/>
+                <mass value="${module['dynamics']['body_1']['mass']}"/>
+                <inertia
+                    ixx="${module['dynamics']['body_1']['inertia_tensor']['I_xx']}"
+                    ixy="${module['dynamics']['body_1']['inertia_tensor']['I_xy']}"
+                    ixz="${module['dynamics']['body_1']['inertia_tensor']['I_xz']}"
+                    iyy="${module['dynamics']['body_1']['inertia_tensor']['I_yy']}"
+                    iyz="${module['dynamics']['body_1']['inertia_tensor']['I_yz']}"
+                    izz="${module['dynamics']['body_1']['inertia_tensor']['I_zz']}"/>
             </inertial>
         </link>

Commit message: change color of modules

File: urdf/ModularBot_new.urdf.xacro (robot description, xacro)
@@ -40,4 +40,7 @@
         <color rgba="1 1 0 1"/>
     </material>
+    <material name="tree_green">
+        <color rgba="0.13 0.54 0.13 1"/>
+    </material>
     <xacro:macro name="default_inertial" params="mass">
         <inertial>
@@ -501,4 +504,5 @@
                         <mesh filename="${module['visual']['mesh_body_2']}" scale="0.001 0.001 0.001"/>
                     </geometry>
+                    <material name="tree_green"/>
                 </visual>
                 <collision>
@@ -552,5 +556,5 @@
                         <mesh filename="${module['visual']['mesh_body_1']}" scale="0.001 0.001 0.001"/>
                     </geometry>
-                    <material name="yellow"/>
+                    <material name="black"/>
                 </visual>
                 <collision>
@@ -640,5 +644,5 @@
                         <mesh filename="${module['visual']['mesh_body_1']}" scale="0.001 0.001 0.001"/>
                     </geometry>
-                    <material name="grey"/>
+                    <material name="tree_green"/>
                 </visual>
                 <collision>

Commit message: HACK: add pen to tool-exchanger

File: urdf/ModularBot_new.urdf.xacro (robot description, xacro)
@@ -591,4 +591,13 @@
         </link>
     </xacro:macro>
+    <xacro:macro name="add_pen" params="type name father">
+        <link name="${name}">
+        <joint name="fixed_${name}" type="fixed">
+            <axis xyz="0 0 1" rpy="0 0 0" />
+            <parent link="${father}"/>
+            <child link="pen"/>
+            <origin xyz="0.0 0.0 0.0" rpy="0.0 0.0 0.0"/>
+        </joint>
+    <xacro:macro/>
     <!-- Macro for adding the physical module housing the actuator -->
     <xacro:macro name="add_joint_stator" params="type name filename size_y size_z size">

Commit message: correct pen length

File: urdf/ModularBot_new.urdf.xacro (robot description, xacro)
@@ -592,12 +592,12 @@
     </xacro:macro>
     <xacro:macro name="add_pen" params="type name father">
-        <link name="${name}">
+        <link name="${name}"/>
         <joint name="fixed_${name}" type="fixed">
             <axis xyz="0 0 1" rpy="0 0 0" />
             <parent link="${father}"/>
-            <child link="pen"/>
-            <origin xyz="0.0 0.0 0.0" rpy="0.0 0.0 0.0"/>
-        </joint>
-    <xacro:macro/>
+            <child link="${name}"/>
+            <origin xyz="0.0 0.0 0.222" rpy="0.0 0.0 0.0"/>
+        </joint>
+    </xacro:macro>
     <!-- Macro for adding the physical module housing the actuator -->
     <xacro:macro name="add_joint_stator" params="type name filename size_y size_z size">

Commit message: remove world from urdf -> conflict with RBDL

File: urdf/ModularBot_new.urdf.xacro (robot description, xacro)
@@ -50,9 +50,9 @@
     </xacro:macro>
     <!-- adding world link for Gazebo simulation -->
-    <link name="world"/>
+    <!-- <link name="world"/>
     <joint name="world" type="fixed">
         <parent link="world"/>
         <child link="base_link"/>
-    </joint>
+    </joint> -->
     <link name="base_link"/>
     <!-- Macro for adding a fixed joint (rigid interconnection between links) -->
