Commit message: wip - Fixed connectors for cube module

File: urdf/ModularBot_new.urdf.xacro (robot description, xacro)
@@ -95,5 +95,116 @@
     <xacro:macro name="add_connectors" params="name filename type">
         <xacro:property name="module" value="${load_yaml(filename)}"/>
-        <link name="${name}_con1">
+        <xacro:if value="${'connector_1' in module['kinematics']}">
+            <link name="${name}_con1">
+                <visual>
+                    <origin rpy="0 0 0" xyz="0 0 0.05"/>
+                    <geometry>
+                        <cylinder length="0.1" radius="${size_interface}"/>
+                    </geometry>
+                    <material name="green"/>
+                </visual>
+            </link>
+            <joint name="${name}_fixed_1" type="fixed">
+                <parent link="${name}"/>
+                <child link="${name}_con1"/>
+                <axis rpy="0 0 0" xyz="0 0 1"/>
+                <origin rpy="${module['kinematics']['connector_1']['roll']} ${module['kinematics']['connector_1']['pitch']} ${module['kinematics']['connector_1']['yaw']}"
+                        xyz="${module['kinematics']['connector_1']['x']} ${module['kinematics']['connector_1']['y']} ${module['kinematics']['connector_1']['z']}"/>
+            </joint>
+        </xacro:if>
+        <xacro:if value="${'connector_2' in module['kinematics']}">
+            <link name="${name}_con2">
+                <visual>
+                    <origin rpy="0 0 0" xyz="0 0 0.05"/>
+                    <geometry>
+                        <cylinder length="0.1" radius="${size_interface}"/>
+                    </geometry>
+                    <material name="green"/>
+                </visual>
+            </link>
+            <joint name="${name}_fixed_2" type="fixed">
+                <parent link="${name}"/>
+                <child link="${name}_con2"/>
+                <axis rpy="0 0 0" xyz="0 0 1"/>
+                <origin rpy="${module['kinematics']['connector_2']['roll']} ${module['kinematics']['connector_2']['pitch']} ${module['kinematics']['connector_2']['yaw']}"
+                        xyz="${module['kinematics']['connector_2']['x']} ${module['kinematics']['connector_2']['y']} ${module['kinematics']['connector_2']['z']}"/>
+            </joint>
+        </xacro:if>
+        <xacro:if value="${'connector_3' in module['kinematics']}">
+            <link name="${name}_con3">
+                <visual>
+                    <origin rpy="0 0 0" xyz="0 0 0.05"/>
+                    <geometry>
+                        <cylinder length="0.1" radius="${size_interface}"/>
+                    </geometry>
+                    <material name="green"/>
+                </visual>
+            </link>
+            <joint name="${name}_fixed_3" type="fixed">
+                <parent link="${name}"/>
+                <child link="${name}_con3"/>
+                <axis rpy="0 0 0" xyz="0 0 1"/>
+                <origin rpy="${module['kinematics']['connector_3']['roll']} ${module['kinematics']['connector_3']['pitch']} ${module['kinematics']['connector_3']['yaw']}"
+                        xyz="${module['kinematics']['connector_3']['x']} ${module['kinematics']['connector_3']['y']} ${module['kinematics']['connector_3']['z']}"/>
+            </joint>
+        </xacro:if>
+        <xacro:if value="${'connector_4' in module['kinematics']}">
+            <link name="${name}_con4">
+                <visual>
+                    <origin rpy="0 0 0" xyz="0 0 0.05"/>
+                    <geometry>
+                        <cylinder length="0.1" radius="${size_interface}"/>
+                    </geometry>
+                    <material name="green"/>
+                </visual>
+            </link>
+            <joint name="${name}_fixed_4" type="fixed">
+                <parent link="${name}"/>
+                <child link="${name}_con4"/>
+                <axis rpy="0 0 0" xyz="0 0 1"/>
+                <origin rpy="${module['kinematics']['connector_4']['roll']} ${module['kinematics']['connector_4']['pitch']} ${module['kinematics']['connector_4']['yaw']}"
+                        xyz="${module['kinematics']['connector_4']['x']} ${module['kinematics']['connector_4']['y']} ${module['kinematics']['connector_4']['z']}"/>
+            </joint>
+        </xacro:if>
+    </xacro:macro>
+    <!-- Macro for adding a slave cube -->
+    <xacro:macro name="add_slave_cube" params="name filename type">
+        <xacro:property name="module" value="${load_yaml(filename)}"/>
+        <link name="${name}">
+            <visual>
+                <origin rpy="0 0 0" xyz="0 0 0.17"/>
+                <geometry>
+                    <!-- <box size="0.34 0.34 0.34"/> -->
+                    <mesh filename="${module['visual']['mesh_body_1']}" scale="0.001 0.001 0.001"/>
+                </geometry>
+                <!-- <material name="grey"/> -->
+            </visual>
+            <collision>
+                <geometry>
+                    <!-- <box size="0.34 0.34 0.34"/> -->
+                    <mesh filename="${module['visual']['mesh_body_1']}" scale="0.001 0.001 0.001"/>
+                </geometry>
+            </collision>
+            <xacro:default_inertial mass="2.0"/>
+        </link>
+        <xacro:add_connectors name="${name}" filename="${filename}" type="${type}"/>
+        <!-- <xacro:if value="1"> -->
+            <!-- <link name="${name}_con1">
+                <visual>
+                    <origin rpy="0 0 0" xyz="0 0 0.05"/>
+                    <geometry>
+                        <cylinder length="0.1" radius="${size_interface}"/>
+                    </geometry>
+                    <material name="green"/>
+                </visual>
+            </link>
+            <joint name="${name}_fixed_1" type="fixed">
+                <parent link="${name}_con1"/>
+                <child link="${name}"/>
+                <origin rpy="${module['kinematics']['connector_1']['roll']} ${module['kinematics']['connector_1']['pitch']} ${module['kinematics']['connector_1']['yaw']}"
+                        xyz="${module['kinematics']['connector_1']['x']} ${module['kinematics']['connector_1']['y']} ${module['kinematics']['connector_1']['z']}"/>
+            </joint> -->
+        <!-- </xacro:if> -->
+        <!-- <link name="${name}_con2">
             <visual>
                 <origin rpy="0 0 0" xyz="0 0 0.05"/>
@@ -104,38 +215,4 @@
             </visual>
         </link>
-        <link name="${name}_con2">
-            <visual>
-                <origin rpy="0 0 0" xyz="0 0 0.05"/>
-                <geometry>
-                    <cylinder length="0.1" radius="${size_interface}"/>
-                </geometry>
-                <material name="green"/>
-            </visual>
-        </link>
-        <link name="${name}_con3">
-            <visual>
-                <origin rpy="0 0 0" xyz="0 0 0.05"/>
-                <geometry>
-                    <cylinder length="0.1" radius="${size_interface}"/>
-                </geometry>
-                <material name="green"/>
-            </visual>
-        </link>
-        <link name="${name}_con4">
-            <visual>
-                <origin rpy="0 0 0" xyz="0 0 0.05"/>
-                <geometry>
-                    <cylinder length="0.1" radius="${size_interface}"/>
-                </geometry>
-                <material name="green"/>
-            </visual>
-        </link>
-        <joint name="${name}_fixed_1" type="fixed">
-            <parent link="${name}"/>
-            <child link="${name}_con1"/>
-            <axis rpy="0 0 0" xyz="0 0 1"/>
-            <origin rpy="${module['kinematics']['connector_1']['roll']} ${module['kinematics']['connector_1']['pitch']} ${module['kinematics']['connector_1']['yaw']}"
-                    xyz="${module['kinematics']['connector_1']['x']} ${module['kinematics']['connector_1']['y']} ${module['kinematics']['connector_1']['z']}"/>
-        </joint>
         <joint name="${name}_fixed_2" type="fixed">
             <parent link="${name}"/>
@@ -145,4 +222,13 @@
                     xyz="${module['kinematics']['connector_2']['x']} ${module['kinematics']['connector_2']['y']} ${module['kinematics']['connector_2']['z']}"/>
         </joint>
+        <link name="${name}_con3">
+            <visual>
+                <origin rpy="0 0 0" xyz="0 0 0.05"/>
+                <geometry>
+                    <cylinder length="0.1" radius="${size_interface}"/>
+                </geometry>
+                <material name="green"/>
+            </visual>
+        </link>
         <joint name="${name}_fixed_3" type="fixed">
             <parent link="${name}"/>
@@ -151,6 +237,15 @@
             <origin rpy="${module['kinematics']['connector_3']['roll']} ${module['kinematics']['connector_3']['pitch']} ${module['kinematics']['connector_3']['yaw']}"
                     xyz="${module['kinematics']['connector_3']['x']} ${module['kinematics']['connector_3']['y']} ${module['kinematics']['connector_3']['z']}"/>
-        </joint>
-        <joint name="${name}_fixed_4" type="fixed">
+        </joint> -->
+        <!-- <link name="${name}_con4">
+            <visual>
+                <origin rpy="0 0 0" xyz="0 0 0.05"/>
+                <geometry>
+                    <cylinder length="0.1" radius="${size_interface}"/>
+                </geometry>
+                <material name="green"/>
+            </visual>
+        </link> -->
+        <!-- <joint name="${name}_fixed_4" type="fixed">
             <parent link="${name}"/>
             <child link="${name}_con4"/>
@@ -158,89 +253,5 @@
             <origin rpy="${module['kinematics']['connector_4']['roll']} ${module['kinematics']['connector_4']['pitch']} ${module['kinematics']['connector_4']['yaw']}"
                     xyz="${module['kinematics']['connector_4']['x']} ${module['kinematics']['connector_4']['y']} ${module['kinematics']['connector_4']['z']}"/>
-        </joint>
-    </xacro:macro>
-    <!-- Macro for adding a slave cube -->
-    <xacro:macro name="add_slave_cube" params="name filename type">
-        <xacro:property name="module" value="${load_yaml(filename)}"/>
-        <link name="${name}">
-            <visual>
-                <origin rpy="0 0 0" xyz="0 0 0.17"/>
-                <geometry>
-                    <!-- <box size="0.34 0.34 0.34"/> -->
-                    <mesh filename="${module['visual']['mesh_body_1']}" scale="0.001 0.001 0.001"/>
-                </geometry>
-                <!-- <material name="grey"/> -->
-            </visual>
-            <collision>
-                <geometry>
-                    <!-- <box size="0.34 0.34 0.34"/> -->
-                    <mesh filename="${module['visual']['mesh_body_1']}" scale="0.001 0.001 0.001"/>
-                </geometry>
-            </collision>
-            <xacro:default_inertial mass="2.0"/>
-        </link>
-        <link name="${name}_con1">
-            <visual>
-                <origin rpy="0 0 0" xyz="0 0 0.05"/>
-                <geometry>
-                    <cylinder length="0.1" radius="${size_interface}"/>
-                </geometry>
-                <material name="green"/>
-            </visual>
-        </link>
-        <link name="${name}_con2">
-            <visual>
-                <origin rpy="0 0 0" xyz="0 0 0.05"/>
-                <geometry>
-                    <cylinder length="0.1" radius="${size_interface}"/>
-                </geometry>
-                <material name="green"/>
-            </visual>
-        </link>
-        <link name="${name}_con3">
-            <visual>
-                <origin rpy="0 0 0" xyz="0 0 0.05"/>
-                <geometry>
-                    <cylinder length="0.1" radius="${size_interface}"/>
-                </geometry>
-                <material name="green"/>
-            </visual>
-        </link>
-        <link name="${name}_con4">
-            <visual>
-                <origin rpy="0 0 0" xyz="0 0 0.05"/>
-                <geometry>
-                    <cylinder length="0.1" radius="${size_interface}"/>
-                </geometry>
-                <material name="green"/>
-            </visual>
-        </link>
-        <joint name="${name}_fixed_1" type="fixed">
-            <parent link="${name}_con1"/>
-            <child link="${name}"/>
-            <axis rpy="0 0 0" xyz="0 0 1"/>
-            <origin rpy="0 0 0" xyz="0 0 0.0"/>
-        </joint>
-        <joint name="${name}_fixed_2" type="fixed">
-            <parent link="${name}"/>
-            <child link="${name}_con2"/>
-            <axis rpy="0 0 0" xyz="0 0 1"/>
-            <origin rpy="${module['kinematics']['connector_2']['roll']} ${module['kinematics']['connector_2']['pitch']} ${module['kinematics']['connector_2']['yaw']}"
-                    xyz="${module['kinematics']['connector_2']['x']} ${module['kinematics']['connector_2']['y']} ${module['kinematics']['connector_2']['z']}"/>
-        </joint>
-        <joint name="${name}_fixed_3" type="fixed">
-            <parent link="${name}"/>
-            <child link="${name}_con3"/>
-            <axis rpy="0 0 0" xyz="0 0 1"/>
-            <origin rpy="${module['kinematics']['connector_3']['roll']} ${module['kinematics']['connector_3']['pitch']} ${module['kinematics']['connector_3']['yaw']}"
-                    xyz="${module['kinematics']['connector_3']['x']} ${module['kinematics']['connector_3']['y']} ${module['kinematics']['connector_3']['z']}"/>
-        </joint>
-        <joint name="${name}_fixed_4" type="fixed">
-            <parent link="${name}"/>
-            <child link="${name}_con4"/>
-            <axis rpy="0 0 0" xyz="0 0 1"/>
-            <origin rpy="${module['kinematics']['connector_4']['roll']} ${module['kinematics']['connector_4']['pitch']} ${module['kinematics']['connector_4']['yaw']}"
-                    xyz="${module['kinematics']['connector_4']['x']} ${module['kinematics']['connector_4']['y']} ${module['kinematics']['connector_4']['z']}"/>
-        </joint>
+        </joint> -->
     </xacro:macro>
     <!-- Macro for adding a straight link -->
@@ -559,5 +570,5 @@
                         <mesh filename="${module['visual']['mesh_body_1']}" scale="0.001 0.001 0.001"/>
                     </geometry>
-                    <material name="black"/>
+                    <material name="tree_green"/>
                 </visual>
                 <collision>

Commit message: inertia scaled by the gear ratio: this is a workaround until we get the required parameters on xbotcore level

File: urdf/ModularBot_new.urdf.xacro (robot description, xacro)
@@ -483,8 +483,8 @@
                         ixz="${module['dynamics']['body_2_fast']['inertia_tensor']['I_xz'] }"
                         iyz="${module['dynamics']['body_2_fast']['inertia_tensor']['I_yz'] }"
-                        izz="${module['dynamics']['body_2_fast']['inertia_tensor']['I_zz'] }"/>
+                        izz="${ gear_ratio * gear_ratio * module['dynamics']['body_2_fast']['inertia_tensor']['I_zz'] }"/>
                         <!-- ixz="${ gear_ratio * module['dynamics']['body_2_fast']['inertia_tensor']['I_xz'] }" -->
                         <!-- iyz="${ gear_ratio * module['dynamics']['body_2_fast']['inertia_tensor']['I_yz'] }" -->
-                        <!-- izz="${ gear_ratio * gear_ratio * module['dynamics']['body_2_fast']['inertia_tensor']['I_zz'] }" -->
+                        <!-- izz="${module['dynamics']['body_2_fast']['inertia_tensor']['I_zz'] }" -->
             </inertial>
         </link>
@@ -601,5 +601,5 @@
             <parent link="${father}"/>
             <child link="${name}"/>
-            <origin xyz="0.0 0.0 0.222" rpy="0.0 0.0 0.0"/>
+            <origin xyz="0.0 0.0 0.233" rpy="0.0 0.0 0.0"/>
         </joint>
     </xacro:macro>

Commit message: wip

File: urdf/ModularBot_new.urdf.xacro (robot description, xacro)
@@ -56,4 +56,33 @@
     </joint> -->
     <link name="base_link"/>
+    <!-- Macro for adding a table -->
+    <xacro:macro name="add_table" params="type name father">
+        <joint name="fixed_table" type="fixed">
+            <axis rpy="0 0 0" xyz="0 0 1"/>
+            <parent link="${father}"/>
+            <child link="${name}"/>
+            <origin rpy="0.0 -0.0 0.0" xyz="0.0 0.0 0.0"/>
+        </joint>
+        <link name="${name}">
+            <visual>
+                <origin rpy="0 0 0" xyz="0.25 0 0.005"/>
+                <geometry>
+                    <box size="0.5 0.5 0.01"/>
+                </geometry>
+                <material name="gray"/>
+            </visual>
+            <collision>
+                <origin rpy="0 0 0" xyz="0.25 0 0.005"/>
+                <geometry>
+                    <box size="0.5 0.5 0.01"/>
+                </geometry>
+            </collision>
+            <inertial>
+                <origin rpy="0 0 0" xyz="0 0 0.00"/>
+                <mass value="0.5"/>
+                <inertia ixx="0.0006" ixy="0.0" ixz="0.0" iyy="0.0006" iyz="0.0" izz="0.0006"/>
+            </inertial>
+        </link>
+    </xacro:macro>
     <!-- Macro for adding a fixed joint (rigid interconnection between links) -->
     <xacro:macro name="add_fixed_joint" params="type name father child x y z roll pitch yaw">

Commit message: wip

File: urdf/ModularBot_new.urdf.xacro (robot description, xacro)
@@ -66,14 +66,14 @@
         <link name="${name}">
             <visual>
-                <origin rpy="0 0 0" xyz="0.25 0 0.005"/>
-                <geometry>
-                    <box size="0.5 0.5 0.01"/>
+                <origin rpy="0 0 0" xyz="0.3 0 -0.005"/>
+                <geometry>
+                    <box size="0.6 0.6 0.01"/>
                 </geometry>
                 <material name="gray"/>
             </visual>
             <collision>
-                <origin rpy="0 0 0" xyz="0.25 0 0.005"/>
-                <geometry>
-                    <box size="0.5 0.5 0.01"/>
+                <origin rpy="0 0 0" xyz="0.25 0 -0.005"/>
+                <geometry>
+                    <box size="0.6 0.6 0.01"/>
                 </geometry>
             </collision>
@@ -497,5 +497,5 @@
                 <!--</collision>-->
             <!--</xacro:if>-->
-            <!--&lt;!&ndash; inertial parameters for avocado rotating part. wrt a point on one end of the rod &ndash;&gt;-->
+            <!--&lt;!&ndash; inertial parameters for ORANGE rotating part. wrt a point on one end of the rod &ndash;&gt;-->
             <!--<inertial>-->
                 <!--<origin xyz="0 0 -0.0635" rpy="0 0 0"/>-->
@@ -558,5 +558,5 @@
                 </collision>
             </xacro:if>
-            <!--inertial parameters for avocado rotating part. wrt a point on one end of the rod-->
+            <!--inertial parameters for ORANGE rotating part. wrt a point on one end of the rod-->
             <!-- <inertial>
                 <origin xyz="0 0 -0.002265" rpy="0 0 0"/>
@@ -610,5 +610,5 @@
                 </collision>
             </xacro:if>
-            <!--inertial parameters for avocado rotating part. wrt a point on one end of the rod-->
+            <!--inertial parameters for ORANGE rotating part. wrt a point on one end of the rod-->
             <!-- <inertial>
                 <origin xyz="0 0 -0.002265" rpy="0 0 0"/>
@@ -643,4 +643,17 @@
             <origin xyz="0.0 0.0 0.222" rpy="0.0 0.0 0.0"/>
         </joint>
+    </xacro:macro>
+    <!-- Add a simple frame ("end-effector") for simulation purposes -->
+    <xacro:macro name="add_simple_ee" params="type name size_z">
+        <link name="${name}">
+            <inertial>
+                <origin xyz="0 0 ${size_z/2}" rpy="0 0 0"/>
+                <mass value="0.848"/>
+                <inertia
+                        ixx="1.1564566e-03" ixy="0.0" ixz="0.0"
+                        iyy="1.2469918e-03" iyz="0.0"
+                        izz="5.7388903e-04"/>
+            </inertial>
+        </link>
     </xacro:macro>
     <!-- Macro for adding the physical module housing the actuator -->
