Commit message: Add gripper support

File: urdf/ModularBot_new.urdf.xacro (robot description, xacro)
@@ -603,4 +603,76 @@
             <origin xyz="0.0 0.0 0.222" rpy="0.0 0.0 0.0"/>
         </joint>
+    </xacro:macro>
+    <xacro:macro name="add_gripper" params="type name filename">
+        <xacro:property name="module" value="${load_yaml(filename)}"/>
+        <!-- <xacro:property name="visual" value="${module['visual']['mesh_body_1']}"/> -->
+        <xacro:property name="mesh_bool" value="false"/>
+        <xacro:unless value="${ module['visual']['mesh_body_1'] == '' }">
+            <xacro:property name="mesh_bool" value="true"/>
+        </xacro:unless>
+        <link name="${name}">
+            <xacro:if value="${ mesh_bool }">
+                <visual>
+                    <!-- Load mesh. Rotate the origin frame (this is because of how the .stl was saved) -->
+                    <origin
+                        rpy="${module['visual']['tf_mesh_1']['roll']} ${module['visual']['tf_mesh_1']['pitch']} ${module['visual']['tf_mesh_1']['yaw']}"
+                        xyz="${module['visual']['tf_mesh_1']['x']} ${module['visual']['tf_mesh_1']['y']} ${module['visual']['tf_mesh_1']['z']}"/>
+                    <geometry>
+                        <mesh filename="${module['visual']['mesh_body_1']}" scale="0.001 0.001 0.001"/>
+                    </geometry>
+                    <material name="tree_green"/>
+                </visual>
+                <collision>
+                    <origin
+                        rpy="${module['visual']['tf_mesh_1']['roll']} ${module['visual']['tf_mesh_1']['pitch']} ${module['visual']['tf_mesh_1']['yaw']}"
+                        xyz="${module['visual']['tf_mesh_1']['x']} ${module['visual']['tf_mesh_1']['y']} ${module['visual']['tf_mesh_1']['z']}"/>
+                    <geometry>
+                        <mesh filename="${module['visual']['mesh_collision_1']}" scale="0.001 0.001 0.001"/>
+                    </geometry>
+                </collision>
+            </xacro:if>
+            <!--inertial parameters for ORANGE rotating part. wrt a point on one end of the rod-->
+            <!-- <inertial>
+                <origin xyz="0 0 -0.002265" rpy="0 0 0"/>
+                <mass value="0.153466"/>
+                <inertia
+                        ixx="0.000034763" ixy="0.0" ixz="0.0"
+                        iyy="0.000034827" iyz="0.0"
+                        izz="0.000031822"/>
+            </inertial> -->
+            <inertial>
+                <origin
+                    xyz="${module['dynamics']['body_1']['CoM']['x']} ${module['dynamics']['body_1']['CoM']['y']} ${module['dynamics']['body_1']['CoM']['z']}"
+                    rpy="0 0 0"/>
+                <mass value="${module['dynamics']['body_1']['mass']}"/>
+                <inertia
+                    ixx="${module['dynamics']['body_1']['inertia_tensor']['I_xx']}"
+                    ixy="${module['dynamics']['body_1']['inertia_tensor']['I_xy']}"
+                    ixz="${module['dynamics']['body_1']['inertia_tensor']['I_xz']}"
+                    iyy="${module['dynamics']['body_1']['inertia_tensor']['I_yy']}"
+                    iyz="${module['dynamics']['body_1']['inertia_tensor']['I_yz']}"
+                    izz="${module['dynamics']['body_1']['inertia_tensor']['I_zz']}"/>
+            </inertial>
+        </link>
+        <link name="TCP_${name}"/>
+        <joint name="fixed_TCP_${name}" type="fixed">
+            <axis xyz="0 0 1" rpy="0 0 0" />
+            <parent link="${name}"/>
+            <child link="TCP_${name}"/>
+            <origin xyz="0.0 0.0 0.1985" rpy="0.0 0.0 0.0"/>
+        </joint>
+    </xacro:macro>
+    <!-- Add a simple frame ("end-effector") for simulation purposes -->
+    <xacro:macro name="add_simple_ee" params="type name size_z">
+        <link name="${name}">
+            <inertial>
+                <origin xyz="0 0 ${size_z/2}" rpy="0 0 0"/>
+                <mass value="0.848"/>
+                <inertia
+                        ixx="1.1564566e-03" ixy="0.0" ixz="0.0"
+                        iyy="1.2469918e-03" iyz="0.0"
+                        izz="5.7388903e-04"/>
+            </inertial>
+        </link>
     </xacro:macro>
     <!-- Macro for adding the physical module housing the actuator -->

Commit message: refactor(xbot2): wip add_socket (to improve)
Co-authored-by: Edoardo Romiti <edoardo.romiti@iit.it>

File: urdf/ModularBot_new.urdf.xacro (robot description, xacro)
@@ -332,4 +332,55 @@
         </gazebo>
     </xacro:macro>
+    <!-- Macro for adding a straight link -->
+    <xacro:macro name="add_socket" params="name type filename size_z size">
+        <xacro:property name="module" value="${load_yaml(filename)}"/>
+        <xacro:property name="mesh_bool" value="false"/>
+        <!-- <xacro:unless value="${ module['visual']['mesh_body_1'] == '' }">
+            <xacro:property name="mesh_bool" value="true"/>
+        </xacro:unless> -->
+        <xacro:if value="${size==1}">
+            <xacro:property name="radius" value="${size1}" />
+        </xacro:if>
+        <xacro:unless value="${size==1}">
+            <xacro:if value="${size==2}">
+                <xacro:property name="radius" value="${size2}" />
+            </xacro:if>
+            <xacro:unless value="${size==2}">
+                <xacro:property name="radius" value="${size3}" />
+            </xacro:unless>
+        </xacro:unless>
+        <link name="${name}">
+            <visual>
+                <origin xyz="0 0 ${size_z/2}" rpy="0 0 0" />
+                <geometry>
+                    <cylinder radius="${radius}" length="${size_z}"/>
+                </geometry>
+                <material name="white"/>
+            </visual>
+            <collision>
+                <origin xyz="0 0 ${size_z/2}" rpy="0 0 0" />
+                <geometry>
+                    <cylinder radius="${radius}" length="${size_z}"/>
+                </geometry>
+            </collision>
+            <inertial>
+                <origin xyz="0 0 ${size_z/2}" rpy="0 0 0"/>
+                <mass value="${mass}"/>
+                <inertia
+                ixx="${mass / 12.0 * (3*radius*radius + size_z*size_z)}" ixy="0.0" ixz="0.0"
+                iyy="${mass / 12.0 * (size_z*size_z + 3*radius*radius)}" iyz="0.0"
+                izz="${mass / 2.0 * (radius*radius)}"/>
+            </inertial>
+        </link>
+        <gazebo reference="${name}">
+            <mu1>0.2</mu1>
+            <mu2>0.2</mu2>
+            <kp>1000000.0</kp>
+            <kd>1.0</kd>
+            <maxVel>0.0</maxVel>
+            <minDepth>0.0001</minDepth>
+            <material>Gazebo/White</material>
+        </gazebo>
+    </xacro:macro>
     <!-- Macro for adding a size adapter -->
     <xacro:macro name="add_size_adapter" params="type name size_z size_in size_out">
