Commit message: Updated URDF_writer.py and read_yaml.py
Computation of kin. param.  needed to write the URDF is updated to work with joint, link and elbow modules

File: web/static/urdf/elbow_module.urdf (robot description, URDF)
Before this commit: robot link_module, 1 links, 0 joints
Links:
- link None: geometry collision box size=0.1 0.1 0.2; collision box size=0.1 0.2 0.1

File: web/static/urdf/joint_module.urdf (robot description, URDF)
Before this commit: robot joint_module, 1 links, 1 joints
Joints:
- joint None: limit lower=-3.14 upper=3.14 -> lower=-3.14 upper=3.14 effort=35 velocity=5.7
