Commit message: Add gripper support
(includes bugfix from commit c3633161a83985c1e8f3d5f130dde6c81736dc5d)

File: src/modular/modular_data/urdf/ModularBot_library.urdf.xacro (robot description, xacro)
@@ -644,4 +644,63 @@
         </joint>
     </xacro:macro>
+    <xacro:macro name="add_gripper" params="type name filename">
+        <xacro:property name="module" value="${load_yaml(filename)}"/>
+        <!-- <xacro:property name="visual" value="${module['visual']['mesh_body_1']}"/> -->
+        <xacro:property name="mesh_bool" value="false"/>
+        <xacro:unless value="${ module['visual']['mesh_body_1'] == '' }">
+            <xacro:property name="mesh_bool" value="true"/>
+        </xacro:unless>
+        <link name="${name}">
+            <xacro:if value="${ mesh_bool }">
+                <visual>
+                    <!-- Load mesh. Rotate the origin frame (this is because of how the .stl was saved) -->
+                    <origin
+                        rpy="${module['visual']['tf_mesh_1']['roll']} ${module['visual']['tf_mesh_1']['pitch']} ${module['visual']['tf_mesh_1']['yaw']}"
+                        xyz="${module['visual']['tf_mesh_1']['x']} ${module['visual']['tf_mesh_1']['y']} ${module['visual']['tf_mesh_1']['z']}"/>
+                    <geometry>
+                        <mesh filename="${module['visual']['mesh_body_1']}" scale="0.001 0.001 0.001"/>
+                    </geometry>
+                    <material name="tree_green"/>
+                </visual>
+                <collision>
+                    <origin
+                        rpy="${module['visual']['tf_mesh_1']['roll']} ${module['visual']['tf_mesh_1']['pitch']} ${module['visual']['tf_mesh_1']['yaw']}"
+                        xyz="${module['visual']['tf_mesh_1']['x']} ${module['visual']['tf_mesh_1']['y']} ${module['visual']['tf_mesh_1']['z']}"/>
+                    <geometry>
+                        <mesh filename="${module['visual']['mesh_collision_1']}" scale="0.001 0.001 0.001"/>
+                    </geometry>
+                </collision>
+            </xacro:if>
+            <!--inertial parameters for ORANGE rotating part. wrt a point on one end of the rod-->
+            <!-- <inertial>
+                <origin xyz="0 0 -0.002265" rpy="0 0 0"/>
+                <mass value="0.153466"/>
+                <inertia
+                        ixx="0.000034763" ixy="0.0" ixz="0.0"
+                        iyy="0.000034827" iyz="0.0"
+                        izz="0.000031822"/>
+            </inertial> -->
+            <inertial>
+                <origin
+                    xyz="${module['dynamics']['body_1']['CoM']['x']} ${module['dynamics']['body_1']['CoM']['y']} ${module['dynamics']['body_1']['CoM']['z']}"
+                    rpy="0 0 0"/>
+                <mass value="${module['dynamics']['body_1']['mass']}"/>
+                <inertia
+                    ixx="${module['dynamics']['body_1']['inertia_tensor']['I_xx']}"
+                    ixy="${module['dynamics']['body_1']['inertia_tensor']['I_xy']}"
+                    ixz="${module['dynamics']['body_1']['inertia_tensor']['I_xz']}"
+                    iyy="${module['dynamics']['body_1']['inertia_tensor']['I_yy']}"
+                    iyz="${module['dynamics']['body_1']['inertia_tensor']['I_yz']}"
+                    izz="${module['dynamics']['body_1']['inertia_tensor']['I_zz']}"/>
+            </inertial>
+        </link>
+        <link name="TCP_${name}"/>
+        <joint name="fixed_TCP_${name}" type="fixed">
+            <axis xyz="0 0 1" rpy="0 0 0" />
+            <parent link="${name}"/>
+            <child link="TCP_${name}"/>
+            <origin xyz="0.0 0.0 0.1985" rpy="0.0 0.0 0.0"/>
+        </joint>
+    </xacro:macro>
     <!-- Add a simple frame ("end-effector") for simulation purposes -->
     <xacro:macro name="add_simple_ee" params="type name size_z">

Commit message: update urdf generation x xbot2 + config_file

File: src/modular/modular_data/urdf/ModularBot_library.urdf.xacro (robot description, xacro)
@@ -4,9 +4,14 @@
     <xacro:include filename="$(find modular)/urdf/modular.gazebo" /> -->
     <gazebo>
-        <plugin name="gazebo_xbot_plugin" filename="libGazeboXBotPlugin.so">
-            <!-- <path_to_config_file>${xbot_config_file}</path_to_config_file> -->
-            <path_to_config_file>configs/ADVR_shared/ModularBot/configs/config_ModularBot.yaml</path_to_config_file>
-        </plugin>
+        <plugin name="xbot2_gz_joint_server" filename="libxbot2_gz_joint_server.so">
+	        <pid>
+                <gain name="small_mot"  p="100"  d="5"/>
+                <!-- <pid name="J1_A" profile="small_mot"/> -->
+	        </pid>
+	    </plugin>
     </gazebo>
+    <xacro:macro name="add_xbot2_pid" params="name profile">
+        <pid name="${name}" profile="${profile}"/>
+    </xacro:macro>
     <xacro:property name="size1" value="0.05" />
     <xacro:property name="size2" value="0.055" />

Commit message: BUGFIX: solved error 'XacroException: unknown macro name: add_xbot2_pid'

File: src/modular/modular_data/urdf/ModularBot_library.urdf.xacro (robot description, xacro)
@@ -3,4 +3,7 @@
     <!-- <xacro:include filename="$(find modular)/urdf/config.xacro" />
     <xacro:include filename="$(find modular)/urdf/modular.gazebo" /> -->
+    <xacro:macro name="add_xbot2_pid" params="name profile">
+        <pid name="${name}" profile="${profile}"/>
+    </xacro:macro>
     <gazebo>
         <plugin name="xbot2_gz_joint_server" filename="libxbot2_gz_joint_server.so">
@@ -11,7 +14,4 @@
 	    </plugin>
     </gazebo>
-    <xacro:macro name="add_xbot2_pid" params="name profile">
-        <pid name="${name}" profile="${profile}"/>
-    </xacro:macro>
     <xacro:property name="size1" value="0.05" />
     <xacro:property name="size2" value="0.055" />

Commit message: update gripper to have indipendent fingers (xbot2-core gives errors)
updated meshes, added fingers as indipendent joints.
NOTE: xbot2 files need an update (probably the joint_map) because when xbot2-core is running, it print:
ERROR in getJointByName. Joint gripper_A_finger_joint1 is NOT defined!
[err ] in init_internal: model interface could not be loaded!
Model joint ordering must be chain-by-chain and inside each chain joints must go from base link to tip link!
[ok  ][xbot2-core] started running
[warn][jm_cli_homing] received aggregated rx with size 8 != 6
[warn][jm_cli_ros_ctrl] received aggregated rx with size 8 != 6

File: src/modular/modular_data/urdf/ModularBot_library.urdf.xacro (robot description, xacro)
@@ -651,5 +651,4 @@
     <xacro:macro name="add_gripper" params="type name filename">
         <xacro:property name="module" value="${load_yaml(filename)}"/>
-        <!-- <xacro:property name="visual" value="${module['visual']['mesh_body_1']}"/> -->
         <xacro:property name="mesh_bool" value="false"/>
         <xacro:unless value="${ module['visual']['mesh_body_1'] == '' }">
@@ -677,13 +676,4 @@
                 </collision>
             </xacro:if>
-            <!--inertial parameters for ORANGE rotating part. wrt a point on one end of the rod-->
-            <!-- <inertial>
-                <origin xyz="0 0 -0.002265" rpy="0 0 0"/>
-                <mass value="0.153466"/>
-                <inertia
-                        ixx="0.000034763" ixy="0.0" ixz="0.0"
-                        iyy="0.000034827" iyz="0.0"
-                        izz="0.000031822"/>
-            </inertial> -->
             <inertial>
                 <origin
@@ -700,4 +690,89 @@
             </inertial>
         </link>
+        <!-- add fingers -->
+        <link name="${name}_leftfinger">
+            <xacro:if value="${ mesh_bool }">
+                <visual>
+                    <geometry>
+                    <mesh filename="${module['visual']['mesh_body_2']}" scale="0.001 0.001 0.001"/>
+                    </geometry>
+                    <material name="grey"/>
+                </visual>
+                <collision>
+                    <geometry>
+                    <mesh filename="${module['visual']['mesh_collision_2']}" scale="0.001 0.001 0.001"/>
+                    </geometry>
+                </collision>
+            </xacro:if>
+            <!-- for simulation -->
+            <inertial>
+                <origin
+                    xyz="${module['dynamics']['body_2']['CoM']['x']} ${module['dynamics']['body_2']['CoM']['y']} ${module['dynamics']['body_2']['CoM']['z']}"
+                    rpy="0 0 0"/>
+                <mass value="${module['dynamics']['body_2']['mass']}"/>
+                <inertia
+                    ixx="${module['dynamics']['body_2']['inertia_tensor']['I_xx']}"
+                    ixy="${module['dynamics']['body_2']['inertia_tensor']['I_xy']}"
+                    ixz="${module['dynamics']['body_2']['inertia_tensor']['I_xz']}"
+                    iyy="${module['dynamics']['body_2']['inertia_tensor']['I_yy']}"
+                    iyz="${module['dynamics']['body_2']['inertia_tensor']['I_yz']}"
+                    izz="${module['dynamics']['body_2']['inertia_tensor']['I_zz']}"/>
+            </inertial>
+        </link>
+        <link name="${name}_rightfinger">
+            <xacro:if value="${ mesh_bool }">
+                <visual>
+                    <origin xyz="0 0 0" rpy="0 0 ${pi}"/>
+                    <geometry>
+                    <mesh filename="${module['visual']['mesh_body_2']}" scale="0.001 0.001 0.001"/>
+                    </geometry>
+                    <material name="grey"/>
+                </visual>
+                <collision>
+                    <origin xyz="0 0 0" rpy="0 0 ${pi}"/>
+                    <geometry>
+                    <mesh filename="${module['visual']['mesh_collision_2']}" scale="0.001 0.001 0.001"/>
+                    </geometry>
+                </collision>
+            </xacro:if>
+            <!-- for simulation -->
+            <inertial>
+                <origin
+                    xyz="${module['dynamics']['body_2']['CoM']['x']} ${module['dynamics']['body_2']['CoM']['y']} ${module['dynamics']['body_2']['CoM']['z']}"
+                    rpy="0 0 0"/>
+                <mass value="${module['dynamics']['body_2']['mass']}"/>
+                <inertia
+                    ixx="${module['dynamics']['body_2']['inertia_tensor']['I_xx']}"
+                    ixy="${module['dynamics']['body_2']['inertia_tensor']['I_xy']}"
+                    ixz="${module['dynamics']['body_2']['inertia_tensor']['I_xz']}"
+                    iyy="${module['dynamics']['body_2']['inertia_tensor']['I_yy']}"
+                    iyz="${module['dynamics']['body_2']['inertia_tensor']['I_yz']}"
+                    izz="${module['dynamics']['body_2']['inertia_tensor']['I_zz']}"/>
+            </inertial>
+        </link>
+        <!-- Add joints -->
+        <joint name="${name}_finger_joint1" type="${module['kinematics']['joint']['joint']['type']}">
+            <parent link="${name}"/>
+            <child link="${name}_leftfinger"/>
+            <origin xyz="0 0 ${module['kinematics']['joint']['proximal']['p_pl']}" rpy="0 0 0"/>
+            <axis xyz="0 -1 0"/>
+            <limit effort="${module['kinematics']['joint']['joint']['effort']}"
+                lower="${module['kinematics']['joint']['joint']['lower_limit']}"
+                upper="${module['kinematics']['joint']['joint']['upper_limit']}"
+                velocity="${module['kinematics']['joint']['joint']['velocity']}"
+            />
+        </joint>
+        <joint name="${name}_finger_joint2" type="${module['kinematics']['joint']['joint']['type']}">
+            <parent link="${name}"/>
+            <child link="${name}_rightfinger"/>
+            <origin xyz="0 0 ${module['kinematics']['joint']['proximal']['p_pl']}" rpy="0 0 0"/>
+            <limit effort="${module['kinematics']['joint']['joint']['effort']}"
+                lower="${module['kinematics']['joint']['joint']['lower_limit']}"
+                upper="${module['kinematics']['joint']['joint']['upper_limit']}"
+                velocity="${module['kinematics']['joint']['joint']['velocity']}"
+            />
+            <axis xyz="0 1 0"/>
+        </joint>
+        <!-- Add TCP -->
         <link name="TCP_${name}"/>
         <joint name="fixed_TCP_${name}" type="fixed">
