Commit message: change height of robot origin

File: src/modular/modular_data/urdf/template.urdf.xacro (robot description, xacro)
@@ -16,5 +16,5 @@
             </joint>
         </xacro:unless>
-        <origin xyz="0.0 0.0 1.2" rpy="0 0 0" />
+        <origin xyz="0.0 0.0 0.8" rpy="0 0 0" />
     </xacro:if>
     <xacro:unless value="${ADD_FLOATING_BASE}">

Commit message: refactor(URDFWriter): `process_urdf` accepts args for xacro substitution

File: src/modular/modular_data/urdf/template.urdf.xacro (robot description, xacro)
@@ -3,6 +3,6 @@
     <xacro:include filename="ModularBot.library.urdf.xacro"/>
     <xacro:include filename="ModularBot.control.urdf.xacro"/>
-    <xacro:arg name="floating_joint" default="false"/>
-    <xacro:property name="ADD_FLOATING_BASE" value="$(arg floating_joint)" />
+    <xacro:arg name="floating_base" default="false"/>
+    <xacro:property name="ADD_FLOATING_BASE" value="$(arg floating_base)" />
     <xacro:arg name="gazebo_urdf" default="false"/>
     <xacro:property name="GAZEBO_URDF" value="$(arg gazebo_urdf)" />
