Commit message: feat (concert): add velodyne to concert mobile base

File: src/modular/modular_data/urdf/concert.sensors.urdf.xacro (robot description, xacro)
@@ -10,4 +10,10 @@
     <xacro:property name="ADD_T265_LEFT" value="true" />
     <xacro:property name="ADD_T265_RIGHT" value="true" />
+</xacro:if>
+<xacro:property name="ADD_VELODYNE_FRONT" value="false" />
+<xacro:property name="ADD_VELODYNE_BACK" value="false" />
+<xacro:if value="${ADD_VELODYNE}">
+    <xacro:property name="ADD_VELODYNE_FRONT" value="true" />
+    <xacro:property name="ADD_VELODYNE_BACK" value="true" />
 </xacro:if>
 <xacro:macro name="add_mobile_base_sensors" params="parent_name">
@@ -152,4 +158,46 @@
         <link name="${t265_right_name}_bottom_screw_frame"/>
     </xacro:unless>
+    <!-- Add Velodyne front -->
+    <xacro:property name="velodyne_front_name" value="velodyne_front" />
+    <xacro:property name="velodyne_front_parent_name" value="${parent_name}" />
+    <xacro:property name="velodyne_front_origin">
+        <origin xyz="0.5305 0.315 -0.1" rpy="0.0 0.0 -1.570796"/>
+    </xacro:property>
+    <xacro:if value="${ADD_VELODYNE_FRONT}">
+        <xacro:include filename="$(find velodyne_description)/urdf/VLP-16.urdf.xacro"/>
+        <xacro:VLP-16 parent="${velodyne_front_parent_name}" name="${velodyne_front_name}" topic="/${velodyne_front_name}_points" hz="10" samples="440">
+            <xacro:insert_block name="velodyne_front_origin" />
+        </xacro:VLP-16>
+    </xacro:if>
+    <xacro:unless value="${ADD_VELODYNE_FRONT}">
+        <!-- camera body, with origin at bottom screw mount -->
+        <joint name="${velodyne_front_name}_base_mount_joint" type="fixed">
+            <xacro:insert_block name="velodyne_front_origin"/>
+            <parent link="${velodyne_front_parent_name}"/>
+            <child link="${velodyne_front_name}_base_link"/>
+        </joint>
+        <link name="${velodyne_front_name}_base_link"/>
+    </xacro:unless>
+    <!-- Add Velodyne back -->
+    <xacro:property name="velodyne_back_name" value="velodyne_back" />
+    <xacro:property name="velodyne_back_parent_name" value="${parent_name}" />
+    <xacro:property name="velodyne_back_origin">
+        <origin xyz="-0.5305 -0.315 -0.1" rpy="0.0 0.0 1.570796"/>
+    </xacro:property>
+    <xacro:if value="${ADD_VELODYNE_BACK}">
+        <xacro:include filename="$(find velodyne_description)/urdf/VLP-16.urdf.xacro"/>
+        <xacro:VLP-16 parent="${velodyne_back_parent_name}" name="${velodyne_back_name}" topic="/${velodyne_back_name}_points" hz="10" samples="440">
+            <xacro:insert_block name="velodyne_back_origin" />
+        </xacro:VLP-16>
+    </xacro:if>
+    <xacro:unless value="${ADD_VELODYNE_BACK}">
+        <!-- camera body, with origin at bottom screw mount -->
+        <joint name="${velodyne_back_name}_base_mount_joint" type="fixed">
+            <xacro:insert_block name="velodyne_back_origin"/>
+            <parent link="${velodyne_back_parent_name}"/>
+            <child link="${velodyne_back_name}_base_link"/>
+        </joint>
+        <link name="${velodyne_back_name}_base_link"/>
+    </xacro:unless>
 </xacro:macro>
 </robot>

File: src/modular/modular_data/urdf/template.urdf.xacro (robot description, xacro)
@@ -9,4 +9,6 @@
     <xacro:arg name="realsense" default="false"/>
     <xacro:property name="ADD_CAMERAS" value="$(arg realsense)" />
+    <xacro:arg name="velodyne" default="false"/>
+    <xacro:property name="ADD_VELODYNE" value="$(arg velodyne)" />
     <!-- adding (or not) world link for Gazebo simulation -->
     <xacro:if value="${ADD_FLOATING_BASE}">

Commit message: feat(concert): add ultrasound sensor pose frames
No gazebo plugin is provided, so for now just the pose of each sensor has been added to the URDF

File: src/modular/modular_data/urdf/concert.sensors.urdf.xacro (robot description, xacro)
@@ -200,4 +200,60 @@
         <link name="${velodyne_back_name}_base_link"/>
     </xacro:unless>
+    <!-- Add front-left Bosch USS5 -->
+    <joint name="bosch_uss5_front_left_joint" type="fixed">
+        <origin xyz="0.5105 0.315 -0.129" rpy="0.0 1.963496 0.0"/>
+        <parent link="${parent_name}"/>
+        <child link="bosch_uss5_front_left"/>
+    </joint>
+    <link name="bosch_uss5_front_left"/>
+    <!-- Add front-right Bosch USS5 -->
+    <joint name="bosch_uss5_front_right_joint" type="fixed">
+        <origin xyz="0.5105 -0.315 -0.129" rpy="0.0 1.963496 0.0"/>
+        <parent link="${parent_name}"/>
+        <child link="bosch_uss5_front_right"/>
+    </joint>
+    <link name="bosch_uss5_front_right"/>
+    <!-- Add back-left Bosch USS5 -->
+    <joint name="bosch_uss5_back_left_joint" type="fixed">
+        <origin xyz="-0.5105 0.315 -0.129" rpy="0.0 1.963496 3.141593"/>
+        <parent link="${parent_name}"/>
+        <child link="bosch_uss5_back_left"/>
+    </joint>
+    <link name="bosch_uss5_back_left"/>
+    <!-- Add back-right Bosch USS5 -->
+    <joint name="bosch_uss5_back_right_joint" type="fixed">
+        <origin xyz="-0.5105 -0.315 -0.129" rpy="0.0 1.963496 3.141593"/>
+        <parent link="${parent_name}"/>
+        <child link="bosch_uss5_back_right"/>
+    </joint>
+    <link name="bosch_uss5_back_right"/>
+    <!-- Add left-front Bosch USS5 -->
+    <joint name="bosch_uss5_left_front_joint" type="fixed">
+        <origin xyz="0.4515 0.365 -0.117" rpy="0.0 1.963496 1.570796"/>
+        <parent link="${parent_name}"/>
+        <child link="bosch_uss5_left_front"/>
+    </joint>
+    <link name="bosch_uss5_left_front"/>
+    <!-- Add left-back Bosch USS5 -->
+    <joint name="bosch_uss5_left_back_joint" type="fixed">
+        <origin xyz="-0.4515 0.365 -0.117" rpy="0.0 1.963496 1.570796"/>
+        <parent link="${parent_name}"/>
+        <child link="bosch_uss5_left_back"/>
+    </joint>
+    <link name="bosch_uss5_left_back"/>
+    <!-- Add right-front Bosch USS5 -->
+    <joint name="bosch_uss5_right_front_joint" type="fixed">
+        <origin xyz="0.4515 -0.365 -0.117" rpy="0.0 1.963496 -1.570796"/>
+        <parent link="${parent_name}"/>
+        <child link="bosch_uss5_right_front"/>
+    </joint>
+    <link name="bosch_uss5_right_front"/>
+    <!-- Add right-back Bosch USS5 -->
+    <joint name="bosch_uss5_right_back_joint" type="fixed">
+        <origin xyz="-0.4515 -0.365 -0.117" rpy="0.0 1.963496 -1.570796"/>
+        <parent link="${parent_name}"/>
+        <child link="bosch_uss5_right_back"/>
+    </joint>
+    <link name="bosch_uss5_right_back"/>
 </xacro:macro>
 </robot>

Commit message: fix(concert): T265 `pose_frame` instead of `bottom_screw_frame`

File: src/modular/modular_data/urdf/concert.sensors.urdf.xacro (robot description, xacro)
@@ -122,7 +122,7 @@
             <xacro:insert_block name="t265_left_origin"/>
             <parent link="${t265_left_parent_name}"/>
-            <child link="${t265_left_name}_bottom_screw_frame"/>
-        </joint>
-        <link name="${t265_left_name}_bottom_screw_frame"/>
+            <child link="${t265_left_name}_pose_frame"/>
+        </joint>
+        <link name="${t265_left_name}_pose_frame"/>
     </xacro:unless>
     <!-- Add right T265 camera -->
@@ -154,7 +154,7 @@
             <xacro:insert_block name="t265_right_origin"/>
             <parent link="${t265_right_parent_name}"/>
-            <child link="${t265_right_name}_bottom_screw_frame"/>
-        </joint>
-        <link name="${t265_right_name}_bottom_screw_frame"/>
+            <child link="${t265_right_name}_pose_frame"/>
+        </joint>
+        <link name="${t265_right_name}_pose_frame"/>
     </xacro:unless>
     <!-- Add Velodyne front -->

Commit message: fix T left camera pose (hw change)

File: src/modular/modular_data/urdf/concert.sensors.urdf.xacro (robot description, xacro)
@@ -98,5 +98,5 @@
     <xacro:property name="t265_left_parent_name" value="${parent_name}" />
     <xacro:property name="t265_left_origin">
-        <origin xyz="-0.02375 0.37245 -0.062" rpy="0 0.0 1.570796"/>
+        <origin xyz="0.02375 0.37245 -0.062" rpy="3.141593 0.0 1.570796"/>
     </xacro:property>
     <xacro:if value="${ADD_T265_LEFT}">

Commit message: add `use_gpu_ray` flag to `xacro_mappings`

File: src/modular/modular_data/urdf/concert.sensors.urdf.xacro (robot description, xacro)
@@ -166,5 +166,5 @@
     <xacro:if value="${ADD_VELODYNE_FRONT}">
         <xacro:include filename="$(find velodyne_description)/urdf/VLP-16.urdf.xacro"/>
-        <xacro:VLP-16 parent="${velodyne_front_parent_name}" name="${velodyne_front_name}" topic="/${velodyne_front_name}_points" hz="10" samples="440">
+        <xacro:VLP-16 parent="${velodyne_front_parent_name}" name="${velodyne_front_name}" topic="/${velodyne_front_name}_points" hz="10" samples="440" gpu="${USE_GPU_RAY}">
             <xacro:insert_block name="velodyne_front_origin" />
         </xacro:VLP-16>
@@ -187,5 +187,5 @@
     <xacro:if value="${ADD_VELODYNE_BACK}">
         <xacro:include filename="$(find velodyne_description)/urdf/VLP-16.urdf.xacro"/>
-        <xacro:VLP-16 parent="${velodyne_back_parent_name}" name="${velodyne_back_name}" topic="/${velodyne_back_name}_points" hz="10" samples="440">
+        <xacro:VLP-16 parent="${velodyne_back_parent_name}" name="${velodyne_back_name}" topic="/${velodyne_back_name}_points" hz="10" samples="440" gpu="${USE_GPU_RAY}">
             <xacro:insert_block name="velodyne_back_origin" />
         </xacro:VLP-16>

File: src/modular/modular_data/urdf/template.urdf.xacro (robot description, xacro)
@@ -13,4 +13,6 @@
     <xacro:arg name="velodyne" default="false"/>
     <xacro:property name="ADD_VELODYNE" value="$(arg velodyne)" />
+    <xacro:arg name="use_gpu_ray" default="false"/>
+    <xacro:property name="USE_GPU_RAY" value="$(arg use_gpu_ray)" />
     <!-- adding (or not) world link for Gazebo simulation -->
     <xacro:if value="${ADD_FLOATING_BASE}">

Commit message: update reference frame for velodynes

File: src/modular/modular_data/urdf/concert.sensors.urdf.xacro (robot description, xacro)
@@ -162,5 +162,5 @@
     <xacro:property name="velodyne_front_parent_name" value="${parent_name}" />
     <xacro:property name="velodyne_front_origin">
-        <origin xyz="0.5305 0.315 -0.1" rpy="0.0 0.0 -1.570796"/>
+        <origin xyz="0.5305 0.315 -0.1" rpy="0.0 0.0 0.0"/>
     </xacro:property>
     <xacro:if value="${ADD_VELODYNE_FRONT}">
@@ -183,5 +183,5 @@
     <xacro:property name="velodyne_back_parent_name" value="${parent_name}" />
     <xacro:property name="velodyne_back_origin">
-        <origin xyz="-0.5305 -0.315 -0.1" rpy="0.0 0.0 1.570796"/>
+        <origin xyz="-0.5305 -0.315 -0.1" rpy="0.0 0.0 3.141593"/>
     </xacro:property>
     <xacro:if value="${ADD_VELODYNE_BACK}">

Commit message: upd velodyne topic names same as hw

File: src/modular/modular_data/urdf/concert.sensors.urdf.xacro (robot description, xacro)
@@ -159,5 +159,5 @@
     </xacro:unless>
     <!-- Add Velodyne front -->
-    <xacro:property name="velodyne_front_name" value="velodyne_front" />
+    <xacro:property name="velodyne_front_name" value="front_base" />
     <xacro:property name="velodyne_front_parent_name" value="${parent_name}" />
     <xacro:property name="velodyne_front_origin">
@@ -166,5 +166,5 @@
     <xacro:if value="${ADD_VELODYNE_FRONT}">
         <xacro:include filename="$(find velodyne_description)/urdf/VLP-16.urdf.xacro"/>
-        <xacro:VLP-16 parent="${velodyne_front_parent_name}" name="${velodyne_front_name}" topic="/${velodyne_front_name}_points" hz="10" samples="440" gpu="${USE_GPU_RAY}">
+        <xacro:VLP-16 parent="${velodyne_front_parent_name}" name="${velodyne_front_name}" topic="/${velodyne_front_name}/velodyne_points" hz="10" samples="440" gpu="${USE_GPU_RAY}">
             <xacro:insert_block name="velodyne_front_origin" />
         </xacro:VLP-16>
@@ -180,5 +180,5 @@
     </xacro:unless>
     <!-- Add Velodyne back -->
-    <xacro:property name="velodyne_back_name" value="velodyne_back" />
+    <xacro:property name="velodyne_back_name" value="back_base" />
     <xacro:property name="velodyne_back_parent_name" value="${parent_name}" />
     <xacro:property name="velodyne_back_origin">
@@ -187,5 +187,5 @@
     <xacro:if value="${ADD_VELODYNE_BACK}">
         <xacro:include filename="$(find velodyne_description)/urdf/VLP-16.urdf.xacro"/>
-        <xacro:VLP-16 parent="${velodyne_back_parent_name}" name="${velodyne_back_name}" topic="/${velodyne_back_name}_points" hz="10" samples="440" gpu="${USE_GPU_RAY}">
+        <xacro:VLP-16 parent="${velodyne_back_parent_name}" name="${velodyne_back_name}" topic="/${velodyne_back_name}/velodyne_points" hz="10" samples="440" gpu="${USE_GPU_RAY}">
             <xacro:insert_block name="velodyne_back_origin" />
         </xacro:VLP-16>
