Commit message: feat(concert.sensors): add Bosch USS5 ultrasound

File: src/modular/modular_data/urdf/concert.sensors.urdf.xacro (robot description, xacro)
@@ -192,5 +192,4 @@
     </xacro:if>
     <xacro:unless value="${ADD_VELODYNE_BACK}">
-        <!-- camera body, with origin at bottom screw mount -->
         <joint name="${velodyne_back_name}_base_mount_joint" type="fixed">
             <xacro:insert_block name="velodyne_back_origin"/>
@@ -200,60 +199,144 @@
         <link name="${velodyne_back_name}_base_link"/>
     </xacro:unless>
-    <!-- Add front-left Bosch USS5 -->
-    <joint name="bosch_uss5_front_left_joint" type="fixed">
+    <!-- Ultrasound sensors -->
+    <xacro:property name="ultrasound_parent_name" value="${parent_name}" />
+    <xacro:property name="ultrasound_ns" value="bosch_uss5" />
+    <!-- Macro for adding ultrasound sensor -->
+    <xacro:macro name="add_ultrasound_sensor" params="parent_name name topic *origin">
+        <joint name="${name}_base_mount_joint" type="fixed">
+            <xacro:insert_block name="origin" />
+            <parent link="${parent_name}"/>
+            <child link="${name}_base_link"/>
+        </joint>
+        <link name="${name}_base_link"/>
+        <!-- Rotate sensor frame (readings are on x axis instead of z) -->
+        <joint name="${name}_joint" type="fixed">
+            <origin xyz="0 0 0" rpy="0.0 -1.57 0.0"/>
+            <parent link="${name}_base_link"/>
+            <child link="${name}"/>
+        </joint>
+        <link name="${name}"/>
+        <xacro:if value="${ADD_ULTRASOUND}">
+            <xacro:add_ultrasound_gazebo name="${name}" topic="${topic}" />
+        </xacro:if>
+    </xacro:macro>
+    <!-- Macro for adding gazebo plugin for ultrasound sensors -->
+    <xacro:macro name="add_ultrasound_gazebo" params="name topic">
+        <gazebo reference="${name}">
+            <sensor type="ray" name="sonar">
+                <update_rate>5</update_rate>
+                <ray>
+                    <scan>
+                        <horizontal>
+                            <samples>5</samples>
+                            <resolution>1.0</resolution>
+                            <min_angle>-1.0</min_angle>
+                            <max_angle>1.0</max_angle>
+                        </horizontal>
+                        <vertical>
+                            <samples>5</samples>
+                            <resolution>1</resolution>
+                            <min_angle>-0.5</min_angle>
+                            <max_angle>0.5</max_angle>
+                        </vertical>
+                    </scan>
+                    <range>
+                        <min>0.2</min>
+                        <max>3.0</max>
+                        <resolution>0.01</resolution>
+                    </range>
+                </ray>
+                <plugin filename="libgazebo_ros_range.so" name="gazebo_ros_range">
+                    <gaussianNoise>0.005</gaussianNoise>
+                    <alwaysOn>true</alwaysOn>
+                    <updateRate>5</updateRate>
+                    <topicName>${topic}</topicName>
+                    <frameName>${name}</frameName>
+                    <fov>2.3</fov>
+                    <radiation>ultrasound</radiation>
+                </plugin>
+            </sensor>
+        </gazebo>
+    </xacro:macro>
+    <!-- Add front-left Bosch USS5 ultrasound sensor -->
+    <xacro:property name="ultrasound_front_left_sagittal_name" value="ultrasound_fl_sag" />
+    <xacro:property name="ultrasound_front_left_sagittal_origin">
         <origin xyz="0.5105 0.315 -0.129" rpy="0.0 1.963496 0.0"/>
-        <parent link="${parent_name}"/>
-        <child link="bosch_uss5_front_left"/>
-    </joint>
-    <link name="bosch_uss5_front_left"/>
-    <!-- Add front-right Bosch USS5 -->
-    <joint name="bosch_uss5_front_right_joint" type="fixed">
+    </xacro:property>
+    <xacro:add_ultrasound_sensor parent_name="${ultrasound_parent_name}"
+                            name="${ultrasound_front_left_sagittal_name}"
+                            topic="/${ultrasound_ns}/${ultrasound_front_left_sagittal_name}">
+        <xacro:insert_block name="ultrasound_front_left_sagittal_origin" />
+    </xacro:add_ultrasound_sensor>
+    <!-- Add front-right Bosch USS5 ultrasound sensor -->
+    <xacro:property name="ultrasound_front_right_sagittal_name" value="ultrasound_fr_sag" />
+    <xacro:property name="ultrasound_front_right_sagittal_origin">
         <origin xyz="0.5105 -0.315 -0.129" rpy="0.0 1.963496 0.0"/>
-        <parent link="${parent_name}"/>
-        <child link="bosch_uss5_front_right"/>
-    </joint>
-    <link name="bosch_uss5_front_right"/>
-    <!-- Add back-left Bosch USS5 -->
-    <joint name="bosch_uss5_back_left_joint" type="fixed">
+    </xacro:property>
+    <xacro:add_ultrasound_sensor parent_name="${ultrasound_parent_name}"
+                            name="${ultrasound_front_right_sagittal_name}"
+                            topic="/${ultrasound_ns}/${ultrasound_front_right_sagittal_name}">
+        <xacro:insert_block name="ultrasound_front_right_sagittal_origin" />
+    </xacro:add_ultrasound_sensor>
+    <!-- Add back-left Bosch USS5 ultrasound sensor -->
+    <xacro:property name="ultrasound_rear_left_sagittal_name" value="ultrasound_rl_sag" />
+    <xacro:property name="ultrasound_rear_left_sagittal_origin">
         <origin xyz="-0.5105 0.315 -0.129" rpy="0.0 1.963496 3.141593"/>
-        <parent link="${parent_name}"/>
-        <child link="bosch_uss5_back_left"/>
-    </joint>
-    <link name="bosch_uss5_back_left"/>
-    <!-- Add back-right Bosch USS5 -->
-    <joint name="bosch_uss5_back_right_joint" type="fixed">
+    </xacro:property>
+    <xacro:add_ultrasound_sensor parent_name="${ultrasound_parent_name}"
+                            name="${ultrasound_rear_left_sagittal_name}"
+                            topic="/${ultrasound_ns}/${ultrasound_rear_left_sagittal_name}">
+        <xacro:insert_block name="ultrasound_rear_left_sagittal_origin" />
+    </xacro:add_ultrasound_sensor>
+    <!-- Add back-right Bosch USS5 ultrasound sensor -->
+    <xacro:property name="ultrasound_rear_right_sagittal_name" value="ultrasound_rr_sag" />
+    <xacro:property name="ultrasound_rear_right_sagittal_origin">
         <origin xyz="-0.5105 -0.315 -0.129" rpy="0.0 1.963496 3.141593"/>
-        <parent link="${parent_name}"/>
-        <child link="bosch_uss5_back_right"/>
-    </joint>
-    <link name="bosch_uss5_back_right"/>
-    <!-- Add left-front Bosch USS5 -->
-    <joint name="bosch_uss5_left_front_joint" type="fixed">
+    </xacro:property>
+    <xacro:add_ultrasound_sensor parent_name="${ultrasound_parent_name}"
+                            name="${ultrasound_rear_right_sagittal_name}"
+                            topic="/${ultrasound_ns}/${ultrasound_rear_right_sagittal_name}">
+        <xacro:insert_block name="ultrasound_rear_right_sagittal_origin" />
+    </xacro:add_ultrasound_sensor>
+    <!-- Add left-front Bosch USS5 ultrasound sensor -->
+    <xacro:property name="ultrasound_front_left_lateral_name" value="ultrasound_fl_lat" />
+    <xacro:property name="ultrasound_front_left_lateral_origin">
         <origin xyz="0.4515 0.365 -0.117" rpy="0.0 1.963496 1.570796"/>
-        <parent link="${parent_name}"/>
-        <child link="bosch_uss5_left_front"/>
-    </joint>
-    <link name="bosch_uss5_left_front"/>
-    <!-- Add left-back Bosch USS5 -->
-    <joint name="bosch_uss5_left_back_joint" type="fixed">
+    </xacro:property>
+    <xacro:add_ultrasound_sensor parent_name="${ultrasound_parent_name}"
+                            name="${ultrasound_front_left_lateral_name}"
+                            topic="/${ultrasound_ns}/${ultrasound_front_left_lateral_name}">
+        <xacro:insert_block name="ultrasound_front_left_lateral_origin" />
+    </xacro:add_ultrasound_sensor>
+    <!-- Add left-back Bosch USS5 ultrasound sensor -->
+    <xacro:property name="ultrasound_rear_left_lateral_name" value="ultrasound_rl_lat" />
+    <xacro:property name="ultrasound_rear_left_lateral_origin">
         <origin xyz="-0.4515 0.365 -0.117" rpy="0.0 1.963496 1.570796"/>
-        <parent link="${parent_name}"/>
-        <child link="bosch_uss5_left_back"/>
-    </joint>
-    <link name="bosch_uss5_left_back"/>
-    <!-- Add right-front Bosch USS5 -->
-    <joint name="bosch_uss5_right_front_joint" type="fixed">
+    </xacro:property>
+    <xacro:add_ultrasound_sensor parent_name="${ultrasound_parent_name}"
+                            name="${ultrasound_rear_left_lateral_name}"
+                            topic="/${ultrasound_ns}/${ultrasound_rear_left_lateral_name}">
+        <xacro:insert_block name="ultrasound_rear_left_lateral_origin" />
+    </xacro:add_ultrasound_sensor>
+    <!-- Add right-front Bosch USS5 ultrasound sensor -->
+    <xacro:property name="ultrasound_front_right_lateral_name" value="ultrasound_fr_lat" />
+    <xacro:property name="ultrasound_front_right_lateral_origin">
         <origin xyz="0.4515 -0.365 -0.117" rpy="0.0 1.963496 -1.570796"/>
-        <parent link="${parent_name}"/>
-        <child link="bosch_uss5_right_front"/>
-    </joint>
-    <link name="bosch_uss5_right_front"/>
-    <!-- Add right-back Bosch USS5 -->
-    <joint name="bosch_uss5_right_back_joint" type="fixed">
+    </xacro:property>
+    <xacro:add_ultrasound_sensor parent_name="${ultrasound_parent_name}"
+                            name="${ultrasound_front_right_lateral_name}"
+                            topic="/${ultrasound_ns}/${ultrasound_front_right_lateral_name}">
+        <xacro:insert_block name="ultrasound_front_right_lateral_origin" />
+    </xacro:add_ultrasound_sensor>
+    <!-- Add right-back Bosch USS5 ultrasound sensor -->
+    <xacro:property name="ultrasound_rear_right_lateral_name" value="ultrasound_rr_lat" />
+    <xacro:property name="ultrasound_rear_right_lateral_origin">
         <origin xyz="-0.4515 -0.365 -0.117" rpy="0.0 1.963496 -1.570796"/>
-        <parent link="${parent_name}"/>
-        <child link="bosch_uss5_right_back"/>
-    </joint>
-    <link name="bosch_uss5_right_back"/>
+    </xacro:property>
+    <xacro:add_ultrasound_sensor parent_name="${ultrasound_parent_name}"
+                            name="${ultrasound_rear_right_lateral_name}"
+                            topic="/${ultrasound_ns}/${ultrasound_rear_right_lateral_name}">
+        <xacro:insert_block name="ultrasound_rear_right_lateral_origin" />
+    </xacro:add_ultrasound_sensor>
 </xacro:macro>
 </robot>

File: src/modular/modular_data/urdf/template.urdf.xacro (robot description, xacro)
@@ -13,4 +13,6 @@
     <xacro:arg name="velodyne" default="false"/>
     <xacro:property name="ADD_VELODYNE" value="$(arg velodyne)" />
+    <xacro:arg name="ultrasound" default="false"/>
+    <xacro:property name="ADD_ULTRASOUND" value="$(arg ultrasound)" />
     <xacro:arg name="use_gpu_ray" default="false"/>
     <xacro:property name="USE_GPU_RAY" value="$(arg use_gpu_ray)" />

Commit message: update velodynes ns and names

File: src/modular/modular_data/urdf/concert.sensors.urdf.xacro (robot description, xacro)
@@ -159,5 +159,5 @@
     </xacro:unless>
     <!-- Add Velodyne front -->
-    <xacro:property name="velodyne_front_name" value="front_base" />
+    <xacro:property name="velodyne_front_name" value="VLP16_lidar_front" />
     <xacro:property name="velodyne_front_parent_name" value="${parent_name}" />
     <xacro:property name="velodyne_front_origin">
@@ -180,5 +180,5 @@
     </xacro:unless>
     <!-- Add Velodyne back -->
-    <xacro:property name="velodyne_back_name" value="back_base" />
+    <xacro:property name="velodyne_back_name" value="VLP16_lidar_back" />
     <xacro:property name="velodyne_back_parent_name" value="${parent_name}" />
     <xacro:property name="velodyne_back_origin">

Commit message: add dalsa cameras frames to urdf

File: src/modular/modular_data/urdf/concert.sensors.urdf.xacro (robot description, xacro)
@@ -339,4 +339,19 @@
         <xacro:insert_block name="ultrasound_rear_right_lateral_origin" />
     </xacro:add_ultrasound_sensor>
+    <!-- Add Dalsa Cameras -->
+    <joint name="fixed_dalsa_camera_right" type="fixed">
+        <axis xyz="0 0 1" rpy="0 0 0" />
+        <parent link="base_link"/>
+        <child link="dalsa_camera_right"/>
+        <origin xyz="0.445 -0.285 0.074" rpy="0.0 -0.26179278697487707 -0.5235508063884032"/>
+    </joint>
+    <link name="dalsa_camera_right"/>
+    <joint name="fixed_dalsa_camera_left" type="fixed">
+        <axis xyz="0 0 1" rpy="0 0 0" />
+        <parent link="base_link"/>
+        <child link="dalsa_camera_left"/>
+        <origin xyz="0.445 0.285 0.074" rpy="0.0 -0.26179278697487707 0.5235508063884032"/>
+    </joint>
+    <link name="dalsa_camera_left"/>
 </xacro:macro>
 </robot>
