Commit message: refactor `concert.sensors`

File: src/modular/modular_data/urdf/concert.sensors.urdf.xacro (robot description, xacro)
@@ -24,36 +24,9 @@
         <origin xyz="0.402872 0.0 -0.078218" rpy="0 0.261799 0"/>
     </xacro:property>
-    <xacro:if value="${ADD_D435I_FRONT}">
-        <xacro:include filename="$(find realsense_gazebo_description)/urdf/_d435i.urdf.xacro" />
-        <xacro:sensor_d435i parent="${d435i_front_parent_name}"
-                            name="${d435i_front_name}"
-                            topics_ns="${d435i_front_name}"
-                            enable_pointCloud="true"
-                            align_depth="true"
-                            unite_imu_method="false"
-                            visualize="true"
-                            accel_fps="300"
-                            gyro_fps="300"
-                            depth_width="1280"
-                            depth_height="720"
-                            depth_fps="90"
-                            infra_width="1280"
-                            infra_height="720"
-                            infra_fps="90"
-                            color_width="1280"
-                            color_height="720"
-                            color_fps="30">
-            <xacro:insert_block name="d435i_front_origin" />
-        </xacro:sensor_d435i>
-    </xacro:if>
-    <xacro:unless value="${ADD_D435I_FRONT}">
-        <!-- camera body, with origin at bottom screw mount -->
-        <joint name="${d435i_front_name}_joint" type="fixed">
-            <xacro:insert_block name="d435i_front_origin"/>
-            <parent link="${d435i_front_parent_name}"/>
-            <child link="${d435i_front_name}_bottom_screw_frame"/>
-        </joint>
-        <link name="${d435i_front_name}_bottom_screw_frame"/>
-    </xacro:unless>
+    <xacro:add_realsense_d_camera name="${d435i_front_name}"
+                                parent_name="${d435i_front_parent_name}"
+                                add_gazebo_sensor="${ADD_D435I_FRONT}">
+        <xacro:insert_block name="d435i_front_origin" />
+    </xacro:add_realsense_d_camera>
     <!-- Add back D435i camera -->
     <xacro:property name="d435i_back_name" value="D435i_camera_back" />
@@ -62,36 +35,9 @@
         <origin xyz="-0.402872 0.0 -0.078218" rpy="0 0.261799 3.141593"/>
     </xacro:property>
-    <xacro:if value="${ADD_D435I_BACK}">
-        <xacro:include filename="$(find realsense_gazebo_description)/urdf/_d435i.urdf.xacro" />
-        <xacro:sensor_d435i parent="${d435i_back_parent_name}"
-                            name="${d435i_back_name}"
-                            topics_ns="${d435i_back_name}"
-                            enable_pointCloud="true"
-                            align_depth="true"
-                            unite_imu_method="false"
-                            visualize="true"
-                            accel_fps="300"
-                            gyro_fps="300"
-                            depth_width="1280"
-                            depth_height="720"
-                            depth_fps="90"
-                            infra_width="1280"
-                            infra_height="720"
-                            infra_fps="90"
-                            color_width="1280"
-                            color_height="720"
-                            color_fps="30">
-            <xacro:insert_block name="d435i_back_origin" />
-        </xacro:sensor_d435i>
-    </xacro:if>
-    <xacro:unless value="${ADD_D435I_BACK}">
-        <!-- camera body, with origin at bottom screw mount -->
-        <joint name="${d435i_back_name}_joint" type="fixed">
-            <xacro:insert_block name="d435i_back_origin"/>
-            <parent link="${d435i_back_parent_name}"/>
-            <child link="${d435i_back_name}_bottom_screw_frame"/>
-        </joint>
-        <link name="${d435i_back_name}_bottom_screw_frame"/>
-    </xacro:unless>
+    <xacro:add_realsense_d_camera name="${d435i_back_name}"
+                                parent_name="${d435i_back_parent_name}"
+                                add_gazebo_sensor="${ADD_D435I_BACK}">
+        <xacro:insert_block name="d435i_back_origin" />
+    </xacro:add_realsense_d_camera>
     <!-- Add left T265 camera -->
     <xacro:property name="t265_left_name" value="T265_camera_left" />
@@ -100,30 +46,9 @@
         <origin xyz="0.02375 0.37245 -0.062" rpy="3.141593 0.0 1.570796"/>
     </xacro:property>
-    <xacro:if value="${ADD_T265_LEFT}">
-        <xacro:include filename="$(find realsense_gazebo_description)/urdf/_t265.urdf.xacro" />
-        <xacro:sensor_t265  parent="${t265_left_parent_name}"
-                            name="${t265_left_name}"
-                            topics_ns="${t265_left_name}"
-                            odom_xyz="0.0 0.0 0.25"
-                            odom_rpy="0.0 0.0 0.0"
-                            odom_fps="262"
-                            fisheye_width="848"
-                            fisheye_height="800"
-                            fisheye_fps="30"
-                            unite_imu_method="false"
-                            accel_fps="62.5"
-                            gyro_fps="200">
-            <xacro:insert_block name="t265_left_origin" />
-        </xacro:sensor_t265>
-    </xacro:if>
-    <xacro:unless value="${ADD_T265_LEFT}">
-        <!-- camera body, with origin at bottom screw mount -->
-        <joint name="${t265_left_name}_joint" type="fixed">
-            <xacro:insert_block name="t265_left_origin"/>
-            <parent link="${t265_left_parent_name}"/>
-            <child link="${t265_left_name}_pose_frame"/>
-        </joint>
-        <link name="${t265_left_name}_pose_frame"/>
-    </xacro:unless>
+    <xacro:add_realsense_t_camera name="${t265_left_name}"
+                                parent_name="${t265_left_parent_name}"
+                                add_gazebo_sensor="${ADD_T265_LEFT}">
+        <xacro:insert_block name="t265_left_origin" />
+    </xacro:add_realsense_t_camera>
     <!-- Add right T265 camera -->
     <xacro:property name="t265_right_name" value="T265_camera_right" />
@@ -132,30 +57,9 @@
         <origin xyz="0.02375 -0.37245 -0.062" rpy="0 0.0 -1.570796"/>
     </xacro:property>
-    <xacro:if value="${ADD_T265_RIGHT}">
-        <xacro:include filename="$(find realsense_gazebo_description)/urdf/_t265.urdf.xacro" />
-        <xacro:sensor_t265  parent="${t265_right_parent_name}"
-                            name="${t265_right_name}"
-                            topics_ns="${t265_right_name}"
-                            odom_xyz="0.0 0.0 0.25"
-                            odom_rpy="0.0 0.0 0.0"
-                            odom_fps="262"
-                            fisheye_width="848"
-                            fisheye_height="800"
-                            fisheye_fps="30"
-                            unite_imu_method="false"
-                            accel_fps="62.5"
-                            gyro_fps="200">
-            <xacro:insert_block name="t265_right_origin" />
-        </xacro:sensor_t265>
-    </xacro:if>
-    <xacro:unless value="${ADD_T265_RIGHT}">
-        <!-- camera body, with origin at bottom screw mount -->
-        <joint name="${t265_right_name}_joint" type="fixed">
-            <xacro:insert_block name="t265_right_origin"/>
-            <parent link="${t265_right_parent_name}"/>
-            <child link="${t265_right_name}_pose_frame"/>
-        </joint>
-        <link name="${t265_right_name}_pose_frame"/>
-    </xacro:unless>
+    <xacro:add_realsense_t_camera name="${t265_right_name}"
+                                parent_name="${t265_right_parent_name}"
+                                add_gazebo_sensor="${ADD_T265_RIGHT}">
+        <xacro:insert_block name="t265_right_origin" />
+    </xacro:add_realsense_t_camera>
     <!-- Add Velodyne front -->
     <xacro:property name="velodyne_front_name" value="VLP16_lidar_front" />
@@ -221,5 +125,101 @@
         </xacro:if>
     </xacro:macro>
-    <!-- Macro for adding gazebo plugin for ultrasound sensors -->
+    <!-- Add front-left Bosch USS5 ultrasound sensor -->
+    <xacro:property name="ultrasound_front_left_sagittal_name" value="ultrasound_fl_sag" />
+    <xacro:property name="ultrasound_front_left_sagittal_origin">
+        <origin xyz="0.5105 0.315 -0.129" rpy="0.0 1.963496 0.0"/>
+    </xacro:property>
+    <xacro:add_ultrasound_sensor parent_name="${ultrasound_parent_name}"
+                            name="${ultrasound_front_left_sagittal_name}"
+                            topic="/${ultrasound_ns}/${ultrasound_front_left_sagittal_name}">
+        <xacro:insert_block name="ultrasound_front_left_sagittal_origin" />
+    </xacro:add_ultrasound_sensor>
+    <!-- Add front-right Bosch USS5 ultrasound sensor -->
+    <xacro:property name="ultrasound_front_right_sagittal_name" value="ultrasound_fr_sag" />
+    <xacro:property name="ultrasound_front_right_sagittal_origin">
+        <origin xyz="0.5105 -0.315 -0.129" rpy="0.0 1.963496 0.0"/>
+    </xacro:property>
+    <xacro:add_ultrasound_sensor parent_name="${ultrasound_parent_name}"
+                            name="${ultrasound_front_right_sagittal_name}"
+                            topic="/${ultrasound_ns}/${ultrasound_front_right_sagittal_name}">
+        <xacro:insert_block name="ultrasound_front_right_sagittal_origin" />
+    </xacro:add_ultrasound_sensor>
+    <!-- Add back-left Bosch USS5 ultrasound sensor -->
+    <xacro:property name="ultrasound_rear_left_sagittal_name" value="ultrasound_rl_sag" />
+    <xacro:property name="ultrasound_rear_left_sagittal_origin">
+        <origin xyz="-0.5105 0.315 -0.129" rpy="0.0 1.963496 3.141593"/>
+    </xacro:property>
+    <xacro:add_ultrasound_sensor parent_name="${ultrasound_parent_name}"
+                            name="${ultrasound_rear_left_sagittal_name}"
+                            topic="/${ultrasound_ns}/${ultrasound_rear_left_sagittal_name}">
+        <xacro:insert_block name="ultrasound_rear_left_sagittal_origin" />
+    </xacro:add_ultrasound_sensor>
+    <!-- Add back-right Bosch USS5 ultrasound sensor -->
+    <xacro:property name="ultrasound_rear_right_sagittal_name" value="ultrasound_rr_sag" />
+    <xacro:property name="ultrasound_rear_right_sagittal_origin">
+        <origin xyz="-0.5105 -0.315 -0.129" rpy="0.0 1.963496 3.141593"/>
+    </xacro:property>
+    <xacro:add_ultrasound_sensor parent_name="${ultrasound_parent_name}"
+                            name="${ultrasound_rear_right_sagittal_name}"
+                            topic="/${ultrasound_ns}/${ultrasound_rear_right_sagittal_name}">
+        <xacro:insert_block name="ultrasound_rear_right_sagittal_origin" />
+    </xacro:add_ultrasound_sensor>
+    <!-- Add left-front Bosch USS5 ultrasound sensor -->
+    <xacro:property name="ultrasound_front_left_lateral_name" value="ultrasound_fl_lat" />
+    <xacro:property name="ultrasound_front_left_lateral_origin">
+        <origin xyz="0.4515 0.365 -0.117" rpy="0.0 1.963496 1.570796"/>
+    </xacro:property>
+    <xacro:add_ultrasound_sensor parent_name="${ultrasound_parent_name}"
+                            name="${ultrasound_front_left_lateral_name}"
+                            topic="/${ultrasound_ns}/${ultrasound_front_left_lateral_name}">
+        <xacro:insert_block name="ultrasound_front_left_lateral_origin" />
+    </xacro:add_ultrasound_sensor>
+    <!-- Add left-back Bosch USS5 ultrasound sensor -->
+    <xacro:property name="ultrasound_rear_left_lateral_name" value="ultrasound_rl_lat" />
+    <xacro:property name="ultrasound_rear_left_lateral_origin">
+        <origin xyz="-0.4515 0.365 -0.117" rpy="0.0 1.963496 1.570796"/>
+    </xacro:property>
+    <xacro:add_ultrasound_sensor parent_name="${ultrasound_parent_name}"
+                            name="${ultrasound_rear_left_lateral_name}"
+                            topic="/${ultrasound_ns}/${ultrasound_rear_left_lateral_name}">
+        <xacro:insert_block name="ultrasound_rear_left_lateral_origin" />
+    </xacro:add_ultrasound_sensor>
+    <!-- Add right-front Bosch USS5 ultrasound sensor -->
+    <xacro:property name="ultrasound_front_right_lateral_name" value="ultrasound_fr_lat" />
+    <xacro:property name="ultrasound_front_right_lateral_origin">
+        <origin xyz="0.4515 -0.365 -0.117" rpy="0.0 1.963496 -1.570796"/>
+    </xacro:property>
+    <xacro:add_ultrasound_sensor parent_name="${ultrasound_parent_name}"
+                            name="${ultrasound_front_right_lateral_name}"
+                            topic="/${ultrasound_ns}/${ultrasound_front_right_lateral_name}">
+        <xacro:insert_block name="ultrasound_front_right_lateral_origin" />
+    </xacro:add_ultrasound_sensor>
+    <!-- Add right-back Bosch USS5 ultrasound sensor -->
+    <xacro:property name="ultrasound_rear_right_lateral_name" value="ultrasound_rr_lat" />
+    <xacro:property name="ultrasound_rear_right_lateral_origin">
+        <origin xyz="-0.4515 -0.365 -0.117" rpy="0.0 1.963496 -1.570796"/>
+    </xacro:property>
+    <xacro:add_ultrasound_sensor parent_name="${ultrasound_parent_name}"
+                            name="${ultrasound_rear_right_lateral_name}"
+                            topic="/${ultrasound_ns}/${ultrasound_rear_right_lateral_name}">
+        <xacro:insert_block name="ultrasound_rear_right_lateral_origin" />
+    </xacro:add_ultrasound_sensor>
+    <!-- Add Dalsa Cameras -->
+    <joint name="fixed_dalsa_camera_right" type="fixed">
+        <axis xyz="0 0 1" rpy="0 0 0" />
+        <parent link="base_link"/>
+        <child link="dalsa_camera_right"/>
+        <origin xyz="0.445 -0.285 0.074" rpy="0.0 -0.26179278697487707 -0.5235508063884032"/>
+    </joint>
+    <link name="dalsa_camera_right"/>
+    <joint name="fixed_dalsa_camera_left" type="fixed">
+        <axis xyz="0 0 1" rpy="0 0 0" />
+        <parent link="base_link"/>
+        <child link="dalsa_camera_left"/>
+        <origin xyz="0.445 0.285 0.074" rpy="0.0 -0.26179278697487707 0.5235508063884032"/>
+    </joint>
+    <link name="dalsa_camera_left"/>
+</xacro:macro>
+<!-- Macro for adding gazebo plugin for ultrasound sensors -->
     <xacro:macro name="add_ultrasound_gazebo" params="name topic">
         <gazebo reference="${name}">
@@ -259,99 +259,67 @@
         </gazebo>
     </xacro:macro>
-    <!-- Add front-left Bosch USS5 ultrasound sensor -->
-    <xacro:property name="ultrasound_front_left_sagittal_name" value="ultrasound_fl_sag" />
-    <xacro:property name="ultrasound_front_left_sagittal_origin">
-        <origin xyz="0.5105 0.315 -0.129" rpy="0.0 1.963496 0.0"/>
-    </xacro:property>
-    <xacro:add_ultrasound_sensor parent_name="${ultrasound_parent_name}"
-                            name="${ultrasound_front_left_sagittal_name}"
-                            topic="/${ultrasound_ns}/${ultrasound_front_left_sagittal_name}">
-        <xacro:insert_block name="ultrasound_front_left_sagittal_origin" />
-    </xacro:add_ultrasound_sensor>
-    <!-- Add front-right Bosch USS5 ultrasound sensor -->
-    <xacro:property name="ultrasound_front_right_sagittal_name" value="ultrasound_fr_sag" />
-    <xacro:property name="ultrasound_front_right_sagittal_origin">
-        <origin xyz="0.5105 -0.315 -0.129" rpy="0.0 1.963496 0.0"/>
-    </xacro:property>
-    <xacro:add_ultrasound_sensor parent_name="${ultrasound_parent_name}"
-                            name="${ultrasound_front_right_sagittal_name}"
-                            topic="/${ultrasound_ns}/${ultrasound_front_right_sagittal_name}">
-        <xacro:insert_block name="ultrasound_front_right_sagittal_origin" />
-    </xacro:add_ultrasound_sensor>
-    <!-- Add back-left Bosch USS5 ultrasound sensor -->
-    <xacro:property name="ultrasound_rear_left_sagittal_name" value="ultrasound_rl_sag" />
-    <xacro:property name="ultrasound_rear_left_sagittal_origin">
-        <origin xyz="-0.5105 0.315 -0.129" rpy="0.0 1.963496 3.141593"/>
-    </xacro:property>
-    <xacro:add_ultrasound_sensor parent_name="${ultrasound_parent_name}"
-                            name="${ultrasound_rear_left_sagittal_name}"
-                            topic="/${ultrasound_ns}/${ultrasound_rear_left_sagittal_name}">
-        <xacro:insert_block name="ultrasound_rear_left_sagittal_origin" />
-    </xacro:add_ultrasound_sensor>
-    <!-- Add back-right Bosch USS5 ultrasound sensor -->
-    <xacro:property name="ultrasound_rear_right_sagittal_name" value="ultrasound_rr_sag" />
-    <xacro:property name="ultrasound_rear_right_sagittal_origin">
-        <origin xyz="-0.5105 -0.315 -0.129" rpy="0.0 1.963496 3.141593"/>
-    </xacro:property>
-    <xacro:add_ultrasound_sensor parent_name="${ultrasound_parent_name}"
-                            name="${ultrasound_rear_right_sagittal_name}"
-                            topic="/${ultrasound_ns}/${ultrasound_rear_right_sagittal_name}">
-        <xacro:insert_block name="ultrasound_rear_right_sagittal_origin" />
-    </xacro:add_ultrasound_sensor>
-    <!-- Add left-front Bosch USS5 ultrasound sensor -->
-    <xacro:property name="ultrasound_front_left_lateral_name" value="ultrasound_fl_lat" />
-    <xacro:property name="ultrasound_front_left_lateral_origin">
-        <origin xyz="0.4515 0.365 -0.117" rpy="0.0 1.963496 1.570796"/>
-    </xacro:property>
-    <xacro:add_ultrasound_sensor parent_name="${ultrasound_parent_name}"
-                            name="${ultrasound_front_left_lateral_name}"
-                            topic="/${ultrasound_ns}/${ultrasound_front_left_lateral_name}">
-        <xacro:insert_block name="ultrasound_front_left_lateral_origin" />
-    </xacro:add_ultrasound_sensor>
-    <!-- Add left-back Bosch USS5 ultrasound sensor -->
-    <xacro:property name="ultrasound_rear_left_lateral_name" value="ultrasound_rl_lat" />
-    <xacro:property name="ultrasound_rear_left_lateral_origin">
-        <origin xyz="-0.4515 0.365 -0.117" rpy="0.0 1.963496 1.570796"/>
-    </xacro:property>
-    <xacro:add_ultrasound_sensor parent_name="${ultrasound_parent_name}"
-                            name="${ultrasound_rear_left_lateral_name}"
-                            topic="/${ultrasound_ns}/${ultrasound_rear_left_lateral_name}">
-        <xacro:insert_block name="ultrasound_rear_left_lateral_origin" />
-    </xacro:add_ultrasound_sensor>
-    <!-- Add right-front Bosch USS5 ultrasound sensor -->
-    <xacro:property name="ultrasound_front_right_lateral_name" value="ultrasound_fr_lat" />
-    <xacro:property name="ultrasound_front_right_lateral_origin">
-        <origin xyz="0.4515 -0.365 -0.117" rpy="0.0 1.963496 -1.570796"/>
-    </xacro:property>
-    <xacro:add_ultrasound_sensor parent_name="${ultrasound_parent_name}"
-                            name="${ultrasound_front_right_lateral_name}"
-                            topic="/${ultrasound_ns}/${ultrasound_front_right_lateral_name}">
-        <xacro:insert_block name="ultrasound_front_right_lateral_origin" />
-    </xacro:add_ultrasound_sensor>
-    <!-- Add right-back Bosch USS5 ultrasound sensor -->
-    <xacro:property name="ultrasound_rear_right_lateral_name" value="ultrasound_rr_lat" />
-    <xacro:property name="ultrasound_rear_right_lateral_origin">
-        <origin xyz="-0.4515 -0.365 -0.117" rpy="0.0 1.963496 -1.570796"/>
-    </xacro:property>
-    <xacro:add_ultrasound_sensor parent_name="${ultrasound_parent_name}"
-                            name="${ultrasound_rear_right_lateral_name}"
-                            topic="/${ultrasound_ns}/${ultrasound_rear_right_lateral_name}">
-        <xacro:insert_block name="ultrasound_rear_right_lateral_origin" />
-    </xacro:add_ultrasound_sensor>
-    <!-- Add Dalsa Cameras -->
-    <joint name="fixed_dalsa_camera_right" type="fixed">
-        <axis xyz="0 0 1" rpy="0 0 0" />
-        <parent link="base_link"/>
-        <child link="dalsa_camera_right"/>
-        <origin xyz="0.445 -0.285 0.074" rpy="0.0 -0.26179278697487707 -0.5235508063884032"/>
-    </joint>
-    <link name="dalsa_camera_right"/>
-    <joint name="fixed_dalsa_camera_left" type="fixed">
-        <axis xyz="0 0 1" rpy="0 0 0" />
-        <parent link="base_link"/>
-        <child link="dalsa_camera_left"/>
-        <origin xyz="0.445 0.285 0.074" rpy="0.0 -0.26179278697487707 0.5235508063884032"/>
-    </joint>
-    <link name="dalsa_camera_left"/>
+<!-- Macro for adding realsense D camera -->
+<xacro:macro name="add_realsense_d_camera" params="name parent_name *origin add_gazebo_sensor">
+    <xacro:if value="${add_gazebo_sensor}">
+        <xacro:include filename="$(find realsense_gazebo_description)/urdf/_d435i.urdf.xacro" />
+        <xacro:sensor_d435i parent="${parent_name}"
+                            name="${name}"
+                            topics_ns="${name}"
+                            enable_pointCloud="true"
+                            align_depth="true"
+                            unite_imu_method="false"
+                            visualize="true"
+                            accel_fps="300"
+                            gyro_fps="300"
+                            depth_width="1280"
+                            depth_height="720"
+                            depth_fps="90"
+                            infra_width="1280"
+                            infra_height="720"
+                            infra_fps="90"
+                            color_width="1280"
+                            color_height="720"
+                            color_fps="30">
+            <xacro:insert_block name="origin" />
+        </xacro:sensor_d435i>
+    </xacro:if>
+    <xacro:unless value="${add_gazebo_sensor}">
+        <!-- camera body, with origin at bottom screw mount -->
+        <joint name="${name}_joint" type="fixed">
+            <xacro:insert_block name="origin"/>
+            <parent link="${parent_name}"/>
+            <child link="${name}_bottom_screw_frame"/>
+        </joint>
+        <link name="${name}_bottom_screw_frame"/>
+    </xacro:unless>
+</xacro:macro>
+<!-- Macro for adding realsense T camera -->
+<xacro:macro name="add_realsense_t_camera" params="name parent_name *origin add_gazebo_sensor">
+    <xacro:if value="${add_gazebo_sensor}">
+        <xacro:include filename="$(find realsense_gazebo_description)/urdf/_t265.urdf.xacro" />
+        <xacro:sensor_t265  parent="${parent_name}"
+                            name="${name}"
+                            topics_ns="${name}"
+                            odom_xyz="0.0 0.0 0.25"
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