Commit message: upd concert lidar poses

File: src/modular/modular_data/urdf/concert.sensors.urdf.xacro (robot description, xacro)
@@ -73,5 +73,5 @@
     <xacro:property name="velodyne_front_parent_name" value="${parent_name}" />
     <xacro:property name="velodyne_front_origin">
-        <origin xyz="0.5305 0.315 -0.1" rpy="0.0 0.0 0.0"/>
+        <origin xyz="0.5305 0.315 -0.0627" rpy="3.141593 0.0 1.570796"/>
     </xacro:property>
     <xacro:if value="${ADD_VELODYNE_FRONT}">
@@ -94,5 +94,5 @@
     <xacro:property name="velodyne_back_parent_name" value="${parent_name}" />
     <xacro:property name="velodyne_back_origin">
-        <origin xyz="-0.5305 -0.315 -0.1" rpy="0.0 0.0 3.141593"/>
+        <origin xyz="-0.5305 -0.315 -0.0627" rpy="3.141593 0.0 -1.570796"/>
     </xacro:property>
     <xacro:if value="${ADD_VELODYNE_BACK}">

Commit message: upd concert lidar poses

File: src/modular/modular_data/urdf/concert.sensors.urdf.xacro (robot description, xacro)
@@ -67,5 +67,5 @@
     <xacro:property name="velodyne_front_parent_name" value="${parent_name}" />
     <xacro:property name="velodyne_front_origin">
-        <origin xyz="0.5305 0.315 -0.1" rpy="0.0 0.0 0.0"/>
+        <origin xyz="0.5305 0.315 -0.0627" rpy="3.141593 0.0 1.570796"/>
     </xacro:property>
     <xacro:if value="${ADD_VELODYNE_FRONT}">
@@ -88,5 +88,5 @@
     <xacro:property name="velodyne_back_parent_name" value="${parent_name}" />
     <xacro:property name="velodyne_back_origin">
-        <origin xyz="-0.5305 -0.315 -0.1" rpy="0.0 0.0 3.141593"/>
+        <origin xyz="-0.5305 -0.315 -0.0627" rpy="3.141593 0.0 -1.570796"/>
     </xacro:property>
     <xacro:if value="${ADD_VELODYNE_BACK}">

Commit message: add `base_link_projected` frame

File: src/modular/modular_data/urdf/concert.sensors.urdf.xacro (robot description, xacro)
@@ -19,4 +19,10 @@
 </xacro:if>
 <xacro:macro name="add_mobile_base_sensors" params="parent_name">
+	<joint name="base_link_projected_joint" type="fixed">
+        <parent link="base_link"/>
+        <child link="base_link_projected"/>
+        <origin xyz="0 0 -0.747" rpy="0 0 0"/>
+    </joint>
+    <link name="base_link_projected"/>
     <!-- Add front D435i camera -->
     <xacro:property name="d435i_front_name" value="D435i_camera_front" />

Commit message: Updated URDF file: Added IMU sensor and modified Velodyne lidar parameters
- Added IMU sensor with properties:
  - Included IMU xacro file.
  - Defined origin for the IMU sensor.
  - Attached IMU sensor to the robot with parent-child configuration.

- Modified Velodyne lidar sensor parameters:
  - Updated 'VLP-16-gz-sensor' for front and back lidar with 'min_angle' (-1.04) and 'max_angle' (3.66) fields.

- Minor adjustments to existing D435i camera properties and structure.

File: src/modular/modular_data/urdf/concert.sensors.urdf.xacro (robot description, xacro)
@@ -69,4 +69,15 @@
         <xacro:insert_block name="t265_right_origin" />
     </xacro:add_realsense_t_camera>
+    <!-- Add IMU sensor -->
+    <xacro:include filename="$(find imu_simulator)/urdf/imu.urdf.xacro" />
+    <xacro:property name="imu_name" value="imu" />
+    <xacro:property name="imu_parent_name" value="${parent_name}" />
+    <xacro:property name="imu_origin">
+        <origin xyz="0 0 0.1" rpy="0 0 0"/>
+    </xacro:property>
+    <xacro:add_imu_sensor name="${imu_name}"
+                        parent="${imu_parent_name}">
+        <xacro:insert_block name="imu_origin" />
+    </xacro:add_imu_sensor>
     <!-- Add Velodyne front -->
     <xacro:property name="velodyne_front_name" value="VLP16_lidar_front" />
@@ -80,5 +91,5 @@
             <xacro:insert_block name="velodyne_front_origin" />
         </xacro:VLP-16>
-        <xacro:VLP-16-gz-sensor name="${velodyne_front_name}" topic="/${velodyne_front_name}" hz="10" samples="440" gpu="${USE_GPU_RAY}">
+        <xacro:VLP-16-gz-sensor name="${velodyne_front_name}" topic="/${velodyne_front_name}" hz="10" samples="440" gpu="${USE_GPU_RAY}" min_angle="-1.04" max_angle="3.66">
         </xacro:VLP-16-gz-sensor>
     </xacro:if>
@@ -103,5 +114,5 @@
             <xacro:insert_block name="velodyne_back_origin" />
         </xacro:VLP-16>
-        <xacro:VLP-16-gz-sensor name="${velodyne_back_name}" topic="/${velodyne_back_name}" hz="10" samples="440" gpu="${USE_GPU_RAY}">
+        <xacro:VLP-16-gz-sensor name="${velodyne_back_name}" topic="/${velodyne_back_name}" hz="10" samples="440" gpu="${USE_GPU_RAY}" min_angle="-1.04" max_angle="3.66">
         </xacro:VLP-16-gz-sensor>
     </xacro:if>

Commit message: added camera

File: src/modular/modular_data/urdf/concert.sensors.urdf.xacro (robot description, xacro)
@@ -8,6 +8,6 @@
     <xacro:property name="ADD_D435I_FRONT" value="true" />
     <xacro:property name="ADD_D435I_BACK" value="true" />
-    <xacro:property name="ADD_T265_LEFT" value="true" />
-    <xacro:property name="ADD_T265_RIGHT" value="true" />
+    <!-- <xacro:property name="ADD_T265_LEFT" value="true" />
+    <xacro:property name="ADD_T265_RIGHT" value="true" /> -->
     <xacro:property name="ADD_DRILL_CAMERA" value="true" />
 </xacro:if>
@@ -19,5 +19,5 @@
 </xacro:if>
 <xacro:macro name="add_mobile_base_sensors" params="parent_name">
-	<joint name="base_link_projected_joint" type="fixed">
+    <joint name="base_link_projected_joint" type="fixed">
         <parent link="base_link"/>
         <child link="base_link_projected"/>
@@ -95,5 +95,4 @@
     </xacro:if>
     <xacro:unless value="${ADD_VELODYNE_FRONT}">
-        <!-- camera body, with origin at bottom screw mount -->
         <joint name="${velodyne_front_name}_base_mount_joint" type="fixed">
             <xacro:insert_block name="velodyne_front_origin"/>
@@ -136,5 +135,4 @@
         </joint>
         <link name="${name}_base_link"/>
-        <!-- Rotate sensor frame (readings are on x axis instead of z) -->
         <joint name="${name}_joint" type="fixed">
             <origin xyz="0 0 0" rpy="0.0 -1.57 0.0"/>
@@ -244,104 +242,187 @@
 </xacro:macro>
 <!-- Macro for adding gazebo plugin for ultrasound sensors -->
-    <xacro:macro name="add_ultrasound_gazebo" params="name topic">
-        <gazebo reference="${name}">
-            <sensor type="ray" name="sonar">
-                <update_rate>5</update_rate>
-                <ray>
-                    <scan>
-                        <horizontal>
-                            <samples>5</samples>
-                            <resolution>1.0</resolution>
-                            <min_angle>-1.0</min_angle>
-                            <max_angle>1.0</max_angle>
-                        </horizontal>
-                        <vertical>
-                            <samples>5</samples>
-                            <resolution>1</resolution>
-                            <min_angle>-0.5</min_angle>
-                            <max_angle>0.5</max_angle>
-                        </vertical>
-                    </scan>
-                    <range>
-                        <min>0.2</min>
-                        <max>3.0</max>
-                        <resolution>0.01</resolution>
-                    </range>
-                </ray>
-                <plugin filename="libgazebo_ros_range.so" name="gazebo_ros_range">
-                    <gaussianNoise>0.005</gaussianNoise>
-                    <alwaysOn>true</alwaysOn>
-                    <updateRate>5</updateRate>
-                    <topicName>${topic}</topicName>
-                    <frameName>${name}</frameName>
-                    <fov>2.3</fov>
-                    <radiation>ultrasound</radiation>
-                </plugin>
+<xacro:macro name="add_ultrasound_gazebo" params="name topic">
+    <gazebo reference="${name}">
+        <sensor type="ray" name="sonar">
+            <update_rate>5</update_rate>
+            <ray>
+                <scan>
+                    <horizontal>
+                        <samples>5</samples>
+                        <resolution>1.0</resolution>
+                        <min_angle>-1.0</min_angle>
+                        <max_angle>1.0</max_angle>
+                    </horizontal>
+                    <vertical>
+                        <samples>5</samples>
+                        <resolution>1</resolution>
+                        <min_angle>-0.5</min_angle>
+                        <max_angle>0.5</max_angle>
+                    </vertical>
+                </scan>
+                <range>
+                    <min>0.2</min>
+                    <max>3.0</max>
+                    <resolution>0.01</resolution>
+                </range>
+            </ray>
+            <plugin filename="libgazebo_ros_range.so" name="gazebo_ros_range">
+                <gaussianNoise>0.005</gaussianNoise>
+                <alwaysOn>true</alwaysOn>
+                <updateRate>5</updateRate>
+                <topicName>${topic}</topicName>
+                <frameName>${name}</frameName>
+                <fov>2.3</fov>
+                <radiation>ultrasound</radiation>
+            </plugin>
+        </sensor>
+    </gazebo>
+</xacro:macro>
+<!-- ============================================================ -->
+<!-- Macro for RealSense D435i - NATIVE GAZEBO RENDERING          -->
+<!-- This uses Gazebo's built-in camera rendering, NOT test data  -->
+<!-- ============================================================ -->
+<xacro:macro name="add_realsense_d_camera" params="name parent_name *origin add_gazebo_sensor">
+    <!-- Camera body link -->
+    <link name="${name}_bottom_screw_frame">
+        <visual>
+            <origin xyz="0 0 0" rpy="${-pi/2} 0 ${-pi/2}"/>
+            <geometry>
+                <box size="0.025 0.090 0.025"/>
+            </geometry>
+            <material name="gray">
+                <color rgba="0.5 0.5 0.5 1"/>
+            </material>
+        </visual>
+        <collision>
+            <origin xyz="0 0 0" rpy="${-pi/2} 0 ${-pi/2}"/>
+            <geometry>
+                <box size="0.02505 0.090 0.025"/>
+            </geometry>
+        </collision>
+        <inertial>
+            <mass value="0.072"/>
+            <inertia ixx="0.0001" ixy="0" ixz="0" iyy="0.0001" iyz="0" izz="0.0001"/>
+        </inertial>
+    </link>
+    <!-- Joint to parent -->
+    <joint name="${name}_joint" type="fixed">
+        <xacro:insert_block name="origin"/>
+        <parent link="${parent_name}"/>
+        <child link="${name}_bottom_screw_frame"/>
+    </joint>
+    <!-- Camera link (sensor reference frame) -->
+    <link name="${name}_link"/>
+    <joint name="${name}_link_joint" type="fixed">
+        <origin xyz="0 0.0175 0.0125" rpy="0 0 0"/>
+        <parent link="${name}_bottom_screw_frame"/>
+        <child link="${name}_link"/>
+    </joint>
+    <!-- Depth frame -->
+    <link name="${name}_depth_frame"/>
+    <joint name="${name}_depth_joint" type="fixed">
+        <origin xyz="0 0 0" rpy="0 0 0"/>
+        <parent link="${name}_link"/>
+        <child link="${name}_depth_frame"/>
+    </joint>
+    <!-- Depth optical frame -->
+    <link name="${name}_depth_optical_frame"/>
+    <joint name="${name}_depth_optical_joint" type="fixed">
+        <origin xyz="0 0 0" rpy="${-pi/2} 0 ${-pi/2}"/>
+        <parent link="${name}_depth_frame"/>
+        <child link="${name}_depth_optical_frame"/>
+    </joint>
+    <!-- Color frame -->
+    <link name="${name}_color_frame"/>
+    <joint name="${name}_color_joint" type="fixed">
+        <origin xyz="0 0.015 0" rpy="0 0 0"/>
+        <parent link="${name}_depth_frame"/>
+        <child link="${name}_color_frame"/>
+    </joint>
+    <!-- Color optical frame -->
+    <link name="${name}_color_optical_frame"/>
+    <joint name="${name}_color_optical_joint" type="fixed">
+        <origin xyz="0 0 0" rpy="${-pi/2} 0 ${-pi/2}"/>
+        <parent link="${name}_color_frame"/>
+        <child link="${name}_color_optical_frame"/>
+    </joint>
+    <!-- Left IR frame -->
+    <link name="${name}_left_ir_frame"/>
+    <joint name="${name}_left_ir_joint" type="fixed">
+        <origin xyz="0 0 0" rpy="0 0 0"/>
+        <parent link="${name}_depth_frame"/>
+        <child link="${name}_left_ir_frame"/>
+    </joint>
+    <!-- Left IR optical frame -->
+    <link name="${name}_left_ir_optical_frame"/>
+    <joint name="${name}_left_ir_optical_joint" type="fixed">
+        <origin xyz="0 0 0" rpy="${-pi/2} 0 ${-pi/2}"/>
+        <parent link="${name}_left_ir_frame"/>
+        <child link="${name}_left_ir_optical_frame"/>
+    </joint>
+    <!-- Right IR frame -->
+    <link name="${name}_right_ir_frame"/>
+    <joint name="${name}_right_ir_joint" type="fixed">
+        <origin xyz="0 -0.050 0" rpy="0 0 0"/>
+        <parent link="${name}_depth_frame"/>
+        <child link="${name}_right_ir_frame"/>
+    </joint>
+    <!-- Right IR optical frame -->
+    <link name="${name}_right_ir_optical_frame"/>
+    <joint name="${name}_right_ir_optical_joint" type="fixed">
+        <origin xyz="0 0 0" rpy="${-pi/2} 0 ${-pi/2}"/>
+        <parent link="${name}_right_ir_frame"/>
+        <child link="${name}_right_ir_optical_frame"/>
+    </joint>
+    <!-- ========================================== -->
+    <!-- NATIVE GAZEBO RGBD CAMERA - REAL RENDERING -->
+    <!-- Uses rgbd_camera type for combined RGB+Depth -->
+    <!-- Topics: /{name}/image, /{name}/depth_image, /{name}/points -->
+    <!-- ========================================== -->
+    <xacro:if value="${add_gazebo_sensor}">
+        <gazebo reference="${name}_link">
+            <!-- RGBD Camera (combined RGB + Depth + PointCloud) -->
+            <sensor name="${name}_rgbd" type="rgbd_camera">
+                <always_on>1</always_on>
+                <update_rate>30</update_rate>
+                <visualize>true</visualize>
+                <topic>${name}</topic>
+                <gz_frame_id>${name}_depth_optical_frame</gz_frame_id>
+                <camera name="${name}">
+                    <horizontal_fov>1.211259</horizontal_fov>
+                    <image>
+                        <width>640</width>
+                        <height>480</height>
+                        <format>R8G8B8</format>
+                    </image>
+                    <clip>
+                        <near>0.1</near>
+                        <far>100</far>
+                    </clip>
+                    <depth_camera>
+                        <clip>
+                            <near>0.1</near>
+                            <far>10</far>
+                        </clip>
+                    </depth_camera>
+                    <noise>
+                        <type>gaussian</type>
+                        <mean>0.0</mean>
+                        <stddev>0.007</stddev>
+                    </noise>
+                    <optical_frame_id>${name}_depth_optical_frame</optical_frame_id>
+                </camera>
             </sensor>
         </gazebo>
-    </xacro:macro>
-<!-- Macro for adding realsense D camera -->
-<xacro:macro name="add_realsense_d_camera" params="name parent_name *origin add_gazebo_sensor">
-    <xacro:if value="${add_gazebo_sensor}">
-        <xacro:include filename="$(find realsense_gazebo_description)/urdf/_d435i.urdf.xacro" />
-        <xacro:sensor_d435i parent="${parent_name}"
-                            name="${name}"
-                            topics_ns="${name}"
-                            enable_pointCloud="true"
-                            align_depth="true"
-                            unite_imu_method="false"
-                            visualize="true"
-                            accel_fps="300"
-                            gyro_fps="300"
-                            depth_width="1280"
-                            depth_height="720"
-                            depth_fps="90"
-                            infra_width="1280"
-                            infra_height="720"
-                            infra_fps="90"
-                            color_width="1280"
-                            color_height="720"
-                            color_fps="30">
-            <xacro:insert_block name="origin" />
-        </xacro:sensor_d435i>
     </xacro:if>
-    <xacro:unless value="${add_gazebo_sensor}">
-        <!-- camera body, with origin at bottom screw mount -->
-        <joint name="${name}_joint" type="fixed">
-            <xacro:insert_block name="origin"/>
-            <parent link="${parent_name}"/>
-            <child link="${name}_bottom_screw_frame"/>
-        </joint>
-        <link name="${name}_bottom_screw_frame"/>
-    </xacro:unless>
 </xacro:macro>
-<!-- Macro for adding realsense T camera -->
+<!-- Macro for T265 camera - Dummy frames only (discontinued) -->
 <xacro:macro name="add_realsense_t_camera" params="name parent_name *origin add_gazebo_sensor">
-    <xacro:if value="${add_gazebo_sensor}">
-        <xacro:include filename="$(find realsense_gazebo_description)/urdf/_t265.urdf.xacro" />
-        <xacro:sensor_t265  parent="${parent_name}"
-                            name="${name}"
-                            topics_ns="${name}"
-                            odom_xyz="0.0 0.0 0.25"
-                            odom_rpy="0.0 0.0 0.0"
-                            odom_fps="262"
-                            fisheye_width="848"
-                            fisheye_height="800"
-                            fisheye_fps="30"
-                            unite_imu_method="false"
-                            accel_fps="62.5"
-                            gyro_fps="200">
-            <xacro:insert_block name="origin" />
-        </xacro:sensor_t265>
-    </xacro:if>
-    <xacro:unless value="${add_gazebo_sensor}">
-        <!-- camera body, with origin at bottom screw mount -->
-        <joint name="${name}_joint" type="fixed">
-            <xacro:insert_block name="origin"/>
-            <parent link="${parent_name}"/>
-            <child link="${name}_pose_frame"/>
-        </joint>
-        <link name="${name}_pose_frame"/>
-    </xacro:unless>
+    <joint name="${name}_joint" type="fixed">
+        <xacro:insert_block name="origin"/>
+        <parent link="${parent_name}"/>
+        <child link="${name}_pose_frame"/>
+    </joint>
+    <link name="${name}_pose_frame"/>
 </xacro:macro>
 </robot>

Commit message: made IMU sensor simulator optional

File: src/modular/modular_data/urdf/concert.sensors.urdf.xacro (robot description, xacro)
@@ -70,14 +70,16 @@
     </xacro:add_realsense_t_camera>
     <!-- Add IMU sensor -->
-    <xacro:include filename="$(find imu_simulator)/urdf/imu.urdf.xacro" />
-    <xacro:property name="imu_name" value="imu" />
-    <xacro:property name="imu_parent_name" value="${parent_name}" />
-    <xacro:property name="imu_origin">
-        <origin xyz="0 0 0.1" rpy="0 0 0"/>
-    </xacro:property>
-    <xacro:add_imu_sensor name="${imu_name}"
-                        parent="${imu_parent_name}">
-        <xacro:insert_block name="imu_origin" />
-    </xacro:add_imu_sensor>
+    <xacro:if value="${ADD_IMU}">
+        <xacro:include filename="$(find imu_simulator)/urdf/imu.urdf.xacro" />
+        <xacro:property name="imu_name" value="imu" />
+        <xacro:property name="imu_parent_name" value="${parent_name}" />
+        <xacro:property name="imu_origin">
+            <origin xyz="0 0 0.1" rpy="0 0 0"/>
+        </xacro:property>
+        <xacro:add_imu_sensor name="${imu_name}"
+                            parent="${imu_parent_name}">
+            <xacro:insert_block name="imu_origin" />
+        </xacro:add_imu_sensor>
+    </xacro:if>
     <!-- Add Velodyne front -->
     <xacro:property name="velodyne_front_name" value="VLP16_lidar_front" />

File: src/modular/modular_data/urdf/template.urdf.xacro (robot description, xacro)
@@ -15,4 +15,6 @@
     <xacro:arg name="ultrasound" default="false"/>
     <xacro:property name="ADD_ULTRASOUND" value="$(arg ultrasound)" />
+    <xacro:arg name="imu" default="false"/>
+    <xacro:property name="ADD_IMU" value="$(arg imu)" />
     <xacro:arg name="use_gpu_ray" default="false"/>
     <xacro:property name="USE_GPU_RAY" value="$(arg use_gpu_ray)" />

Commit message: feat(URDF_writer): enhance camera and addon handling. load cameras from JSON

File: src/modular/modular_data/urdf/concert.sensors.urdf.xacro (robot description, xacro)
@@ -26,5 +26,5 @@
     <link name="base_link_projected"/>
     <!-- Add front D435i camera -->
-    <xacro:property name="d435i_front_name" value="D435i_camera_front" />
+    <!-- <xacro:property name="d435i_front_name" value="D435i_camera_front" />
     <xacro:property name="d435i_front_parent_name" value="${parent_name}" />
     <xacro:property name="d435i_front_origin">
@@ -35,16 +35,16 @@
                                 add_gazebo_sensor="${ADD_D435I_FRONT}">
         <xacro:insert_block name="d435i_front_origin" />
-    </xacro:add_realsense_d_camera>
+    </xacro:add_realsense_d_camera> -->
     <!-- Add back D435i camera -->
-    <xacro:property name="d435i_back_name" value="D435i_camera_back" />
+    <!-- <xacro:property name="d435i_back_name" value="D435i_camera_back" />
     <xacro:property name="d435i_back_parent_name" value="${parent_name}" />
     <xacro:property name="d435i_back_origin">
         <origin xyz="-0.402872 0.0 -0.078218" rpy="0 0.261799 3.141593"/>
-    </xacro:property>
-    <xacro:add_realsense_d_camera name="${d435i_back_name}"
+    </xacro:property> -->
+    <!-- <xacro:add_realsense_d_camera name="${d435i_back_name}"
                                 parent_name="${d435i_back_parent_name}"
                                 add_gazebo_sensor="${ADD_D435I_BACK}">
         <xacro:insert_block name="d435i_back_origin" />
-    </xacro:add_realsense_d_camera>
+    </xacro:add_realsense_d_camera> -->
     <!-- Add left T265 camera -->
     <xacro:property name="t265_left_name" value="T265_camera_left" />
