Commit message: Add Plugin abstract class to switch between ros_control, xbotcore, xbot2
Ref: https://refactoring.guru/design-patterns/state/python/example

File: src/modular/modular_data/urdf/ModularBot.library.urdf.xacro (robot description, xacro)
@@ -1,17 +1,6 @@
 <?xml version="1.0"?>
-<robot name="ModularBot" xmlns:xacro="http://ros.org/wiki/xacro">
+<robot name="ModularBot" xmlns:xacro="http://www.ros.org/wiki/xacro">
     <!-- <xacro:include filename="$(find modular)/urdf/config.xacro" />
     <xacro:include filename="$(find modular)/urdf/modular.gazebo" /> -->
-    <xacro:macro name="add_xbot2_pid" params="name profile">
-        <pid name="${name}" profile="${profile}"/>
-    </xacro:macro>
-    <gazebo>
-        <plugin name="xbot2_gz_joint_server" filename="libxbot2_gz_joint_server.so">
-	        <pid>
-                <gain name="small_mot"  p="100"  d="5"/>
-                <!-- <pid name="J1_A" profile="small_mot"/> -->
-	        </pid>
-	    </plugin>
-    </gazebo>
     <xacro:property name="size1" value="0.05" />
     <xacro:property name="size2" value="0.055" />
@@ -486,30 +475,4 @@
             <limit lower="${lower_lim}" upper="${upper_lim}" effort="${effort}" velocity="${velocity}"/>
         </joint>
-        <!--<link name="${child}">-->
-            <!--<xacro:if value="${type==joint_mesh}">-->
-                <!--<visual>-->
-                    <!--&lt;!&ndash; Load mesh. Rotate the origin frame (this is because of how the .stl was saved) &ndash;&gt;-->
-                    <!--<origin rpy="${roll} ${pitch} ${yaw}" xyz="${x} ${y} ${z}"/>-->
-                    <!--<geometry>-->
-                        <!--<mesh filename="package://modular/meshes/asm0001.stl" scale="0.001 0.001 0.001"/>-->
-                    <!--</geometry>-->
-                <!--</visual>-->
-                <!--<collision>-->
-                    <!--<origin rpy="${roll} ${pitch} ${yaw}" xyz="${x} ${y} ${z}"/>-->
-                    <!--<geometry>-->
-                        <!--<mesh filename="package://modular/meshes/asm0001.stl" scale="0.001 0.001 0.001"/>-->
-                    <!--</geometry>-->
-                <!--</collision>-->
-            <!--</xacro:if>-->
-            <!--&lt;!&ndash; inertial parameters for ORANGE rotating part. wrt a point on one end of the rod &ndash;&gt;-->
-            <!--<inertial>-->
-                <!--<origin xyz="0 0 -0.0635" rpy="0 0 0"/>-->
-                <!--<mass value="${mass}"/>-->
-                <!--<inertia-->
-                <!--ixx="${mass / 3.0 * (0.127*0.127)}" ixy="0.0" ixz="0.0"-->
-                <!--iyy="${mass / 3.0 * (0.127*0.127)}" iyz="0.0"-->
-                <!--izz="0.0000148"/>-->
-            <!--</inertial>-->
-        <!--</link>-->
     </xacro:macro>
     <xacro:macro name="add_rotor_fast" params="type name filename x y z roll pitch yaw">

Commit message: wip: movit config auto-generation

File: src/modular/modular_data/urdf/ModularBot.library.urdf.xacro (robot description, xacro)
@@ -56,18 +56,18 @@
             <parent link="${father}"/>
             <child link="${name}"/>
-            <origin rpy="0.0 -0.0 0.0" xyz="0.0 0.0 0.0"/>
+            <origin rpy="0.0 0.0 0.0" xyz="0.0 0.0 0.01"/>
         </joint>
         <link name="${name}">
             <visual>
-                <origin rpy="0 0 0" xyz="0.3 0 -0.005"/>
-                <geometry>
-                    <box size="0.6 0.6 0.01"/>
+                <origin rpy="0 0 0" xyz="0.6 0 -0.005"/>
+                <geometry>
+                    <box size="1.2 0.6 0.01"/>
                 </geometry>
                 <material name="gray"/>
             </visual>
             <collision>
-                <origin rpy="0 0 0" xyz="0.25 0 -0.005"/>
-                <geometry>
-                    <box size="0.6 0.6 0.01"/>
+                <origin rpy="0 0 0" xyz="0.6 0 -0.005"/>
+                <geometry>
+                    <box size="1.2 0.6 0.01"/>
                 </geometry>
             </collision>

Commit message: add passive links yamls and meshes

File: src/modular/modular_data/urdf/ModularBot.library.urdf.xacro (robot description, xacro)
@@ -279,5 +279,10 @@
     </xacro:macro>
     <!-- Macro for adding a straight link -->
-    <xacro:macro name="add_link" params="name type size_z size">
+    <xacro:macro name="add_link" params="name type filename size_z size">
+        <xacro:property name="module" value="${load_yaml(filename)}"/>
+        <xacro:property name="mesh_bool" value="false"/>
+        <xacro:unless value="${ module['visual']['mesh_body_1'] == '' }">
+            <xacro:property name="mesh_bool" value="true"/>
+        </xacro:unless>
         <xacro:if value="${size==1}">
             <xacro:property name="radius" value="${size1}" />
@@ -291,27 +296,64 @@
             </xacro:unless>
         </xacro:unless>
-        <link name="${name}">
-            <visual>
-                <origin xyz="0 0 ${size_z/2}" rpy="0 0 0" />
-                <geometry>
-                    <cylinder radius="${radius}" length="${size_z}"/>
-                </geometry>
-                <material name="white"/>
-            </visual>
-            <collision>
-                <origin xyz="0 0 ${size_z/2}" rpy="0 0 0" />
-                <geometry>
-                    <cylinder radius="${radius}" length="${size_z}"/>
-                </geometry>
-            </collision>
-            <inertial>
-                <origin xyz="0 0 ${size_z/2}" rpy="0 0 0"/>
-                <mass value="${mass}"/>
-                <inertia
-                ixx="${mass / 12.0 * (3*radius*radius + size_z*size_z)}" ixy="0.0" ixz="0.0"
-                iyy="${mass / 12.0 * (size_z*size_z + 3*radius*radius)}" iyz="0.0"
-                izz="${mass / 2.0 * (radius*radius)}"/>
-            </inertial>
-        </link>
+        <xacro:if value="${mesh_bool == 'false' }">
+            <link name="${name}">
+                <visual>
+                    <origin xyz="0 0 ${size_z/2}" rpy="0 0 0" />
+                    <geometry>
+                        <cylinder radius="${radius}" length="${size_z}"/>
+                    </geometry>
+                    <material name="white"/>
+                </visual>
+                <collision>
+                    <origin xyz="0 0 ${size_z/2}" rpy="0 0 0" />
+                    <geometry>
+                        <cylinder radius="${radius}" length="${size_z}"/>
+                    </geometry>
+                </collision>
+                <inertial>
+                    <origin xyz="0 0 ${size_z/2}" rpy="0 0 0"/>
+                    <mass value="${mass}"/>
+                    <inertia
+                    ixx="${mass / 12.0 * (3*radius*radius + size_z*size_z)}" ixy="0.0" ixz="0.0"
+                    iyy="${mass / 12.0 * (size_z*size_z + 3*radius*radius)}" iyz="0.0"
+                    izz="${mass / 2.0 * (radius*radius)}"/>
+                </inertial>
+            </link>
+        </xacro:if>
+        <xacro:unless value="${mesh_bool == 'false'}">
+            <link name="${name}">
+                <visual>
+                    <!-- Load mesh. Rotate the origin frame (this is because of how the .stl was saved) -->
+                    <origin
+                        rpy="${module['visual']['tf_mesh_1']['roll']} ${module['visual']['tf_mesh_1']['pitch']} ${module['visual']['tf_mesh_1']['yaw']}"
+                        xyz="${module['visual']['tf_mesh_1']['x']} ${module['visual']['tf_mesh_1']['y']} ${module['visual']['tf_mesh_1']['z']}"/>
+                    <geometry>
+                        <mesh filename="${module['visual']['mesh_body_1']}" scale="0.001 0.001 0.001"/>
+                    </geometry>
+                    <material name="tree_green"/>
+                </visual>
+                <collision>
+                    <origin
+                        rpy="${module['visual']['tf_mesh_1']['roll']} ${module['visual']['tf_mesh_1']['pitch']} ${module['visual']['tf_mesh_1']['yaw']}"
+                        xyz="${module['visual']['tf_mesh_1']['x']} ${module['visual']['tf_mesh_1']['y']} ${module['visual']['tf_mesh_1']['z']}"/>
+                    <geometry>
+                        <mesh filename="${module['visual']['mesh_collision_1']}" scale="0.001 0.001 0.001"/>
+                    </geometry>
+                </collision>
+                <inertial>
+                    <origin
+                        xyz="${module['dynamics']['body_1']['CoM']['x']} ${module['dynamics']['body_1']['CoM']['y']} ${module['dynamics']['body_1']['CoM']['z']}"
+                        rpy="0 0 0"/>
+                    <mass value="${module['dynamics']['body_1']['mass']}"/>
+                    <inertia
+                        ixx="${module['dynamics']['body_1']['inertia_tensor']['I_xx']}"
+                        ixy="${module['dynamics']['body_1']['inertia_tensor']['I_xy']}"
+                        ixz="${module['dynamics']['body_1']['inertia_tensor']['I_xz']}"
+                        iyy="${module['dynamics']['body_1']['inertia_tensor']['I_yy']}"
+                        iyz="${module['dynamics']['body_1']['inertia_tensor']['I_yz']}"
+                        izz="${module['dynamics']['body_1']['inertia_tensor']['I_zz']}"/>
+                </inertial>
+            </link>
+        </xacro:unless>
         <gazebo reference="${name}">
             <mu1>0.2</mu1>
@@ -822,5 +864,4 @@
                     </geometry>
                 </collision>
-                <!-- TODO: change inertial parameters with the one from CAD. This will be the inertia tensor of only the housing/stator part -->
                 <inertial>
                     <origin

Commit message: wip

File: src/modular/modular_data/urdf/ModularBot.library.urdf.xacro (robot description, xacro)
@@ -60,5 +60,5 @@
         <link name="${name}">
             <visual>
-                <origin rpy="0 0 0" xyz="0.6 0 -0.005"/>
+                <origin rpy="0 0 0" xyz="0.6 0.3 -0.005"/>
                 <geometry>
                     <box size="1.2 0.6 0.01"/>
@@ -67,5 +67,5 @@
             </visual>
             <collision>
-                <origin rpy="0 0 0" xyz="0.6 0 -0.005"/>
+                <origin rpy="0 0 0" xyz="0.6 0.3 -0.005"/>
                 <geometry>
                     <box size="1.2 0.6 0.01"/>
@@ -296,30 +296,5 @@
             </xacro:unless>
         </xacro:unless>
-        <xacro:if value="${mesh_bool == 'false' }">
-            <link name="${name}">
-                <visual>
-                    <origin xyz="0 0 ${size_z/2}" rpy="0 0 0" />
-                    <geometry>
-                        <cylinder radius="${radius}" length="${size_z}"/>
-                    </geometry>
-                    <material name="white"/>
-                </visual>
-                <collision>
-                    <origin xyz="0 0 ${size_z/2}" rpy="0 0 0" />
-                    <geometry>
-                        <cylinder radius="${radius}" length="${size_z}"/>
-                    </geometry>
-                </collision>
-                <inertial>
-                    <origin xyz="0 0 ${size_z/2}" rpy="0 0 0"/>
-                    <mass value="${mass}"/>
-                    <inertia
-                    ixx="${mass / 12.0 * (3*radius*radius + size_z*size_z)}" ixy="0.0" ixz="0.0"
-                    iyy="${mass / 12.0 * (size_z*size_z + 3*radius*radius)}" iyz="0.0"
-                    izz="${mass / 2.0 * (radius*radius)}"/>
-                </inertial>
-            </link>
-        </xacro:if>
-        <xacro:unless value="${mesh_bool == 'false'}">
+        <xacro:if value="${mesh_bool}">
             <link name="${name}">
                 <visual>
@@ -353,4 +328,29 @@
                         iyz="${module['dynamics']['body_1']['inertia_tensor']['I_yz']}"
                         izz="${module['dynamics']['body_1']['inertia_tensor']['I_zz']}"/>
+                </inertial>
+            </link>
+        </xacro:if>
+        <xacro:unless value="${mesh_bool}">
+            <link name="${name}">
+                <visual>
+                    <origin xyz="0 0 ${size_z/2}" rpy="0 0 0" />
+                    <geometry>
+                        <cylinder radius="${radius}" length="${size_z}"/>
+                    </geometry>
+                    <material name="white"/>
+                </visual>
+                <collision>
+                    <origin xyz="0 0 ${size_z/2}" rpy="0 0 0" />
+                    <geometry>
+                        <cylinder radius="${radius}" length="${size_z}"/>
+                    </geometry>
+                </collision>
+                <inertial>
+                    <origin xyz="0 0 ${size_z/2}" rpy="0 0 0"/>
+                    <mass value="${mass}"/>
+                    <inertia
+                    ixx="${mass / 12.0 * (3*radius*radius + size_z*size_z)}" ixy="0.0" ixz="0.0"
+                    iyy="${mass / 12.0 * (size_z*size_z + 3*radius*radius)}" iyz="0.0"
+                    izz="${mass / 2.0 * (radius*radius)}"/>
                 </inertial>
             </link>
@@ -791,4 +791,17 @@
     <xacro:macro name="add_simple_ee" params="type name size_z">
         <link name="${name}">
+            <visual>
+                <origin xyz="0 0 ${size_z/2}" rpy="0 0 0" />
+                <geometry>
+                    <cylinder radius="0.05" length="${size_z}"/>
+                </geometry>
+                <material name="blue"/>
+            </visual>
+            <collision>
+                <origin xyz="0 0 ${size_z/2}" rpy="0 0 0" />
+                <geometry>
+                    <cylinder radius="0.05" length="${size_z}"/>
+                </geometry>
+            </collision>
             <inertial>
                 <origin xyz="0 0 ${size_z/2}" rpy="0 0 0"/>

Commit message: wippao

File: src/modular/modular_data/urdf/ModularBot.library.urdf.xacro (robot description, xacro)
@@ -792,23 +792,23 @@
         <link name="${name}">
             <visual>
-                <origin xyz="0 0 ${size_z/2}" rpy="0 0 0" />
-                <geometry>
-                    <cylinder radius="0.05" length="${size_z}"/>
+                <origin xyz="0 0 -${size_z/2}" rpy="0 0 0" />
+                <geometry>
+                    <cylinder radius="0.02" length="${size_z}"/>
                 </geometry>
                 <material name="blue"/>
             </visual>
             <collision>
-                <origin xyz="0 0 ${size_z/2}" rpy="0 0 0" />
-                <geometry>
-                    <cylinder radius="0.05" length="${size_z}"/>
+                <origin xyz="0 0 -${size_z/2}" rpy="0 0 0" />
+                <geometry>
+                    <cylinder radius="0.02" length="${size_z}"/>
                 </geometry>
             </collision>
             <inertial>
-                <origin xyz="0 0 ${size_z/2}" rpy="0 0 0"/>
-                <mass value="0.848"/>
+                <origin xyz="-0.007 0 0.044" rpy="0 0 0"/>
+                <mass value="1.305"/>
                 <inertia
-                        ixx="1.1564566e-03" ixy="0.0" ixz="0.0"
-                        iyy="1.2469918e-03" iyz="0.0"
-                        izz="5.7388903e-04"/>
+                        ixx="1.8769887e-03" ixy="0.0" ixz="0.0"
+                        iyy="2.2629779e-03" iyz="0.0"
+                        izz="1.8887550e-03"/>
             </inertial>
         </link>

Commit message: add passive links

File: src/modular/modular_data/urdf/ModularBot.library.urdf.xacro (robot description, xacro)
@@ -245,5 +245,10 @@
     </xacro:macro>
     <!-- Macro for adding a straight link -->
-    <xacro:macro name="add_link" params="name type size_z size">
+    <xacro:macro name="add_link" params="name type filename size_z size">
+        <xacro:property name="module" value="${load_yaml(filename)}"/>
+        <xacro:property name="mesh_bool" value="false"/>
+        <xacro:unless value="${ module['visual']['mesh_body_1'] == '' }">
+            <xacro:property name="mesh_bool" value="true"/>
+        </xacro:unless>
         <xacro:if value="${size==1}">
             <xacro:property name="radius" value="${size1}" />
@@ -257,27 +262,64 @@
             </xacro:unless>
         </xacro:unless>
-        <link name="${name}">
-            <visual>
-                <origin xyz="0 0 ${size_z/2}" rpy="0 0 0" />
-                <geometry>
-                    <cylinder radius="${radius}" length="${size_z}"/>
-                </geometry>
-                <material name="white"/>
-            </visual>
-            <collision>
-                <origin xyz="0 0 ${size_z/2}" rpy="0 0 0" />
-                <geometry>
-                    <cylinder radius="${radius}" length="${size_z}"/>
-                </geometry>
-            </collision>
-            <inertial>
-                <origin xyz="0 0 ${size_z/2}" rpy="0 0 0"/>
-                <mass value="${mass}"/>
-                <inertia
-                ixx="${mass / 12.0 * (3*radius*radius + size_z*size_z)}" ixy="0.0" ixz="0.0"
-                iyy="${mass / 12.0 * (size_z*size_z + 3*radius*radius)}" iyz="0.0"
-                izz="${mass / 2.0 * (radius*radius)}"/>
-            </inertial>
-        </link>
+        <xacro:if value="${mesh_bool == 'false' }">
+            <link name="${name}">
+                <visual>
+                    <origin xyz="0 0 ${size_z/2}" rpy="0 0 0" />
+                    <geometry>
+                        <cylinder radius="${radius}" length="${size_z}"/>
+                    </geometry>
+                    <material name="white"/>
+                </visual>
+                <collision>
+                    <origin xyz="0 0 ${size_z/2}" rpy="0 0 0" />
+                    <geometry>
+                        <cylinder radius="${radius}" length="${size_z}"/>
+                    </geometry>
+                </collision>
+                <inertial>
+                    <origin xyz="0 0 ${size_z/2}" rpy="0 0 0"/>
+                    <mass value="${mass}"/>
+                    <inertia
+                    ixx="${mass / 12.0 * (3*radius*radius + size_z*size_z)}" ixy="0.0" ixz="0.0"
+                    iyy="${mass / 12.0 * (size_z*size_z + 3*radius*radius)}" iyz="0.0"
+                    izz="${mass / 2.0 * (radius*radius)}"/>
+                </inertial>
+            </link>
+        </xacro:if>
+        <xacro:unless value="${mesh_bool == 'false'}">
+            <link name="${name}">
+                <visual>
+                    <!-- Load mesh. Rotate the origin frame (this is because of how the .stl was saved) -->
+                    <origin
+                        rpy="${module['visual']['tf_mesh_1']['roll']} ${module['visual']['tf_mesh_1']['pitch']} ${module['visual']['tf_mesh_1']['yaw']}"
+                        xyz="${module['visual']['tf_mesh_1']['x']} ${module['visual']['tf_mesh_1']['y']} ${module['visual']['tf_mesh_1']['z']}"/>
+                    <geometry>
+                        <mesh filename="${module['visual']['mesh_body_1']}" scale="0.001 0.001 0.001"/>
+                    </geometry>
+                    <material name="tree_green"/>
+                </visual>
+                <collision>
+                    <origin
+                        rpy="${module['visual']['tf_mesh_1']['roll']} ${module['visual']['tf_mesh_1']['pitch']} ${module['visual']['tf_mesh_1']['yaw']}"
+                        xyz="${module['visual']['tf_mesh_1']['x']} ${module['visual']['tf_mesh_1']['y']} ${module['visual']['tf_mesh_1']['z']}"/>
+                    <geometry>
+                        <mesh filename="${module['visual']['mesh_collision_1']}" scale="0.001 0.001 0.001"/>
+                    </geometry>
+                </collision>
+                <inertial>
+                    <origin
+                        xyz="${module['dynamics']['body_1']['CoM']['x']} ${module['dynamics']['body_1']['CoM']['y']} ${module['dynamics']['body_1']['CoM']['z']}"
+                        rpy="0 0 0"/>
+                    <mass value="${module['dynamics']['body_1']['mass']}"/>
+                    <inertia
+                        ixx="${module['dynamics']['body_1']['inertia_tensor']['I_xx']}"
+                        ixy="${module['dynamics']['body_1']['inertia_tensor']['I_xy']}"
+                        ixz="${module['dynamics']['body_1']['inertia_tensor']['I_xz']}"
+                        iyy="${module['dynamics']['body_1']['inertia_tensor']['I_yy']}"
+                        iyz="${module['dynamics']['body_1']['inertia_tensor']['I_yz']}"
+                        izz="${module['dynamics']['body_1']['inertia_tensor']['I_zz']}"/>
+                </inertial>
+            </link>
+        </xacro:unless>
         <gazebo reference="${name}">
             <mu1>0.2</mu1>
