Commit message: chore (ModularBot): remove unused files

File: src/modular/modular_data/urdf/ModularBot.library.urdf.xacro (robot description, xacro)
@@ -366,4 +366,55 @@
         </gazebo>
     </xacro:macro>
+    <!-- Macro for adding a socket -->
+    <xacro:macro name="add_socket" params="name type filename size_z size">
+        <xacro:property name="module" value="${load_yaml(filename)}"/>
+        <xacro:property name="mesh_bool" value="false"/>
+        <!-- <xacro:unless value="${ module['visual']['mesh_body_1'] == '' }">
+            <xacro:property name="mesh_bool" value="true"/>
+        </xacro:unless> -->
+        <xacro:if value="${size==1}">
+            <xacro:property name="radius" value="${size1}" />
+        </xacro:if>
+        <xacro:unless value="${size==1}">
+            <xacro:if value="${size==2}">
+                <xacro:property name="radius" value="${size2}" />
+            </xacro:if>
+            <xacro:unless value="${size==2}">
+                <xacro:property name="radius" value="${size3}" />
+            </xacro:unless>
+        </xacro:unless>
+        <link name="${name}">
+            <visual>
+                <origin xyz="0 0 ${size_z/2}" rpy="0 0 0" />
+                <geometry>
+                    <cylinder radius="${radius}" length="${size_z}"/>
+                </geometry>
+                <material name="white"/>
+            </visual>
+            <collision>
+                <origin xyz="0 0 ${size_z/2}" rpy="0 0 0" />
+                <geometry>
+                    <cylinder radius="${radius}" length="${size_z}"/>
+                </geometry>
+            </collision>
+            <inertial>
+                <origin xyz="0 0 ${size_z/2}" rpy="0 0 0"/>
+                <mass value="${mass}"/>
+                <inertia
+                ixx="${mass / 12.0 * (3*radius*radius + size_z*size_z)}" ixy="0.0" ixz="0.0"
+                iyy="${mass / 12.0 * (size_z*size_z + 3*radius*radius)}" iyz="0.0"
+                izz="${mass / 2.0 * (radius*radius)}"/>
+            </inertial>
+        </link>
+        <gazebo reference="${name}">
+            <mu1>0.2</mu1>
+            <mu2>0.2</mu2>
+            <kp>1000000.0</kp>
+            <kd>1.0</kd>
+            <maxVel>0.0</maxVel>
+            <minDepth>0.0001</minDepth>
+            <material>Gazebo/White</material>
+        </gazebo>
+    </xacro:macro>
     <!-- Macro for adding a size adapter -->
     <xacro:macro name="add_size_adapter" params="type name size_z size_in size_out">

Commit message: fix (sim/dummy): fix urdf, srdf and meshes path for simulation and dummy

File: src/modular/modular_data/urdf/ModularBot.library.urdf.xacro (robot description, xacro)
@@ -43,11 +43,4 @@
         </inertial>
     </xacro:macro>
-    <!-- adding world link for Gazebo simulation -->
-    <!-- <link name="world"/>
-    <joint name="world" type="fixed">
-        <parent link="world"/>
-        <child link="base_link"/>
-    </joint> -->
-    <link name="base_link"/>
     <!-- Macro for adding a table -->
     <xacro:macro name="add_table" params="type name father">

File: src/modular/modular_data/urdf/template.urdf.xacro (robot description, xacro)
@@ -3,3 +3,12 @@
     <xacro:include filename="ModularBot.library.urdf.xacro"/>
     <xacro:include filename="ModularBot.control.urdf.xacro"/>
+    <!-- adding world link for Gazebo simulation -->
+    <link name="world"/>
+    <joint name="world" type="fixed">
+        <parent link="world"/>
+        <child link="base_link"/>
+    </joint>
+    <link name="base_link">
+        <xacro:default_inertial mass="10.0"/>
+    </link>
 </robot>

Commit message: feat: add_size adapters and links

File: src/modular/modular_data/urdf/ModularBot.library.urdf.xacro (robot description, xacro)
@@ -3,7 +3,13 @@
     <!-- <xacro:include filename="$(find modular)/urdf/config.xacro" />
     <xacro:include filename="$(find modular)/urdf/modular.gazebo" /> -->
+<!--
     <xacro:property name="size1" value="0.05" />
     <xacro:property name="size2" value="0.055" />
-    <xacro:property name="size3" value="0.06" />
+    <xacro:property name="size3" value="0.06" /> -->
+    <xacro:property name="size1" value="0.0335" />
+    <xacro:property name="size2" value="0.038" />
+    <xacro:property name="size3" value="0.043" />
+    <xacro:property name="size4" value="0.053" />
+    <xacro:property name="size5" value="0.069" />
     <xacro:property name="size_interface" value="0.045" />
     <!-- <xacro:property name="leglen" value="0.3" /> -->
@@ -286,5 +292,15 @@
             </xacro:if>
             <xacro:unless value="${size==2}">
-                <xacro:property name="radius" value="${size3}" />
+                <xacro:if value="${size==3}">
+                    <xacro:property name="radius" value="${size3}" />
+                </xacro:if>
+                <xacro:unless value="${size==3}">
+                    <xacro:if value="${size==4}">
+                        <xacro:property name="radius" value="${size4}" />
+                    </xacro:if>
+                    <xacro:unless value="${size==4}">
+                        <xacro:property name="radius" value="${size5}" />
+                    </xacro:unless>
+                </xacro:unless>
             </xacro:unless>
         </xacro:unless>
@@ -411,63 +427,105 @@
     </xacro:macro>
     <!-- Macro for adding a size adapter -->
-    <xacro:macro name="add_size_adapter" params="type name size_z size_in size_out">
-        <xacro:if value="${size_in==3}">
-            <xacro:property name="radius1" value="${size3}" />
+    <xacro:macro name="add_size_adapter" params="type name filename size_z">
+         <xacro:property name="module" value="${load_yaml(filename)}"/>
+        <xacro:property name="mesh_bool" value="false"/>
+        <xacro:unless value="${ module['visual']['mesh_body_1'] == '' }">
+            <xacro:property name="mesh_bool" value="true"/>
+        </xacro:unless>
+        <xacro:if value="${mesh_bool}">
+            <link name="${name}">
+                <visual>
+                    <!-- Load mesh. Rotate the origin frame (this is because of how the .stl was saved) -->
+                    <origin
+                        rpy="${module['visual']['tf_mesh_1']['roll']} ${module['visual']['tf_mesh_1']['pitch']} ${module['visual']['tf_mesh_1']['yaw']}"
+                        xyz="${module['visual']['tf_mesh_1']['x']} ${module['visual']['tf_mesh_1']['y']} ${module['visual']['tf_mesh_1']['z']}"/>
+                    <geometry>
+                        <mesh filename="${module['visual']['mesh_body_1']}" scale="0.001 0.001 0.001"/>
+                    </geometry>
+                    <material name="tree_green"/>
+                </visual>
+                <collision>
+                    <origin
+                        rpy="${module['visual']['tf_mesh_1']['roll']} ${module['visual']['tf_mesh_1']['pitch']} ${module['visual']['tf_mesh_1']['yaw']}"
+                        xyz="${module['visual']['tf_mesh_1']['x']} ${module['visual']['tf_mesh_1']['y']} ${module['visual']['tf_mesh_1']['z']}"/>
+                    <geometry>
+                        <mesh filename="${module['visual']['mesh_collision_1']}" scale="0.001 0.001 0.001"/>
+                    </geometry>
+                </collision>
+                <inertial>
+                    <origin
+                        xyz="${module['dynamics']['body_1']['CoM']['x']} ${module['dynamics']['body_1']['CoM']['y']} ${module['dynamics']['body_1']['CoM']['z']}"
+                        rpy="0 0 0"/>
+                    <mass value="${module['dynamics']['body_1']['mass']}"/>
+                    <inertia
+                        ixx="${module['dynamics']['body_1']['inertia_tensor']['I_xx']}"
+                        ixy="${module['dynamics']['body_1']['inertia_tensor']['I_xy']}"
+                        ixz="${module['dynamics']['body_1']['inertia_tensor']['I_xz']}"
+                        iyy="${module['dynamics']['body_1']['inertia_tensor']['I_yy']}"
+                        iyz="${module['dynamics']['body_1']['inertia_tensor']['I_yz']}"
+                        izz="${module['dynamics']['body_1']['inertia_tensor']['I_zz']}"/>
+                </inertial>
+            </link>
         </xacro:if>
-        <xacro:unless value="${size_in==3}">
-            <xacro:if value="${size_in==2}">
-                <xacro:property name="radius1" value="${size2}" />
+        <xacro:unless value="${mesh_bool}">
+            <xacro:if value="${module['size_in']=='big'}">
+                <xacro:property name="radius3" value="${size3}" />
             </xacro:if>
-            <xacro:unless value="${size_in==2}">
+            <xacro:unless value="${module['size_in']=='big'}">
+                <xacro:if value="${module['size_in']=='medium'}">
+                    <xacro:property name="radius2" value="${size2}" />
+                </xacro:if>
+                <xacro:unless value="${module['size_in']=='medium}">
+                    <!-- ERROR! -->
+                </xacro:unless>
+            </xacro:unless>
+            <xacro:if value="${module['size_out']=='big'}">
                 <!-- ERROR! -->
+            </xacro:if>
+            <xacro:unless value="${module['size_out']=='big'}">
+                <xacro:if value="${module['size_out']=='medium'}">
+                    <xacro:property name="radius2" value="${size2}" />
+                </xacro:if>
+                <xacro:unless value="${module['size_out']=='medium'}">
+                    <xacro:property name="radius1" value="${size1}" />
+                </xacro:unless>
             </xacro:unless>
-        </xacro:unless>
-        <xacro:if value="${size_out==3}">
-            <!-- ERROR! -->
-        </xacro:if>
-        <xacro:unless value="${size_out==3}">
-            <xacro:if value="${size_out==2}">
-                <xacro:property name="radius2" value="${size2}" />
-            </xacro:if>
-            <xacro:unless value="${size_out==2}">
-                <xacro:property name="radius2" value="${size1}" />
-            </xacro:unless>
-        </xacro:unless>
-        <link name="${name}">
-            <visual>
-                <origin xyz="0 0 ${size_z/4}" rpy="0 0 0" />
-                <geometry>
-                    <cylinder radius="${radius1}" length="${size_z/2}"/>
-                </geometry>
-                <material name="grey"/>
-            </visual>
-            <visual>
-                <origin xyz="0 0 ${3*size_z/4}" rpy="0 0 0" />
-                <geometry>
-                    <cylinder radius="${radius2}" length="${size_z/2}"/>
-                </geometry>
-                <material name="grey"/>
-            </visual>
-            <collision>
-                <origin xyz="0 0 ${size_z/4}" rpy="0 0 0" />
-                <geometry>
-                    <cylinder radius="${radius1}" length="${size_z/2}"/>
-                </geometry>
-            </collision>
-            <collision>
-                <origin xyz="0 0 ${3*size_z/4}" rpy="0 0 0" />
-                <geometry>
-                    <cylinder radius="${radius2}" length="${size_z/2}"/>
-                </geometry>
-            </collision>
-            <inertial>
-                <origin xyz="0 0 ${size_z/2}" rpy="0 0 0"/>
-                <mass value="${mass}"/>
-                <inertia
-                ixx="${mass / 12.0 * (3*radius1*radius1 + 4*size_z/2*size_z/2) + mass / 12.0 * (3*radius2*radius2 + 4*size_z/2*size_z/2)}" ixy="0.0" ixz="0.0"
-                iyy="${mass / 12.0 * (3*radius1*radius1 + 4*size_z/2*size_z/2) + mass / 12.0 * (3*radius2*radius2 + 4*size_z/2*size_z/2)}" iyz="0.0"
-                izz="${mass / 4.0 * (radius1*radius1) + mass / 4.0 * (radius2*radius2)}"/>
-            </inertial>
-        </link>
+            <link name="${name}">
+                <visual>
+                    <origin xyz="0 0 ${size_z/4}" rpy="0 0 0" />
+                    <geometry>
+                        <cylinder radius="${radius1}" length="${size_z/2}"/>
+                    </geometry>
+                    <material name="grey"/>
+                </visual>
+                <visual>
+                    <origin xyz="0 0 ${3*size_z/4}" rpy="0 0 0" />
+                    <geometry>
+                        <cylinder radius="${radius2}" length="${size_z/2}"/>
+                    </geometry>
+                    <material name="grey"/>
+                </visual>
+                <collision>
+                    <origin xyz="0 0 ${size_z/4}" rpy="0 0 0" />
+                    <geometry>
+                        <cylinder radius="${radius1}" length="${size_z/2}"/>
+                    </geometry>
+                </collision>
+                <collision>
+                    <origin xyz="0 0 ${3*size_z/4}" rpy="0 0 0" />
+                    <geometry>
+                        <cylinder radius="${radius2}" length="${size_z/2}"/>
+                    </geometry>
+                </collision>
+                <inertial>
+                    <origin xyz="0 0 ${size_z/2}" rpy="0 0 0"/>
+                    <mass value="${mass}"/>
+                    <inertia
+                    ixx="${mass / 12.0 * (3*radius1*radius1 + 4*size_z/2*size_z/2) + mass / 12.0 * (3*radius2*radius2 + 4*size_z/2*size_z/2)}" ixy="0.0" ixz="0.0"
+                    iyy="${mass / 12.0 * (3*radius1*radius1 + 4*size_z/2*size_z/2) + mass / 12.0 * (3*radius2*radius2 + 4*size_z/2*size_z/2)}" iyz="0.0"
+                    izz="${mass / 4.0 * (radius1*radius1) + mass / 4.0 * (radius2*radius2)}"/>
+                </inertial>
+            </link>
+        </xacro:unless>
         <gazebo reference="${name}">
             <mu1>0.2</mu1>

Commit message: fix : fix wrong meshes orientation

File: src/modular/modular_data/urdf/ModularBot.library.urdf.xacro (robot description, xacro)
@@ -315,5 +315,5 @@
                         <mesh filename="${module['visual']['mesh_body_1']}" scale="0.001 0.001 0.001"/>
                     </geometry>
-                    <material name="tree_green"/>
+                    <material name="white"/>
                 </visual>
                 <collision>
@@ -382,5 +382,5 @@
             <xacro:property name="mesh_bool" value="true"/>
         </xacro:unless> -->
-        <xacro:if value="${size==1}">
+        <!-- <xacro:if value="${size==1}">
             <xacro:property name="radius" value="${size1}" />
         </xacro:if>
@@ -392,5 +392,6 @@
                 <xacro:property name="radius" value="${size3}" />
             </xacro:unless>
-        </xacro:unless>
+        </xacro:unless> -->
+        <xacro:property name="radius" value="${size4}" />
         <link name="${name}">
             <visual>

Commit message: fix : fix wrong meshes orientation

File: src/modular/modular_data/urdf/ModularBot.library.urdf.xacro (robot description, xacro)
@@ -299,5 +299,5 @@
                         <mesh filename="${module['visual']['mesh_body_1']}" scale="0.001 0.001 0.001"/>
                     </geometry>
-                    <material name="tree_green"/>
+                    <material name="white"/>
                 </visual>
                 <collision>
@@ -366,5 +366,5 @@
             <xacro:property name="mesh_bool" value="true"/>
         </xacro:unless> -->
-        <xacro:if value="${size==1}">
+        <!-- <xacro:if value="${size==1}">
             <xacro:property name="radius" value="${size1}" />
         </xacro:if>
@@ -376,5 +376,6 @@
                 <xacro:property name="radius" value="${size3}" />
             </xacro:unless>
-        </xacro:unless>
+        </xacro:unless> -->
+        <xacro:property name="radius" value="${size4}" />
         <link name="${name}">
             <visual>

Commit message: quick fix(xacro)

File: src/modular/modular_data/urdf/ModularBot.library.urdf.xacro (robot description, xacro)
@@ -377,5 +377,5 @@
             </xacro:unless>
         </xacro:unless> -->
-        <xacro:property name="radius" value="${size4}" />
+        <xacro:property name="radius" value="${size_interface}" />
         <link name="${name}">
             <visual>

Commit message: fix warning: deprecated usage of load_yaml
(cherry picked from commit c98892a469bb9eef65e7ad55511c6e83f644c920)

File: src/modular/modular_data/urdf/ModularBot.library.urdf.xacro (robot description, xacro)
@@ -89,5 +89,5 @@
     <!-- Macro for adding a master cube -->
     <xacro:macro name="add_master_cube" params="name filename type">
-        <xacro:property name="module" value="${load_yaml(filename)}"/>
+        <xacro:property name="module" value="${xacro.load_yaml(filename)}"/>
         <joint name="fixed" type="fixed">
             <parent link="base_link"/>
@@ -116,5 +116,5 @@
     </xacro:macro>
     <xacro:macro name="add_connectors" params="name filename type">
-        <xacro:property name="module" value="${load_yaml(filename)}"/>
+        <xacro:property name="module" value="${xacro.load_yaml(filename)}"/>
         <xacro:if value="${'connector_1' in module['kinematics']}">
             <link name="${name}_con1">
@@ -192,5 +192,5 @@
     <!-- Macro for adding a slave cube -->
     <xacro:macro name="add_slave_cube" params="name filename type">
-        <xacro:property name="module" value="${load_yaml(filename)}"/>
+        <xacro:property name="module" value="${xacro.load_yaml(filename)}"/>
         <link name="${name}">
             <visual>
@@ -279,5 +279,5 @@
     <!-- Macro for adding a straight link -->
     <xacro:macro name="add_link" params="name type filename size_z size">
-        <xacro:property name="module" value="${load_yaml(filename)}"/>
+        <xacro:property name="module" value="${xacro.load_yaml(filename)}"/>
         <xacro:property name="mesh_bool" value="false"/>
         <xacro:unless value="${ module['visual']['mesh_body_1'] == '' }">
@@ -377,20 +377,5 @@
     <!-- Macro for adding a socket -->
     <xacro:macro name="add_socket" params="name type filename size_z size">
-        <xacro:property name="module" value="${load_yaml(filename)}"/>
-        <xacro:property name="mesh_bool" value="false"/>
-        <!-- <xacro:unless value="${ module['visual']['mesh_body_1'] == '' }">
-            <xacro:property name="mesh_bool" value="true"/>
-        </xacro:unless> -->
-        <!-- <xacro:if value="${size==1}">
-            <xacro:property name="radius" value="${size1}" />
-        </xacro:if>
-        <xacro:unless value="${size==1}">
-            <xacro:if value="${size==2}">
-                <xacro:property name="radius" value="${size2}" />
-            </xacro:if>
-            <xacro:unless value="${size==2}">
-                <xacro:property name="radius" value="${size3}" />
-            </xacro:unless>
-        </xacro:unless> -->
+        <xacro:property name="module" value="${xacro.load_yaml(filename)}"/>
         <xacro:property name="radius" value="${size_interface}" />
         <link name="${name}">
@@ -429,5 +414,5 @@
     <!-- Macro for adding a size adapter -->
     <xacro:macro name="add_size_adapter" params="type name filename size_z">
-         <xacro:property name="module" value="${load_yaml(filename)}"/>
+         <xacro:property name="module" value="${xacro.load_yaml(filename)}"/>
         <xacro:property name="mesh_bool" value="false"/>
         <xacro:unless value="${ module['visual']['mesh_body_1'] == '' }">
@@ -622,5 +607,5 @@
     </xacro:macro>
     <xacro:macro name="add_rotor_fast" params="type name filename x y z roll pitch yaw">
-        <xacro:property name="module" value="${load_yaml(filename)}"/>
+        <xacro:property name="module" value="${xacro.load_yaml(filename)}"/>
         <xacro:property name="gear_ratio" value="${module['control']['nu']}"/>
         <link name="${name}">
@@ -644,6 +629,5 @@
     </xacro:macro>
     <xacro:macro name="add_distal" params="type name filename">
-        <xacro:property name="module" value="${load_yaml(filename)}"/>
-        <!-- <xacro:property name="visual" value="${module['visual']['mesh_body_1']}"/> -->
+        <xacro:property name="module" value="${xacro.load_yaml(filename)}"/>
         <xacro:property name="mesh_bool" value="false"/>
         <xacro:unless value="${ module['visual']['mesh_body_2'] == '' }">
@@ -696,6 +680,5 @@
     </xacro:macro>
     <xacro:macro name="add_tool_exchanger" params="type name filename">
-        <xacro:property name="module" value="${load_yaml(filename)}"/>
-        <!-- <xacro:property name="visual" value="${module['visual']['mesh_body_1']}"/> -->
+        <xacro:property name="module" value="${xacro.load_yaml(filename)}"/>
         <xacro:property name="mesh_bool" value="false"/>
         <xacro:unless value="${ module['visual']['mesh_body_1'] == '' }">
@@ -758,5 +741,5 @@
     </xacro:macro>
     <xacro:macro name="add_gripper" params="type name filename">
-        <xacro:property name="module" value="${load_yaml(filename)}"/>
+        <xacro:property name="module" value="${xacro.load_yaml(filename)}"/>
         <xacro:property name="mesh_bool" value="false"/>
         <xacro:unless value="${ module['visual']['mesh_body_1'] == '' }">
@@ -919,5 +902,5 @@
     <!-- Macro for adding the physical module housing the actuator -->
     <xacro:macro name="add_joint_stator" params="type name filename size_y size_z size">
-        <xacro:property name="module" value="${load_yaml(filename)}"/>
+        <xacro:property name="module" value="${xacro.load_yaml(filename)}"/>
         <xacro:property name="mesh_bool" value="false"/>
         <xacro:unless value="${ module['visual']['mesh_body_1'] == '' }">
