Commit message: feat: add concert modules

File: src/modular/modular_data/urdf/ModularBot.library.urdf.xacro (robot description, xacro)
@@ -87,4 +87,46 @@
         </joint>
     </xacro:macro>
+    <!-- Macro for adding a mobile base -->
+    <xacro:macro name="add_mobile_base" params="name filename type">
+        <xacro:property name="module" value="${load_yaml(filename)}"/>
+        <joint name="floating" type="floating">
+            <parent link="base_link"/>
+            <child link="${name}"/>
+            <axis rpy="0 0 0" xyz="0 0 1"/>
+            <origin rpy="0.0 0.0 0.0" xyz="0.0 0.0 0.0"/>
+        </joint>
+        <link name="${name}">
+            <visual>
+                <origin rpy="${module['visual']['tf_mesh_1']['roll']} ${module['visual']['tf_mesh_1']['pitch']} ${module['visual']['tf_mesh_1']['yaw']}"
+                        xyz="${module['visual']['tf_mesh_1']['x']} ${module['visual']['tf_mesh_1']['y']} ${module['visual']['tf_mesh_1']['z']}"/>
+                <geometry>
+                    <!-- <box size="0.34 0.34 0.34"/> -->
+                    <mesh filename="${module['visual']['mesh_body_1']}" scale="0.001 0.001 0.001"/>
+                </geometry>
+                <!-- <material name="gray"/> -->
+            </visual>
+            <collision>
+                <origin rpy="${module['visual']['tf_mesh_1']['roll']} ${module['visual']['tf_mesh_1']['pitch']} ${module['visual']['tf_mesh_1']['yaw']}"
+                        xyz="${module['visual']['tf_mesh_1']['x']} ${module['visual']['tf_mesh_1']['y']} ${module['visual']['tf_mesh_1']['z']}"/>
+                <geometry>
+                    <!-- <box size="0.34 0.34 0.34"/> -->
+                    <mesh filename="${module['visual']['mesh_collision_1']}" scale="0.001 0.001 0.001"/>
+                </geometry>
+            </collision>
+            <inertial>
+                <origin
+                    xyz="${module['dynamics']['body_1']['CoM']['x']} ${module['dynamics']['body_1']['CoM']['y']} ${module['dynamics']['body_1']['CoM']['z']}"
+                    rpy="0 0 0"/>
+                <mass value="${module['dynamics']['body_1']['mass']}"/>
+                <inertia
+                    ixx="${module['dynamics']['body_1']['inertia_tensor']['I_xx']}"
+                    ixy="${module['dynamics']['body_1']['inertia_tensor']['I_xy']}"
+                    ixz="${module['dynamics']['body_1']['inertia_tensor']['I_xz']}"
+                    iyy="${module['dynamics']['body_1']['inertia_tensor']['I_yy']}"
+                    iyz="${module['dynamics']['body_1']['inertia_tensor']['I_yz']}"
+                    izz="${module['dynamics']['body_1']['inertia_tensor']['I_zz']}"/>
+            </inertial>
+        </link>
+    </xacro:macro>
     <!-- Macro for adding a master cube -->
     <xacro:macro name="add_master_cube" params="name filename type">
@@ -98,5 +140,6 @@
         <link name="${name}">
             <visual>
-                <origin rpy="0 0 0" xyz="0 0 0.17"/>
+                <origin rpy="${module['visual']['tf_mesh_1']['roll']} ${module['visual']['tf_mesh_1']['pitch']} ${module['visual']['tf_mesh_1']['yaw']}"
+                        xyz="${module['visual']['tf_mesh_1']['x']} ${module['visual']['tf_mesh_1']['y']} ${module['visual']['tf_mesh_1']['z']}"/>
                 <geometry>
                     <!-- <box size="0.34 0.34 0.34"/> -->
@@ -106,5 +149,6 @@
             </visual>
             <collision>
-                <origin rpy="0 0 0" xyz="0 0 0.17"/>
+                <origin rpy="${module['visual']['tf_mesh_1']['roll']} ${module['visual']['tf_mesh_1']['pitch']} ${module['visual']['tf_mesh_1']['yaw']}"
+                        xyz="${module['visual']['tf_mesh_1']['x']} ${module['visual']['tf_mesh_1']['y']} ${module['visual']['tf_mesh_1']['z']}"/>
                 <geometry>
                     <!-- <box size="0.34 0.34 0.34"/> -->
@@ -189,4 +233,22 @@
             </joint>
         </xacro:if>
+        <xacro:if value="${'connector_5' in module['kinematics']}">
+            <link name="${name}_con5">
+                <visual>
+                    <origin rpy="0 0 0" xyz="0 0 0.05"/>
+                    <geometry>
+                        <cylinder length="0.1" radius="${size_interface}"/>
+                    </geometry>
+                    <material name="green"/>
+                </visual>
+            </link>
+            <joint name="${name}_fixed_5" type="fixed">
+                <parent link="${name}"/>
+                <child link="${name}_con5"/>
+                <axis rpy="0 0 0" xyz="0 0 1"/>
+                <origin rpy="${module['kinematics']['connector_5']['roll']} ${module['kinematics']['connector_5']['pitch']} ${module['kinematics']['connector_5']['yaw']}"
+                        xyz="${module['kinematics']['connector_5']['x']} ${module['kinematics']['connector_5']['y']} ${module['kinematics']['connector_5']['z']}"/>
+            </joint>
+        </xacro:if>
     </xacro:macro>
     <!-- Macro for adding a slave cube -->
@@ -195,5 +257,6 @@
         <link name="${name}">
             <visual>
-                <origin rpy="0 0 0" xyz="0 0 0.17"/>
+                <origin rpy="${module['visual']['tf_mesh_1']['roll']} ${module['visual']['tf_mesh_1']['pitch']} ${module['visual']['tf_mesh_1']['yaw']}"
+                        xyz="${module['visual']['tf_mesh_1']['x']} ${module['visual']['tf_mesh_1']['y']} ${module['visual']['tf_mesh_1']['z']}"/>
                 <geometry>
                     <!-- <box size="0.34 0.34 0.34"/> -->
@@ -203,4 +266,6 @@
             </visual>
             <collision>
+                <origin rpy="${module['visual']['tf_mesh_1']['roll']} ${module['visual']['tf_mesh_1']['pitch']} ${module['visual']['tf_mesh_1']['yaw']}"
+                        xyz="${module['visual']['tf_mesh_1']['x']} ${module['visual']['tf_mesh_1']['y']} ${module['visual']['tf_mesh_1']['z']}"/>
                 <geometry>
                     <!-- <box size="0.34 0.34 0.34"/> -->

Commit message: misc fixes

File: src/modular/modular_data/urdf/ModularBot.library.urdf.xacro (robot description, xacro)
@@ -89,5 +89,5 @@
     <!-- Macro for adding a mobile base -->
     <xacro:macro name="add_mobile_base" params="name filename type">
-        <xacro:property name="module" value="${load_yaml(filename)}"/>
+        <xacro:property name="module" value="${xacro.load_yaml(filename)}"/>
         <joint name="floating" type="floating">
             <parent link="base_link"/>

Commit message: feat(URDFWriter): write a second urdf for Gazebo
adding methods:
- `set_floating_base`: for setting the floating base flag
- `update_xacro_mappings`: to update the `URDFWriter` attribute `xacro_mappings`. These are used to perform arg substitution in the xacro file, so that different urdf can be written depending on the flags value

modified methods:
- `write_urdf`: writes two different urdf, one for xbot and one for gazebo. Uses the value of `URDFWriter.xacro_mappings` to set flags

modified files:
- `ModularBot_gazebo.launch`: to use the gazebo urdf
- `deploy.sh`: to copy the gazebo urdf as well
- `ModularBot.library.urdf.xacro`: change floating joint to fixed
-`template.urdf.xacro`: add arguments to set flags for `floating_joint` and `gazebo_urdf`

File: src/modular/modular_data/urdf/ModularBot.library.urdf.xacro (robot description, xacro)
@@ -90,5 +90,5 @@
     <xacro:macro name="add_mobile_base" params="name filename type">
         <xacro:property name="module" value="${xacro.load_yaml(filename)}"/>
-        <joint name="floating" type="floating">
+        <joint name="fixed" type="fixed">
             <parent link="base_link"/>
             <child link="${name}"/>

File: src/modular/modular_data/urdf/template.urdf.xacro (robot description, xacro)
@@ -3,10 +3,26 @@
     <xacro:include filename="ModularBot.library.urdf.xacro"/>
     <xacro:include filename="ModularBot.control.urdf.xacro"/>
-    <!-- adding world link for Gazebo simulation -->
-    <link name="world"/>
-    <joint name="world" type="fixed">
-        <parent link="world"/>
-        <child link="base_link"/>
-    </joint>
+    <xacro:arg name="floating_joint" default="false"/>
+    <xacro:property name="ADD_FLOATING_BASE" value="$(arg floating_joint)" />
+    <xacro:arg name="gazebo_urdf" default="false"/>
+    <xacro:property name="GAZEBO_URDF" value="$(arg gazebo_urdf)" />
+    <!-- adding (or not) world link for Gazebo simulation -->
+    <xacro:if value="${ADD_FLOATING_BASE}">
+        <xacro:unless value="${GAZEBO_URDF}">
+            <link name="world"/>
+            <joint name="reference" type="floating">
+                <parent link="world"/>
+                <child link="base_link"/>
+            </joint>
+        </xacro:unless>
+        <origin xyz="0.0 0.0 1.2" rpy="0 0 0" />
+    </xacro:if>
+    <xacro:unless value="${ADD_FLOATING_BASE}">
+        <link name="world"/>
+        <joint name="reference" type="fixed">
+            <parent link="world"/>
+            <child link="base_link"/>
+        </joint>
+    </xacro:unless>
     <link name="base_link">
         <xacro:default_inertial mass="0.1"/>

Commit message: wip: handle non-mesh collision geometries for distal links and wheels
to be updated also for other links

File: src/modular/modular_data/urdf/ModularBot.library.urdf.xacro (robot description, xacro)
@@ -715,7 +715,26 @@
                         rpy="${module['visual']['tf_mesh_2']['roll']} ${module['visual']['tf_mesh_2']['pitch']} ${module['visual']['tf_mesh_2']['yaw']}"
                         xyz="${module['visual']['tf_mesh_2']['x']} ${module['visual']['tf_mesh_2']['y']} ${module['visual']['tf_mesh_2']['z']}"/>
-                    <geometry>
-                        <mesh filename="${module['visual']['mesh_collision_2']}" scale="0.001 0.001 0.001"/>
-                    </geometry>
+                    <xacro:if value="${'type' in module['visual']['mesh_collision_2']}">
+                        <xacro:if value="${module['visual']['mesh_collision_2']['type'] == 'box'}">
+                            <geometry>
+                                <box size="${module['visual']['mesh_collision_2']['parameters']['size']}"/>
+                            </geometry>
+                        </xacro:if>
+                        <xacro:if value="${module['visual']['mesh_collision_2']['type'] == 'cylinder'}">
+                            <geometry>
+                                <cylinder radius="${module['visual']['mesh_collision_2']['parameters']['radius']}" length="${module['visual']['mesh_collision_2']['parameters']['length']}"/>
+                            </geometry>
+                        </xacro:if>
+                        <xacro:if value="${module['visual']['mesh_collision_2']['type'] == 'sphere'}">
+                            <geometry>
+                                <sphere radius="${module['visual']['mesh_collision_2']['parameters']['radius']}"/>
+                            </geometry>
+                        </xacro:if>
+                    </xacro:if>
+                    <xacro:unless value="${'type' in module['visual']['mesh_collision_2']}">
+                        <geometry>
+                            <mesh filename="${module['visual']['mesh_collision_2']}" scale="0.001 0.001 0.001"/>
+                        </geometry>
+                    </xacro:unless>
                 </collision>
             </xacro:if>

Commit message: feat: add `<gazebo>` tag according to YAML description
- modified YAML. If no gazebo tag is needed the value associated to a gazebo key is an empty string
- modified xacro library. add gazebo tag only if the `gazebo_urdf` flag is set to true

File: src/modular/modular_data/urdf/ModularBot.library.urdf.xacro (robot description, xacro)
@@ -430,13 +430,15 @@
             </link>
         </xacro:unless>
-        <gazebo reference="${name}">
-            <mu1>0.2</mu1>
-            <mu2>0.2</mu2>
-            <kp>1000000.0</kp>
-            <kd>1.0</kd>
-            <maxVel>0.0</maxVel>
-            <minDepth>0.0001</minDepth>
-            <material>Gazebo/White</material>
-        </gazebo>
+        <xacro:if value="${ GAZEBO_URDF }">
+            <gazebo reference="${name}">
+                <mu1>0.2</mu1>
+                <mu2>0.2</mu2>
+                <kp>1000000.0</kp>
+                <kd>1.0</kd>
+                <maxVel>0.0</maxVel>
+                <minDepth>0.0001</minDepth>
+                <material>Gazebo/White</material>
+            </gazebo>
+        </xacro:if>
     </xacro:macro>
     <!-- Macro for adding a socket -->
@@ -467,13 +469,15 @@
             </inertial>
         </link>
-        <gazebo reference="${name}">
-            <mu1>0.2</mu1>
-            <mu2>0.2</mu2>
-            <kp>1000000.0</kp>
-            <kd>1.0</kd>
-            <maxVel>0.0</maxVel>
-            <minDepth>0.0001</minDepth>
-            <material>Gazebo/White</material>
-        </gazebo>
+        <xacro:if value="${ GAZEBO_URDF }">
+            <gazebo reference="${name}">
+                <mu1>0.2</mu1>
+                <mu2>0.2</mu2>
+                <kp>1000000.0</kp>
+                <kd>1.0</kd>
+                <maxVel>0.0</maxVel>
+                <minDepth>0.0001</minDepth>
+                <material>Gazebo/White</material>
+            </gazebo>
+        </xacro:if>
     </xacro:macro>
     <!-- Macro for adding a size adapter -->
@@ -579,13 +583,15 @@
             </link>
         </xacro:unless>
-        <gazebo reference="${name}">
-            <mu1>0.2</mu1>
-            <mu2>0.2</mu2>
-            <kp>1000000.0</kp>
-            <kd>1.0</kd>
-            <maxVel>0.0</maxVel>
-            <minDepth>0.0001</minDepth>
-            <material>Gazebo/Grey</material>
-        </gazebo>
+        <xacro:if value="${ GAZEBO_URDF }">
+            <gazebo reference="${name}">
+                <mu1>0.2</mu1>
+                <mu2>0.2</mu2>
+                <kp>1000000.0</kp>
+                <kd>1.0</kd>
+                <maxVel>0.0</maxVel>
+                <minDepth>0.0001</minDepth>
+                <material>Gazebo/Grey</material>
+            </gazebo>
+        </xacro:if>
     </xacro:macro>
     <!-- Macro for adding an elbow module (90° link) -->
@@ -651,13 +657,15 @@
             </collision>
         </link>
-        <gazebo reference="${name}">
-            <mu1>0.2</mu1>
-            <mu2>0.2</mu2>
-            <kp>1000000.0</kp>
-            <kd>1.0</kd>
-            <maxVel>0.0</maxVel>
-            <minDepth>0.0001</minDepth>
-            <material>Gazebo/White</material>
-        </gazebo>
+        <xacro:if value="${ GAZEBO_URDF }">
+            <gazebo reference="${name}">
+                <mu1>0.2</mu1>
+                <mu2>0.2</mu2>
+                <kp>1000000.0</kp>
+                <kd>1.0</kd>
+                <maxVel>0.0</maxVel>
+                <minDepth>0.0001</minDepth>
+                <material>Gazebo/White</material>
+            </gazebo>
+        </xacro:if>
     </xacro:macro>
     <!-- Macro for adding the joint. A dummy link is also added with no visual tag, but with inertial parameters corresponding to the rotating part -->
@@ -762,4 +770,50 @@
             </inertial>
         </link>
+        <xacro:if value="${ GAZEBO_URDF }">
+            <xacro:unless value="${ module['gazebo'] == '' }">
+                <gazebo reference="${name}">
+                    <material>${ module['gazebo']['material']}</material>
+                    <collision>
+                        <surface>
+                            <friction>
+                                <!-- <torsional>
+                                    <coefficient> 1.0 </coefficient>
+                                    <use_patch_radius>true</use_patch_radius>
+                                    <patch_radius>0.2</patch_radius>
+                                </torsional> -->
+                                <ode>
+                                    <mu>${ module['gazebo']['collision']['surface']['friction']['ode']['mu']}</mu>
+                                    <mu2>${ module['gazebo']['collision']['surface']['friction']['ode']['mu2']}</mu2>
+                                </ode>
+                                <bullet>
+                                    <friction>${ module['gazebo']['collision']['surface']['friction']['bullet']['friction']}</friction>
+                                    <friction2>${ module['gazebo']['collision']['surface']['friction']['bullet']['friction2']}</friction2>
+                                </bullet>
+                            </friction>
+                            <contact>
+                                <ode>
+                                    <kp>${ module['gazebo']['collision']['surface']['contact']['ode']['kp']}</kp>
+                                    <kd>${ module['gazebo']['collision']['surface']['contact']['ode']['kd']}</kd>
+                                    <max_vel>${ module['gazebo']['collision']['surface']['contact']['ode']['max_vel']}</max_vel>
+                                </ode>
+                                <bullet>
+                                    <soft_cfm>${ module['gazebo']['collision']['surface']['contact']['bullet']['soft_cfm']}</soft_cfm>
+                                    <soft_erp>${ module['gazebo']['collision']['surface']['contact']['bullet']['soft_erp']}</soft_erp>
+                                    <kp>${ module['gazebo']['collision']['surface']['contact']['bullet']['kp']}</kp>
+                                    <kd>${ module['gazebo']['collision']['surface']['contact']['bullet']['kd']}</kd>
+                                </bullet>
+                            </contact>
+                        </surface>
+                    </collision>
+                </gazebo>
+            </xacro:unless>
+        </xacro:if>
+    </xacro:macro>
+    <xacro:macro name="gazebo_element" params="name">
+        <xacro:property name="GAZEBO_URDF" value="$(arg gazebo_urdf)" />
+        <xacro:if value="${GAZEBO_URDF}">
+            <gazebo reference="${name}">
+            </gazebo>
+        </xacro:if>
     </xacro:macro>
     <xacro:macro name="add_tool_exchanger" params="type name filename">
@@ -1062,13 +1116,15 @@
             </link>
         </xacro:unless>
-        <gazebo reference="${name}">
-            <mu1>0.2</mu1>
-            <mu2>0.2</mu2>
-            <kp>1000000.0</kp>
-            <kd>1.0</kd>
-            <maxVel>0.0</maxVel>
-            <minDepth>0.0001</minDepth>
-            <material>Gazebo/Blue</material>
-        </gazebo>
+        <xacro:if value="${ GAZEBO_URDF }">
+            <gazebo reference="${name}">
+                <mu1>0.2</mu1>
+                <mu2>0.2</mu2>
+                <kp>1000000.0</kp>
+                <kd>1.0</kd>
+                <maxVel>0.0</maxVel>
+                <minDepth>0.0001</minDepth>
+                <material>Gazebo/Blue</material>
+            </gazebo>
+        </xacro:if>
     </xacro:macro>
     <!-- Macro for adding a fixed joint (rigid interconnection between links and statoric part of the joint) -->
