Commit message: feat: gazebo tags are added by `add_gazebo_element`
- Only python handles the gazebo tags. removed all `<gazebo>` from xacro.
- modified YAML gazebo fields to be consistent with python

File: src/modular/modular_data/urdf/ModularBot.library.urdf.xacro (robot description, xacro)
@@ -430,15 +430,4 @@
             </link>
         </xacro:unless>
-        <xacro:if value="${ GAZEBO_URDF }">
-            <gazebo reference="${name}">
-                <mu1>0.2</mu1>
-                <mu2>0.2</mu2>
-                <kp>1000000.0</kp>
-                <kd>1.0</kd>
-                <maxVel>0.0</maxVel>
-                <minDepth>0.0001</minDepth>
-                <material>Gazebo/White</material>
-            </gazebo>
-        </xacro:if>
     </xacro:macro>
     <!-- Macro for adding a socket -->
@@ -469,15 +458,4 @@
             </inertial>
         </link>
-        <xacro:if value="${ GAZEBO_URDF }">
-            <gazebo reference="${name}">
-                <mu1>0.2</mu1>
-                <mu2>0.2</mu2>
-                <kp>1000000.0</kp>
-                <kd>1.0</kd>
-                <maxVel>0.0</maxVel>
-                <minDepth>0.0001</minDepth>
-                <material>Gazebo/White</material>
-            </gazebo>
-        </xacro:if>
     </xacro:macro>
     <!-- Macro for adding a size adapter -->
@@ -491,5 +469,4 @@
             <link name="${name}">
                 <visual>
-                    <!-- Load mesh. Rotate the origin frame (this is because of how the .stl was saved) -->
                     <origin
                         rpy="${module['visual']['tf_mesh_1']['roll']} ${module['visual']['tf_mesh_1']['pitch']} ${module['visual']['tf_mesh_1']['yaw']}"
@@ -583,15 +560,4 @@
             </link>
         </xacro:unless>
-        <xacro:if value="${ GAZEBO_URDF }">
-            <gazebo reference="${name}">
-                <mu1>0.2</mu1>
-                <mu2>0.2</mu2>
-                <kp>1000000.0</kp>
-                <kd>1.0</kd>
-                <maxVel>0.0</maxVel>
-                <minDepth>0.0001</minDepth>
-                <material>Gazebo/Grey</material>
-            </gazebo>
-        </xacro:if>
     </xacro:macro>
     <!-- Macro for adding an elbow module (90° link) -->
@@ -657,15 +623,4 @@
             </collision>
         </link>
-        <xacro:if value="${ GAZEBO_URDF }">
-            <gazebo reference="${name}">
-                <mu1>0.2</mu1>
-                <mu2>0.2</mu2>
-                <kp>1000000.0</kp>
-                <kd>1.0</kd>
-                <maxVel>0.0</maxVel>
-                <minDepth>0.0001</minDepth>
-                <material>Gazebo/White</material>
-            </gazebo>
-        </xacro:if>
     </xacro:macro>
     <!-- Macro for adding the joint. A dummy link is also added with no visual tag, but with inertial parameters corresponding to the rotating part -->
@@ -710,5 +665,4 @@
             <xacro:if value="${ mesh_bool }">
                 <visual>
-                    <!-- Load mesh. Rotate the origin frame (this is because of how the .stl was saved) -->
                     <origin
                         rpy="${module['visual']['tf_mesh_2']['roll']} ${module['visual']['tf_mesh_2']['pitch']} ${module['visual']['tf_mesh_2']['yaw']}"
@@ -747,13 +701,4 @@
                 </collision>
             </xacro:if>
-            <!--inertial parameters for ORANGE rotating part. wrt a point on one end of the rod-->
-            <!-- <inertial>
-                <origin xyz="0 0 -0.002265" rpy="0 0 0"/>
-                <mass value="0.153466"/>
-                <inertia
-                        ixx="0.000034763" ixy="0.0" ixz="0.0"
-                        iyy="0.000034827" iyz="0.0"
-                        izz="0.000031822"/>
-            </inertial> -->
             <inertial>
                 <origin
@@ -770,50 +715,4 @@
             </inertial>
         </link>
-        <xacro:if value="${ GAZEBO_URDF }">
-            <xacro:unless value="${ module['gazebo'] == '' }">
-                <gazebo reference="${name}">
-                    <material>${ module['gazebo']['material']}</material>
-                    <collision>
-                        <surface>
-                            <friction>
-                                <!-- <torsional>
-                                    <coefficient> 1.0 </coefficient>
-                                    <use_patch_radius>true</use_patch_radius>
-                                    <patch_radius>0.2</patch_radius>
-                                </torsional> -->
-                                <ode>
-                                    <mu>${ module['gazebo']['collision']['surface']['friction']['ode']['mu']}</mu>
-                                    <mu2>${ module['gazebo']['collision']['surface']['friction']['ode']['mu2']}</mu2>
-                                </ode>
-                                <bullet>
-                                    <friction>${ module['gazebo']['collision']['surface']['friction']['bullet']['friction']}</friction>
-                                    <friction2>${ module['gazebo']['collision']['surface']['friction']['bullet']['friction2']}</friction2>
-                                </bullet>
-                            </friction>
-                            <contact>
-                                <ode>
-                                    <kp>${ module['gazebo']['collision']['surface']['contact']['ode']['kp']}</kp>
-                                    <kd>${ module['gazebo']['collision']['surface']['contact']['ode']['kd']}</kd>
-                                    <max_vel>${ module['gazebo']['collision']['surface']['contact']['ode']['max_vel']}</max_vel>
-                                </ode>
-                                <bullet>
-                                    <soft_cfm>${ module['gazebo']['collision']['surface']['contact']['bullet']['soft_cfm']}</soft_cfm>
-                                    <soft_erp>${ module['gazebo']['collision']['surface']['contact']['bullet']['soft_erp']}</soft_erp>
-                                    <kp>${ module['gazebo']['collision']['surface']['contact']['bullet']['kp']}</kp>
-                                    <kd>${ module['gazebo']['collision']['surface']['contact']['bullet']['kd']}</kd>
-                                </bullet>
-                            </contact>
-                        </surface>
-                    </collision>
-                </gazebo>
-            </xacro:unless>
-        </xacro:if>
-    </xacro:macro>
-    <xacro:macro name="gazebo_element" params="name">
-        <xacro:property name="GAZEBO_URDF" value="$(arg gazebo_urdf)" />
-        <xacro:if value="${GAZEBO_URDF}">
-            <gazebo reference="${name}">
-            </gazebo>
-        </xacro:if>
     </xacro:macro>
     <xacro:macro name="add_tool_exchanger" params="type name filename">
@@ -826,5 +725,4 @@
             <xacro:if value="${ mesh_bool }">
                 <visual>
-                    <!-- Load mesh. Rotate the origin frame (this is because of how the .stl was saved) -->
                     <origin
                         rpy="${module['visual']['tf_mesh_1']['roll']} ${module['visual']['tf_mesh_1']['pitch']} ${module['visual']['tf_mesh_1']['yaw']}"
@@ -844,13 +742,4 @@
                 </collision>
             </xacro:if>
-            <!--inertial parameters for ORANGE rotating part. wrt a point on one end of the rod-->
-            <!-- <inertial>
-                <origin xyz="0 0 -0.002265" rpy="0 0 0"/>
-                <mass value="0.153466"/>
-                <inertia
-                        ixx="0.000034763" ixy="0.0" ixz="0.0"
-                        iyy="0.000034827" iyz="0.0"
-                        izz="0.000031822"/>
-            </inertial> -->
             <inertial>
                 <origin
@@ -1116,15 +1005,4 @@
             </link>
         </xacro:unless>
-        <xacro:if value="${ GAZEBO_URDF }">
-            <gazebo reference="${name}">
-                <mu1>0.2</mu1>
-                <mu2>0.2</mu2>
-                <kp>1000000.0</kp>
-                <kd>1.0</kd>
-                <maxVel>0.0</maxVel>
-                <minDepth>0.0001</minDepth>
-                <material>Gazebo/Blue</material>
-            </gazebo>
-        </xacro:if>
     </xacro:macro>
     <!-- Macro for adding a fixed joint (rigid interconnection between links and statoric part of the joint) -->
