Commit message: refactor `library.urdf.xacro` and YAML structure

File: src/modular/modular_data/urdf/ModularBot.library.urdf.xacro (robot description, xacro)
@@ -49,34 +49,99 @@
         </inertial>
     </xacro:macro>
-    <!-- Macro for adding a table -->
-    <xacro:macro name="add_table" params="type name father">
-        <joint name="fixed_table" type="fixed">
-            <axis rpy="0 0 0" xyz="0 0 1"/>
+    <xacro:macro name="add_geometry" params="body">
+        <geometry>
+            <xacro:if value="${body['type'] == 'mesh'}">
+                <mesh filename="${body['parameters']['file']}" scale="${' '.join(str(x) for x in body['parameters']['scale'])}"/>
+            </xacro:if>
+            <xacro:if value="${body['type'] == 'cylinder'}">
+                <cylinder radius="${body['parameters']['radius']}" length="${body['parameters']['length']}"/>
+            </xacro:if>
+            <xacro:if value="${body['type'] == 'box'}">
+                <box size="${body['parameters']['size']}"/>
+            </xacro:if>
+            <xacro:if value="${body['type'] == 'sphere'}">
+                <sphere radius="${body['parameters']['radius']}"/>
+            </xacro:if>
+        </geometry>
+    </xacro:macro>
+    <xacro:macro name="add_origin" params="body_pose">
+        <origin
+            rpy="${body_pose['roll']} ${body_pose['pitch']} ${body_pose['yaw']}"
+            xyz="${body_pose['x']} ${body_pose['y']} ${body_pose['z']}"/>
+    </xacro:macro>
+    <xacro:macro name="add_link_element" params="name type module body_name">
+        <xacro:property name="visual_bool" value="false"/>
+        <xacro:unless value="${module['visual'][body_name] == '' }">
+            <xacro:property name="visual_bool" value="true"/>
+            <xacro:property name="visual_body" value="${module['visual'][body_name]}"/>
+        </xacro:unless>
+        <xacro:property name="collision_bool" value="false"/>
+        <xacro:unless value="${module['collision'][body_name] == '' }">
+            <xacro:property name="collision_bool" value="true"/>
+            <xacro:property name="collision_body" value="${module['collision'][body_name]}"/>
+        </xacro:unless>
+        <xacro:property name="dynamics_body" value="${module['dynamics'][body_name]}"/>
+        <link name="${name}">
+            <xacro:unless value="${visual_bool == 0}">
+                <visual>
+                    <xacro:add_origin body_pose="${visual_body['pose']}"/>
+                    <xacro:add_geometry body="${visual_body}"/>
+                    <material name="${visual_body['color']}"/>
+                </visual>
+            </xacro:unless>
+            <xacro:unless value="${collision_bool == 0}">
+                <collision>
+                    <xacro:add_origin body_pose="${collision_body['pose']}"/>
+                    <xacro:add_geometry body="${collision_body}"/>
+                </collision>
+            </xacro:unless>
+            <xacro:if value="${dynamics_body['mass'] == 0.0}">
+                <xacro:default_inertial mass="${mass}"/>
+            </xacro:if>
+            <xacro:unless value="${dynamics_body['mass'] == 0.0}">
+                <inertial>
+                    <origin
+                        xyz="${dynamics_body['CoM']['x']} ${dynamics_body['CoM']['y']} ${dynamics_body['CoM']['z']}"
+                        rpy="0 0 0"/>
+                    <mass value="${dynamics_body['mass']}"/>
+                    <inertia
+                        ixx="${dynamics_body['inertia_tensor']['I_xx']}"
+                        ixy="${dynamics_body['inertia_tensor']['I_xy']}"
+                        ixz="${dynamics_body['inertia_tensor']['I_xz']}"
+                        iyy="${dynamics_body['inertia_tensor']['I_yy']}"
+                        iyz="${dynamics_body['inertia_tensor']['I_yz']}"
+                        izz="${dynamics_body['inertia_tensor']['I_zz']}"/>
+                </inertial>
+            </xacro:unless>
+        </link>
+    </xacro:macro>
+    <!-- Macro for adding a straight link -->
+    <xacro:macro name="add_link" params="name type filename">
+        <xacro:property name="module" value="${xacro.load_yaml(filename)}"/>
+        <xacro:property name="body_name" value="body_1"/>
+        <xacro:add_link_element name="${name}" type="${type}" module="${module}" body_name="${body_name}"/>
+    </xacro:macro>
+    <!-- Macro for adding the physical module housing the actuator -->
+    <xacro:macro name="add_joint_stator" params="type name filename">
+        <xacro:property name="module" value="${xacro.load_yaml(filename)}"/>
+        <xacro:property name="body_name" value="body_1"/>
+        <xacro:add_link_element name="${name}" type="${type}" module="${module}" body_name="${body_name}"/>
+    </xacro:macro>
+    <xacro:macro name="add_distal" params="type name filename">
+        <xacro:property name="module" value="${xacro.load_yaml(filename)}"/>
+        <xacro:property name="body_name" value="body_2"/>
+        <xacro:add_link_element name="${name}" type="${type}" module="${module}" body_name="${body_name}"/>
+    </xacro:macro>
+    <!-- Macro for adding the joint. A dummy link is also added with no visual tag, but with inertial parameters corresponding to the rotating part -->
+    <xacro:macro name="add_joint" params="type name father child x y z roll pitch yaw upper_lim lower_lim effort velocity">
+        <joint name="${name}" type="revolute">
+            <axis xyz="0 0 1" rpy="0 0 0" />
             <parent link="${father}"/>
-            <child link="${name}"/>
-            <origin rpy="0.0 0.0 0.0" xyz="0.0 0.0 0.01"/>
-        </joint>
-        <link name="${name}">
-            <visual>
-                <origin rpy="0 0 0" xyz="0.6 0.3 -0.005"/>
-                <geometry>
-                    <box size="1.2 0.6 0.01"/>
-                </geometry>
-                <material name="gray"/>
-            </visual>
-            <collision>
-                <origin rpy="0 0 0" xyz="0.6 0.3 -0.005"/>
-                <geometry>
-                    <box size="1.2 0.6 0.01"/>
-                </geometry>
-            </collision>
-            <inertial>
-                <origin rpy="0 0 0" xyz="0 0 0.00"/>
-                <mass value="0.5"/>
-                <inertia ixx="0.0006" ixy="0.0" ixz="0.0" iyy="0.0006" iyz="0.0" izz="0.0006"/>
-            </inertial>
-        </link>
-    </xacro:macro>
-    <!-- Macro for adding a fixed joint (rigid interconnection between links) -->
+            <child link="${child}"/>
+            <origin xyz="${x} ${y} ${z}" rpy="${roll} ${pitch} ${yaw}"/>
+            <limit lower="${lower_lim}" upper="${upper_lim}" effort="${effort}" velocity="${velocity}"/>
+        </joint>
+    </xacro:macro>
+    <!-- Macro for adding a fixed joint (rigid interconnection between links and statoric part of the joint) -->
     <xacro:macro name="add_fixed_joint" params="type name father child x y z roll pitch yaw">
         <joint name="${name}" type="fixed">
@@ -87,4 +152,26 @@
         </joint>
     </xacro:macro>
+    <xacro:macro name="add_rotor_fast" params="type name filename x y z roll pitch yaw">
+        <xacro:property name="module" value="${xacro.load_yaml(filename)}"/>
+        <xacro:property name="gear_ratio" value="${module['control']['nu']}"/>
+        <link name="${name}">
+            <inertial>
+                <origin
+                        xyz="${module['dynamics']['body_2_fast']['CoM']['x']} ${module['dynamics']['body_2_fast']['CoM']['y']} ${module['dynamics']['body_2_fast']['CoM']['z']}"
+                        rpy="0 0 0"/>
+                    <mass value="${module['dynamics']['body_2_fast']['mass']}"/>
+                    <inertia
+                        ixx="${module['dynamics']['body_2_fast']['inertia_tensor']['I_xx']}"
+                        ixy="${module['dynamics']['body_2_fast']['inertia_tensor']['I_xy']}"
+                        iyy="${module['dynamics']['body_2_fast']['inertia_tensor']['I_yy']}"
+                        ixz="${module['dynamics']['body_2_fast']['inertia_tensor']['I_xz'] }"
+                        iyz="${module['dynamics']['body_2_fast']['inertia_tensor']['I_yz'] }"
+                        izz="${ gear_ratio * gear_ratio * module['dynamics']['body_2_fast']['inertia_tensor']['I_zz'] }"/>
+                        <!-- ixz="${ gear_ratio * module['dynamics']['body_2_fast']['inertia_tensor']['I_xz'] }" -->
+                        <!-- iyz="${ gear_ratio * module['dynamics']['body_2_fast']['inertia_tensor']['I_yz'] }" -->
+                        <!-- izz="${module['dynamics']['body_2_fast']['inertia_tensor']['I_zz'] }" -->
+            </inertial>
+        </link>
+    </xacro:macro>
     <!-- Macro for adding a mobile base -->
     <xacro:macro name="add_mobile_base" params="name filename type">
@@ -96,36 +183,6 @@
             <origin rpy="0.0 0.0 0.0" xyz="0.0 0.0 0.0"/>
         </joint>
-        <link name="${name}">
-            <visual>
-                <origin rpy="${module['visual']['tf_mesh_1']['roll']} ${module['visual']['tf_mesh_1']['pitch']} ${module['visual']['tf_mesh_1']['yaw']}"
-                        xyz="${module['visual']['tf_mesh_1']['x']} ${module['visual']['tf_mesh_1']['y']} ${module['visual']['tf_mesh_1']['z']}"/>
-                <geometry>
-                    <!-- <box size="0.34 0.34 0.34"/> -->
-                    <mesh filename="${module['visual']['mesh_body_1']}" scale="0.001 0.001 0.001"/>
-                </geometry>
-                <!-- <material name="gray"/> -->
-            </visual>
-            <collision>
-                <origin rpy="${module['visual']['tf_mesh_1']['roll']} ${module['visual']['tf_mesh_1']['pitch']} ${module['visual']['tf_mesh_1']['yaw']}"
-                        xyz="${module['visual']['tf_mesh_1']['x']} ${module['visual']['tf_mesh_1']['y']} ${module['visual']['tf_mesh_1']['z']}"/>
-                <geometry>
-                    <!-- <box size="0.34 0.34 0.34"/> -->
-                    <mesh filename="${module['visual']['mesh_collision_1']}" scale="0.001 0.001 0.001"/>
-                </geometry>
-            </collision>
-            <inertial>
-                <origin
-                    xyz="${module['dynamics']['body_1']['CoM']['x']} ${module['dynamics']['body_1']['CoM']['y']} ${module['dynamics']['body_1']['CoM']['z']}"
-                    rpy="0 0 0"/>
-                <mass value="${module['dynamics']['body_1']['mass']}"/>
-                <inertia
-                    ixx="${module['dynamics']['body_1']['inertia_tensor']['I_xx']}"
-                    ixy="${module['dynamics']['body_1']['inertia_tensor']['I_xy']}"
-                    ixz="${module['dynamics']['body_1']['inertia_tensor']['I_xz']}"
-                    iyy="${module['dynamics']['body_1']['inertia_tensor']['I_yy']}"
-                    iyz="${module['dynamics']['body_1']['inertia_tensor']['I_yz']}"
-                    izz="${module['dynamics']['body_1']['inertia_tensor']['I_zz']}"/>
-            </inertial>
-        </link>
+        <xacro:property name="body_name" value="body_1"/>
+        <xacro:add_link_element name="${name}" type="${type}" module="${module}" body_name="${body_name}"/>
     </xacro:macro>
     <!-- Macro for adding a master cube -->
@@ -143,8 +200,6 @@
                         xyz="${module['visual']['tf_mesh_1']['x']} ${module['visual']['tf_mesh_1']['y']} ${module['visual']['tf_mesh_1']['z']}"/>
                 <geometry>
-                    <!-- <box size="0.34 0.34 0.34"/> -->
                     <mesh filename="${module['visual']['mesh_body_1']}" scale="0.001 0.001 0.001"/>
                 </geometry>
-                <!-- <material name="gray"/> -->
             </visual>
             <collision>
@@ -152,5 +207,4 @@
                         xyz="${module['visual']['tf_mesh_1']['x']} ${module['visual']['tf_mesh_1']['y']} ${module['visual']['tf_mesh_1']['z']}"/>
                 <geometry>
-                    <!-- <box size="0.34 0.34 0.34"/> -->
                     <mesh filename="${module['visual']['mesh_collision_1']}" scale="0.001 0.001 0.001"/>
                 </geometry>
@@ -260,8 +314,6 @@
                         xyz="${module['visual']['tf_mesh_1']['x']} ${module['visual']['tf_mesh_1']['y']} ${module['visual']['tf_mesh_1']['z']}"/>
                 <geometry>
-                    <!-- <box size="0.34 0.34 0.34"/> -->
                     <mesh filename="${module['visual']['mesh_body_1']}" scale="0.001 0.001 0.001"/>
                 </geometry>
-                <!-- <material name="grey"/> -->
             </visual>
             <collision>
@@ -269,5 +321,4 @@
                         xyz="${module['visual']['tf_mesh_1']['x']} ${module['visual']['tf_mesh_1']['y']} ${module['visual']['tf_mesh_1']['z']}"/>
                 <geometry>
-                    <!-- <box size="0.34 0.34 0.34"/> -->
                     <mesh filename="${module['visual']['mesh_body_1']}" scale="0.001 0.001 0.001"/>
                 </geometry>
@@ -341,93 +392,4 @@
                     xyz="${module['kinematics']['connector_4']['x']} ${module['kinematics']['connector_4']['y']} ${module['kinematics']['connector_4']['z']}"/>
         </joint> -->
-    </xacro:macro>
-    <!-- Macro for adding a straight link -->
-    <xacro:macro name="add_link" params="name type filename size_z size">
-        <xacro:property name="module" value="${xacro.load_yaml(filename)}"/>
-        <xacro:property name="mesh_bool" value="false"/>
-        <xacro:unless value="${ module['visual']['mesh_body_1'] == '' }">
-            <xacro:property name="mesh_bool" value="true"/>
-        </xacro:unless>
-        <xacro:if value="${size==1}">
-            <xacro:property name="radius" value="${size1}" />
-        </xacro:if>
-        <xacro:unless value="${size==1}">
-            <xacro:if value="${size==2}">
-                <xacro:property name="radius" value="${size2}" />
-            </xacro:if>
-            <xacro:unless value="${size==2}">
-                <xacro:if value="${size==3}">
-                    <xacro:property name="radius" value="${size3}" />
-                </xacro:if>
-                <xacro:unless value="${size==3}">
-                    <xacro:if value="${size==4}">
-                        <xacro:property name="radius" value="${size4}" />
-                    </xacro:if>
-                    <xacro:unless value="${size==4}">
-                        <xacro:property name="radius" value="${size5}" />
-                    </xacro:unless>
-                </xacro:unless>
-            </xacro:unless>
-        </xacro:unless>
-        <xacro:if value="${mesh_bool}">
-            <link name="${name}">
-                <visual>
-                    <!-- Load mesh. Rotate the origin frame (this is because of how the .stl was saved) -->
-                    <origin
-                        rpy="${module['visual']['tf_mesh_1']['roll']} ${module['visual']['tf_mesh_1']['pitch']} ${module['visual']['tf_mesh_1']['yaw']}"
-                        xyz="${module['visual']['tf_mesh_1']['x']} ${module['visual']['tf_mesh_1']['y']} ${module['visual']['tf_mesh_1']['z']}"/>
-                    <geometry>
-                        <mesh filename="${module['visual']['mesh_body_1']}" scale="0.001 0.001 0.001"/>
-                    </geometry>
-                    <material name="white"/>
-                </visual>
-                <collision>
-                    <origin
-                        rpy="${module['visual']['tf_mesh_1']['roll']} ${module['visual']['tf_mesh_1']['pitch']} ${module['visual']['tf_mesh_1']['yaw']}"
-                        xyz="${module['visual']['tf_mesh_1']['x']} ${module['visual']['tf_mesh_1']['y']} ${module['visual']['tf_mesh_1']['z']}"/>
-                    <geometry>
-                        <mesh filename="${module['visual']['mesh_collision_1']}" scale="0.001 0.001 0.001"/>
-                    </geometry>
-                </collision>
-                <inertial>
-                    <origin
-                        xyz="${module['dynamics']['body_1']['CoM']['x']} ${module['dynamics']['body_1']['CoM']['y']} ${module['dynamics']['body_1']['CoM']['z']}"
-                        rpy="0 0 0"/>
-                    <mass value="${module['dynamics']['body_1']['mass']}"/>
-                    <inertia
-                        ixx="${module['dynamics']['body_1']['inertia_tensor']['I_xx']}"
-                        ixy="${module['dynamics']['body_1']['inertia_tensor']['I_xy']}"
-                        ixz="${module['dynamics']['body_1']['inertia_tensor']['I_xz']}"
-                        iyy="${module['dynamics']['body_1']['inertia_tensor']['I_yy']}"
-                        iyz="${module['dynamics']['body_1']['inertia_tensor']['I_yz']}"
-                        izz="${module['dynamics']['body_1']['inertia_tensor']['I_zz']}"/>
-                </inertial>
-            </link>
-        </xacro:if>
-        <xacro:unless value="${mesh_bool}">
-            <link name="${name}">
-                <visual>
-                    <origin xyz="0 0 ${size_z/2}" rpy="0 0 0" />
-                    <geometry>
-                        <cylinder radius="${radius}" length="${size_z}"/>
-                    </geometry>
-                    <material name="white"/>
-                </visual>
-                <collision>
-                    <origin xyz="0 0 ${size_z/2}" rpy="0 0 0" />
-                    <geometry>
-                        <cylinder radius="${radius}" length="${size_z}"/>
-                    </geometry>
-                </collision>
-                <inertial>
-                    <origin xyz="0 0 ${size_z/2}" rpy="0 0 0"/>
-                    <mass value="${mass}"/>
-                    <inertia
-                    ixx="${mass / 12.0 * (3*radius*radius + size_z*size_z)}" ixy="0.0" ixz="0.0"
-                    iyy="${mass / 12.0 * (size_z*size_z + 3*radius*radius)}" iyz="0.0"
-                    izz="${mass / 2.0 * (radius*radius)}"/>
-                </inertial>
-            </link>
-        </xacro:unless>
     </xacro:macro>
     <!-- Macro for adding a socket -->
@@ -624,40 +586,8 @@
         </link>
     </xacro:macro>
-    <!-- Macro for adding the joint. A dummy link is also added with no visual tag, but with inertial parameters corresponding to the rotating part -->
-    <xacro:macro name="add_joint" params="type name father child x y z roll pitch yaw upper_lim lower_lim effort velocity">
-        <joint name="${name}" type="revolute">
-            <axis xyz="0 0 1" rpy="0 0 0" />
-            <parent link="${father}"/>
-            <child link="${child}"/>
-            <origin xyz="${x} ${y} ${z}" rpy="${roll} ${pitch} ${yaw}"/>
-            <limit lower="${lower_lim}" upper="${upper_lim}" effort="${effort}" velocity="${velocity}"/>
-        </joint>
-    </xacro:macro>
-    <xacro:macro name="add_rotor_fast" params="type name filename x y z roll pitch yaw">
-        <xacro:property name="module" value="${xacro.load_yaml(filename)}"/>
-        <xacro:property name="gear_ratio" value="${module['control']['nu']}"/>
-        <link name="${name}">
-            <inertial>
-                <origin
-                        xyz="${module['dynamics']['body_2_fast']['CoM']['x']} ${module['dynamics']['body_2_fast']['CoM']['y']} ${module['dynamics']['body_2_fast']['CoM']['z']}"
-                        rpy="0 0 0"/>
-                    <mass value="${module['dynamics']['body_2_fast']['mass']}"/>
-                    <inertia
-                        ixx="${module['dynamics']['body_2_fast']['inertia_tensor']['I_xx']}"
-                        ixy="${module['dynamics']['body_2_fast']['inertia_tensor']['I_xy']}"
-                        iyy="${module['dynamics']['body_2_fast']['inertia_tensor']['I_yy']}"
-                        ixz="${module['dynamics']['body_2_fast']['inertia_tensor']['I_xz'] }"
-                        iyz="${module['dynamics']['body_2_fast']['inertia_tensor']['I_yz'] }"
-                        izz="${ gear_ratio * gear_ratio * module['dynamics']['body_2_fast']['inertia_tensor']['I_zz'] }"/>
-                        <!-- ixz="${ gear_ratio * module['dynamics']['body_2_fast']['inertia_tensor']['I_xz'] }" -->
-                        <!-- iyz="${ gear_ratio * module['dynamics']['body_2_fast']['inertia_tensor']['I_yz'] }" -->
-                        <!-- izz="${module['dynamics']['body_2_fast']['inertia_tensor']['I_zz'] }" -->
-            </inertial>
-        </link>
-    </xacro:macro>
-    <xacro:macro name="add_distal" params="type name filename">
+    <xacro:macro name="add_tool_exchanger" params="type name filename">
         <xacro:property name="module" value="${xacro.load_yaml(filename)}"/>
         <xacro:property name="mesh_bool" value="false"/>
-        <xacro:unless value="${ module['visual']['mesh_body_2'] == '' }">
+        <xacro:unless value="${ module['visual']['mesh_body_1'] == '' }">
             <xacro:property name="mesh_bool" value="true"/>
         </xacro:unless>
@@ -666,8 +596,8 @@
                 <visual>
                     <origin
-                        rpy="${module['visual']['tf_mesh_2']['roll']} ${module['visual']['tf_mesh_2']['pitch']} ${module['visual']['tf_mesh_2']['yaw']}"
-                        xyz="${module['visual']['tf_mesh_2']['x']} ${module['visual']['tf_mesh_2']['y']} ${module['visual']['tf_mesh_2']['z']}"/>
-                    <geometry>
-                        <mesh filename="${module['visual']['mesh_body_2']}" scale="0.001 0.001 0.001"/>
+                        rpy="${module['visual']['tf_mesh_1']['roll']} ${module['visual']['tf_mesh_1']['pitch']} ${module['visual']['tf_mesh_1']['yaw']}"
+                        xyz="${module['visual']['tf_mesh_1']['x']} ${module['visual']['tf_mesh_1']['y']} ${module['visual']['tf_mesh_1']['z']}"/>
+                    <geometry>
+                        <mesh filename="${module['visual']['mesh_body_1']}" scale="0.001 0.001 0.001"/>
                     </geometry>
                     <material name="tree_green"/>
@@ -675,30 +605,92 @@
                 <collision>
                     <origin
-                        rpy="${module['visual']['tf_mesh_2']['roll']} ${module['visual']['tf_mesh_2']['pitch']} ${module['visual']['tf_mesh_2']['yaw']}"
-                        xyz="${module['visual']['tf_mesh_2']['x']} ${module['visual']['tf_mesh_2']['y']} ${module['visual']['tf_mesh_2']['z']}"/>
-                    <xacro:if value="${'type' in module['visual']['mesh_collision_2']}">
-                        <xacro:if value="${module['visual']['mesh_collision_2']['type'] == 'box'}">
-                            <geometry>
-                                <box size="${module['visual']['mesh_collision_2']['parameters']['size']}"/>
-                            </geometry>
-                        </xacro:if>
-                        <xacro:if value="${module['visual']['mesh_collision_2']['type'] == 'cylinder'}">
-                            <geometry>
-                                <cylinder radius="${module['visual']['mesh_collision_2']['parameters']['radius']}" length="${module['visual']['mesh_collision_2']['parameters']['length']}"/>
-                            </geometry>
-                        </xacro:if>
-                        <xacro:if value="${module['visual']['mesh_collision_2']['type'] == 'sphere'}">
-                            <geometry>
-                                <sphere radius="${module['visual']['mesh_collision_2']['parameters']['radius']}"/>
-                            </geometry>
-                        </xacro:if>
-                    </xacro:if>
-                    <xacro:unless value="${'type' in module['visual']['mesh_collision_2']}">
-                        <geometry>
-                            <mesh filename="${module['visual']['mesh_collision_2']}" scale="0.001 0.001 0.001"/>
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