Commit message: chore: remove deprecated `elbow` type

File: src/modular/modular_data/urdf/ModularBot.library.urdf.xacro (robot description, xacro)
@@ -523,67 +523,4 @@
         </xacro:unless>
     </xacro:macro>
-    <!-- Macro for adding an elbow module (90° link) -->
-    <xacro:macro name="add_elbow" params="type name size_y size_z size">
-        <xacro:if value="${size==1}">
-            <xacro:property name="radius" value="${size1}" />
-        </xacro:if>
-        <xacro:unless value="${size==1}">
-            <xacro:if value="${size==2}">
-                <xacro:property name="radius" value="${size2}" />
-            </xacro:if>
-            <xacro:unless value="${size==2}">
-                <xacro:property name="radius" value="${size3}" />
-            </xacro:unless>
-        </xacro:unless>
-        <link name="${name}">
-            <visual>
-                <origin xyz="0 0 ${size_z/2}" rpy="0 0 0" />
-                <geometry>
-                    <cylinder radius="${radius}" length="${size_z}"/>
-                </geometry>
-                <material name="blue"/>
-            </visual>
-            <visual>
-                <origin xyz="0 ${size_y/2} ${size_z}" rpy="1.57 0 0" />
-                <geometry>
-                    <cylinder radius="${radius}" length="${size_y}"/>
-                </geometry>
-                <material name="blue"/>
-            </visual>
-            <visual>
-                <origin xyz="0 0 ${size_z}" rpy="0 0 0" />
-                <geometry>
-                    <sphere radius="${radius}" />
-                </geometry>
-                <material name="blue"/>
-            </visual>
-            <collision>
-                <origin xyz="0 0 ${size_z/2}" rpy="0 0 0" />
-                <geometry>
-                    <cylinder radius="${radius}" length="${size_z}"/>
-                </geometry>
-            </collision>
-            <inertial>
-                <origin xyz="0 0 ${size_z/2}" rpy="0 0 0"/>
-                <mass value="${mass}"/>
-                <inertia
-                ixx="${mass / 2 *( 1 / 12.0 * (3*radius*radius + 4*size_y*size_y) + size_z*size_z) + mass / 24.0 * (3*radius*radius + 4*size_z*size_z)}" ixy="0.0" ixz="0.0"
-                iyy="${mass / 24.0 * (3*radius*radius + 4*size_z*size_z) + mass / 2 *( 1 / 2 *radius*radius + size_z*size_z)}" iyz="0.0"
-                izz="${mass / 4.0 * (radius*radius) + mass / 24.0 * (3*radius*radius + 4*size_y*size_y)}"/>
-            </inertial>
-            <collision>
-                <origin xyz="0 ${size_y/2} ${size_z}" rpy="1.57 0 0" />
-                <geometry>
-                    <cylinder radius="${radius}" length="${size_y}"/>
-                </geometry>
-            </collision>
-            <collision>
-                <origin xyz="0 0 ${size_z}" rpy="0 0 0" />
-                <geometry>
-                    <sphere radius="${radius}" />
-                </geometry>
-            </collision>
-        </link>
-    </xacro:macro>
     <xacro:macro name="add_tool_exchanger" params="type name filename">
         <xacro:property name="module" value="${xacro.load_yaml(filename)}"/>

Commit message: updated structure of YAML: `kinematics_convention` and `actuator_data`

File: src/modular/modular_data/urdf/ModularBot.library.urdf.xacro (robot description, xacro)
@@ -154,5 +154,5 @@
     <xacro:macro name="add_rotor_fast" params="type name filename x y z roll pitch yaw">
         <xacro:property name="module" value="${xacro.load_yaml(filename)}"/>
-        <xacro:property name="gear_ratio" value="${module['control']['nu']}"/>
+        <xacro:property name="gear_ratio" value="${module['actuator_data']['gear_ratio']}"/>
         <link name="${name}">
             <inertial>

Commit message: huge refactor of `ModuleNode` and added `JSONInterpreter`

File: src/modular/modular_data/urdf/ModularBot.library.urdf.xacro (robot description, xacro)
@@ -17,5 +17,5 @@
     <xacro:property name="len2" value="0.6" />
     <xacro:property name="len3" value="0.8" />
-    <xacro:property name="mass" value="0.5" />
+    <xacro:property name="mass" value="0.001" />
     <!-- <xacro:property name="pi" value="3.1415" /> -->
     <material name="blue">
@@ -46,5 +46,5 @@
         <inertial>
             <mass value="${mass}" />
-            <inertia ixx="1.0e-03" ixy="0.0" ixz="0.0" iyy="1.0e-03" iyz="0.0" izz="1.0e-03" />
+            <inertia ixx="1.0e-06" ixy="0.0" ixz="0.0" iyy="1.0e-06" iyz="0.0" izz="1.0e-06" />
         </inertial>
     </xacro:macro>
@@ -72,14 +72,18 @@
     <xacro:macro name="add_link_element" params="name type module body_name">
         <xacro:property name="visual_bool" value="false"/>
-        <xacro:unless value="${module['visual'][body_name] == '' }">
+        <xacro:unless value="${not module['visual'][body_name]}">
             <xacro:property name="visual_bool" value="true"/>
             <xacro:property name="visual_body" value="${module['visual'][body_name]}"/>
         </xacro:unless>
         <xacro:property name="collision_bool" value="false"/>
-        <xacro:unless value="${module['collision'][body_name] == '' }">
+        <xacro:unless value="${not module['collision'][body_name]}">
             <xacro:property name="collision_bool" value="true"/>
             <xacro:property name="collision_body" value="${module['collision'][body_name]}"/>
         </xacro:unless>
-        <xacro:property name="dynamics_body" value="${module['dynamics'][body_name]}"/>
+        <xacro:property name="dynamics_bool" value="false"/>
+        <xacro:unless value="${module['dynamics'][body_name]['mass'] is None }">
+            <xacro:property name="dynamics_bool" value="true"/>
+            <xacro:property name="dynamics_body" value="${module['dynamics'][body_name]}"/>
+        </xacro:unless>
         <link name="${name}">
             <xacro:unless value="${visual_bool == 0}">
@@ -87,5 +91,10 @@
                     <xacro:add_origin body_pose="${visual_body['pose']}"/>
                     <xacro:add_geometry body="${visual_body}"/>
-                    <material name="${visual_body['color']}"/>
+                    <!-- <xacro:unless value="${visual_body['color'] is None }">
+                        <material name="${visual_body['color']}"/>
+                    </xacro:unless> -->
+                    <xacro:if value="${'color' in visual_body}">
+                        <material name="${visual_body['color']}"/>
+                    </xacro:if>
                 </visual>
             </xacro:unless>
@@ -96,8 +105,8 @@
                 </collision>
             </xacro:unless>
-            <xacro:if value="${dynamics_body['mass'] == 0.0}">
+            <xacro:if value="${dynamics_bool == 0}">
                 <xacro:default_inertial mass="${mass}"/>
             </xacro:if>
-            <xacro:unless value="${dynamics_body['mass'] == 0.0}">
+            <xacro:unless value="${dynamics_bool == 0}">
                 <inertial>
                     <origin
@@ -195,5 +204,7 @@
             <origin rpy="0.0 0.0 0.0" xyz="0.0 0.0 0.0"/>
         </joint>
-        <link name="${name}">
+        <xacro:property name="body_name" value="body_1"/>
+        <xacro:add_link_element name="${name}" type="${type}" module="${module}" body_name="${body_name}"/>
+        <!-- <link name="${name}">
             <visual>
                 <origin rpy="${module['visual']['tf_mesh_1']['roll']} ${module['visual']['tf_mesh_1']['pitch']} ${module['visual']['tf_mesh_1']['yaw']}"
@@ -211,5 +222,5 @@
             </collision>
             <xacro:default_inertial mass="2"/>
-        </link>
+        </link> -->
     </xacro:macro>
     <xacro:macro name="add_connectors" params="name filename type">
@@ -309,5 +320,7 @@
     <xacro:macro name="add_slave_cube" params="name filename type">
         <xacro:property name="module" value="${xacro.load_yaml(filename)}"/>
-        <link name="${name}">
+        <xacro:property name="body_name" value="body_1"/>
+        <xacro:add_link_element name="${name}" type="${type}" module="${module}" body_name="${body_name}"/>
+        <!-- <link name="${name}">
             <visual>
                 <origin rpy="${module['visual']['tf_mesh_1']['roll']} ${module['visual']['tf_mesh_1']['pitch']} ${module['visual']['tf_mesh_1']['yaw']}"
@@ -325,5 +338,5 @@
             </collision>
             <xacro:default_inertial mass="2.0"/>
-        </link>
+        </link> -->
         <xacro:add_connectors name="${name}" filename="${filename}" type="${type}"/>
         <!-- <xacro:if value="1"> -->
@@ -394,8 +407,10 @@
     </xacro:macro>
     <!-- Macro for adding a socket -->
-    <xacro:macro name="add_socket" params="name type filename size_z size">
-        <xacro:property name="module" value="${xacro.load_yaml(filename)}"/>
+    <xacro:macro name="add_socket" params="name type filename size">
+        <xacro:property name="module" value="${xacro.load_yaml(filename)}"/>
+        <xacro:property name="body_name" value="body_1"/>
+        <xacro:add_link_element name="${name}" type="${type}" module="${module}" body_name="${body_name}"/>
         <xacro:property name="radius" value="${size_interface}" />
-        <link name="${name}">
+        <!-- <link name="${name}">
             <visual>
                 <origin xyz="0 0 ${size_z/2}" rpy="0 0 0" />
@@ -419,5 +434,5 @@
                 izz="${mass / 2.0 * (radius*radius)}"/>
             </inertial>
-        </link>
+        </link> -->
     </xacro:macro>
     <!-- Macro for adding a size adapter -->

Commit message: feat (concert): adding cameras to concert mobile base

File: src/modular/modular_data/urdf/ModularBot.library.urdf.xacro (robot description, xacro)
@@ -194,4 +194,6 @@
         <xacro:property name="body_name" value="body_1"/>
         <xacro:add_link_element name="${name}" type="${type}" module="${module}" body_name="${body_name}"/>
+        <xacro:include filename="$(find modular)/src/modular/modular_data/urdf/concert.sensors.urdf.xacro"/>
+        <xacro:add_mobile_base_sensors parent_name="${name}"/>
     </xacro:macro>
     <!-- Macro for adding a master cube -->

File: src/modular/modular_data/urdf/template.urdf.xacro (robot description, xacro)
@@ -1,10 +1,12 @@
 <?xml version="1.0"?>
 <robot name="ModularBot" xmlns:xacro="http://www.ros.org/wiki/xacro">
-    <xacro:include filename="ModularBot.library.urdf.xacro"/>
-    <xacro:include filename="ModularBot.control.urdf.xacro"/>
+    <xacro:include filename="$(find modular)/src/modular/modular_data/urdf/ModularBot.library.urdf.xacro"/>
+    <xacro:include filename="$(find modular)/src/modular/modular_data/urdf/ModularBot.control.urdf.xacro"/>
     <xacro:arg name="floating_base" default="false"/>
     <xacro:property name="ADD_FLOATING_BASE" value="$(arg floating_base)" />
     <xacro:arg name="gazebo_urdf" default="false"/>
     <xacro:property name="GAZEBO_URDF" value="$(arg gazebo_urdf)" />
+    <xacro:arg name="realsense" default="false"/>
+    <xacro:property name="ADD_CAMERAS" value="$(arg realsense)" />
     <!-- adding (or not) world link for Gazebo simulation -->
     <xacro:if value="${ADD_FLOATING_BASE}">
@@ -26,5 +28,5 @@
     </xacro:unless>
     <link name="base_link">
-        <xacro:default_inertial mass="0.1"/>
+        <xacro:default_inertial mass="0.001"/>
     </link>
 </robot>

Commit message: fix: avoid finding `modular` via ROS

File: src/modular/modular_data/urdf/ModularBot.library.urdf.xacro (robot description, xacro)
@@ -194,5 +194,5 @@
         <xacro:property name="body_name" value="body_1"/>
         <xacro:add_link_element name="${name}" type="${type}" module="${module}" body_name="${body_name}"/>
-        <xacro:include filename="$(find modular)/src/modular/modular_data/urdf/concert.sensors.urdf.xacro"/>
+        <xacro:include filename="${MODULAR_PATH}/src/modular/modular_data/urdf/concert.sensors.urdf.xacro"/>
         <xacro:add_mobile_base_sensors parent_name="${name}"/>
     </xacro:macro>

File: src/modular/modular_data/urdf/template.urdf.xacro (robot description, xacro)
@@ -1,6 +1,8 @@
 <?xml version="1.0"?>
 <robot name="ModularBot" xmlns:xacro="http://www.ros.org/wiki/xacro">
-    <xacro:include filename="$(find modular)/src/modular/modular_data/urdf/ModularBot.library.urdf.xacro"/>
-    <xacro:include filename="$(find modular)/src/modular/modular_data/urdf/ModularBot.control.urdf.xacro"/>
+    <xacro:arg name="modular_path" default="missing_argument_modular_path"/>
+    <xacro:property name="MODULAR_PATH" value="$(arg modular_path)" />
+    <xacro:include filename="${MODULAR_PATH}/src/modular/modular_data/urdf/ModularBot.library.urdf.xacro"/>
+    <xacro:include filename="${MODULAR_PATH}/src/modular/modular_data/urdf/ModularBot.control.urdf.xacro"/>
     <xacro:arg name="floating_base" default="false"/>
     <xacro:property name="ADD_FLOATING_BASE" value="$(arg floating_base)" />

Commit message: fix gripper (changes after upd yaml structure)

File: src/modular/modular_data/urdf/ModularBot.library.urdf.xacro (robot description, xacro)
@@ -693,23 +693,23 @@
         </link>
         <!-- Add joints -->
-        <joint name="${name}_finger_joint1" type="${module['kinematics']['joint']['joint']['type']}">
+        <joint name="${name}_finger_joint1" type="${module['actuator_data']['type']}">
             <parent link="${name}"/>
             <child link="${name}_leftfinger"/>
             <origin xyz="0 0 ${module['kinematics']['joint']['proximal']['p_pl']}" rpy="0 0 0"/>
             <axis xyz="0 -1 0"/>
-            <limit effort="${module['kinematics']['joint']['joint']['effort']}"
-                lower="${module['kinematics']['joint']['joint']['lower_limit']}"
-                upper="${module['kinematics']['joint']['joint']['upper_limit']}"
-                velocity="${module['kinematics']['joint']['joint']['velocity']}"
+            <limit effort="${module['actuator_data']['effort']}"
+                lower="${module['actuator_data']['lower_limit']}"
+                upper="${module['actuator_data']['upper_limit']}"
+                velocity="${module['actuator_data']['velocity']}"
             />
         </joint>
-        <joint name="${name}_finger_joint2" type="${module['kinematics']['joint']['joint']['type']}">
+        <joint name="${name}_finger_joint2" type="${module['actuator_data']['type']}">
             <parent link="${name}"/>
             <child link="${name}_rightfinger"/>
             <origin xyz="0 0 ${module['kinematics']['joint']['proximal']['p_pl']}" rpy="0 0 0"/>
-            <limit effort="${module['kinematics']['joint']['joint']['effort']}"
-                lower="${module['kinematics']['joint']['joint']['lower_limit']}"
-                upper="${module['kinematics']['joint']['joint']['upper_limit']}"
-                velocity="${module['kinematics']['joint']['joint']['velocity']}"
+            <limit effort="${module['actuator_data']['effort']}"
+                lower="${module['actuator_data']['lower_limit']}"
+                upper="${module['actuator_data']['upper_limit']}"
+                velocity="${module['actuator_data']['velocity']}"
             />
             <axis xyz="0 1 0"/>

Commit message: fix add_connectors()

File: src/modular/modular_data/urdf/ModularBot.library.urdf.xacro (robot description, xacro)
@@ -226,96 +226,21 @@
         </link> -->
     </xacro:macro>
-    <xacro:macro name="add_connectors" params="name filename type">
-        <xacro:property name="module" value="${xacro.load_yaml(filename)}"/>
-        <xacro:if value="${'connector_1' in module['kinematics']}">
-            <link name="${name}_con1">
-                <visual>
-                    <origin rpy="0 0 0" xyz="0 0 0.05"/>
-                    <geometry>
-                        <cylinder length="0.1" radius="${size_interface}"/>
-                    </geometry>
-                    <material name="green"/>
-                </visual>
-            </link>
-            <joint name="${name}_fixed_1" type="fixed">
-                <parent link="${name}"/>
-                <child link="${name}_con1"/>
-                <axis rpy="0 0 0" xyz="0 0 1"/>
-                <origin rpy="${module['kinematics']['connector_1']['roll']} ${module['kinematics']['connector_1']['pitch']} ${module['kinematics']['connector_1']['yaw']}"
-                        xyz="${module['kinematics']['connector_1']['x']} ${module['kinematics']['connector_1']['y']} ${module['kinematics']['connector_1']['z']}"/>
-            </joint>
-        </xacro:if>
-        <xacro:if value="${'connector_2' in module['kinematics']}">
-            <link name="${name}_con2">
-                <visual>
-                    <origin rpy="0 0 0" xyz="0 0 0.05"/>
-                    <geometry>
-                        <cylinder length="0.1" radius="${size_interface}"/>
-                    </geometry>
-                    <material name="green"/>
-                </visual>
-            </link>
-            <joint name="${name}_fixed_2" type="fixed">
-                <parent link="${name}"/>
-                <child link="${name}_con2"/>
-                <axis rpy="0 0 0" xyz="0 0 1"/>
-                <origin rpy="${module['kinematics']['connector_2']['roll']} ${module['kinematics']['connector_2']['pitch']} ${module['kinematics']['connector_2']['yaw']}"
-                        xyz="${module['kinematics']['connector_2']['x']} ${module['kinematics']['connector_2']['y']} ${module['kinematics']['connector_2']['z']}"/>
-            </joint>
-        </xacro:if>
-        <xacro:if value="${'connector_3' in module['kinematics']}">
-            <link name="${name}_con3">
-                <visual>
-                    <origin rpy="0 0 0" xyz="0 0 0.05"/>
-                    <geometry>
-                        <cylinder length="0.1" radius="${size_interface}"/>
-                    </geometry>
-                    <material name="green"/>
-                </visual>
-            </link>
-            <joint name="${name}_fixed_3" type="fixed">
-                <parent link="${name}"/>
-                <child link="${name}_con3"/>
-                <axis rpy="0 0 0" xyz="0 0 1"/>
-                <origin rpy="${module['kinematics']['connector_3']['roll']} ${module['kinematics']['connector_3']['pitch']} ${module['kinematics']['connector_3']['yaw']}"
-                        xyz="${module['kinematics']['connector_3']['x']} ${module['kinematics']['connector_3']['y']} ${module['kinematics']['connector_3']['z']}"/>
-            </joint>
-        </xacro:if>
-        <xacro:if value="${'connector_4' in module['kinematics']}">
-            <link name="${name}_con4">
-                <visual>
-                    <origin rpy="0 0 0" xyz="0 0 0.05"/>
-                    <geometry>
-                        <cylinder length="0.1" radius="${size_interface}"/>
-                    </geometry>
-                    <material name="green"/>
-                </visual>
-            </link>
-            <joint name="${name}_fixed_4" type="fixed">
-                <parent link="${name}"/>
-                <child link="${name}_con4"/>
-                <axis rpy="0 0 0" xyz="0 0 1"/>
-                <origin rpy="${module['kinematics']['connector_4']['roll']} ${module['kinematics']['connector_4']['pitch']} ${module['kinematics']['connector_4']['yaw']}"
-                        xyz="${module['kinematics']['connector_4']['x']} ${module['kinematics']['connector_4']['y']} ${module['kinematics']['connector_4']['z']}"/>
-            </joint>
-        </xacro:if>
-        <xacro:if value="${'connector_5' in module['kinematics']}">
-            <link name="${name}_con5">
-                <visual>
-                    <origin rpy="0 0 0" xyz="0 0 0.05"/>
-                    <geometry>
-                        <cylinder length="0.1" radius="${size_interface}"/>
-                    </geometry>
-                    <material name="green"/>
-                </visual>
-            </link>
-            <joint name="${name}_fixed_5" type="fixed">
-                <parent link="${name}"/>
-                <child link="${name}_con5"/>
-                <axis rpy="0 0 0" xyz="0 0 1"/>
-                <origin rpy="${module['kinematics']['connector_5']['roll']} ${module['kinematics']['connector_5']['pitch']} ${module['kinematics']['connector_5']['yaw']}"
-                        xyz="${module['kinematics']['connector_5']['x']} ${module['kinematics']['connector_5']['y']} ${module['kinematics']['connector_5']['z']}"/>
-            </joint>
-        </xacro:if>
+    <xacro:macro name="add_connector" params="name type parent_name x y z roll pitch yaw">
+        <link name="${name}">
+            <visual>
+                <origin rpy="0 0 0" xyz="0 0 0.05"/>
+                <geometry>
+                    <cylinder length="0.1" radius="${size_interface}"/>
+                </geometry>
+                <material name="green"/>
+            </visual>
+        </link>
+        <joint name="${name}_fixed" type="fixed">
+            <parent link="${parent_name}"/>
+            <child link="${name}"/>
+            <axis rpy="0 0 0" xyz="0 0 1"/>
+            <origin rpy="${roll} ${pitch} ${yaw}"
+                    xyz="${x} ${y} ${z}"/>
+        </joint>
     </xacro:macro>
     <!-- Macro for adding a slave cube -->

Commit message: simple_ee module should have negligible mass
previously this one would have the same mass of the tool-exchanger

File: src/modular/modular_data/urdf/ModularBot.library.urdf.xacro (robot description, xacro)
@@ -667,9 +667,9 @@
             <inertial>
                 <origin xyz="-0.007 0 0.044" rpy="0 0 0"/>
-                <mass value="1.305"/>
+                <mass value="0.001305"/>
                 <inertia
-                        ixx="1.8769887e-03" ixy="0.0" ixz="0.0"
-                        iyy="2.2629779e-03" iyz="0.0"
-                        izz="1.8887550e-03"/>
+                        ixx="1.8769887e-05" ixy="0.0" ixz="0.0"
+                        iyy="2.2629779e-05" iyz="0.0"
+                        izz="1.8887550e-05"/>
             </inertial>
         </link>
