Commit message: wip: better handling of end-effectors
(to be refactored)

File: src/modular/modular_data/urdf/ModularBot.library.urdf.xacro (robot description, xacro)
@@ -468,8 +468,10 @@
         <xacro:property name="module" value="${xacro.load_yaml(filename)}"/>
         <xacro:property name="mesh_bool" value="false"/>
-        <xacro:unless value="${ module['visual']['mesh_body_1'] == '' }">
+        <xacro:property name="body_name" value="body_1"/>
+        <xacro:unless value="${not module['visual'][body_name]}">
             <xacro:property name="mesh_bool" value="true"/>
         </xacro:unless>
-        <link name="${name}">
+        <xacro:add_link_element name="${name}" type="${type}" module="${module}" body_name="${body_name}"/>
+        <!-- <link name="${name}">
             <xacro:if value="${ mesh_bool }">
                 <visual>
@@ -504,5 +506,5 @@
                     izz="${module['dynamics']['body_1']['inertia_tensor']['I_zz']}"/>
             </inertial>
-        </link>
+        </link> -->
     </xacro:macro>
     <!-- Add a pen to the tool-exchanger. Length may vary -->
@@ -519,8 +521,10 @@
         <xacro:property name="module" value="${xacro.load_yaml(filename)}"/>
         <xacro:property name="mesh_bool" value="false"/>
-        <xacro:unless value="${ module['visual']['mesh_body_1'] == '' }">
+        <xacro:property name="body_name" value="body_1"/>
+        <xacro:unless value="${not module['visual'][body_name]}">
             <xacro:property name="mesh_bool" value="true"/>
         </xacro:unless>
-        <link name="${name}">
+        <xacro:add_link_element name="${name}" type="${type}" module="${module}" body_name="${body_name}"/>
+        <!-- <link name="${name}">
             <xacro:if value="${ mesh_bool }">
                 <visual>
@@ -529,5 +533,5 @@
                         xyz="${module['visual']['tf_mesh_1']['x']} ${module['visual']['tf_mesh_1']['y']} ${module['visual']['tf_mesh_1']['z']}"/>
                     <geometry>
-                        <mesh filename="${module['visual']['mesh_body_1']}" scale="0.001 0.001 0.001"/>
+                        <mesh filename="${module['visual'][body_1']['parameters']['file']}" scale="0.001 0.001 0.001"/>
                     </geometry>
                     <material name="tree_green"/>
@@ -538,5 +542,5 @@
                         xyz="${module['visual']['tf_mesh_1']['x']} ${module['visual']['tf_mesh_1']['y']} ${module['visual']['tf_mesh_1']['z']}"/>
                     <geometry>
-                        <mesh filename="${module['visual']['mesh_collision_1']}" scale="0.001 0.001 0.001"/>
+                        <mesh filename="${module['collision'][body_1']['parameters']['file']}" scale="0.001 0.001 0.001"/>
                     </geometry>
                 </collision>
@@ -555,5 +559,5 @@
                     izz="${module['dynamics']['body_1']['inertia_tensor']['I_zz']}"/>
             </inertial>
-        </link>
+        </link> -->
         <!-- add fingers -->
         <link name="${name}_leftfinger">

Commit message: fix and refactor `add_gripper` and `add_tool_exchanger`

File: src/modular/modular_data/urdf/ModularBot.library.urdf.xacro (robot description, xacro)
@@ -467,44 +467,6 @@
     <xacro:macro name="add_tool_exchanger" params="type name filename">
         <xacro:property name="module" value="${xacro.load_yaml(filename)}"/>
-        <xacro:property name="mesh_bool" value="false"/>
         <xacro:property name="body_name" value="body_1"/>
-        <xacro:unless value="${not module['visual'][body_name]}">
-            <xacro:property name="mesh_bool" value="true"/>
-        </xacro:unless>
-        <xacro:add_link_element name="${name}" type="${type}" module="${module}" body_name="${body_name}"/>
-        <!-- <link name="${name}">
-            <xacro:if value="${ mesh_bool }">
-                <visual>
-                    <origin
-                        rpy="${module['visual']['tf_mesh_1']['roll']} ${module['visual']['tf_mesh_1']['pitch']} ${module['visual']['tf_mesh_1']['yaw']}"
-                        xyz="${module['visual']['tf_mesh_1']['x']} ${module['visual']['tf_mesh_1']['y']} ${module['visual']['tf_mesh_1']['z']}"/>
-                    <geometry>
-                        <mesh filename="${module['visual']['mesh_body_1']}" scale="0.001 0.001 0.001"/>
-                    </geometry>
-                    <material name="tree_green"/>
-                </visual>
-                <collision>
-                    <origin
-                        rpy="${module['visual']['tf_mesh_1']['roll']} ${module['visual']['tf_mesh_1']['pitch']} ${module['visual']['tf_mesh_1']['yaw']}"
-                        xyz="${module['visual']['tf_mesh_1']['x']} ${module['visual']['tf_mesh_1']['y']} ${module['visual']['tf_mesh_1']['z']}"/>
-                    <geometry>
-                        <mesh filename="${module['visual']['mesh_collision_1']}" scale="0.001 0.001 0.001"/>
-                    </geometry>
-                </collision>
-            </xacro:if>
-            <inertial>
-                <origin
-                    xyz="${module['dynamics']['body_1']['CoM']['x']} ${module['dynamics']['body_1']['CoM']['y']} ${module['dynamics']['body_1']['CoM']['z']}"
-                    rpy="0 0 0"/>
-                <mass value="${module['dynamics']['body_1']['mass']}"/>
-                <inertia
-                    ixx="${module['dynamics']['body_1']['inertia_tensor']['I_xx']}"
-                    ixy="${module['dynamics']['body_1']['inertia_tensor']['I_xy']}"
-                    ixz="${module['dynamics']['body_1']['inertia_tensor']['I_xz']}"
-                    iyy="${module['dynamics']['body_1']['inertia_tensor']['I_yy']}"
-                    iyz="${module['dynamics']['body_1']['inertia_tensor']['I_yz']}"
-                    izz="${module['dynamics']['body_1']['inertia_tensor']['I_zz']}"/>
-            </inertial>
-        </link> -->
+        <xacro:add_link_element name="${name}" type="${type}" module="${module}" body_name="${body_name}"/>
     </xacro:macro>
     <!-- Add a pen to the tool-exchanger. Length may vary -->
@@ -518,111 +480,45 @@
         </joint>
     </xacro:macro>
-    <xacro:macro name="add_gripper" params="type name filename">
-        <xacro:property name="module" value="${xacro.load_yaml(filename)}"/>
-        <xacro:property name="mesh_bool" value="false"/>
+    <xacro:macro name="add_gripper_body" params="type name filename">
+        <xacro:property name="module" value="${xacro.load_yaml(filename)}"/>
         <xacro:property name="body_name" value="body_1"/>
-        <xacro:unless value="${not module['visual'][body_name]}">
-            <xacro:property name="mesh_bool" value="true"/>
-        </xacro:unless>
-        <xacro:add_link_element name="${name}" type="${type}" module="${module}" body_name="${body_name}"/>
-        <!-- <link name="${name}">
-            <xacro:if value="${ mesh_bool }">
-                <visual>
-                    <origin
-                        rpy="${module['visual']['tf_mesh_1']['roll']} ${module['visual']['tf_mesh_1']['pitch']} ${module['visual']['tf_mesh_1']['yaw']}"
-                        xyz="${module['visual']['tf_mesh_1']['x']} ${module['visual']['tf_mesh_1']['y']} ${module['visual']['tf_mesh_1']['z']}"/>
-                    <geometry>
-                        <mesh filename="${module['visual'][body_1']['parameters']['file']}" scale="0.001 0.001 0.001"/>
-                    </geometry>
-                    <material name="tree_green"/>
-                </visual>
-                <collision>
-                    <origin
-                        rpy="${module['visual']['tf_mesh_1']['roll']} ${module['visual']['tf_mesh_1']['pitch']} ${module['visual']['tf_mesh_1']['yaw']}"
-                        xyz="${module['visual']['tf_mesh_1']['x']} ${module['visual']['tf_mesh_1']['y']} ${module['visual']['tf_mesh_1']['z']}"/>
-                    <geometry>
-                        <mesh filename="${module['collision'][body_1']['parameters']['file']}" scale="0.001 0.001 0.001"/>
-                    </geometry>
-                </collision>
-            </xacro:if>
+        <xacro:add_link_element name="${name}" type="${type}" module="${module}" body_name="${body_name}"/>
+    </xacro:macro>
+    <xacro:macro name="add_gripper_fingers" params="type name joint_name_finger1 joint_name_finger2 TCP_name filename">
+        <!-- add fingers -->
+        <xacro:property name="module" value="${xacro.load_yaml(filename)}"/>
+        <xacro:property name="body_name" value="body_2"/>
+        <xacro:add_link_element name="${name}_finger1" type="${type}" module="${module}" body_name="${body_name}"/>
+        <!-- add the right finger (same mesh rotated by pi!) -->
+        <link name="${name}_finger2">
+            <visual>
+                <xacro:add_origin body_pose="${dict(x=0.0, y=0.0, z=0.0, roll=0.0, pitch=0.0, yaw=pi)}"/>
+                <xacro:add_geometry body="${module['visual'][body_name]}"/>
+                <xacro:if value="${'color' in module['visual'][body_name]}">
+                    <material name="${module['visual'][body_name]['color']}"/>
+                </xacro:if>
+            </visual>
+            <collision>
+                <xacro:add_origin body_pose="${dict(x=0.0, y=0.0, z=0.0, roll=0.0, pitch=0.0, yaw=pi)}"/>
+                <xacro:add_geometry body="${module['collision'][body_name]}"/>
+            </collision>
             <inertial>
                 <origin
-                    xyz="${module['dynamics']['body_1']['CoM']['x']} ${module['dynamics']['body_1']['CoM']['y']} ${module['dynamics']['body_1']['CoM']['z']}"
+                    xyz="${module['dynamics'][body_name]['CoM']['x']} ${module['dynamics'][body_name]['CoM']['y']} ${module['dynamics'][body_name]['CoM']['z']}"
                     rpy="0 0 0"/>
-                <mass value="${module['dynamics']['body_1']['mass']}"/>
+                <mass value="${module['dynamics'][body_name]['mass']}"/>
                 <inertia
-                    ixx="${module['dynamics']['body_1']['inertia_tensor']['I_xx']}"
-                    ixy="${module['dynamics']['body_1']['inertia_tensor']['I_xy']}"
-                    ixz="${module['dynamics']['body_1']['inertia_tensor']['I_xz']}"
-                    iyy="${module['dynamics']['body_1']['inertia_tensor']['I_yy']}"
-                    iyz="${module['dynamics']['body_1']['inertia_tensor']['I_yz']}"
-                    izz="${module['dynamics']['body_1']['inertia_tensor']['I_zz']}"/>
-            </inertial>
-        </link> -->
-        <!-- add fingers -->
-        <link name="${name}_leftfinger">
-            <xacro:if value="${ mesh_bool }">
-                <visual>
-                    <geometry>
-                    <mesh filename="${module['visual']['mesh_body_2']}" scale="0.001 0.001 0.001"/>
-                    </geometry>
-                    <material name="grey"/>
-                </visual>
-                <collision>
-                    <geometry>
-                    <mesh filename="${module['visual']['mesh_collision_2']}" scale="0.001 0.001 0.001"/>
-                    </geometry>
-                </collision>
-            </xacro:if>
-            <!-- for simulation -->
-            <inertial>
-                <origin
-                    xyz="${module['dynamics']['body_2']['CoM']['x']} ${module['dynamics']['body_2']['CoM']['y']} ${module['dynamics']['body_2']['CoM']['z']}"
-                    rpy="0 0 0"/>
-                <mass value="${module['dynamics']['body_2']['mass']}"/>
-                <inertia
-                    ixx="${module['dynamics']['body_2']['inertia_tensor']['I_xx']}"
-                    ixy="${module['dynamics']['body_2']['inertia_tensor']['I_xy']}"
-                    ixz="${module['dynamics']['body_2']['inertia_tensor']['I_xz']}"
-                    iyy="${module['dynamics']['body_2']['inertia_tensor']['I_yy']}"
-                    iyz="${module['dynamics']['body_2']['inertia_tensor']['I_yz']}"
-                    izz="${module['dynamics']['body_2']['inertia_tensor']['I_zz']}"/>
-            </inertial>
-        </link>
-        <link name="${name}_rightfinger">
-            <xacro:if value="${ mesh_bool }">
-                <visual>
-                    <origin xyz="0 0 0" rpy="0 0 ${pi}"/>
-                    <geometry>
-                    <mesh filename="${module['visual']['mesh_body_2']}" scale="0.001 0.001 0.001"/>
-                    </geometry>
-                    <material name="grey"/>
-                </visual>
-                <collision>
-                    <origin xyz="0 0 0" rpy="0 0 ${pi}"/>
-                    <geometry>
-                    <mesh filename="${module['visual']['mesh_collision_2']}" scale="0.001 0.001 0.001"/>
-                    </geometry>
-                </collision>
-            </xacro:if>
-            <!-- for simulation -->
-            <inertial>
-                <origin
-                    xyz="${module['dynamics']['body_2']['CoM']['x']} ${module['dynamics']['body_2']['CoM']['y']} ${module['dynamics']['body_2']['CoM']['z']}"
-                    rpy="0 0 0"/>
-                <mass value="${module['dynamics']['body_2']['mass']}"/>
-                <inertia
-                    ixx="${module['dynamics']['body_2']['inertia_tensor']['I_xx']}"
-                    ixy="${module['dynamics']['body_2']['inertia_tensor']['I_xy']}"
-                    ixz="${module['dynamics']['body_2']['inertia_tensor']['I_xz']}"
-                    iyy="${module['dynamics']['body_2']['inertia_tensor']['I_yy']}"
-                    iyz="${module['dynamics']['body_2']['inertia_tensor']['I_yz']}"
-                    izz="${module['dynamics']['body_2']['inertia_tensor']['I_zz']}"/>
+                    ixx="${module['dynamics'][body_name]['inertia_tensor']['I_xx']}"
+                    ixy="${module['dynamics'][body_name]['inertia_tensor']['I_xy']}"
+                    ixz="${module['dynamics'][body_name]['inertia_tensor']['I_xz']}"
+                    iyy="${module['dynamics'][body_name]['inertia_tensor']['I_yy']}"
+                    iyz="${module['dynamics'][body_name]['inertia_tensor']['I_yz']}"
+                    izz="${module['dynamics'][body_name]['inertia_tensor']['I_zz']}"/>
             </inertial>
         </link>
         <!-- Add joints -->
-        <joint name="${name}_finger_joint1" type="${module['actuator_data']['type']}">
+        <joint name="${joint_name_finger1}" type="${module['actuator_data']['type']}">
             <parent link="${name}"/>
-            <child link="${name}_leftfinger"/>
+            <child link="${name}_finger1"/>
             <origin xyz="0 0 ${module['kinematics']['joint']['proximal']['p_pl']}" rpy="0 0 0"/>
             <axis xyz="0 -1 0"/>
@@ -633,8 +529,9 @@
             />
         </joint>
-        <joint name="${name}_finger_joint2" type="${module['actuator_data']['type']}">
+        <joint name="${joint_name_finger2}" type="${module['actuator_data']['type']}">
             <parent link="${name}"/>
-            <child link="${name}_rightfinger"/>
+            <child link="${name}_finger2"/>
             <origin xyz="0 0 ${module['kinematics']['joint']['proximal']['p_pl']}" rpy="0 0 0"/>
+            <axis xyz="0 1 0"/>
             <limit effort="${module['actuator_data']['effort']}"
                 lower="${module['actuator_data']['lower_limit']}"
@@ -642,12 +539,11 @@
                 velocity="${module['actuator_data']['velocity']}"
             />
-            <axis xyz="0 1 0"/>
         </joint>
         <!-- Add TCP -->
-        <link name="TCP_${name}"/>
-        <joint name="fixed_TCP_${name}" type="fixed">
+        <link name="${TCP_name}"/>
+        <joint name="fixed_${name}" type="fixed">
             <axis xyz="0 0 1" rpy="0 0 0" />
             <parent link="${name}"/>
-            <child link="TCP_${name}"/>
+            <child link="${TCP_name}"/>
             <origin xyz="0.0 0.0 0.1985" rpy="0.0 0.0 0.0"/>
         </joint>

Commit message: refactor (URDF_writer): add mass and radius arguments to  `add_simple_ee`

File: src/modular/modular_data/urdf/ModularBot.library.urdf.xacro (robot description, xacro)
@@ -549,11 +549,11 @@
         </joint>
     </xacro:macro>
-    <!-- Add a simple frame ("end-effector") for simulation purposes -->
-    <xacro:macro name="add_simple_ee" params="type name size_z">
+    <!-- Add a cylinder -->
+    <xacro:macro name="add_cylinder" params="type name size_z mass radius">
         <link name="${name}">
             <visual>
                 <origin xyz="0 0 -${size_z/2}" rpy="0 0 0" />
                 <geometry>
-                    <cylinder radius="0.02" length="${size_z}"/>
+                    <cylinder radius="${radius}" length="${size_z}"/>
                 </geometry>
                 <material name="blue"/>
@@ -562,14 +562,14 @@
                 <origin xyz="0 0 -${size_z/2}" rpy="0 0 0" />
                 <geometry>
-                    <cylinder radius="0.02" length="${size_z}"/>
+                    <cylinder radius="${radius}" length="${size_z}"/>
                 </geometry>
             </collision>
             <inertial>
-                <origin xyz="-0.007 0 0.044" rpy="0 0 0"/>
-                <mass value="0.001305"/>
+                <origin xyz="0 0 ${size_z/2}" rpy="0 0 0"/>
+                <mass value="${mass}"/>
                 <inertia
-                        ixx="1.8769887e-05" ixy="0.0" ixz="0.0"
-                        iyy="2.2629779e-05" iyz="0.0"
-                        izz="1.8887550e-05"/>
+                ixx="${mass / 12.0 * (3*radius*radius + size_z*size_z)}" ixy="0.0" ixz="0.0"
+                iyy="${mass / 12.0 * (size_z*size_z + 3*radius*radius)}" iyz="0.0"
+                izz="${mass / 2.0 * (radius*radius)}"/>
             </inertial>
         </link>
