Commit message: refactor(Modularbot.library): general refactor and cleanup

File: src/modular/modular_data/urdf/ModularBot.library.urdf.xacro (robot description, xacro)
@@ -1,10 +1,4 @@
 <?xml version="1.0"?>
 <robot name="ModularBot" xmlns:xacro="http://www.ros.org/wiki/xacro">
-    <!-- <xacro:include filename="$(find modular)/urdf/config.xacro" />
-    <xacro:include filename="$(find modular)/urdf/modular.gazebo" /> -->
-<!--
-    <xacro:property name="size1" value="0.05" />
-    <xacro:property name="size2" value="0.055" />
-    <xacro:property name="size3" value="0.06" /> -->
     <xacro:property name="size1" value="0.0335" />
     <xacro:property name="size2" value="0.038" />
@@ -13,10 +7,8 @@
     <xacro:property name="size5" value="0.069" />
     <xacro:property name="size_interface" value="0.045" />
-    <!-- <xacro:property name="leglen" value="0.3" /> -->
     <xacro:property name="len1" value="0.4" />
     <xacro:property name="len2" value="0.6" />
     <xacro:property name="len3" value="0.8" />
     <xacro:property name="mass" value="0.001" />
-    <!-- <xacro:property name="pi" value="3.1415" /> -->
     <material name="blue">
         <color rgba="0 0 0.8 1"/>
@@ -91,7 +83,4 @@
                     <xacro:add_origin body_pose="${visual_body['pose']}"/>
                     <xacro:add_geometry body="${visual_body}"/>
-                    <!-- <xacro:unless value="${visual_body['color'] is None }">
-                        <material name="${visual_body['color']}"/>
-                    </xacro:unless> -->
                     <xacro:if value="${'color' in visual_body}">
                         <material name="${visual_body['color']}"/>
@@ -125,5 +114,5 @@
         </link>
     </xacro:macro>
-    <!-- Macro for adding a straight link -->
+    <!-- Macro for adding a generic link -->
     <xacro:macro name="add_link" params="name type filename">
         <xacro:property name="module" value="${xacro.load_yaml(filename)}"/>
@@ -131,10 +120,11 @@
         <xacro:add_link_element name="${name}" type="${type}" module="${module}" body_name="${body_name}"/>
     </xacro:macro>
-    <!-- Macro for adding the physical module housing the actuator -->
-    <xacro:macro name="add_joint_stator" params="type name filename">
-        <xacro:property name="module" value="${xacro.load_yaml(filename)}"/>
-        <xacro:property name="body_name" value="body_1"/>
-        <xacro:add_link_element name="${name}" type="${type}" module="${module}" body_name="${body_name}"/>
-    </xacro:macro>
+    <!-- Macro for adding the proximal part of the joint (the physical module housing the actuator) -->
+    <xacro:macro name="add_proximal" params="type name filename">
+        <xacro:property name="module" value="${xacro.load_yaml(filename)}"/>
+        <xacro:property name="body_name" value="body_1"/>
+        <xacro:add_link_element name="${name}" type="${type}" module="${module}" body_name="${body_name}"/>
+    </xacro:macro>
+    <!-- Macro for adding the distal part of the joint -->
     <xacro:macro name="add_distal" params="type name filename">
         <xacro:property name="module" value="${xacro.load_yaml(filename)}"/>
@@ -177,7 +167,4 @@
                         iyz="${module['dynamics']['body_2_fast']['inertia_tensor']['I_yz'] }"
                         izz="${ gear_ratio * gear_ratio * module['dynamics']['body_2_fast']['inertia_tensor']['I_zz'] }"/>
-                        <!-- ixz="${ gear_ratio * module['dynamics']['body_2_fast']['inertia_tensor']['I_xz'] }" -->
-                        <!-- iyz="${ gear_ratio * module['dynamics']['body_2_fast']['inertia_tensor']['I_yz'] }" -->
-                        <!-- izz="${module['dynamics']['body_2_fast']['inertia_tensor']['I_zz'] }" -->
             </inertial>
         </link>
@@ -208,21 +195,4 @@
         <xacro:property name="body_name" value="body_1"/>
         <xacro:add_link_element name="${name}" type="${type}" module="${module}" body_name="${body_name}"/>
-        <!-- <link name="${name}">
-            <visual>
-                <origin rpy="${module['visual']['tf_mesh_1']['roll']} ${module['visual']['tf_mesh_1']['pitch']} ${module['visual']['tf_mesh_1']['yaw']}"
-                        xyz="${module['visual']['tf_mesh_1']['x']} ${module['visual']['tf_mesh_1']['y']} ${module['visual']['tf_mesh_1']['z']}"/>
-                <geometry>
-                    <mesh filename="${module['visual']['mesh_body_1']}" scale="0.001 0.001 0.001"/>
-                </geometry>
-            </visual>
-            <collision>
-                <origin rpy="${module['visual']['tf_mesh_1']['roll']} ${module['visual']['tf_mesh_1']['pitch']} ${module['visual']['tf_mesh_1']['yaw']}"
-                        xyz="${module['visual']['tf_mesh_1']['x']} ${module['visual']['tf_mesh_1']['y']} ${module['visual']['tf_mesh_1']['z']}"/>
-                <geometry>
-                    <mesh filename="${module['visual']['mesh_collision_1']}" scale="0.001 0.001 0.001"/>
-                </geometry>
-            </collision>
-            <xacro:default_inertial mass="2"/>
-        </link> -->
     </xacro:macro>
     <xacro:macro name="add_connector" params="name type parent_name x y z roll pitch yaw">
@@ -249,87 +219,4 @@
         <xacro:property name="body_name" value="body_1"/>
         <xacro:add_link_element name="${name}" type="${type}" module="${module}" body_name="${body_name}"/>
-        <!-- <link name="${name}">
-            <visual>
-                <origin rpy="${module['visual']['tf_mesh_1']['roll']} ${module['visual']['tf_mesh_1']['pitch']} ${module['visual']['tf_mesh_1']['yaw']}"
-                        xyz="${module['visual']['tf_mesh_1']['x']} ${module['visual']['tf_mesh_1']['y']} ${module['visual']['tf_mesh_1']['z']}"/>
-                <geometry>
-                    <mesh filename="${module['visual']['mesh_body_1']}" scale="0.001 0.001 0.001"/>
-                </geometry>
-            </visual>
-            <collision>
-                <origin rpy="${module['visual']['tf_mesh_1']['roll']} ${module['visual']['tf_mesh_1']['pitch']} ${module['visual']['tf_mesh_1']['yaw']}"
-                        xyz="${module['visual']['tf_mesh_1']['x']} ${module['visual']['tf_mesh_1']['y']} ${module['visual']['tf_mesh_1']['z']}"/>
-                <geometry>
-                    <mesh filename="${module['visual']['mesh_body_1']}" scale="0.001 0.001 0.001"/>
-                </geometry>
-            </collision>
-            <xacro:default_inertial mass="2.0"/>
-        </link> -->
-        <xacro:add_connectors name="${name}" filename="${filename}" type="${type}"/>
-        <!-- <xacro:if value="1"> -->
-            <!-- <link name="${name}_con1">
-                <visual>
-                    <origin rpy="0 0 0" xyz="0 0 0.05"/>
-                    <geometry>
-                        <cylinder length="0.1" radius="${size_interface}"/>
-                    </geometry>
-                    <material name="green"/>
-                </visual>
-            </link>
-            <joint name="${name}_fixed_1" type="fixed">
-                <parent link="${name}_con1"/>
-                <child link="${name}"/>
-                <origin rpy="${module['kinematics']['connector_1']['roll']} ${module['kinematics']['connector_1']['pitch']} ${module['kinematics']['connector_1']['yaw']}"
-                        xyz="${module['kinematics']['connector_1']['x']} ${module['kinematics']['connector_1']['y']} ${module['kinematics']['connector_1']['z']}"/>
-            </joint> -->
-        <!-- </xacro:if> -->
-        <!-- <link name="${name}_con2">
-            <visual>
-                <origin rpy="0 0 0" xyz="0 0 0.05"/>
-                <geometry>
-                    <cylinder length="0.1" radius="${size_interface}"/>
-                </geometry>
-                <material name="green"/>
-            </visual>
-        </link>
-        <joint name="${name}_fixed_2" type="fixed">
-            <parent link="${name}"/>
-            <child link="${name}_con2"/>
-            <axis rpy="0 0 0" xyz="0 0 1"/>
-            <origin rpy="${module['kinematics']['connector_2']['roll']} ${module['kinematics']['connector_2']['pitch']} ${module['kinematics']['connector_2']['yaw']}"
-                    xyz="${module['kinematics']['connector_2']['x']} ${module['kinematics']['connector_2']['y']} ${module['kinematics']['connector_2']['z']}"/>
-        </joint>
-        <link name="${name}_con3">
-            <visual>
-                <origin rpy="0 0 0" xyz="0 0 0.05"/>
-                <geometry>
-                    <cylinder length="0.1" radius="${size_interface}"/>
-                </geometry>
-                <material name="green"/>
-            </visual>
-        </link>
-        <joint name="${name}_fixed_3" type="fixed">
-            <parent link="${name}"/>
-            <child link="${name}_con3"/>
-            <axis rpy="0 0 0" xyz="0 0 1"/>
-            <origin rpy="${module['kinematics']['connector_3']['roll']} ${module['kinematics']['connector_3']['pitch']} ${module['kinematics']['connector_3']['yaw']}"
-                    xyz="${module['kinematics']['connector_3']['x']} ${module['kinematics']['connector_3']['y']} ${module['kinematics']['connector_3']['z']}"/>
-        </joint> -->
-        <!-- <link name="${name}_con4">
-            <visual>
-                <origin rpy="0 0 0" xyz="0 0 0.05"/>
-                <geometry>
-                    <cylinder length="0.1" radius="${size_interface}"/>
-                </geometry>
-                <material name="green"/>
-            </visual>
-        </link> -->
-        <!-- <joint name="${name}_fixed_4" type="fixed">
-            <parent link="${name}"/>
-            <child link="${name}_con4"/>
-            <axis rpy="0 0 0" xyz="0 0 1"/>
-            <origin rpy="${module['kinematics']['connector_4']['roll']} ${module['kinematics']['connector_4']['pitch']} ${module['kinematics']['connector_4']['yaw']}"
-                    xyz="${module['kinematics']['connector_4']['x']} ${module['kinematics']['connector_4']['y']} ${module['kinematics']['connector_4']['z']}"/>
-        </joint> -->
     </xacro:macro>
     <!-- Macro for adding a socket -->
@@ -338,28 +225,4 @@
         <xacro:property name="body_name" value="body_1"/>
         <xacro:add_link_element name="${name}" type="${type}" module="${module}" body_name="${body_name}"/>
-        <xacro:property name="radius" value="${size_interface}" />
-        <!-- <link name="${name}">
-            <visual>
-                <origin xyz="0 0 ${size_z/2}" rpy="0 0 0" />
-                <geometry>
-                    <cylinder radius="${radius}" length="${size_z}"/>
-                </geometry>
-                <material name="white"/>
-            </visual>
-            <collision>
-                <origin xyz="0 0 ${size_z/2}" rpy="0 0 0" />
-                <geometry>
-                    <cylinder radius="${radius}" length="${size_z}"/>
-                </geometry>
-            </collision>
-            <inertial>
-                <origin xyz="0 0 ${size_z/2}" rpy="0 0 0"/>
-                <mass value="${mass}"/>
-                <inertia
-                ixx="${mass / 12.0 * (3*radius*radius + size_z*size_z)}" ixy="0.0" ixz="0.0"
-                iyy="${mass / 12.0 * (size_z*size_z + 3*radius*radius)}" iyz="0.0"
-                izz="${mass / 2.0 * (radius*radius)}"/>
-            </inertial>
-        </link> -->
     </xacro:macro>
     <!-- Macro for adding a size adapter -->

Commit message: feat(ModuleNode): multiple geometries per body are accepted
both in the visual and collision tags

File: src/modular/modular_data/urdf/ModularBot.library.urdf.xacro (robot description, xacro)
@@ -66,10 +66,10 @@
         <xacro:unless value="${not module['visual'][body_name]}">
             <xacro:property name="visual_bool" value="true"/>
-            <xacro:property name="visual_body" value="${module['visual'][body_name]}"/>
+            <xacro:property name="visual_bodies" value="${module['visual'][body_name]}"/>
         </xacro:unless>
         <xacro:property name="collision_bool" value="false"/>
         <xacro:unless value="${not module['collision'][body_name]}">
             <xacro:property name="collision_bool" value="true"/>
-            <xacro:property name="collision_body" value="${module['collision'][body_name]}"/>
+            <xacro:property name="collision_bodies" value="${module['collision'][body_name]}"/>
         </xacro:unless>
         <xacro:property name="dynamics_bool" value="false"/>
@@ -80,17 +80,37 @@
         <link name="${name}">
             <xacro:unless value="${visual_bool == 0}">
-                <visual>
-                    <xacro:add_origin body_pose="${visual_body['pose']}"/>
-                    <xacro:add_geometry body="${visual_body}"/>
-                    <xacro:if value="${'color' in visual_body}">
-                        <material name="${visual_body['color']}"/>
-                    </xacro:if>
-                </visual>
+                <!-- xacro loop -->
+                <xacro:macro name="visual_loop" params="visual_bodies n_bodies">
+                    <xacro:property name="i_bodies" value="${n_bodies-1}"/>
+                    <xacro:unless value="${i_bodies == -1}">
+                        <visual>
+                            <xacro:property name="body" value="${visual_bodies[i_bodies]}"/>
+                            <xacro:add_origin body_pose="${body['pose']}"/>
+                            <xacro:add_geometry body="${body}"/>
+                            <xacro:if value="${'color' in body}">
+                                <material name="${body['color']}"/>
+                            </xacro:if>
+                        </visual>
+                        <xacro:visual_loop visual_bodies="${visual_bodies}" n_bodies="${i_bodies}"/>
+                    </xacro:unless>
+                </xacro:macro>
+                <!-- call the macro -->
+                <xacro:visual_loop visual_bodies="${visual_bodies}" n_bodies="${len(visual_bodies)}"/>
             </xacro:unless>
             <xacro:unless value="${collision_bool == 0}">
-                <collision>
-                    <xacro:add_origin body_pose="${collision_body['pose']}"/>
-                    <xacro:add_geometry body="${collision_body}"/>
-                </collision>
+                <!-- xacro loop -->
+                <xacro:macro name="collision_loop" params="collision_bodies n_bodies">
+                    <xacro:property name="i_bodies" value="${n_bodies-1}"/>
+                    <xacro:unless value="${i_bodies == -1}">
+                        <collision>
+                            <xacro:property name="body" value="${collision_bodies[i_bodies]}"/>
+                            <xacro:add_origin body_pose="${body['pose']}"/>
+                            <xacro:add_geometry body="${body}"/>
+                        </collision>
+                        <xacro:collision_loop collision_bodies="${collision_bodies}" n_bodies="${i_bodies}"/>
+                    </xacro:unless>
+                </xacro:macro>
+                <!-- call the macro -->
+                <xacro:collision_loop collision_bodies="${collision_bodies}" n_bodies="${len(collision_bodies)}"/>
             </xacro:unless>
             <xacro:if value="${dynamics_bool == 0}">
@@ -357,12 +377,12 @@
             <visual>
                 <xacro:add_origin body_pose="${dict(x=0.0, y=0.0, z=0.0, roll=0.0, pitch=0.0, yaw=pi)}"/>
-                <xacro:add_geometry body="${module['visual'][body_name]}"/>
-                <xacro:if value="${'color' in module['visual'][body_name]}">
-                    <material name="${module['visual'][body_name]['color']}"/>
+                <xacro:add_geometry body="${module['visual'][body_name][0]}"/>
+                <xacro:if value="${'color' in module['visual'][body_name][0]}">
+                    <material name="${module['visual'][body_name]['color'][0]}"/>
                 </xacro:if>
             </visual>
             <collision>
                 <xacro:add_origin body_pose="${dict(x=0.0, y=0.0, z=0.0, roll=0.0, pitch=0.0, yaw=pi)}"/>
-                <xacro:add_geometry body="${module['collision'][body_name]}"/>
+                <xacro:add_geometry body="${module['collision'][body_name][0]}"/>
             </collision>
             <inertial>

Commit message: modify add_tcp for end-effectors

File: src/modular/modular_data/urdf/ModularBot.library.urdf.xacro (robot description, xacro)
@@ -363,4 +363,17 @@
         </joint>
     </xacro:macro>
+    <!-- Add a tcp. Length may vary -->
+    <xacro:macro name="add_tcp" params="type name father filename x y z roll pitch yaw">
+        <xacro:property name="module" value="${xacro.load_yaml(filename)}"/>
+        <link name="${name}"/>
+        <joint name="fixed_${name}" type="fixed">
+            <axis xyz="0 0 1" rpy="0 0 0" />
+            <parent link="${father}"/>
+            <child link="${name}"/>
+            <origin
+            rpy="${roll} ${pitch} ${yaw}"
+            xyz="${x} ${y} ${z}"/>
+        </joint>
+    </xacro:macro>
     <xacro:macro name="add_gripper_body" params="type name filename">
         <xacro:property name="module" value="${xacro.load_yaml(filename)}"/>

Commit message: dagana integration

File: src/modular/modular_data/urdf/ModularBot.library.urdf.xacro (robot description, xacro)
@@ -133,4 +133,11 @@
             </xacro:unless>
         </link>
+    </xacro:macro>
+    <!-- Macro for adding a generic link -->
+    <xacro:macro name="add_dagana" params="name type father x y z roll pitch yaw">
+        <xacro:include filename="$(find dagana_urdf)/urdf/dagana_macro.urdf.xacro" />
+        <xacro:dagana_gripper name="${name}" parent_link="${father}" joint_type="revolute">
+            <origin xyz="${x} ${y} ${z}" rpy="${roll} ${pitch} ${yaw}"/>
+        </xacro:dagana_gripper>
     </xacro:macro>
     <!-- Macro for adding a generic link -->

Commit message: fix bug in color visualization

File: src/modular/modular_data/urdf/ModularBot.library.urdf.xacro (robot description, xacro)
@@ -88,6 +88,10 @@
                             <xacro:add_origin body_pose="${body['pose']}"/>
                             <xacro:add_geometry body="${body}"/>
-                            <xacro:if value="${'color' in body}">
-                                <material name="${body['color']}"/>
+                            <xacro:if value="${'color' in body['parameters']}">
+                                <material name="${body['parameters']['color']['material_name']}">
+                                <xacro:if value="${'rgba' in body['parameters']['color']}">
+                                    <color rgba="${' '.join(str(x) for x in body['parameters']['color']['rgba'])}"/>
+                                </xacro:if>
+                                </material>
                             </xacro:if>
                         </visual>
@@ -398,6 +402,6 @@
                 <xacro:add_origin body_pose="${dict(x=0.0, y=0.0, z=0.0, roll=0.0, pitch=0.0, yaw=pi)}"/>
                 <xacro:add_geometry body="${module['visual'][body_name][0]}"/>
-                <xacro:if value="${'color' in module['visual'][body_name][0]}">
-                    <material name="${module['visual'][body_name]['color'][0]}"/>
+                <xacro:if value="${'color' in module['visual'][body_name][0]['parameters']}">
+                    <material name="${module['visual'][body_name][0]['parameters']['color']}"/>
                 </xacro:if>
             </visual>

Commit message: wip: camera drill integration

File: src/modular/modular_data/urdf/ModularBot.library.urdf.xacro (robot description, xacro)
@@ -138,5 +138,5 @@
         </link>
     </xacro:macro>
-    <!-- Macro for adding a generic link -->
+    <!-- Macro for adding dagana -->
     <xacro:macro name="add_dagana" params="name type father x y z roll pitch yaw">
         <xacro:include filename="$(find dagana_urdf)/urdf/dagana_macro.urdf.xacro" />
@@ -144,4 +144,15 @@
             <origin xyz="${x} ${y} ${z}" rpy="${roll} ${pitch} ${yaw}"/>
         </xacro:dagana_gripper>
+    </xacro:macro>
+    <!-- Macro for adding the drill module -->
+    <xacro:macro name="add_drill" params="name type filename">
+        <xacro:property name="module" value="${xacro.load_yaml(filename)}"/>
+        <xacro:property name="body_name" value="body_1"/>
+        <xacro:add_link_element name="${name}" type="${type}" module="${module}" body_name="${body_name}"/>
+        <!-- Add realsense D camera -->
+        <xacro:include filename="${MODULAR_PATH}/modular_data/urdf/concert.sensors.urdf.xacro"/>
+        <xacro:add_realsense_d_camera name="drill_camera" parent_name="${name}" add_gazebo_sensor="${ADD_DRILL_CAMERA}">
+            <origin xyz="0.103 0.0 0.25" rpy="0.0 0.0 0.0"/>
+        </xacro:add_realsense_d_camera>
     </xacro:macro>
     <!-- Macro for adding a generic link -->

File: src/modular/modular_data/urdf/concert.sensors.urdf.xacro (robot description, xacro)
@@ -10,4 +10,5 @@
     <xacro:property name="ADD_T265_LEFT" value="true" />
     <xacro:property name="ADD_T265_RIGHT" value="true" />
+    <xacro:property name="ADD_DRILL_CAMERA" value="true" />
 </xacro:if>
 <xacro:property name="ADD_VELODYNE_FRONT" value="false" />

File: src/modular/modular_data/urdf/template.urdf.xacro (robot description, xacro)
@@ -17,4 +17,6 @@
     <xacro:arg name="use_gpu_ray" default="false"/>
     <xacro:property name="USE_GPU_RAY" value="$(arg use_gpu_ray)" />
+    <xacro:arg name="drill_camera" default="false"/>
+    <xacro:property name="ADD_DRILL_CAMERA" value="$(arg drill_camera)" />
     <!-- adding (or not) world link for Gazebo simulation -->
     <xacro:if value="${ADD_FLOATING_BASE}">

Commit message: fhi pino compatibility

File: src/modular/modular_data/urdf/ModularBot.library.urdf.xacro (robot description, xacro)
@@ -221,5 +221,5 @@
     </xacro:macro>
     <!-- Macro for adding a socket -->
-    <xacro:macro name="add_socket" params="name type filename size">
+    <xacro:macro name="add_socket" params="name type filename flange_size">
         <xacro:property name="module" value="${xacro.load_yaml(filename)}"/>
         <xacro:property name="body_name" value="body_1"/>

Commit message: drill camera pose

File: src/modular/modular_data/urdf/ModularBot.library.urdf.xacro (robot description, xacro)
@@ -153,5 +153,5 @@
         <xacro:include filename="${MODULAR_PATH}/modular_data/urdf/concert.sensors.urdf.xacro"/>
         <xacro:add_realsense_d_camera name="drill_camera" parent_name="${name}" add_gazebo_sensor="${ADD_DRILL_CAMERA}">
-            <origin xyz="0.103 0.0 0.25" rpy="0.0 0.0 0.0"/>
+            <origin xyz="0.12 0.0 0.26" rpy="0.05 0.22 0.05"/>
         </xacro:add_realsense_d_camera>
     </xacro:macro>
