Commit message: refactor: avoid loading yaml from xacro (no thread-safe for json files)

File: src/modular/modular_data/urdf/ModularBot.library.urdf.xacro (robot description, xacro)
@@ -156,4 +156,11 @@
         </xacro:add_realsense_d_camera>
     </xacro:macro>
+    <!-- Add realsense D camera -->
+    <xacro:macro name="add_realsense_d_camera" params="name type parent_name">
+        <xacro:include filename="${MODULAR_PATH}/modular_data/urdf/concert.sensors.urdf.xacro" ns="concert_sensors"/>
+        <xacro:concert_sensors.add_realsense_d_camera name="${name}" parent_name="${parent_name}" add_gazebo_sensor="${ADD_DRILL_CAMERA}">
+            <origin xyz="0.12 0.0 0.26" rpy="0.05 0.22 0.05"/>
+        </xacro:concert_sensors.add_realsense_d_camera>
+    </xacro:macro>
     <!-- Macro for adding a generic link -->
     <xacro:macro name="add_link" params="name type filename">
@@ -163,6 +170,6 @@
     </xacro:macro>
     <!-- Macro for adding the proximal part of the joint (the physical module housing the actuator) -->
-    <xacro:macro name="add_proximal" params="type name filename">
-        <xacro:property name="module" value="${xacro.load_yaml(filename)}"/>
+    <xacro:macro name="add_proximal" params="type name module">
+        <!-- <xacro:property name="module" value="${xacro.load_yaml(filename)}"/> -->
         <xacro:property name="body_name" value="body_1"/>
         <xacro:add_link_element name="${name}" type="${type}" module="${module}" body_name="${body_name}"/>
@@ -193,5 +200,5 @@
         </joint>
     </xacro:macro>
-    <xacro:macro name="add_rotor_fast" params="type name filename x y z roll pitch yaw">
+    <xacro:macro name="add_rotor_fast" params="type name filename">
         <xacro:property name="module" value="${xacro.load_yaml(filename)}"/>
         <xacro:property name="gear_ratio" value="${module['actuator_data']['gear_ratio']}"/>
@@ -225,4 +232,8 @@
         <xacro:include filename="${MODULAR_PATH}/modular_data/urdf/concert.sensors.urdf.xacro"/>
         <xacro:add_mobile_base_sensors parent_name="${name}"/>
+    </xacro:macro>
+    <xacro:macro name="add_mobile_base_sensors" params="parent_name">
+        <xacro:include filename="${MODULAR_PATH}/modular_data/urdf/concert.sensors.urdf.xacro" ns="concert_sensors"/>
+        <xacro:concert_sensors.add_mobile_base_sensors parent_name="${parent_name}"/>
     </xacro:macro>
     <!-- Macro for adding a master cube -->
@@ -386,6 +397,5 @@
     </xacro:macro>
     <!-- Add a tcp. Length may vary -->
-    <xacro:macro name="add_tcp" params="type name father filename x y z roll pitch yaw">
-        <xacro:property name="module" value="${xacro.load_yaml(filename)}"/>
+    <xacro:macro name="add_tcp" params="type name father x y z roll pitch yaw">
         <link name="${name}"/>
         <joint name="fixed_${name}" type="fixed">

Commit message: add `xacro_if_guard`. fix removal of gazebo elements (wip in 3aa38684)

File: src/modular/modular_data/urdf/ModularBot.library.urdf.xacro (robot description, xacro)
@@ -40,4 +40,9 @@
             <inertia ixx="1.0e-06" ixy="0.0" ixz="0.0" iyy="1.0e-06" iyz="0.0" izz="1.0e-06" />
         </inertial>
+    </xacro:macro>
+    <xacro:macro name="xacro_if_guard" params="name value *block">
+        <xacro:if value="${value}">
+            <xacro:insert_block name="block"/>
+        </xacro:if>
     </xacro:macro>
     <xacro:macro name="add_geometry" params="body">

Commit message: fix: remove size param from `xacro:add_socket`

File: src/modular/modular_data/urdf/ModularBot.library.urdf.xacro (robot description, xacro)
@@ -263,5 +263,5 @@
     </xacro:macro>
     <!-- Macro for adding a socket -->
-    <xacro:macro name="add_socket" params="name type filename size">
+    <xacro:macro name="add_socket" params="name type filename">
         <xacro:property name="module" value="${xacro.load_yaml(filename)}"/>
         <xacro:property name="body_name" value="body_1"/>

Commit message: fix: remove size param from `xacro:add_socket`

File: src/modular/modular_data/urdf/ModularBot.library.urdf.xacro (robot description, xacro)
@@ -279,5 +279,5 @@
     </xacro:macro>
     <!-- Macro for adding a socket -->
-    <xacro:macro name="add_socket" params="name type filename size">
+    <xacro:macro name="add_socket" params="name type filename">
         <xacro:property name="module" value="${xacro.load_yaml(filename)}"/>
         <xacro:property name="body_name" value="body_1"/>

Commit message: refactor: rmv `add_slave_cube` method and occurances
Now `cube` are supported by `add_module()`. Historic commit :P

File: src/modular/modular_data/urdf/ModularBot.library.urdf.xacro (robot description, xacro)
@@ -242,16 +242,4 @@
         <xacro:concert_sensors.add_mobile_base_sensors parent_name="${parent_name}"/>
     </xacro:macro>
-    <!-- Macro for adding a master cube -->
-    <xacro:macro name="add_master_cube" params="name filename type">
-        <xacro:property name="module" value="${xacro.load_yaml(filename)}"/>
-        <joint name="fixed" type="fixed">
-            <parent link="base_link"/>
-            <child link="${name}"/>
-            <axis rpy="0 0 0" xyz="0 0 1"/>
-            <origin rpy="0.0 0.0 0.0" xyz="0.0 0.0 0.0"/>
-        </joint>
-        <xacro:property name="body_name" value="body_1"/>
-        <xacro:add_link_element name="${name}" type="${type}" module="${module}" body_name="${body_name}"/>
-    </xacro:macro>
     <xacro:macro name="add_connector" params="name type parent_name x y z roll pitch yaw">
         <link name="${name}">
@@ -271,10 +259,4 @@
                     xyz="${x} ${y} ${z}"/>
         </joint>
-    </xacro:macro>
-    <!-- Macro for adding a slave cube -->
-    <xacro:macro name="add_slave_cube" params="name filename type">
-        <xacro:property name="module" value="${xacro.load_yaml(filename)}"/>
-        <xacro:property name="body_name" value="body_1"/>
-        <xacro:add_link_element name="${name}" type="${type}" module="${module}" body_name="${body_name}"/>
     </xacro:macro>
     <!-- Macro for adding a socket -->

Commit message: fix: rmv sensors as well when removing `mobile_base`

File: src/modular/modular_data/urdf/ModularBot.library.urdf.xacro (robot description, xacro)
@@ -238,5 +238,5 @@
         <xacro:add_mobile_base_sensors parent_name="${name}"/>
     </xacro:macro>
-    <xacro:macro name="add_mobile_base_sensors" params="parent_name">
+    <xacro:macro name="add_mobile_base_sensors" params="name parent_name">
         <xacro:include filename="${MODULAR_PATH}/modular_data/urdf/concert.sensors.urdf.xacro" ns="concert_sensors"/>
         <xacro:concert_sensors.add_mobile_base_sensors parent_name="${parent_name}"/>

Commit message: chore: add material color for dagana

File: src/modular/modular_data/urdf/ModularBot.library.urdf.xacro (robot description, xacro)
@@ -146,4 +146,7 @@
     <xacro:macro name="add_dagana" params="name type father x y z roll pitch yaw">
         <xacro:include filename="$(find dagana_urdf)/urdf/dagana_macro.urdf.xacro" />
+        <material name="dark_grey">
+            <color rgba="0.2 0.2 0.2 1"/>
+        </material>
         <xacro:dagana_gripper name="${name}" parent_link="${father}" joint_type="revolute">
             <origin xyz="${x} ${y} ${z}" rpy="${roll} ${pitch} ${yaw}"/>

Commit message: refactor: add `socket` type and uniform to use `add_module()`

File: src/modular/modular_data/urdf/ModularBot.library.urdf.xacro (robot description, xacro)
@@ -262,10 +262,4 @@
                     xyz="${x} ${y} ${z}"/>
         </joint>
-    </xacro:macro>
-    <!-- Macro for adding a socket -->
-    <xacro:macro name="add_socket" params="name type filename">
-        <xacro:property name="module" value="${xacro.load_yaml(filename)}"/>
-        <xacro:property name="body_name" value="body_1"/>
-        <xacro:add_link_element name="${name}" type="${type}" module="${module}" body_name="${body_name}"/>
     </xacro:macro>
     <!-- Macro for adding a size adapter -->

Commit message: upd drill camera calibration

File: src/modular/modular_data/urdf/ModularBot.library.urdf.xacro (robot description, xacro)
@@ -161,5 +161,5 @@
         <xacro:include filename="${MODULAR_PATH}/modular_data/urdf/concert.sensors.urdf.xacro"/>
         <xacro:add_realsense_d_camera name="drill_camera" parent_name="${name}" add_gazebo_sensor="${ADD_DRILL_CAMERA}">
-            <origin xyz="0.12 0.0 0.26" rpy="0.05 0.22 0.05"/>
+            <origin xyz="0.12 0.0 0.26" rpy="0.05 0.22 0.04"/>
         </xacro:add_realsense_d_camera>
     </xacro:macro>

Commit message: fix: allow non-revolute joint types

File: src/modular/modular_data/urdf/ModularBot.library.urdf.xacro (robot description, xacro)
@@ -55,5 +55,5 @@
             </xacro:if>
             <xacro:if value="${body['type'] == 'box'}">
-                <box size="${body['parameters']['size']}"/>
+                <box size="${' '.join(str(x) for x in body['parameters']['size'])}"/>
             </xacro:if>
             <xacro:if value="${body['type'] == 'sphere'}">
@@ -191,5 +191,5 @@
     <!-- Macro for adding the joint. A dummy link is also added with no visual tag, but with inertial parameters corresponding to the rotating part -->
     <xacro:macro name="add_joint" params="type name father child x y z roll pitch yaw upper_lim lower_lim effort velocity">
-        <joint name="${name}" type="revolute">
+        <joint name="${name}" type="${type}">
             <axis xyz="0 0 1" rpy="0 0 0" />
             <parent link="${father}"/>

Commit message: fix inertia reflection for the so-called "rotor_fast" elements

File: src/modular/modular_data/urdf/ModularBot.library.urdf.xacro (robot description, xacro)
@@ -208,20 +208,28 @@
         </joint>
     </xacro:macro>
-    <xacro:macro name="add_rotor_fast" params="type name filename">
-        <xacro:property name="module" value="${xacro.load_yaml(filename)}"/>
+    <!-- Deprecated -->
+    <xacro:macro name="add_rotor" params="type name fixed_joint_rotor_name stator_name distal_link_name x y z roll pitch yaw module">
         <xacro:property name="gear_ratio" value="${module['actuator_data']['gear_ratio']}"/>
+        <xacro:if value="${REFLECT_ROTOR_INERTIA}">
+            <xacro:add_fixed_joint type="fixed_joint" name="${fixed_joint_name}" father="${distal_link_name}" child="${name}" x="0.0" y="0.0" z="0.0" roll="0.0" pitch="0.0" yaw="0.0"/>
+            <xacro:property name="izz" value="${ gear_ratio * gear_ratio * module['dynamics']['body_2_fast']['inertia_tensor']['I_zz'] }"/>
+        </xacro:if>
+        <xacro:unless value="${REFLECT_ROTOR_INERTIA}">
+            <xacro:add_fixed_joint type="fixed_joint" name="${fixed_joint_name}" father="${stator_name}" child="${name}" x="${x}" y="${y}" z="${z}" roll="${roll}" pitch="${pitch}" yaw="${yaw}"/>
+            <xacro:property name="izz" value="${ module['dynamics']['body_2_fast']['inertia_tensor']['I_zz'] }"/>
+        </xacro:unless>
         <link name="${name}">
             <inertial>
                 <origin
-                        xyz="${module['dynamics']['body_2_fast']['CoM']['x']} ${module['dynamics']['body_2_fast']['CoM']['y']} ${module['dynamics']['body_2_fast']['CoM']['z']}"
-                        rpy="0 0 0"/>
-                    <mass value="${module['dynamics']['body_2_fast']['mass']}"/>
-                    <inertia
-                        ixx="${module['dynamics']['body_2_fast']['inertia_tensor']['I_xx']}"
-                        ixy="${module['dynamics']['body_2_fast']['inertia_tensor']['I_xy']}"
-                        iyy="${module['dynamics']['body_2_fast']['inertia_tensor']['I_yy']}"
-                        ixz="${module['dynamics']['body_2_fast']['inertia_tensor']['I_xz'] }"
-                        iyz="${module['dynamics']['body_2_fast']['inertia_tensor']['I_yz'] }"
-                        izz="${ gear_ratio * gear_ratio * module['dynamics']['body_2_fast']['inertia_tensor']['I_zz'] }"/>
+                    xyz="${module['dynamics']['body_2_fast']['CoM']['x']} ${module['dynamics']['body_2_fast']['CoM']['y']} ${module['dynamics']['body_2_fast']['CoM']['z']}"
+                    rpy="0 0 0"/>
+                <mass value="${module['dynamics']['body_2_fast']['mass']}"/>
+                <inertia
+                    ixx="${module['dynamics']['body_2_fast']['inertia_tensor']['I_xx']}"
+                    ixy="${module['dynamics']['body_2_fast']['inertia_tensor']['I_xy']}"
+                    iyy="${module['dynamics']['body_2_fast']['inertia_tensor']['I_yy']}"
+                    ixz="${module['dynamics']['body_2_fast']['inertia_tensor']['I_xz'] }"
+                    iyz="${module['dynamics']['body_2_fast']['inertia_tensor']['I_yz'] }"
+                    izz="${izz}"/>
             </inertial>
         </link>

File: src/modular/modular_data/urdf/template.urdf.xacro (robot description, xacro)
@@ -19,4 +19,6 @@
     <xacro:arg name="drill_camera" default="false"/>
     <xacro:property name="ADD_DRILL_CAMERA" value="$(arg drill_camera)" />
+    <xacro:arg name="reflect_rotor_inertia" default="false"/>
+    <xacro:property name="REFLECT_ROTOR_INERTIA" value="$(arg reflect_rotor_inertia)" />
     <!-- adding (or not) world link for Gazebo simulation -->
     <xacro:if value="${ADD_FLOATING_BASE}">
