Commit message: refactor RGBD camera URDF generation
- Thread `publish_tf` and `gazebo_urdf` controls through camera helpers
- Remove obsolete drill camera xacro wrappers
- Refactor `add_realsense_d_camera` to `add_rgbd_camera`

File: src/modular/modular_data/urdf/ModularBot.library.urdf.xacro (robot description, xacro)
@@ -151,22 +151,4 @@
             <origin xyz="${x} ${y} ${z}" rpy="${roll} ${pitch} ${yaw}"/>
         </xacro:dagana_gripper>
-    </xacro:macro>
-    <!-- Macro for adding the drill module -->
-    <xacro:macro name="add_drill" params="name type filename">
-        <xacro:property name="module" value="${xacro.load_yaml(filename)}"/>
-        <xacro:property name="body_name" value="body_1"/>
-        <xacro:add_link_element name="${name}" type="${type}" module="${module}" body_name="${body_name}"/>
-        <!-- Add realsense D camera -->
-        <xacro:include filename="${MODULAR_PATH}/modular_data/urdf/concert.sensors.urdf.xacro"/>
-        <xacro:add_realsense_d_camera name="drill_camera" parent_name="${name}" add_gazebo_sensor="${ADD_DRILL_CAMERA}">
-            <origin xyz="0.12 0.0 0.26" rpy="0.05 0.22 0.04"/>
-        </xacro:add_realsense_d_camera>
-    </xacro:macro>
-    <!-- Add realsense D camera -->
-    <xacro:macro name="add_realsense_d_camera" params="name type parent_name">
-        <xacro:include filename="${MODULAR_PATH}/modular_data/urdf/concert.sensors.urdf.xacro" ns="concert_sensors"/>
-        <xacro:concert_sensors.add_realsense_d_camera name="${name}" parent_name="${parent_name}" add_gazebo_sensor="${ADD_DRILL_CAMERA}">
-            <origin xyz="0.12 0.0 0.26" rpy="0.05 0.22 0.05"/>
-        </xacro:concert_sensors.add_realsense_d_camera>
     </xacro:macro>
     <!-- Macro for adding a generic link -->

File: src/modular/modular_data/urdf/concert.sensors.urdf.xacro (robot description, xacro)
@@ -10,5 +10,4 @@
     <!-- <xacro:property name="ADD_T265_LEFT" value="true" />
     <xacro:property name="ADD_T265_RIGHT" value="true" /> -->
-    <xacro:property name="ADD_DRILL_CAMERA" value="true" />
 </xacro:if>
 <xacro:property name="ADD_VELODYNE_FRONT" value="false" />
@@ -31,9 +30,10 @@
         <origin xyz="0.402872 0.0 -0.078218" rpy="0 0.261799 0"/>
     </xacro:property>
-    <xacro:add_realsense_d_camera name="${d435i_front_name}"
+    <xacro:add_rgbd_camera name="${d435i_front_name}"
                                 parent_name="${d435i_front_parent_name}"
-                                add_gazebo_sensor="${ADD_D435I_FRONT}">
+                                gazebo_urdf="${GAZEBO_URDF}"
+                                publish_tf="${ADD_D435I_FRONT}">
         <xacro:insert_block name="d435i_front_origin" />
-    </xacro:add_realsense_d_camera> -->
+    </xacro:add_rgbd_camera> -->
     <!-- Add back D435i camera -->
     <!-- <xacro:property name="d435i_back_name" value="D435i_camera_back" />
@@ -42,9 +42,10 @@
         <origin xyz="-0.402872 0.0 -0.078218" rpy="0 0.261799 3.141593"/>
     </xacro:property> -->
-    <!-- <xacro:add_realsense_d_camera name="${d435i_back_name}"
+    <!-- <xacro:add_rgbd_camera name="${d435i_back_name}"
                                 parent_name="${d435i_back_parent_name}"
-                                add_gazebo_sensor="${ADD_D435I_BACK}">
+                                gazebo_urdf="${GAZEBO_URDF}"
+                                publish_tf="${ADD_D435I_BACK}">
         <xacro:insert_block name="d435i_back_origin" />
-    </xacro:add_realsense_d_camera> -->
+    </xacro:add_rgbd_camera> -->
     <!-- Add left T265 camera -->
     <xacro:property name="t265_left_name" value="T265_camera_left" />
@@ -55,5 +56,5 @@
     <xacro:add_realsense_t_camera name="${t265_left_name}"
                                 parent_name="${t265_left_parent_name}"
-                                add_gazebo_sensor="${ADD_T265_LEFT}">
+                                gazebo_urdf="${ADD_T265_LEFT}">
         <xacro:insert_block name="t265_left_origin" />
     </xacro:add_realsense_t_camera>
@@ -66,5 +67,5 @@
     <xacro:add_realsense_t_camera name="${t265_right_name}"
                                 parent_name="${t265_right_parent_name}"
-                                add_gazebo_sensor="${ADD_T265_RIGHT}">
+                                gazebo_urdf="${ADD_T265_RIGHT}">
         <xacro:insert_block name="t265_right_origin" />
     </xacro:add_realsense_t_camera>
@@ -281,31 +282,11 @@
     </gazebo>
 </xacro:macro>
+<!-- Not used: point cloud is wrongly rotated. We use the macro from realsense_gazebo_description -->
 <!-- ============================================================ -->
-<!-- Macro for RealSense D435i - NATIVE GAZEBO RENDERING          -->
-<!-- This uses Gazebo's built-in camera rendering, NOT test data  -->
+<!-- Macro for Gazebo rgbd camera emulating a RealSense D435i -->
 <!-- ============================================================ -->
-<xacro:macro name="add_realsense_d_camera" params="name parent_name *origin add_gazebo_sensor">
+<xacro:macro name="add_rgbd_camera" params="name parent_name *origin publish_tf gazebo_urdf">
     <!-- Camera body link -->
-    <link name="${name}_bottom_screw_frame">
-        <visual>
-            <origin xyz="0 0 0" rpy="${-pi/2} 0 ${-pi/2}"/>
-            <geometry>
-                <box size="0.025 0.090 0.025"/>
-            </geometry>
-            <material name="gray">
-                <color rgba="0.5 0.5 0.5 1"/>
-            </material>
-        </visual>
-        <collision>
-            <origin xyz="0 0 0" rpy="${-pi/2} 0 ${-pi/2}"/>
-            <geometry>
-                <box size="0.02505 0.090 0.025"/>
-            </geometry>
-        </collision>
-        <inertial>
-            <mass value="0.072"/>
-            <inertia ixx="0.0001" ixy="0" ixz="0" iyy="0.0001" iyz="0" izz="0.0001"/>
-        </inertial>
-    </link>
+    <link name="${name}_bottom_screw_frame"/>
     <!-- Joint to parent -->
     <joint name="${name}_joint" type="fixed">
@@ -314,111 +295,133 @@
         <child link="${name}_bottom_screw_frame"/>
     </joint>
-    <!-- Camera link (sensor reference frame) -->
-    <link name="${name}_link"/>
-    <joint name="${name}_link_joint" type="fixed">
-        <origin xyz="0 0.0175 0.0125" rpy="0 0 0"/>
-        <parent link="${name}_bottom_screw_frame"/>
-        <child link="${name}_link"/>
-    </joint>
-    <!-- Depth frame -->
-    <link name="${name}_depth_frame"/>
-    <joint name="${name}_depth_joint" type="fixed">
-        <origin xyz="0 0 0" rpy="0 0 0"/>
-        <parent link="${name}_link"/>
-        <child link="${name}_depth_frame"/>
-    </joint>
-    <!-- Depth optical frame -->
-    <link name="${name}_depth_optical_frame"/>
-    <joint name="${name}_depth_optical_joint" type="fixed">
-        <origin xyz="0 0 0" rpy="${-pi/2} 0 ${-pi/2}"/>
-        <parent link="${name}_depth_frame"/>
-        <child link="${name}_depth_optical_frame"/>
-    </joint>
-    <!-- Color frame -->
-    <link name="${name}_color_frame"/>
-    <joint name="${name}_color_joint" type="fixed">
-        <origin xyz="0 0.015 0" rpy="0 0 0"/>
-        <parent link="${name}_depth_frame"/>
-        <child link="${name}_color_frame"/>
-    </joint>
-    <!-- Color optical frame -->
-    <link name="${name}_color_optical_frame"/>
-    <joint name="${name}_color_optical_joint" type="fixed">
-        <origin xyz="0 0 0" rpy="${-pi/2} 0 ${-pi/2}"/>
-        <parent link="${name}_color_frame"/>
-        <child link="${name}_color_optical_frame"/>
-    </joint>
-    <!-- Left IR frame -->
-    <link name="${name}_left_ir_frame"/>
-    <joint name="${name}_left_ir_joint" type="fixed">
-        <origin xyz="0 0 0" rpy="0 0 0"/>
-        <parent link="${name}_depth_frame"/>
-        <child link="${name}_left_ir_frame"/>
-    </joint>
-    <!-- Left IR optical frame -->
-    <link name="${name}_left_ir_optical_frame"/>
-    <joint name="${name}_left_ir_optical_joint" type="fixed">
-        <origin xyz="0 0 0" rpy="${-pi/2} 0 ${-pi/2}"/>
-        <parent link="${name}_left_ir_frame"/>
-        <child link="${name}_left_ir_optical_frame"/>
-    </joint>
-    <!-- Right IR frame -->
-    <link name="${name}_right_ir_frame"/>
-    <joint name="${name}_right_ir_joint" type="fixed">
-        <origin xyz="0 -0.050 0" rpy="0 0 0"/>
-        <parent link="${name}_depth_frame"/>
-        <child link="${name}_right_ir_frame"/>
-    </joint>
-    <!-- Right IR optical frame -->
-    <link name="${name}_right_ir_optical_frame"/>
-    <joint name="${name}_right_ir_optical_joint" type="fixed">
-        <origin xyz="0 0 0" rpy="${-pi/2} 0 ${-pi/2}"/>
-        <parent link="${name}_right_ir_frame"/>
-        <child link="${name}_right_ir_optical_frame"/>
-    </joint>
-    <!-- ========================================== -->
-    <!-- NATIVE GAZEBO RGBD CAMERA - REAL RENDERING -->
-    <!-- Uses rgbd_camera type for combined RGB+Depth -->
-    <!-- Topics: /{name}/image, /{name}/depth_image, /{name}/points -->
-    <!-- ========================================== -->
-    <xacro:if value="${add_gazebo_sensor}">
-        <gazebo reference="${name}_link">
-            <!-- RGBD Camera (combined RGB + Depth + PointCloud) -->
-            <sensor name="${name}_rgbd" type="rgbd_camera">
-                <always_on>1</always_on>
-                <update_rate>30</update_rate>
-                <visualize>true</visualize>
-                <topic>${name}</topic>
-                <gz_frame_id>${name}_depth_optical_frame</gz_frame_id>
-                <camera name="${name}">
-                    <horizontal_fov>1.211259</horizontal_fov>
-                    <image>
-                        <width>640</width>
-                        <height>480</height>
-                        <format>R8G8B8</format>
-                    </image>
-                    <clip>
-                        <near>0.1</near>
-                        <far>100</far>
-                    </clip>
-                    <depth_camera>
+    <xacro:if value="${publish_tf}">
+        <!-- Camera link (sensor reference frame) -->
+        <link name="${name}_link">
+            <visual>
+                <origin xyz="0 -0.0175 0" rpy="0 0 0"/>
+                <geometry>
+                    <box size="0.025 0.090 0.025"/>
+                </geometry>
+                <material name="gray">
+                    <color rgba="0.5 0.5 0.5 1"/>
+                </material>
+            </visual>
+            <collision>
+                <origin xyz="0 -0.0175 0" rpy="0 0 0"/>
+                <geometry>
+                    <box size="0.02505 0.090 0.025"/>
+                </geometry>
+            </collision>
+            <inertial>
+                <mass value="0.072"/>
+                <inertia ixx="0.0001" ixy="0" ixz="0" iyy="0.0001" iyz="0" izz="0.0001"/>
+            </inertial>
+        </link>
+        <joint name="${name}_link_joint" type="fixed">
+            <origin xyz="0 0.0175 0.0125" rpy="0 0 0"/>
+            <parent link="${name}_bottom_screw_frame"/>
+            <child link="${name}_link"/>
+        </joint>
+        <!-- Depth frame -->
+        <link name="${name}_depth_frame"/>
+        <joint name="${name}_depth_joint" type="fixed">
+            <origin xyz="0 0 0" rpy="0 0 0"/>
+            <parent link="${name}_link"/>
+            <child link="${name}_depth_frame"/>
+        </joint>
+        <!-- Depth optical frame -->
+        <link name="${name}_depth_optical_frame"/>
+        <joint name="${name}_depth_optical_joint" type="fixed">
+            <origin xyz="0 0 0" rpy="${-pi/2} 0 ${-pi/2}"/>
+            <parent link="${name}_depth_frame"/>
+            <child link="${name}_depth_optical_frame"/>
+        </joint>
+        <!-- Color frame -->
+        <link name="${name}_color_frame"/>
+        <joint name="${name}_color_joint" type="fixed">
+            <origin xyz="0 0.015 0" rpy="0 0 0"/>
+            <parent link="${name}_depth_frame"/>
+            <child link="${name}_color_frame"/>
+        </joint>
+        <!-- Color optical frame -->
+        <link name="${name}_color_optical_frame"/>
+        <joint name="${name}_color_optical_joint" type="fixed">
+            <origin xyz="0 0 0" rpy="${-pi/2} 0 ${-pi/2}"/>
+            <parent link="${name}_color_frame"/>
+            <child link="${name}_color_optical_frame"/>
+        </joint>
+        <!-- Left IR frame -->
+        <link name="${name}_left_ir_frame"/>
+        <joint name="${name}_left_ir_joint" type="fixed">
+            <origin xyz="0 0 0" rpy="0 0 0"/>
+            <parent link="${name}_depth_frame"/>
+            <child link="${name}_left_ir_frame"/>
+        </joint>
+        <!-- Left IR optical frame -->
+        <link name="${name}_left_ir_optical_frame"/>
+        <joint name="${name}_left_ir_optical_joint" type="fixed">
+            <origin xyz="0 0 0" rpy="${-pi/2} 0 ${-pi/2}"/>
+            <parent link="${name}_left_ir_frame"/>
+            <child link="${name}_left_ir_optical_frame"/>
+        </joint>
+        <!-- Right IR frame -->
+        <link name="${name}_right_ir_frame"/>
+        <joint name="${name}_right_ir_joint" type="fixed">
+            <origin xyz="0 -0.050 0" rpy="0 0 0"/>
+            <parent link="${name}_depth_frame"/>
+            <child link="${name}_right_ir_frame"/>
+        </joint>
+        <!-- Right IR optical frame -->
+        <link name="${name}_right_ir_optical_frame"/>
+        <joint name="${name}_right_ir_optical_joint" type="fixed">
+            <origin xyz="0 0 0" rpy="${-pi/2} 0 ${-pi/2}"/>
+            <parent link="${name}_right_ir_frame"/>
+            <child link="${name}_right_ir_optical_frame"/>
+        </joint>
+        <!-- ========================================== -->
+        <!-- NATIVE GAZEBO RGBD CAMERA - REAL RENDERING -->
+        <!-- Uses rgbd_camera type for combined RGB+Depth -->
+        <!-- Topics: /{name}/image, /{name}/depth_image, /{name}/points -->
+        <!-- ========================================== -->
+        <xacro:if value="${gazebo_urdf}">
+            <gazebo reference="${name}_link">
+                <!-- RGBD Camera (combined RGB + Depth + PointCloud) -->
+                <sensor name="${name}_rgbd" type="rgbd_camera">
+                    <always_on>1</always_on>
+                    <update_rate>30</update_rate>
+                    <visualize>true</visualize>
+                    <topic>${name}</topic>
+                    <gz_frame_id>${name}_depth_frame</gz_frame_id>
+                    <camera name="${name}">
+                        <horizontal_fov>1.211259</horizontal_fov>
+                        <image>
+                            <width>640</width>
+                            <height>480</height>
+                            <format>R8G8B8</format>
+                        </image>
                         <clip>
                             <near>0.1</near>
-                            <far>10</far>
+                            <far>100</far>
                         </clip>
-                    </depth_camera>
-                    <noise>
-                        <type>gaussian</type>
-                        <mean>0.0</mean>
-                        <stddev>0.007</stddev>
-                    </noise>
-                    <optical_frame_id>${name}_depth_optical_frame</optical_frame_id>
-                </camera>
-            </sensor>
-        </gazebo>
+                        <depth_camera>
+                            <clip>
+                                <near>0.1</near>
+                                <far>10</far>
+                            </clip>
+                        </depth_camera>
+                        <noise>
+                            <type>gaussian</type>
+                            <mean>0.0</mean>
+                            <stddev>0.007</stddev>
+                        </noise>
+                        <optical_frame_id>${name}_depth_optical_frame</optical_frame_id>
+                    </camera>
+                </sensor>
+            </gazebo>
+        </xacro:if>
     </xacro:if>
 </xacro:macro>
 <!-- Macro for T265 camera - Dummy frames only (discontinued) -->
-<xacro:macro name="add_realsense_t_camera" params="name parent_name *origin add_gazebo_sensor">
+<xacro:macro name="add_realsense_t_camera" params="name parent_name *origin gazebo_urdf">
     <joint name="${name}_joint" type="fixed">
         <xacro:insert_block name="origin"/>
